Commit message: u

File: urdf/razbot.urdf (robot description, URDF)
Before this commit: robot razbot, 27 links, 26 joints
Links:
- removed link body_link
- added link base_footprint
- link base_link: mass None -> 0.00001; geometry collision mesh filename=package://robot_gazebo/meshes/razbot/body.stl scale=0.001 0.001 0.001; visual mesh filename=package://robot_gazebo/meshes/razbot/body.stl scale=0.001 0.001 0.001
Joints:
- joint base_joint: child body_link -> base_link; parent base_link -> base_footprint
- joint leg_center_joint_LF: parent body_link -> base_link
- joint leg_center_joint_LM: parent body_link -> base_link
- joint leg_center_joint_LR: parent body_link -> base_link
- joint leg_center_joint_RF: parent body_link -> base_link
- joint leg_center_joint_RM: parent body_link -> base_link
- joint leg_center_joint_RR: parent body_link -> base_link
