Commit message: u

File: urdf/lbr_iiwa_14_r820.urdf (robot description, URDF)
Before this commit: robot lbr_iiwa_14_r820, 10 links, 9 joints
Links:
- link base_link: mass None -> 2
- link link_1: mass None -> 2
- link link_2: mass None -> 2
- link link_3: mass None -> 2
- link link_4: mass None -> 2
- link link_5: mass None -> 2
- link link_6: mass None -> 2
- link link_7: mass None -> 2

File: xacro/lbr_iiwa_14_r820.xacro (robot description, xacro)
@@ -8,4 +8,9 @@
 <!-- ****************************************************** base link **************************************************************** -->
     <link name="${prefix}base_link">
+      <inertial>
+        <origin xyz="0 0 0" rpy="0 0 0"/>
+        <mass value="2"/>
+        <inertia ixx="0.01" ixy="0" ixz="0" iyy="0.01" iyz="0" izz="0.01" />
+      </inertial>
       <visual>
         <origin xyz="0 0 0" rpy="0 0 0" />
@@ -23,4 +28,9 @@
 <!-- ****************************************************** link 1 (A1) ************************************************************** -->
     <link name="${prefix}link_1">
+      <inertial>
+        <origin xyz="0 0 0" rpy="0 0 0"/>
+        <mass value="2"/>
+        <inertia ixx="0.01" ixy="0" ixz="0" iyy="0.01" iyz="0" izz="0.01" />
+      </inertial>
       <visual>
         <origin xyz="0 0 0" rpy="0 0 0" />
@@ -38,4 +48,9 @@
 <!-- ****************************************************** link 2 **************************************************************** -->
     <link name="${prefix}link_2">
+      <inertial>
+        <origin xyz="0 0 0" rpy="0 0 0"/>
+        <mass value="2"/>
+        <inertia ixx="0.01" ixy="0" ixz="0" iyy="0.01" iyz="0" izz="0.01" />
+      </inertial>
       <visual>
         <origin xyz="0 0 0" rpy="0 0 0" />
@@ -53,4 +68,9 @@
 <!-- ****************************************************** link 3 **************************************************************** -->
     <link name="${prefix}link_3">
+      <inertial>
+        <origin xyz="0 0 0" rpy="0 0 0"/>
+        <mass value="2"/>
+        <inertia ixx="0.01" ixy="0" ixz="0" iyy="0.01" iyz="0" izz="0.01" />
+      </inertial>
       <visual>
         <origin xyz="0 0 0" rpy="0 0 0" />
@@ -68,4 +88,9 @@
 <!-- ****************************************************** link 4 **************************************************************** -->
     <link name="${prefix}link_4">
+      <inertial>
+        <origin xyz="0 0 0" rpy="0 0 0"/>
+        <mass value="2"/>
+        <inertia ixx="0.01" ixy="0" ixz="0" iyy="0.01" iyz="0" izz="0.01" />
+      </inertial>
       <visual>
         <origin xyz="0 0 0" rpy="0 0 0" />
@@ -83,4 +108,9 @@
 <!-- ****************************************************** link 5 **************************************************************** -->
     <link name="${prefix}link_5">
+      <inertial>
+        <origin xyz="0 0 0" rpy="0 0 0"/>
+        <mass value="2"/>
+        <inertia ixx="0.01" ixy="0" ixz="0" iyy="0.01" iyz="0" izz="0.01" />
+      </inertial>
       <visual>
         <origin xyz="0 0 0" rpy="0 0 0" />
@@ -98,4 +128,9 @@
 <!-- ****************************************************** link 6 **************************************************************** -->
     <link name="${prefix}link_6">
+      <inertial>
+        <origin xyz="0 0 0" rpy="0 0 0"/>
+        <mass value="2"/>
+        <inertia ixx="0.01" ixy="0" ixz="0" iyy="0.01" iyz="0" izz="0.01" />
+      </inertial>
       <visual>
         <origin xyz="0 0 0" rpy="0 0 0" />
@@ -113,4 +148,9 @@
 <!-- ****************************************************** link 7 **************************************************************** -->
     <link name="${prefix}link_7">
+      <inertial>
+        <origin xyz="0 0 0" rpy="0 0 0"/>
+        <mass value="2"/>
+        <inertia ixx="0.01" ixy="0" ixz="0" iyy="0.01" iyz="0" izz="0.01" />
+      </inertial>
       <visual>
         <origin xyz="0 0 0" rpy="0 0 0" />
