Commit message: u

File: urdf/pxm3.urdf (robot description, URDF)
Before this commit: robot pxm3, 26 links, 25 joints
Links:
- removed link MP_BODY
- added link base_footprint
- link base_link: mass None -> 0.97559947; geometry collision mesh filename=package://robot_gazebo/meshes/pxm3/body_coll.STL scale=1 1 1; visual mesh filename=package://robot_gazebo/meshes/pxm3/body.STL scale=1 1 1
Joints:
- removed joint j_pxm3_attachment
- added joint j_base_base_footprint: type fixed, parent base_footprint, child base_link, origin xyz=0 0 0 rpy=0 0 0
- joint j_c1_LF: parent MP_BODY -> base_link
- joint j_c1_LM: parent MP_BODY -> base_link
- joint j_c1_LR: parent MP_BODY -> base_link
- joint j_c1_RF: parent MP_BODY -> base_link
- joint j_c1_RM: parent MP_BODY -> base_link
- joint j_c1_RR: parent MP_BODY -> base_link

Commit message: u

File: urdf/pxm3.urdf (robot description, URDF)
Before this commit: robot pxm3, 26 links, 25 joints
Joints:
- joint j_c1_LF: origin xyz= 0.1248   0.06164  0.001116 rpy=0 4.7123  2.356194490192345 -> xyz= 0.1248   0.06164  0.001116 rpy=0 4.71238898038469 2.356194490192345
- joint j_c1_LM: origin xyz= 0        0.1034   0.001116 rpy=0 4.7123  3.14159 -> xyz= 0        0.1034   0.001116 rpy=0 4.71238898038469 3.141592653589793
- joint j_c1_LR: origin xyz=-0.1248   0.06164  0.001116 rpy=0 4.7123  3.9269908169872414 -> xyz=-0.1248   0.06164  0.001116 rpy=0 4.71238898038469 3.9269908169872414
- joint j_c1_RF: origin xyz= 0.1248  -0.06164  0.001116 rpy=0 4.7123  0.7853981633974483 -> xyz= 0.1248  -0.06164  0.001116 rpy=0 4.71238898038469 0.7853981633974483
- joint j_c1_RM: origin xyz= 0       -0.1034   0.001116 rpy=0 4.7123  0 -> xyz= 0       -0.1034   0.001116 rpy=0 4.71238898038469 0
- joint j_c1_RR: origin xyz=-0.1248  -0.06164  0.001116 rpy=0 4.7123 -0.7853981633974483 -> xyz=-0.1248  -0.06164  0.001116 rpy=0 4.71238898038469 -0.7853981633974483
- joint j_c2_LF: origin xyz=0 -0.054 0 rpy=0 1.5704 3.14159 -> xyz=0 -0.054 0 rpy=0 1.5707963267948966 3.141592653589793
- joint j_c2_LM: origin xyz=0 -0.054 0 rpy=0 1.5704 3.14159 -> xyz=0 -0.054 0 rpy=0 1.5707963267948966 3.141592653589793
- joint j_c2_LR: origin xyz=0 -0.054 0 rpy=0 1.5704 3.14159 -> xyz=0 -0.054 0 rpy=0 1.5707963267948966 3.141592653589793
- joint j_c2_RF: origin xyz=0 -0.054 0 rpy=0 1.5704 3.14159 -> xyz=0 -0.054 0 rpy=0 1.5707963267948966 3.141592653589793
- joint j_c2_RM: origin xyz=0 -0.054 0 rpy=0 1.5704 3.14159 -> xyz=0 -0.054 0 rpy=0 1.5707963267948966 3.141592653589793
- joint j_c2_RR: origin xyz=0 -0.054 0 rpy=0 1.5704 3.14159 -> xyz=0 -0.054 0 rpy=0 1.5707963267948966 3.141592653589793
- joint j_thigh_LF: origin xyz=0 0 0 rpy= 0 3.14159 3.14159 -> xyz=0 0 0 rpy= 0 3.141592653589793 3.141592653589793
- joint j_thigh_LM: origin xyz=0 0 0 rpy= 0 3.14159 3.14159 -> xyz=0 0 0 rpy= 0 3.141592653589793 3.141592653589793
- joint j_thigh_LR: origin xyz=0 0 0 rpy= 0 3.14159 3.14159 -> xyz=0 0 0 rpy= 0 3.141592653589793 3.141592653589793
- joint j_thigh_RF: origin xyz=0 0 0 rpy= 0 3.14159 3.14159 -> xyz=0 0 0 rpy= 0 3.141592653589793 3.141592653589793
- joint j_thigh_RM: origin xyz=0 0 0 rpy= 0 3.14159 3.14159 -> xyz=0 0 0 rpy= 0 3.141592653589793 3.141592653589793
- joint j_thigh_RR: origin xyz=0 0 0 rpy= 0 3.14159 3.14159 -> xyz=0 0 0 rpy= 0 3.141592653589793 3.141592653589793
- joint j_tibia_LF: origin xyz=0 -0.0645 -0.0145 rpy=-1.5707 0 3.14159 -> xyz=0 -0.0645 -0.0145 rpy=-1.5707963267948966 0 3.141592653589793
- joint j_tibia_LM: origin xyz=0 -0.0645 -0.0145 rpy=-1.5707 0 3.14159 -> xyz=0 -0.0645 -0.0145 rpy=-1.5707963267948966 0 3.141592653589793
- joint j_tibia_LR: origin xyz=0 -0.0645 -0.0145 rpy=-1.5707 0 3.14159 -> xyz=0 -0.0645 -0.0145 rpy=-1.5707963267948966 0 3.141592653589793
- joint j_tibia_RF: origin xyz=0 -0.0645 -0.0145 rpy=-1.5707 0 3.14159 -> xyz=0 -0.0645 -0.0145 rpy=-1.5707963267948966 0 3.141592653589793
- joint j_tibia_RM: origin xyz=0 -0.0645 -0.0145 rpy=-1.5707 0 3.14159 -> xyz=0 -0.0645 -0.0145 rpy=-1.5707963267948966 0 3.141592653589793
- joint j_tibia_RR: origin xyz=0 -0.0645 -0.0145 rpy=-1.5707 0 3.14159 -> xyz=0 -0.0645 -0.0145 rpy=-1.5707963267948966 0 3.141592653589793

File: urdf/razbot.urdf (robot description, URDF)
Before this commit: robot razbot, 27 links, 26 joints
Joints:
- joint base_joint: origin xyz=0.0 0.0 0.0 rpy=0.0 0.0 0.0 -> xyz=0 0 0 rpy=0 0 0
- joint coxa_joint_LF: limit lower=-3.14 upper=3.14 effort=6.0 velocity=0.524 -> lower=-3.141592653589793 upper=3.141592653589793 effort=6.0 velocity=5.235987755982989; origin xyz=0.0 0.0 0.0 rpy=0.0 0.0 0.5235987755982988 -> xyz=0 0 0 rpy=0.0 0.0 0.5235987755982988
- joint coxa_joint_LM: limit lower=-3.14 upper=3.14 effort=6.0 velocity=0.524 -> lower=-3.141592653589793 upper=3.141592653589793 effort=6.0 velocity=5.235987755982989; origin xyz=0.0 0.0 0.0 rpy=0.0 0.0 1.5707963267948966 -> xyz=0 0 0 rpy=0.0 0.0 1.5707963267948966
- joint coxa_joint_LR: limit lower=-3.14 upper=3.14 effort=6.0 velocity=0.524 -> lower=-3.141592653589793 upper=3.141592653589793 effort=6.0 velocity=5.235987755982989; origin xyz=0.0 0.0 0.0 rpy=0.0 0.0 2.6179938779914944 -> xyz=0 0 0 rpy=0.0 0.0 2.6179938779914944
- joint coxa_joint_RF: limit lower=-3.14 upper=3.14 effort=6.0 velocity=0.524 -> lower=-3.141592653589793 upper=3.141592653589793 effort=6.0 velocity=5.235987755982989; origin xyz=0.0 0.0 0.0 rpy=0.0 0.0 -0.5235987755982988 -> xyz=0 0 0 rpy=0.0 0.0 -0.5235987755982988
- joint coxa_joint_RM: limit lower=-3.14 upper=3.14 effort=6.0 velocity=0.524 -> lower=-3.141592653589793 upper=3.141592653589793 effort=6.0 velocity=5.235987755982989; origin xyz=0.0 0.0 0.0 rpy=0.0 0.0 -1.5707963267948966 -> xyz=0 0 0 rpy=0.0 0.0 -1.5707963267948966
- joint coxa_joint_RR: limit lower=-3.14 upper=3.14 effort=6.0 velocity=0.524 -> lower=-3.141592653589793 upper=3.141592653589793 effort=6.0 velocity=5.235987755982989; origin xyz=0.0 0.0 0.0 rpy=0.0 0.0 -2.6179938779914944 -> xyz=0 0 0 rpy=0.0 0.0 -2.6179938779914944
- joint femur_joint_LF: limit lower=-3.14 upper=3.14 effort=6.0 velocity=0.524 -> lower=-3.141592653589793 upper=3.141592653589793 effort=6.0 velocity=5.235987755982989
- joint femur_joint_LM: limit lower=-3.14 upper=3.14 effort=6.0 velocity=0.524 -> lower=-3.141592653589793 upper=3.141592653589793 effort=6.0 velocity=5.235987755982989
- joint femur_joint_LR: limit lower=-3.14 upper=3.14 effort=6.0 velocity=0.524 -> lower=-3.141592653589793 upper=3.141592653589793 effort=6.0 velocity=5.235987755982989
- joint femur_joint_RF: limit lower=-3.14 upper=3.14 effort=6.0 velocity=0.524 -> lower=-3.141592653589793 upper=3.141592653589793 effort=6.0 velocity=5.235987755982989
- joint femur_joint_RM: limit lower=-3.14 upper=3.14 effort=6.0 velocity=0.524 -> lower=-3.141592653589793 upper=3.141592653589793 effort=6.0 velocity=5.235987755982989
- joint femur_joint_RR: limit lower=-3.14 upper=3.14 effort=6.0 velocity=0.524 -> lower=-3.141592653589793 upper=3.141592653589793 effort=6.0 velocity=5.235987755982989
- joint imu_joint: origin xyz=0.0 0.0 0.0 rpy=0.0 0.0 0.0 -> xyz=0 0 0 rpy=0 0 0
- joint leg_center_joint_LF: origin xyz=0.147 0.08475 0.0 rpy=0.0 0.0 0.0 -> xyz=0.147 0.08475 0.0 rpy=0 0 0
- joint leg_center_joint_LM: origin xyz=0.0 0.17 0.0 rpy=0.0 0.0 0.0 -> xyz=0.0 0.17 0.0 rpy=0 0 0
- joint leg_center_joint_LR: origin xyz=-0.147 0.08475 0.0 rpy=0.0 0.0 0.0 -> xyz=-0.147 0.08475 0.0 rpy=0 0 0
- joint leg_center_joint_RF: origin xyz=0.147 -0.08475 0.0 rpy=0.0 0.0 0.0 -> xyz=0.147 -0.08475 0.0 rpy=0 0 0
- joint leg_center_joint_RM: origin xyz=0.0 -0.17 0.0 rpy=0.0 0.0 0.0 -> xyz=0.0 -0.17 0.0 rpy=0 0 0
- joint leg_center_joint_RR: origin xyz=-0.147 -0.08475 0.0 rpy=0.0 0.0 0.0 -> xyz=-0.147 -0.08475 0.0 rpy=0 0 0
- joint tibia_joint_LF: limit lower=-3.14 upper=3.14 effort=6.0 velocity=0.524 -> lower=-3.141592653589793 upper=3.141592653589793 effort=6.0 velocity=5.235987755982989; origin xyz=0.0 -0.065 0.0 rpy=3.141592653589793 0.0 0.0 -> xyz=0.0 -0.065 0.0 rpy=3.141592653589793 0 0
- joint tibia_joint_LM: limit lower=-3.14 upper=3.14 effort=6.0 velocity=0.524 -> lower=-3.141592653589793 upper=3.141592653589793 effort=6.0 velocity=5.235987755982989; origin xyz=0.0 -0.065 0.0 rpy=3.141592653589793 0.0 0.0 -> xyz=0.0 -0.065 0.0 rpy=3.141592653589793 0 0
- joint tibia_joint_LR: limit lower=-3.14 upper=3.14 effort=6.0 velocity=0.524 -> lower=-3.141592653589793 upper=3.141592653589793 effort=6.0 velocity=5.235987755982989; origin xyz=0.0 -0.065 0.0 rpy=3.141592653589793 0.0 0.0 -> xyz=0.0 -0.065 0.0 rpy=3.141592653589793 0 0
- joint tibia_joint_RF: limit lower=-3.14 upper=3.14 effort=6.0 velocity=0.524 -> lower=-3.141592653589793 upper=3.141592653589793 effort=6.0 velocity=5.235987755982989; origin xyz=0.0 -0.065 0.0 rpy=3.141592653589793 0.0 0.0 -> xyz=0.0 -0.065 0.0 rpy=3.141592653589793 0 0
- joint tibia_joint_RM: limit lower=-3.14 upper=3.14 effort=6.0 velocity=0.524 -> lower=-3.141592653589793 upper=3.141592653589793 effort=6.0 velocity=5.235987755982989; origin xyz=0.0 -0.065 0.0 rpy=3.141592653589793 0.0 0.0 -> xyz=0.0 -0.065 0.0 rpy=3.141592653589793 0 0
- joint tibia_joint_RR: limit lower=-3.14 upper=3.14 effort=6.0 velocity=0.524 -> lower=-3.141592653589793 upper=3.141592653589793 effort=6.0 velocity=5.235987755982989; origin xyz=0.0 -0.065 0.0 rpy=3.141592653589793 0.0 0.0 -> xyz=0.0 -0.065 0.0 rpy=3.141592653589793 0 0

File: xacro/pxm3.xacro (robot description, xacro)
@@ -252,5 +252,7 @@
   <link name="base_footprint"/>
 <!-- ****************************************************** Main Macro ***************************************************************  -->
-  <xacro:pxm3 parent="base_footprint" />
+  <xacro:pxm3 parent="base_footprint">
+    <origin xyz="0 0 0" rpy="0 0 0" />
+  </xacro:pxm3>
 <!-- ****************************************************** Gazebo Control ***********************************************************  -->
 <!-- *********************************************************************************************************************************  -->
