Commit message: u

File: urdf/kr3r540.urdf (robot description, URDF)
Before this commit: robot kr16_2, 10 links, 9 joints
Links:
- link base_link: mass 2 -> None; geometry collision mesh filename=package://robot_gazebo/meshes/kr3r540/collision/base_link.s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; visual mesh filename=package://robot_gazebo/meshes/kr3r540/visual/base_link.stl
- link link_1: mass 2 -> None; geometry collision mesh filename=package://robot_gazebo/meshes/kr3r540/collision/link_1.stl; visual mesh filename=package://robot_gazebo/meshes/kr3r540/visual/link_1.stl
- link link_2: mass 2 -> None; geometry collision mesh filename=package://robot_gazebo/meshes/kr3r540/collision/link_2.stl; visual mesh filename=package://robot_gazebo/meshes/kr3r540/visual/link_2.stl
- link link_3: mass 2 -> None; geometry collision mesh filename=package://robot_gazebo/meshes/kr3r540/collision/link_3.stl; visual mesh filename=package://robot_gazebo/meshes/kr3r540/visual/link_3.stl
- link link_4: mass 2 -> None; geometry collision mesh filename=package://robot_gazebo/meshes/kr3r540/collision/link_4.stl; visual mesh filename=package://robot_gazebo/meshes/kr3r540/visual/link_4.stl
- link link_5: mass 2 -> None; geometry collision mesh filename=package://robot_gazebo/meshes/kr3r540/collision/link_5.stl; visual mesh filename=package://robot_gazebo/meshes/kr3r540/visual/link_5.stl
- link link_6: mass 2 -> None; geometry collision mesh filename=package://robot_gazebo/meshes/kr3r540/collision/link_6.stl; visual mesh filename=package://robot_gazebo/meshes/kr3r540/visual/link_6.stl
Joints:
- removed joint joint_a6-flange
- added joint joint_a6-tool0: type fixed, parent link_6, child flange, origin xyz=0 0 0 rpy=0 0 0
- joint joint_a1: limit lower=-3.2288591161895095 upper=3.2288591161895095 effort=0 velocity=2.722713633111154 -> lower=-2.9670597283903604 upper=2.9670597283903604 effort=0 velocity=9.250245035569947; origin xyz=0 0 0.675 rpy=0 0 0 -> xyz=0 0 0.345 rpy=0 0 0
- joint joint_a2: limit lower=-2.705260340591211 upper=0.6108652381980153 effort=0 velocity=2.722713633111154 -> lower=-2.9670597283903604 upper=0.8726646259971648 effort=0 velocity=9.232791743050003; origin xyz=0.26 0 0 rpy=0 0 0 -> xyz=0.020 0 0 rpy=0 0 0
- joint joint_a3: limit lower=-2.2689280275926285 upper=2.6878070480712677 effort=0 velocity=2.722713633111154 -> lower=-1.9198621771937625 upper=2.705260340591211 effort=0 velocity=9.389871375729493; origin xyz=0.68 0 0 rpy=0 0 0 -> xyz=0.260 0 0 rpy=0 0 0
- joint joint_a4: limit lower=-6.1086523819801535 upper=6.1086523819801535 effort=0 velocity=5.759586531581287 -> lower=-3.0543261909900767 upper=3.0543261909900767 effort=0 velocity=10.471975511965978; origin xyz=0.67 0 -0.035 rpy=0 0 0 -> xyz=0 0 0.020 rpy=0 0 0
- joint joint_a5: limit lower=-2.2689280275926285 upper=2.2689280275926285 effort=0 velocity=5.759586531581287 -> lower=-2.0943951023931953 upper=2.0943951023931953 effort=0 velocity=10.471975511965978; origin xyz=0 0 0 rpy=0 0 0 -> xyz=0.260 0 0 rpy=0 0 0
- joint joint_a6: limit lower=-6.1086523819801535 upper=6.1086523819801535 effort=0 velocity=10.733774899765127 -> lower=-6.1086523819801535 upper=6.1086523819801535 effort=0 velocity=13.962634015954636; origin xyz=0 0 0 rpy=0 0 0 -> xyz=0.075 0 0 rpy=0 0 0

Commit message: u

File: urdf/kr3r540.urdf (robot description, URDF)
Before this commit: robot kr3r540, 10 links, 9 joints
Links:
- link base_link: mass None -> 1.0
- link link_1: mass None -> 1.0
- link link_2: mass None -> 1.0
- link link_3: mass None -> 1.0
- link link_4: mass None -> 1.0
- link link_5: mass None -> 1.0
- link link_6: mass None -> 1.0

File: xacro/kr3r540.xacro (robot description, xacro)
@@ -8,4 +8,12 @@
 <!-- ****************************************************** base link **************************************************************** -->
     <link name="${prefix}base_link">
+      <inertial>
+        <origin xyz="0 0 0" rpy="0 0 0" />
+        <mass value="1.0" />
+        <inertia
+            ixx="0" ixy="0" ixz="0"
+            iyy="0" iyz="0"
+            izz="0" />
+      </inertial>
       <visual>
         <origin xyz="0 0 0" rpy="0 0 0" />
@@ -23,8 +31,16 @@
     </link>
     <gazebo reference="${prefix}base_link">
-      <material>Gazebo/Orange</material>
+      <material>Gazebo/Gray</material>
     </gazebo>
 <!-- ****************************************************** link 1 (A1) **************************************************************** -->
     <link name="${prefix}link_1">
+      <inertial>
+        <origin xyz="0 0 0" rpy="0 0 0" />
+        <mass value="1.0" />
+        <inertia
+            ixx="0" ixy="0" ixz="0"
+            iyy="0" iyz="0"
+            izz="0" />
+      </inertial>
       <visual>
         <origin xyz="0 0 0" rpy="0 0 0" />
@@ -46,4 +62,12 @@
 <!-- ****************************************************** link 2 **************************************************************** -->
     <link name="${prefix}link_2">
+      <inertial>
+        <origin xyz="0 0 0" rpy="0 0 0" />
+        <mass value="1.0" />
+        <inertia
+            ixx="0" ixy="0" ixz="0"
+            iyy="0" iyz="0"
+            izz="0" />
+      </inertial>
       <visual>
         <origin xyz="0 0 0" rpy="0 0 0" />
@@ -65,4 +89,12 @@
 <!-- ****************************************************** link 2 **************************************************************** -->
     <link name="${prefix}link_3">
+      <inertial>
+        <origin xyz="0 0 0" rpy="0 0 0" />
+        <mass value="1.0" />
+        <inertia
+            ixx="0" ixy="0" ixz="0"
+            iyy="0" iyz="0"
+            izz="0" />
+      </inertial>
       <visual>
         <origin xyz="0 0 0" rpy="0 0 0" />
@@ -84,4 +116,12 @@
 <!-- ****************************************************** link 4 **************************************************************** -->
     <link name="${prefix}link_4">
+      <inertial>
+        <origin xyz="0 0 0" rpy="0 0 0" />
+        <mass value="1.0" />
+        <inertia
+            ixx="0" ixy="0" ixz="0"
+            iyy="0" iyz="0"
+            izz="0" />
+      </inertial>
       <visual>
         <origin xyz="0 0 0" rpy="0 0 0" />
@@ -103,4 +143,12 @@
 <!-- ****************************************************** link 5 **************************************************************** -->
     <link name="${prefix}link_5">
+      <inertial>
+        <origin xyz="0 0 0" rpy="0 0 0" />
+        <mass value="1.0" />
+        <inertia
+            ixx="0" ixy="0" ixz="0"
+            iyy="0" iyz="0"
+            izz="0" />
+      </inertial>
       <visual>
         <origin xyz="0 0 0" rpy="0 0 0" />
@@ -122,4 +170,12 @@
 <!-- ****************************************************** link 6 **************************************************************** -->
     <link name="${prefix}link_6">
+      <inertial>
+        <origin xyz="0 0 0" rpy="0 0 0" />
+        <mass value="1.0" />
+        <inertia
+            ixx="0" ixy="0" ixz="0"
+            iyy="0" iyz="0"
+            izz="0" />
+      </inertial>
       <visual>
         <origin xyz="0 0 0" rpy="0 0 0" />
@@ -137,5 +193,5 @@
     </link>
     <gazebo reference="${prefix}link_6">
-      <material>Gazebo/Orange</material>
+      <material>Gazebo/Gray</material>
     </gazebo>
 <!-- ****************************************************** tool 0 ******************************************************************* -->

File: xacro/kr5_arc.xacro (robot description, xacro)
@@ -33,5 +33,5 @@
     </link>
     <gazebo reference="${prefix}base_link">
-      <material>Gazebo/Orange</material>
+      <material>Gazebo/Gray</material>
     </gazebo>
 <!-- ****************************************************** link 1 (A1) **************************************************************** -->
@@ -225,5 +225,5 @@
     </link>
     <gazebo reference="${prefix}link_6">
-      <material>Gazebo/Orange</material>
+      <material>Gazebo/Gray</material>
     </gazebo>
 <!-- ****************************************************** tool 0 ******************************************************************* -->
