Commit message: fix to world

File: urdf/kr3r540.urdf (robot description, URDF)
Before this commit: robot kr3r540, 10 links, 9 joints
Links:
- added link world
Joints:
- added joint base_joint: type fixed, parent world, child base_link, origin xyz=0 0 0 rpy=0 0 0

File: xacro/kr120r2500pro.xacro (robot description, xacro)
@@ -4,5 +4,5 @@
   <xacro:property name="mesh_path"        value="package://robot_gazebo/meshes/kr120r2500pro/"/>
 <!-- ****************************************************** Macro ******************************************************************** -->
-  <xacro:macro name="kuka_kr120r2500pro" params="prefix">
+  <xacro:macro name="kuka_kr120r2500pro" params="parent prefix">
 <!-- ****************************************************** LINKS ******************************************************************** -->
 <!-- ****************************************************** base link **************************************************************** -->
@@ -151,4 +151,10 @@
 <!-- ****************************************************** END LINKS **************************************************************** -->
 <!-- ****************************************************** JOINTS ******************************************************************* -->
+<!-- ****************************************************** Base Joint *************************************************************** -->
+    <joint name="${prefix}base_joint" type="fixed">
+      <origin xyz="0 0 0" rpy="0 0 0" />
+      <parent link="${parent}"/>
+      <child link="${prefix}base_link" />
+    </joint>
 <!-- ****************************************************** joint 1 (A1) ************************************************************* -->
     <joint name="${prefix}joint_a1" type="revolute">
@@ -159,5 +165,5 @@
       <limit effort="0" lower="${-radians(185)}" upper="${radians(185)}" velocity="${radians(156)}"/>
     </joint>
-<!-- ****************************************************** joint 2 (A2) **************************************************************** -->
+<!-- ****************************************************** joint 2 (A2) ************************************************************* -->
     <joint name="${prefix}joint_a2" type="revolute">
       <origin xyz="0.35 0 0" rpy="0 0 0"/>
@@ -167,5 +173,5 @@
       <limit effort="0" lower="${-radians(155)}" upper="${radians(35)}" velocity="${radians(156)}"/>
     </joint>
-<!-- ****************************************************** joint 3 (A3) **************************************************************** -->
+<!-- ****************************************************** joint 3 (A3) ************************************************************* -->
     <joint name="${prefix}joint_a3" type="revolute">
       <origin xyz="1.150 0 0" rpy="0 0 0"/>
@@ -175,5 +181,5 @@
       <limit effort="0" lower="${-radians(130)}" upper="${radians(154)}" velocity="${radians(156)}"/>
     </joint>
-<!-- ****************************************************** joint 4 (A4) **************************************************************** -->
+<!-- ****************************************************** joint 4 (A4) ************************************************************* -->
     <joint name="${prefix}joint_a4" type="revolute">
       <origin xyz="1.0 0 -0.041" rpy="0 0 0"/>
@@ -183,5 +189,5 @@
       <limit effort="0" lower="${-radians(350)}" upper="${radians(350)}" velocity="${radians(330)}"/>
     </joint>
-<!-- ****************************************************** joint 5 (A5) **************************************************************** -->
+<!-- ****************************************************** joint 5 (A5) ************************************************************* -->
     <joint name="${prefix}joint_a5" type="revolute">
       <origin xyz="0 0 0" rpy="0 0 0"/>
@@ -191,5 +197,5 @@
       <limit effort="0" lower="${-radians(130)}" upper="${radians(130)}" velocity="${radians(330)}"/>
     </joint>
-<!-- ****************************************************** joint 6 (A6) **************************************************************** -->
+<!-- ****************************************************** joint 6 (A6) ************************************************************* -->
     <joint name="${prefix}joint_a6" type="revolute">
       <origin xyz="0 0 0" rpy="0 0 0"/>
@@ -199,5 +205,5 @@
       <limit effort="0" lower="${-radians(350)}" upper="${radians(350)}" velocity="${radians(615)}"/>
     </joint>
-<!-- ****************************************************** tool frame - fixed frame ********************************************* -->
+<!-- ****************************************************** tool frame - fixed frame ************************************************* -->
     <joint name="${prefix}joint_a6-flange" type="fixed">
       <parent link="${prefix}link_6"/>
@@ -205,6 +211,6 @@
       <origin xyz="0.215 0 0" rpy="0 0 0"/>
     </joint>
-<!-- ****************************************************** END JOINTS *********************************************************** -->
-<!-- ****************************************************** ROS base_link to KUKA $ROBROOT coordinate system transform *********** -->
+<!-- ****************************************************** END JOINTS *************************************************************** -->
+<!-- ****************************************************** ROS base_link to KUKA $ROBROOT coordinate system transform *************** -->
    <link name="${prefix}base" />
     <joint name="${prefix}base_link-base" type="fixed">
@@ -213,5 +219,5 @@
       <child link="${prefix}base"/>
     </joint>
-<!-- ***************** This frame corresponds to the $TOOL coordinate system in KUKA KRC controllers ***************************** -->
+<!-- ***************** This frame corresponds to the $TOOL coordinate system in KUKA KRC controllers ********************************* -->
     <link name="${prefix}tool0" />
     <joint name="${prefix}flange-tool0" type="fixed">
@@ -222,6 +228,11 @@
 <!-- ****************************************************** End Macro **************************************************************** -->
   </xacro:macro>
+<!-- ****************************************************** World Link *************************************************************** -->
+  <link name="world"/>
+  <gazebo reference="world">
+    <static>true</static>
+  </gazebo>
 <!-- ****************************************************** Generates a urdf from macro ********************************************** -->
-  <xacro:kuka_kr120r2500pro prefix=""/>
+  <xacro:kuka_kr120r2500pro parent="world" prefix=""/>
 <!-- ****************************************************** End ********************************************************************** -->
 </robot>

File: xacro/kr16_2.xacro (robot description, xacro)
@@ -4,5 +4,5 @@
   <xacro:property name="mesh_path"        value="package://robot_gazebo/meshes/kr16_2/"/>
 <!-- ****************************************************** Macro ******************************************************************** -->
-  <xacro:macro name="kuka_kr16_2" params="prefix">
+  <xacro:macro name="kuka_kr16_2" params="parent prefix">
 <!-- ****************************************************** LINKS ******************************************************************** -->
 <!-- ****************************************************** base link **************************************************************** -->
@@ -151,4 +151,10 @@
 <!-- ****************************************************** END LINKS **************************************************************** -->
 <!-- ****************************************************** JOINTS ******************************************************************* -->
+<!-- ****************************************************** Base Joint ***************************************************************  -->
+    <joint name="${prefix}base_joint" type="fixed">
+      <origin xyz="0 0 0" rpy="0 0 0" />
+      <parent link="${parent}"/>
+      <child link="${prefix}base_link" />
+    </joint>
 <!-- ****************************************************** joint 1 (A1) ************************************************************* -->
     <joint name="${prefix}joint_a1" type="revolute">
@@ -222,6 +228,11 @@
 <!-- ****************************************************** End Macro **************************************************************** -->
   </xacro:macro>
+<!-- ****************************************************** World Link *************************************************************** -->
+  <link name="world"/>
+  <gazebo reference="world">
+    <static>true</static>
+  </gazebo>
 <!-- ****************************************************** Generates a urdf from macro ********************************************** -->
-<xacro:kuka_kr16_2 prefix=""/>
+<xacro:kuka_kr16_2 parent="world" prefix=""/>
 <!-- ****************************************************** End ********************************************************************** -->
 </robot>

File: xacro/kr3r540.xacro (robot description, xacro)
@@ -5,5 +5,5 @@
   <xacro:property name="mesh_path" value="package://robot_gazebo/meshes/kr3r540/"/>
 <!-- ****************************************************** Macro ******************************************************************** -->
-  <xacro:macro name="kuka_kr3r540" params="prefix">
+  <xacro:macro name="kuka_kr3r540" params="parent prefix">
 <!-- ****************************************************** LINKS ******************************************************************** -->
 <!-- ****************************************************** base link **************************************************************** -->
@@ -201,4 +201,10 @@
 <!-- ****************************************************** END LINKS **************************************************************** -->
 <!-- ****************************************************** JOINTS ******************************************************************* -->
+<!-- ****************************************************** Base Joint ***************************************************************  -->
+    <joint name="${prefix}base_joint" type="fixed">
+      <origin xyz="0 0 0" rpy="0 0 0" />
+      <parent link="${parent}"/>
+      <child link="${prefix}base_link" />
+    </joint>
 <!-- ****************************************************** joint 1 (A1) ************************************************************* -->
     <joint name="${prefix}joint_a1" type="revolute">
@@ -272,6 +278,11 @@
 <!-- ****************************************************** End Macro **************************************************************** -->
   </xacro:macro>
+<!-- ****************************************************** World Link *************************************************************** -->
+  <link name="world"/>
+  <gazebo reference="world">
+    <static>true</static>
+  </gazebo>
 <!-- ****************************************************** Generates a urdf from macro ********************************************** -->
-  <xacro:kuka_kr3r540 prefix=""/>
+  <xacro:kuka_kr3r540 parent="world" prefix=""/>
 <!-- ****************************************************** End ********************************************************************** -->
 </robot>

File: xacro/kr5_arc.xacro (robot description, xacro)
@@ -4,5 +4,5 @@
   <xacro:property name="mesh_path"        value="package://robot_gazebo/meshes/kr5_arc/"/>
 <!-- ****************************************************** Macro ******************************************************************** -->
-  <xacro:macro name="kuka_kr5_arc" params="prefix">
+  <xacro:macro name="kuka_kr5_arc" params="parent prefix">
 <!-- ****************************************************** LINKS ******************************************************************** -->
 <!-- ****************************************************** base link **************************************************************** -->
@@ -233,4 +233,10 @@
 <!-- ****************************************************** END LINKS **************************************************************** -->
 <!-- ****************************************************** JOINTS ******************************************************************* -->
+<!-- ****************************************************** Base Joint ***************************************************************  -->
+    <joint name="${prefix}base_joint" type="fixed">
+      <origin xyz="0 0 0" rpy="0 0 0" />
+      <parent link="${parent}"/>
+      <child link="${prefix}base_link" />
+    </joint>
 <!-- ****************************************************** joint 1 (A1) ************************************************************* -->
     <joint name="${prefix}joint_a1" type="revolute">
@@ -304,4 +310,9 @@
 <!-- ****************************************************** End Macro **************************************************************** -->
   </xacro:macro>
+<!-- ****************************************************** World Link *************************************************************** -->
+  <link name="world"/>
+  <gazebo reference="world">
+    <static>true</static>
+  </gazebo>
 <!-- ****************************************************** Generates a urdf from macro ********************************************** -->
   <xacro:kuka_kr5_arc prefix=""/>

File: xacro/lbr_iiwa_14_r820.xacro (robot description, xacro)
@@ -171,4 +171,10 @@
 <!-- ****************************************************** END LINKS **************************************************************** -->
 <!-- ****************************************************** JOINTS ******************************************************************* -->
+<!-- ****************************************************** Base Joint *************************************************************** -->
+    <joint name="${prefix}base_joint" type="fixed">
+      <origin xyz="0 0 0" rpy="0 0 0" />
+      <parent link="${parent}"/>
+      <child link="${prefix}base_link" />
+    </joint>
 <!-- ****************************************************** joint 1 (A1) ************************************************************* -->
     <joint name="${prefix}joint_a1" type="revolute">
@@ -244,6 +250,11 @@
 <!-- ****************************************************** End Macro **************************************************************** -->
   </xacro:macro>
+<!-- ****************************************************** World Link *************************************************************** -->
+  <link name="world"/>
+  <gazebo reference="world">
+    <static>true</static>
+  </gazebo>
 <!-- ****************************************************** Generates a urdf from macro ********************************************** -->
-  <xacro:kuka_lbr_iiwa_14_r820 prefix=""/>
+  <xacro:kuka_lbr_iiwa_14_r820 parent="world" prefix=""/>
 <!-- ****************************************************** End ********************************************************************** -->
 </robot>
