Commit message: u

File: urdf/kr120r2500pro.urdf (robot description, URDF)
Before this commit: robot kr120r2500pro, 10 links, 9 joints
Links:
- added link world
Joints:
- added joint base_joint: type fixed, parent world, child base_link, origin xyz=0 0 0 rpy=0 0 0

File: urdf/kr16_2.urdf (robot description, URDF)
Before this commit: robot kr16_2, 10 links, 9 joints
Links:
- added link world
Joints:
- added joint base_joint: type fixed, parent world, child base_link, origin xyz=0 0 0 rpy=0 0 0

File: urdf/kr5_arc.urdf (robot description, URDF)
Before this commit: robot kr5_arc, 10 links, 9 joints
Links:
- added link world
Joints:
- added joint base_joint: type fixed, parent world, child base_link, origin xyz=0 0 0 rpy=0 0 0

File: urdf/lbr_iiwa_14_r820.urdf (robot description, URDF)
Before this commit: robot lbr_iiwa_14_r820, 10 links, 9 joints
Links:
- added link world
Joints:
- added joint base_joint: type fixed, parent world, child base_link, origin xyz=0 0 0 rpy=0 0 0

File: xacro/kr5_arc.xacro (robot description, xacro)
@@ -316,5 +316,5 @@
   </gazebo>
 <!-- ****************************************************** Generates a urdf from macro ********************************************** -->
-  <xacro:kuka_kr5_arc prefix=""/>
+  <xacro:kuka_kr5_arc parent="world" prefix=""/>
 <!-- ****************************************************** End ********************************************************************** -->
 </robot>

File: xacro/lbr_iiwa_14_r820.xacro (robot description, xacro)
@@ -4,5 +4,5 @@
   <xacro:property name="mesh_path"        value="package://robot_gazebo/meshes/lbr_iiwa_14_r820/"/>
 <!-- ****************************************************** Macro ******************************************************************** -->
-  <xacro:macro name="kuka_lbr_iiwa_14_r820" params="prefix">
+  <xacro:macro name="kuka_lbr_iiwa_14_r820" params="parent prefix">
 <!-- ****************************************************** LINKS ******************************************************************** -->
 <!-- ****************************************************** base link **************************************************************** -->
