Commit message: u

File: urdf/bocbot.urdf (robot description, URDF)
Before this commit: robot bocbot, 8 links, 7 joints
Links:
- link back_left_wheel: mass 5.0 -> 15.0
- link back_right_wheel: mass 5.0 -> 15.0
- link base: geometry collision mesh filename=package://robot_gazebo/meshes/bocbot/base.stl scale=1 1 1; visual mesh filename=package://robot_gazebo/meshes/bocbot/base.stl scale=1 1 1
- link front_left_wheel: mass 5.0 -> 15.0
- link front_right_wheel: mass 5.0 -> 15.0

File: xacro/bocbot.xacro (robot description, xacro)
@@ -7,5 +7,5 @@
 <!-- ****************************************************** Parameters ***************************************************************  -->
   <xacro:property name="mesh_path"      value="package://robot_gazebo/meshes/bocbot/"/>
-  <xacro:property name="base_mass"      value="15.0"                              />
+  <xacro:property name="base_mass"      value="15.0"                              /> <!-- arbitrary mass value                          -->
   <xacro:property name="base_width"     value="0.20"                              />
   <xacro:property name="base_length"    value="0.40"                              />
@@ -13,5 +13,13 @@
   <xacro:property name="wheel_mass"     value="5.0"                               />
   <xacro:property name="wheel_width"    value="0.05"                              />
-  <xacro:property name="wheel_radius"   value="0.01"                              />
+  <xacro:property name="wheel_radius"   value="0.10"                              />
+  <xacro:property name="camera_mass"    value="0.1"                               />
+  <xacro:property name="camera_width"   value="0.05"                              />
+  <xacro:property name="camera_length"  value="0.05"                              />
+  <xacro:property name="camera_height"  value="0.05"                              />
+  <xacro:property name="hokuyo_mass"    value="1e-5"                              />
+  <xacro:property name="hokuyo_width"   value="0.05"                              />
+  <xacro:property name="hokuyo_length"  value="0.05"                              />
+  <xacro:property name="hokuyo_height"  value="0.080165"                          />
   <xacro:property name="y_offset"       value="${(base_width+wheel_width*1.2)/2}" />
   <xacro:property name="z_offset"       value="${base_height/2}"                  />
@@ -130,6 +138,6 @@
   <link name="camera">
     <inertial>
-      <mass value="0.1"/>
-      <origin xyz="0.05 0.05 0.05" rpy=" 0 0 0"/>
+      <mass value="${camera_mass}"/>
+      <origin xyz="0 0 0" rpy=" 0 0 0"/>
       <inertia ixx="1e-6" ixy="0" ixz="0" iyy="1e-6" iyz="0" izz="1e-6" />
     </inertial>
@@ -137,5 +145,5 @@
       <origin xyz="0 0 0" rpy="0 0 0" />
       <geometry>
-        <box size="0.05 0.05 0.05"/>
+        <box size="${camera_length} ${camera_width} ${camera_height}"/>
       </geometry>
       <material name="green"/>
@@ -144,5 +152,5 @@
       <origin xyz="0 0 0" rpy="0 0 0" />
       <geometry>
-        <box size="0.05 0.05 0.05"/>
+        <box size="${camera_length} ${camera_width} ${camera_height}"/>
       </geometry>
     </collision>
@@ -151,5 +159,5 @@
   <link name="hokuyo">
     <inertial>
-      <mass value="1e-5"/>
+      <mass value="${hokuyo_mass}"/>
       <origin xyz="0 0 0" rpy=" 0 0 0"/>
       <inertia ixx="1e-6" ixy="0" ixz="0" iyy="1e-6" iyz="0" izz="1e-6" />
@@ -158,6 +166,5 @@
       <origin xyz="0 0 0" rpy="0 0 0" />
       <geometry>
-        <mesh filename="${mesh_path}hokuyo.dae"/>
-        <!-- <box size="0.05 0.05 0.05"/> -->
+        <mesh filename="${mesh_path}hokuyo.dae"/> <!--  <box size="${hokuyo_length} ${hokuyo_width} ${hokuyo_height}"/> -->
       </geometry>
       <material name="red"/>
@@ -166,5 +173,5 @@
       <origin xyz="0 0 0" rpy="0 0 0" />
       <geometry>
-        <box size="0.1 0.1 0.1"/>
+        <mesh filename="${mesh_path}hokuyo.dae"/> <!--  <box size="${hokuyo_length} ${hokuyo_width} ${hokuyo_height}"/> -->
       </geometry>
     </collision>
