Commit message: u

File: urdf/diffbot.urdf (robot description, URDF)
Before this commit: robot diffbot, 5 links, 4 joints
Links:
- added link base_footprint
Joints:
- added joint base_joint: type fixed, parent base_footprint, child base_link, origin xyz=0.0 0.0 0.0 rpy=0.0 0.0 0.0

File: xacro/diffbot.xacro (robot description, xacro)
@@ -21,4 +21,12 @@
 <!-- ****************************************************** Macro ********************************************************************  -->
   <xacro:macro name="diffbot" params="prefix">
+<!-- ****************************************************** Base Footprint ***********************************************************  -->
+    <link name="base_footprint"/>
+<!-- ****************************************************** Base Joint ***************************************************************  -->
+    <joint name="base_joint" type="fixed">
+        <parent link="base_footprint"/>
+        <child link="${prefix}base_link"/>
+        <origin xyz="0.0 0.0 0.0" rpy="0.0 0.0 0.0"/>
+    </joint>
 <!-- ****************************************************** Base Link ****************************************************************  -->
   <link name="${prefix}base_link">

Commit message: u

File: urdf/diffbot.urdf (robot description, URDF)
Before this commit: robot diffbot, 6 links, 5 joints
Links:
- link base_link: geometry collision box size=0.2 0.1 0.05; visual box size=0.2 0.1 0.05
- link front_caster: geometry collision sphere radius=0.025; visual sphere radius=0.025
- link left_wheel: geometry collision cylinder length=0.01 radius=0.025; visual cylinder length=0.01 radius=0.025
- link rear_caster: geometry collision sphere radius=0.025; visual sphere radius=0.025
- link right_wheel: geometry collision cylinder length=0.01 radius=0.025; visual cylinder length=0.01 radius=0.025
Joints:
- joint base_joint: origin xyz=0.0 0.0 0.0 rpy=0.0 0.0 0.0 -> xyz=0.0 0.0 0.05 rpy=0.0 0.0 0.0
- joint front_caster_joint: origin xyz=0.0 0 -0.025 rpy=0 0 0 -> xyz=0.07500000000000001 0 -0.025 rpy=0 0 0
- joint left_wheel_joint: origin xyz=0 -0.060000000000000005 -0.025 rpy=0 0 0 -> xyz=0 -0.055 -0.025 rpy=0 0 0
- joint rear_caster_joint: origin xyz=0.0 0 -0.025 rpy=0 0 0 -> xyz=-0.07500000000000001 0 -0.025 rpy=0 0 0
- joint right_wheel_joint: origin xyz=0 0.060000000000000005 -0.025 rpy=0 0 0 -> xyz=0 0.055 -0.025 rpy=0 0 0

File: urdf/twr.urdf (robot description, URDF)
Before this commit: robot twr, 7 links, 6 joints
Joints:
- joint drivewhl_l_joint: limit lower=-3.1415 upper=3.1415 effort=30 velocity=5.0 -> lower=-3.141592653589793 upper=3.141592653589793 effort=30 velocity=5.0
- joint drivewhl_r_joint: limit lower=-3.1415 upper=3.1415 effort=30 velocity=5.0 -> lower=-3.141592653589793 upper=3.141592653589793 effort=30 velocity=5.0

File: xacro/diffbot.xacro (robot description, xacro)
@@ -15,5 +15,5 @@
   <xacro:property name="caster_wheel_mass"    value="0.1"               /> <!-- arbitrary value for caster wheel mass     -->
   <xacro:property name="caster_wheel_radius"  value="${wheel_radius}"   />
-  <xacro:property name="z_offset"             value="-${base_height/2}" /> <!-- Space btw top of beam and the each joint  -->
+  <xacro:property name="z_offset"             value="${base_height/2}" /> <!-- Space btw top of beam and the each joint  -->
 <!-- ****************************************************** Includes *****************************************************************  -->
   <xacro:include filename="$(find robot_gazebo)/xacro/common_rviz_materials.xacro" />   <!-- RVIZ Colors                                -->
@@ -27,5 +27,5 @@
         <parent link="base_footprint"/>
         <child link="${prefix}base_link"/>
-        <origin xyz="0.0 0.0 0.0" rpy="0.0 0.0 0.0"/>
+        <origin xyz="0.0 0.0 ${(wheel_radius+z_offset)}" rpy="0.0 0.0 0.0"/>
     </joint>
 <!-- ****************************************************** Base Link ****************************************************************  -->
@@ -34,5 +34,5 @@
       <origin xyz="0 0 0" rpy="0 0 0"/>
       <geometry>
-        <box size="${base_width} ${base_length} ${base_height}"/>
+        <box size="${base_length} ${base_width} ${base_height}"/>
       </geometry>
     </collision>
@@ -57,5 +57,5 @@
       <parent link="${prefix}base_link"/>
       <child link="${prefix}left_wheel"/>
-      <origin xyz="0 -${(base_width+wheel_width)/2} ${z_offset}" rpy="0 0 0"/>
+      <origin xyz="0 -${(base_width+wheel_width)/2} ${-z_offset}" rpy="0 0 0"/>
       <axis xyz="0 1 0"/>
       <dynamics damping="0.2"/>
@@ -64,5 +64,5 @@
     <link name="${prefix}left_wheel">
       <collision>
-        <origin xyz="0 0 0" rpy="${pi/2} 0 0"/>
+        <origin xyz="0 0 0" rpy="${radians(90)} 0 0"/>
         <geometry>
           <cylinder length="${wheel_width}" radius="${wheel_radius}"/>
@@ -70,5 +70,5 @@
       </collision>
       <visual>
-        <origin xyz="0 0 0" rpy="${pi/2} 0 0"/>
+        <origin xyz="0 0 0" rpy="${radians(90)} 0 0"/>
         <geometry>
           <cylinder length="${wheel_width}" radius="${wheel_radius}"/>
@@ -77,5 +77,5 @@
       </visual>
       <inertial>
-        <origin xyz="0 0 0" rpy="${pi/2} 0 0"/>
+        <origin xyz="0 0 0" rpy="${radians(90)} 0 0"/>
         <mass value="${wheel_mass}"/>
         <inertia
@@ -89,5 +89,5 @@
       <parent link="${prefix}base_link"/>
       <child link="${prefix}right_wheel"/>
-      <origin xyz="0 ${(base_width+wheel_width)/2} ${z_offset}" rpy="0 0 0"/>
+      <origin xyz="0 ${(base_width+wheel_width)/2} ${-z_offset}" rpy="0 0 0"/>
       <axis xyz="0 1 0"/>
       <dynamics damping="0.2"/>
@@ -96,5 +96,5 @@
     <link name="${prefix}right_wheel">
       <collision>
-        <origin xyz="0 0 0" rpy="${pi/2} 0 0"/>
+        <origin xyz="0 0 0" rpy="${radians(90)} 0 0"/>
         <geometry>
           <cylinder length="${wheel_width}" radius="${wheel_radius}"/>
@@ -102,5 +102,5 @@
       </collision>
       <visual>
-        <origin xyz="0 0 0" rpy="${pi/2} 0 0"/>
+        <origin xyz="0 0 0" rpy="${radians(90)} 0 0"/>
         <geometry>
           <cylinder length="${wheel_width}" radius="${wheel_radius}"/>
@@ -109,5 +109,5 @@
       </visual>
       <inertial>
-        <origin xyz="0 0 0" rpy="${pi/2} 0 0"/>
+        <origin xyz="0 0 0" rpy="${radians(90)} 0 0"/>
         <mass value="${wheel_mass}"/>
         <inertia
@@ -121,5 +121,5 @@
       <parent link="${prefix}base_link"/>
       <child link="${prefix}front_caster"/>
-      <origin xyz="${base_length/2 - caster_wheel_radius} 0 ${z_offset}" rpy="0 0 0"/>
+      <origin xyz="${base_length/2 - caster_wheel_radius} 0 ${-z_offset}" rpy="0 0 0"/>
     </joint>
 <!-- ****************************************************** Front caster Link ********************************************************  -->
@@ -151,5 +151,5 @@
       <parent link="${prefix}base_link"/>
       <child link="${prefix}rear_caster"/>
-      <origin xyz="${-base_length/2 + caster_wheel_radius} 0 ${z_offset}" rpy="0 0 0"/>
+      <origin xyz="${-base_length/2 + caster_wheel_radius} 0 ${-z_offset}" rpy="0 0 0"/>
     </joint>
 <!-- ****************************************************** Rear Caster Link *********************************************************  -->

File: xacro/twr.xacro (robot description, xacro)
@@ -13,5 +13,4 @@
   <xacro:property name="wheel_radius" value="0.14"/>
   <xacro:property name="wheel_width"  value="0.06"/>
-<!-- x-axis points forward, y-axis points to left, z-axis points upwards                                                                -->
   <xacro:property name="wheel_ygap"   value="0.035"/> <!-- gap between the wheel and chassis along y-axis in meters                     -->
   <xacro:property name="wheel_zoff"   value="0.05" /> <!-- Position the wheels along the z-axis                                         -->
@@ -80,10 +79,10 @@
       </visual>
       <collision>
-        <origin xyz="0 0 0" rpy="${pi/2} 0 0"/>
+        <origin xyz="0 0 0" rpy="${radians(90)} 0 0"/>
         <geometry>
           <cylinder radius="${wheel_radius}" length="${wheel_width}"/>
         </geometry>
       </collision>
-      <xacro:cylinder_inertia m="110.5" r="${wheel_radius}" h="${wheel_width}"/>
+        <xacro:cylinder_inertia m="110.5" r="${wheel_radius}" h="${wheel_width}"/>
     </link>
 <!-- ****************************************************** Drive Wheels Joint Macro *************************************************  -->
@@ -94,7 +93,8 @@
       <child link="${prefix}_link"/>
       <origin xyz="${x_reflect*wheel_xoff} ${y_reflect*(base_width/2+wheel_ygap)} ${-wheel_zoff}" rpy="0 0 0"/>
-      <limit upper="3.1415" lower="-3.1415" effort="30" velocity="5.0"/>
+      <limit upper="${radians(180)}" lower="-${radians(180)}" effort="30" velocity="5.0"/>
       <axis xyz="0 1 0"/>
     </joint>
+<!-- ****************************************************** End of Macro *************************************************************  -->
   </xacro:macro>
 <!-- ****************************************************** Drive Wheels Link and Joint **********************************************  -->

Commit message: u

File: urdf/diffbot.urdf (robot description, URDF)
Before this commit: robot diffbot, 6 links, 5 joints
Joints:
- joint left_wheel_joint: limit (none) -> lower=-3.141592653589793 upper=3.141592653589793 effort=30 velocity=5.0
- joint right_wheel_joint: limit (none) -> lower=-3.141592653589793 upper=3.141592653589793 effort=30 velocity=5.0

File: xacro/diffbot.xacro (robot description, xacro)
@@ -6,14 +6,14 @@
 <!-- *********************************************************************************************************************************  -->
 <!-- ****************************************************** Parameters ***************************************************************  -->
-  <xacro:property name="base_mass"            value="0.3"               /> <!-- arbitrary value for base mass             -->
-  <xacro:property name="base_width"           value="0.10"              />
-  <xacro:property name="base_length"          value="0.20"              />
-  <xacro:property name="base_height"          value="0.05"              />
-  <xacro:property name="wheel_mass"           value="0.3"               /> <!-- arbitrary value for wheel mass            -->
-  <xacro:property name="wheel_width"          value="0.010"             />
-  <xacro:property name="wheel_radius"         value="0.025"             />
-  <xacro:property name="caster_wheel_mass"    value="0.1"               /> <!-- arbitrary value for caster wheel mass     -->
-  <xacro:property name="caster_wheel_radius"  value="${wheel_radius}"   />
-  <xacro:property name="z_offset"             value="${base_height/2}" /> <!-- Space btw top of beam and the each joint  -->
+  <xacro:property name="base_mass"      value="0.3"               /> <!-- arbitrary value for base mass             -->
+  <xacro:property name="base_width"     value="0.10"              />
+  <xacro:property name="base_length"    value="0.20"              />
+  <xacro:property name="base_height"    value="0.05"              />
+  <xacro:property name="wheel_mass"     value="0.3"               /> <!-- arbitrary value for wheel mass            -->
+  <xacro:property name="wheel_width"    value="0.010"             />
+  <xacro:property name="wheel_radius"   value="0.025"             />
+  <xacro:property name="caster_mass"    value="0.1"               /> <!-- arbitrary value for caster wheel mass     -->
+  <xacro:property name="caster_radius"  value="${wheel_radius}"   />
+  <xacro:property name="z_offset"       value="${base_height/2}" /> <!-- Space btw top of beam and the each joint  -->
 <!-- ****************************************************** Includes *****************************************************************  -->
   <xacro:include filename="$(find robot_gazebo)/xacro/common_rviz_materials.xacro" />   <!-- RVIZ Colors                                -->
@@ -58,4 +58,5 @@
       <child link="${prefix}left_wheel"/>
       <origin xyz="0 -${(base_width+wheel_width)/2} ${-z_offset}" rpy="0 0 0"/>
+      <limit upper="${radians(180)}" lower="-${radians(180)}" effort="30" velocity="5.0"/>
       <axis xyz="0 1 0"/>
       <dynamics damping="0.2"/>
@@ -90,4 +91,5 @@
       <child link="${prefix}right_wheel"/>
       <origin xyz="0 ${(base_width+wheel_width)/2} ${-z_offset}" rpy="0 0 0"/>
+      <limit upper="${radians(180)}" lower="-${radians(180)}" effort="30" velocity="5.0"/>
       <axis xyz="0 1 0"/>
       <dynamics damping="0.2"/>
@@ -121,5 +123,5 @@
       <parent link="${prefix}base_link"/>
       <child link="${prefix}front_caster"/>
-      <origin xyz="${base_length/2 - caster_wheel_radius} 0 ${-z_offset}" rpy="0 0 0"/>
+      <origin xyz="${base_length/2 - caster_radius} 0 ${-z_offset}" rpy="0 0 0"/>
     </joint>
 <!-- ****************************************************** Front caster Link ********************************************************  -->
@@ -128,5 +130,5 @@
         <origin xyz="0 0 0" rpy="0 0 0"/>
         <geometry>
-          <sphere radius="${caster_wheel_radius}"/>
+          <sphere radius="${caster_radius}"/>
         </geometry>
       </collision>
@@ -134,5 +136,5 @@
         <origin xyz="0 0 0" rpy="0 0 0"/>
         <geometry>
-          <sphere radius="${caster_wheel_radius}"/>
+          <sphere radius="${caster_radius}"/>
         </geometry>
         <material name="white"/>
@@ -140,9 +142,9 @@
       <inertial>
         <origin xyz="0 0 0" rpy="0 0 0"/>
-        <mass value="${caster_wheel_mass}"/>
+        <mass value="${caster_mass}"/>
         <inertia
-          ixx="${caster_wheel_mass * 0.4 * (caster_wheel_radius * caster_wheel_radius)}" ixy="0.0" ixz="0.0"
-          iyy="${caster_wheel_mass * 0.4 * (caster_wheel_radius * caster_wheel_radius)}" iyz="0.0"
-          izz="${caster_wheel_mass * 0.4 * (caster_wheel_radius * caster_wheel_radius)}"/>
+          ixx="${caster_mass * 0.4 * (caster_radius * caster_radius)}" ixy="0.0" ixz="0.0"
+          iyy="${caster_mass * 0.4 * (caster_radius * caster_radius)}" iyz="0.0"
+          izz="${caster_mass * 0.4 * (caster_radius * caster_radius)}"/>
       </inertial>
     </link>
@@ -151,5 +153,5 @@
       <parent link="${prefix}base_link"/>
       <child link="${prefix}rear_caster"/>
-      <origin xyz="${-base_length/2 + caster_wheel_radius} 0 ${-z_offset}" rpy="0 0 0"/>
+      <origin xyz="${-base_length/2 + caster_radius} 0 ${-z_offset}" rpy="0 0 0"/>
     </joint>
 <!-- ****************************************************** Rear Caster Link *********************************************************  -->
@@ -158,5 +160,5 @@
         <origin xyz="0 0 0" rpy="0 0 0"/>
         <geometry>
-          <sphere radius="${caster_wheel_radius}"/>
+          <sphere radius="${caster_radius}"/>
         </geometry>
       </collision>
@@ -164,5 +166,5 @@
         <origin xyz="0 0 0" rpy="0 0 0"/>
         <geometry>
-          <sphere radius="${caster_wheel_radius}"/>
+          <sphere radius="${caster_radius}"/>
         </geometry>
         <material name="white"/>
@@ -170,9 +172,9 @@
       <inertial>
         <origin xyz="0 0 0" rpy="0 0 0"/>
-        <mass value="${caster_wheel_mass}"/>
+        <mass value="${caster_mass}"/>
         <inertia
-          ixx="${caster_wheel_mass * 0.4 * (caster_wheel_radius * caster_wheel_radius)}" ixy="0.0" ixz="0.0"
-          iyy="${caster_wheel_mass * 0.4 * (caster_wheel_radius * caster_wheel_radius)}" iyz="0.0"
-          izz="${caster_wheel_mass * 0.4 * (caster_wheel_radius * caster_wheel_radius)}"/>
+          ixx="${caster_mass * 0.4 * (caster_radius * caster_radius)}" ixy="0.0" ixz="0.0"
+          iyy="${caster_mass * 0.4 * (caster_radius * caster_radius)}" iyz="0.0"
+          izz="${caster_mass * 0.4 * (caster_radius * caster_radius)}"/>
       </inertial>
     </link>

Commit message: u

File: urdf/diffbot.urdf (robot description, URDF)
Before this commit: robot diffbot, 6 links, 5 joints
Links:
- link base_link: mass 0.3 -> 0.6; geometry collision box size=0.4 0.2 0.1; visual box size=0.4 0.2 0.1
- link front_caster: geometry collision sphere radius=0.05; visual sphere radius=0.05
- link left_wheel: geometry collision cylinder length=0.03 radius=0.05; visual cylinder length=0.03 radius=0.05
- link rear_caster: geometry collision sphere radius=0.05; visual sphere radius=0.05
- link right_wheel: geometry collision cylinder length=0.03 radius=0.05; visual cylinder length=0.03 radius=0.05
Joints:
- joint base_joint: origin xyz=0.0 0.0 0.05 rpy=0.0 0.0 0.0 -> xyz=0.0 0.0 0.1 rpy=0.0 0.0 0.0
- joint front_caster_joint: origin xyz=0.07500000000000001 0 -0.025 rpy=0 0 0 -> xyz=0.15000000000000002 0 -0.05 rpy=0 0 0
- joint left_wheel_joint: origin xyz=0 -0.055 -0.025 rpy=0 0 0 -> xyz=0 -0.115 -0.05 rpy=0 0 0
- joint rear_caster_joint: origin xyz=-0.07500000000000001 0 -0.025 rpy=0 0 0 -> xyz=-0.15000000000000002 0 -0.05 rpy=0 0 0
- joint right_wheel_joint: origin xyz=0 0.055 -0.025 rpy=0 0 0 -> xyz=0 0.115 -0.05 rpy=0 0 0

File: xacro/diffbot.xacro (robot description, xacro)
@@ -6,14 +6,14 @@
 <!-- *********************************************************************************************************************************  -->
 <!-- ****************************************************** Parameters ***************************************************************  -->
-  <xacro:property name="base_mass"      value="0.3"               /> <!-- arbitrary value for base mass             -->
-  <xacro:property name="base_width"     value="0.10"              />
-  <xacro:property name="base_length"    value="0.20"              />
-  <xacro:property name="base_height"    value="0.05"              />
+  <xacro:property name="base_mass"      value="0.6"               /> <!-- arbitrary value for base mass             -->
+  <xacro:property name="base_width"     value="0.20"              />
+  <xacro:property name="base_length"    value="0.40"              />
+  <xacro:property name="base_height"    value="0.10"              />
   <xacro:property name="wheel_mass"     value="0.3"               /> <!-- arbitrary value for wheel mass            -->
-  <xacro:property name="wheel_width"    value="0.010"             />
-  <xacro:property name="wheel_radius"   value="0.025"             />
+  <xacro:property name="wheel_width"    value="0.030"             />
+  <xacro:property name="wheel_radius"   value="0.050"             />
   <xacro:property name="caster_mass"    value="0.1"               /> <!-- arbitrary value for caster wheel mass     -->
   <xacro:property name="caster_radius"  value="${wheel_radius}"   />
-  <xacro:property name="z_offset"       value="${base_height/2}" /> <!-- Space btw top of beam and the each joint  -->
+  <xacro:property name="z_offset"       value="${base_height/2}"  /> <!-- Space btw top of beam and the each joint  -->
 <!-- ****************************************************** Includes *****************************************************************  -->
   <xacro:include filename="$(find robot_gazebo)/xacro/common_rviz_materials.xacro" />   <!-- RVIZ Colors                                -->

Commit message: u

File: urdf/diffbot.urdf (robot description, URDF)
Before this commit: robot diffbot, 6 links, 5 joints
Joints:
- joint left_wheel_joint: origin xyz=0 -0.115 -0.05 rpy=0 0 0 -> xyz=0 -0.11800000000000001 -0.05 rpy=0 0 0
- joint right_wheel_joint: origin xyz=0 0.115 -0.05 rpy=0 0 0 -> xyz=0 0.11800000000000001 -0.05 rpy=0 0 0

File: xacro/diffbot.xacro (robot description, xacro)
@@ -6,14 +6,15 @@
 <!-- *********************************************************************************************************************************  -->
 <!-- ****************************************************** Parameters ***************************************************************  -->
-  <xacro:property name="base_mass"      value="0.6"               /> <!-- arbitrary value for base mass             -->
-  <xacro:property name="base_width"     value="0.20"              />
-  <xacro:property name="base_length"    value="0.40"              />
-  <xacro:property name="base_height"    value="0.10"              />
-  <xacro:property name="wheel_mass"     value="0.3"               /> <!-- arbitrary value for wheel mass            -->
-  <xacro:property name="wheel_width"    value="0.030"             />
-  <xacro:property name="wheel_radius"   value="0.050"             />
-  <xacro:property name="caster_mass"    value="0.1"               /> <!-- arbitrary value for caster wheel mass     -->
-  <xacro:property name="caster_radius"  value="${wheel_radius}"   />
-  <xacro:property name="z_offset"       value="${base_height/2}"  /> <!-- Space btw top of beam and the each joint  -->
+  <xacro:property name="base_mass"      value="0.6"                               />  <!-- arbitrary value for base mass                -->
+  <xacro:property name="base_width"     value="0.20"                              />
+  <xacro:property name="base_length"    value="0.40"                              />
+  <xacro:property name="base_height"    value="0.10"                              />
+  <xacro:property name="wheel_mass"     value="0.3"                               />  <!-- arbitrary value for wheel mass               -->
+  <xacro:property name="wheel_width"    value="0.030"                             />
+  <xacro:property name="wheel_radius"   value="0.050"                             />
+  <xacro:property name="caster_mass"    value="0.1"                               />  <!-- arbitrary value for caster wheel mass        -->
+  <xacro:property name="caster_radius"  value="${wheel_radius}"                   />
+  <xacro:property name="y_offset"       value="${(base_width+wheel_width*1.2)/2}" />
+  <xacro:property name="z_offset"       value="${base_height/2}"                  />  <!-- Space btw top of beam and the each joint     -->
 <!-- ****************************************************** Includes *****************************************************************  -->
   <xacro:include filename="$(find robot_gazebo)/xacro/common_rviz_materials.xacro" />   <!-- RVIZ Colors                                -->
@@ -57,5 +58,5 @@
       <parent link="${prefix}base_link"/>
       <child link="${prefix}left_wheel"/>
-      <origin xyz="0 -${(base_width+wheel_width)/2} ${-z_offset}" rpy="0 0 0"/>
+      <origin xyz="0 -${y_offset} -${z_offset}" rpy="0 0 0"/>
       <limit upper="${radians(180)}" lower="-${radians(180)}" effort="30" velocity="5.0"/>
       <axis xyz="0 1 0"/>
@@ -90,5 +91,5 @@
       <parent link="${prefix}base_link"/>
       <child link="${prefix}right_wheel"/>
-      <origin xyz="0 ${(base_width+wheel_width)/2} ${-z_offset}" rpy="0 0 0"/>
+      <origin xyz="0 ${y_offset} -${z_offset}" rpy="0 0 0"/>
       <limit upper="${radians(180)}" lower="-${radians(180)}" effort="30" velocity="5.0"/>
       <axis xyz="0 1 0"/>
