Commit message: u

File: urdf/diffbot.urdf (robot description, URDF)
Before this commit: robot diffbot, 6 links, 5 joints
Links:
- link base_link: geometry collision mesh filename=package://robot_gazebo/meshes/diffbot/base.stl scale=1 1 1; visual mesh filename=package://robot_gazebo/meshes/diffbot/base.stl scale=1 1 1

File: xacro/diffbot.xacro (robot description, xacro)
@@ -6,4 +6,5 @@
 <!-- *********************************************************************************************************************************  -->
 <!-- ****************************************************** Parameters ***************************************************************  -->
+  <xacro:property name="mesh_path"      value="package://robot_gazebo/meshes/diffbot/"/>
   <xacro:property name="base_mass"      value="0.6"                               />  <!-- arbitrary value for base mass                -->
   <xacro:property name="base_width"     value="0.20"                              />
@@ -35,5 +36,5 @@
       <origin xyz="0 0 0" rpy="0 0 0"/>
       <geometry>
-        <box size="${base_length} ${base_width} ${base_height}"/>
+        <mesh filename="${mesh_path}base.stl" scale="1 1 1"/>  <!--  <box size="${base_length} ${base_width} ${base_height}"/> -->
       </geometry>
     </collision>
@@ -41,5 +42,5 @@
       <origin xyz="0 0 0" rpy="0 0 0"/>
       <geometry>
-        <box size="${base_length} ${base_width} ${base_height}"/>
+        <mesh filename="${mesh_path}base.stl" scale="1 1 1"/>  <!--  <box size="${base_length} ${base_width} ${base_height}"/> -->
       </geometry>
       <material name="orange"/>

Commit message: u

File: urdf/diffbot.urdf (robot description, URDF)
Before this commit: robot diffbot, 6 links, 5 joints
Links:
- link base_link: geometry collision mesh filename=package://robot_gazebo/meshes/diffbot/base.dae scale=1 1 1; visual mesh filename=package://robot_gazebo/meshes/diffbot/base.dae scale=1 1 1

File: xacro/diffbot.xacro (robot description, xacro)
@@ -36,5 +36,5 @@
       <origin xyz="0 0 0" rpy="0 0 0"/>
       <geometry>
-        <mesh filename="${mesh_path}base.stl" scale="1 1 1"/>  <!--  <box size="${base_length} ${base_width} ${base_height}"/> -->
+        <mesh filename="${mesh_path}base.dae" scale="1 1 1"/>  <!--  <box size="${base_length} ${base_width} ${base_height}"/> -->
       </geometry>
     </collision>
@@ -42,5 +42,5 @@
       <origin xyz="0 0 0" rpy="0 0 0"/>
       <geometry>
-        <mesh filename="${mesh_path}base.stl" scale="1 1 1"/>  <!--  <box size="${base_length} ${base_width} ${base_height}"/> -->
+        <mesh filename="${mesh_path}base.dae" scale="1 1 1"/>  <!--  <box size="${base_length} ${base_width} ${base_height}"/> -->
       </geometry>
       <material name="orange"/>

Commit message: u

File: urdf/diffbot.urdf (robot description, URDF)
Before this commit: robot diffbot, 6 links, 5 joints
Links:
- link base_link: geometry collision mesh filename=package://robot_gazebo/meshes/diffbot/base.stl scale=1 1 1; visual mesh filename=package://robot_gazebo/meshes/diffbot/base.stl scale=1 1 1

Commit message: u

File: urdf/diffbot.urdf (robot description, URDF)
Before this commit: robot diffbot, 6 links, 5 joints
Links:
- link front_caster: geometry collision sphere radius=0.055; visual sphere radius=0.055
- link rear_caster: geometry collision sphere radius=0.055; visual sphere radius=0.055
Joints:
- joint front_caster_joint: origin xyz=0.114 0 -0.025 rpy=0 0 0 -> xyz=0.13775 0 -0.05 rpy=0 0 0
- joint rear_caster_joint: origin xyz=-0.114 0 -0.025 rpy=0 0 0 -> xyz=-0.13775 0 -0.05 rpy=0 0 0

Commit message: u

File: urdf/diffbot.urdf (robot description, URDF)
Before this commit: robot diffbot, 6 links, 5 joints
Links:
- link left_wheel: geometry collision mesh filename=package://robot_gazebo/meshes/diffbot/wheel.dae scale=1 1 1; visual mesh filename=package://robot_gazebo/meshes/diffbot/wheel.dae scale=1 1 1

File: xacro/diffbot.xacro (robot description, xacro)
@@ -73,5 +73,5 @@
         <origin xyz="0 0 0" rpy="${radians(90)} 0 0"/>
         <geometry>
-          <cylinder length="${wheel_width}" radius="${wheel_radius}"/>
+          <mesh filename="${mesh_path}wheel.dae" scale="1 1 1"/> <!-- <cylinder length="${wheel_width}" radius="${wheel_radius}"/> -->
         </geometry>
       </collision>
@@ -79,5 +79,5 @@
         <origin xyz="0 0 0" rpy="${radians(90)} 0 0"/>
         <geometry>
-          <cylinder length="${wheel_width}" radius="${wheel_radius}"/>
+          <mesh filename="${mesh_path}wheel.dae" scale="1 1 1"/> <!-- <cylinder length="${wheel_width}" radius="${wheel_radius}"/> -->
         </geometry>
         <material name="black"/>
@@ -106,5 +106,5 @@
         <origin xyz="0 0 0" rpy="${radians(90)} 0 0"/>
         <geometry>
-          <cylinder length="${wheel_width}" radius="${wheel_radius}"/>
+          <mesh filename="${mesh_path}wheel.dae" scale="1 1 1"/> <!-- <cylinder length="${wheel_width}" radius="${wheel_radius}"/> -->
         </geometry>
       </collision>
@@ -112,5 +112,5 @@
         <origin xyz="0 0 0" rpy="${radians(90)} 0 0"/>
         <geometry>
-          <cylinder length="${wheel_width}" radius="${wheel_radius}"/>
+          <mesh filename="${mesh_path}wheel.dae" scale="1 1 1"/> <!-- <cylinder length="${wheel_width}" radius="${wheel_radius}"/> -->
         </geometry>
         <material name="black"/>

Commit message: u

File: urdf/diffbot.urdf (robot description, URDF)
Before this commit: robot diffbot, 6 links, 5 joints
Links:
- link right_wheel: geometry collision mesh filename=package://robot_gazebo/meshes/diffbot/wheel.dae scale=1 1 1; visual mesh filename=package://robot_gazebo/meshes/diffbot/wheel.dae scale=1 1 1

Commit message: u

File: urdf/diffbot.urdf (robot description, URDF)
Before this commit: robot diffbot, 7 links, 6 joints
Links:
- removed link base_footprint
- removed link base_link
- added link base, mass 0.6; collision mesh filename=package://robot_gazebo/meshes/diffbot/base.stl scale=1 1 1; visual mesh filename=package://robot_gazebo/meshes/diffbot/base.stl scale=1 1 1
- added link camera, mass 0.1; collision box size=0.05 0.05 0.05; visual box size=0.05 0.05 0.05
- added link footprint
Joints:
- removed joint base_joint
- added joint camera_joint: type fixed, parent base, child camera, origin xyz=0.2 0 0 rpy=0 0 0, axis 0 1 0
- added joint footprint_joint: type fixed, parent footprint, child base, origin xyz=0.0 0.0 0.10500000000000001 rpy=0.0 0.0 0.0
- joint front_caster_joint: parent base_link -> base
- joint hokuyo_joint: parent base_link -> base
- joint left_wheel_joint: parent base_link -> base
- joint rear_caster_joint: parent base_link -> base
- joint right_wheel_joint: parent base_link -> base

File: xacro/diffbot.xacro (robot description, xacro)
@@ -23,4 +23,9 @@
   <xacro:property name="caster_x"       value="${(base_length/2 - caster_radius)*0.95}" />
   <xacro:property name="caster_z"       value="${base_height/2}"/>
+  <xacro:property name="camera_mass"    value="0.1"      />
+  <xacro:property name="camera_width"   value="0.05"     />
+  <xacro:property name="camera_length"  value="0.05"     />
+  <xacro:property name="camera_height"  value="0.05"     />
+  <xacro:property name="camera_x"       value="0.2"      /> <!-- x offset from base center -->
   <xacro:property name="hokuyo_mass"    value="1e-5"     />
   <xacro:property name="hokuyo_width"   value="0.05"     />

Commit message: u

File: urdf/diffbot.urdf (robot description, URDF)
Before this commit: robot diffbot, 8 links, 7 joints
Joints:
- joint front_caster_joint: origin xyz=0.13775 0 -0.05 rpy=0 0 0 -> xyz=0.13775 0 -0.04 rpy=0 0 0
- joint rear_caster_joint: origin xyz=-0.13775 0 -0.05 rpy=0 0 0 -> xyz=-0.13775 0 -0.04 rpy=0 0 0

File: xacro/diffbot.xacro (robot description, xacro)
@@ -22,5 +22,5 @@
   <xacro:property name="caster_radius"  value="${wheel_radius-wheel_z}"           />
   <xacro:property name="caster_x"       value="${(base_length/2 - caster_radius)*0.95}" />
-  <xacro:property name="caster_z"       value="${base_height/2}"/>
+  <xacro:property name="caster_z"       value="${base_height/2-0.01}"/>
   <xacro:property name="camera_mass"    value="0.1"      />
   <xacro:property name="camera_width"   value="0.05"     />
