Commit message: u

File: urdf/rrbot.urdf (robot description, URDF)
Before this commit: robot rrbot, 8 links, 7 joints
Links:
- removed link base_link
- removed link camera_link
- removed link camera_link_optical
- removed link hokuyo_link
- removed link tool_link
- added link base, mass 1; collision box size=0.1 0.1 2; visual box size=0.1 0.1 2
- added link camera, mass 1e-05; collision box size=0.05 0.05 0.05; visual box size=0.05 0.05 0.05
- added link camera_optical
- added link hokuyo, mass 1e-5; collision box size=0.1 0.1 0.1; visual mesh filename=package://robot_gazebo/meshes/rrbot/hokuyo.dae
- added link tool
Joints:
- joint base_joint: child base_link -> base
- joint camera_joint: child camera_link -> camera
- joint camera_optical_joint: child camera_link_optical -> camera_optical; parent camera_link -> camera
- joint hokuyo_joint: child hokuyo_link -> hokuyo
- joint joint1: parent base_link -> base
- joint tool_joint: child tool_link -> tool

File: urdf/skidbot.urdf (robot description, URDF)
Before this commit: robot skidbot, 8 links, 7 joints
Links:
- link camera: mass 0.1 -> 1e-05

Commit message: u

File: urdf/rrbot.urdf (robot description, URDF)
Before this commit: robot rrbot, 8 links, 7 joints
Links:
- removed link base
- removed link camera
- removed link camera_optical
- removed link hokuyo
- removed link link3
- removed link tool
- added link base_link, mass 1; collision box size=0.1 0.1 2; visual box size=0.1 0.1 2
- added link camera_link, mass 1e-5; collision box size=0.05 0.05 0.05; visual box size=0.05 0.05 0.05
- added link camera_link_optical
- added link hokuyo_link, mass 1e-5; collision box size=0.1 0.1 0.1; visual box size=0.05 0.05 0.05
- added link link1, mass 1; collision box size=0.1 0.1 1; visual box size=0.1 0.1 1
- added link tool_link
Joints:
- joint base_joint: child base -> base_link
- joint camera_joint: child camera -> camera_link; origin xyz=0.07500000000000001 0 0.9 rpy=0 0 0 -> xyz=0.05 0 0.9 rpy=0 0 0; parent link3 -> link2
- joint camera_optical_joint: child camera_optical -> camera_link_optical; parent camera -> camera_link
- joint hokuyo_joint: child hokuyo -> hokuyo_link; parent link3 -> link2
- joint joint1: child link2 -> link1; parent base -> base_link
- joint joint2: child link3 -> link2; parent link2 -> link1
- joint tool_joint: child tool -> tool_link; parent link3 -> link2

File: xacro/rrbot.xacro (robot description, xacro)
@@ -1,45 +1,22 @@
 <?xml version="1.0"?>
 <robot name="rrbot" xmlns:xacro="http://www.ros.org/wiki/xacro">
-<!-- ****************************************************** RRBot Robot **************************************************************  -->
-<!-- Muthanna Alwahash                                                                                                                  -->
-<!-- March 2022                                                                                                                         -->
-<!-- *********************************************************************************************************************************  -->
-<!-- ****************************************************** Parameters ***************************************************************  -->
   <xacro:property name="mesh_path"      value="package://robot_gazebo/meshes/rrbot/" />
-  <xacro:property name="name_space"     value="rrbot" />
-  <xacro:property name="prefix"         value=""      />
-  <xacro:property name="mass"           value="1"     /> <!-- arbitrary value for mass -->
-  <xacro:property name="width"          value="0.1"   /> <!-- Square dimensions (widthxwidth) of beams -->
-  <xacro:property name="height1"        value="2"     /> <!-- Link 1 (Base) -->
-  <xacro:property name="height2"        value="1"     /> <!-- Link 2 -->
-  <xacro:property name="height3"        value="1"     /> <!-- Link 3 -->
-  <xacro:property name="joint_gap"      value="0.05"                   /> <!-- Space btw top of beam and the each joint -->
-  <xacro:property name="joint1_y"       value="${width}"               />
-  <xacro:property name="joint1_z"       value="${height1-joint_gap}"   />
-  <xacro:property name="joint2_y"       value="${width}"               />
-  <xacro:property name="joint2_z"       value="${height2-joint_gap*2}" />
-  <xacro:property name="camera_mass"    value="1e-5"     />
-  <xacro:property name="camera_width"   value="0.05"     />
-  <xacro:property name="camera_length"  value="0.05"     />
-  <xacro:property name="camera_height"  value="0.05"     />
-  <xacro:property name="camera_x"       value="${(width+camera_width)/2}" />
-  <xacro:property name="camera_z"       value="${height3-joint_gap*2}" />
-  <xacro:property name="hokuyo_mass"    value="1e-5"     />
-  <xacro:property name="hokuyo_width"   value="0.05"     />
-  <xacro:property name="hokuyo_length"  value="0.05"     />
-  <xacro:property name="hokuyo_height"  value="0.0706"   />
-  <xacro:property name="hokuyo_z"       value="${height3-joint_gap/2}" />
-  <xacro:property name="tool_z"         value="${height3}" />
-<!-- ****************************************************** Includes *****************************************************************  -->
   <xacro:include filename="$(find robot_gazebo)/xacro/common_rviz_materials.xacro" />   <!-- RVIZ Colors                                -->
-  <xacro:include filename="$(find robot_gazebo)/gazebo/gz_rrbot.xacro" />               <!--  Gazebo                                    -->
-<!-- ****************************************************** Base Joint ***************************************************************  -->
+  <xacro:macro name="rrbot" params="parent prefix">
+  <!-- Constants for robot dimensions -->
+  <xacro:property name="mass" value="1" /> <!-- arbitrary value for mass -->
+  <xacro:property name="width" value="0.1" /> <!-- Square dimensions (widthxwidth) of beams -->
+  <xacro:property name="height1" value="2" /> <!-- Link 1 -->
+  <xacro:property name="height2" value="1" /> <!-- Link 2 -->
+  <xacro:property name="height3" value="1" /> <!-- Link 3 -->
+  <xacro:property name="camera_link" value="0.05" /> <!-- Size of square 'camera' box -->
+  <xacro:property name="axel_offset" value="0.05" /> <!-- Space btw top of beam and the each joint -->
   <joint name="${prefix}base_joint" type="fixed">
     <origin xyz="0 0 0" rpy="0 0 0" />
-    <parent link="world"/>
-    <child link="${prefix}base" />
+    <parent link="${parent}"/>
+    <child link="${prefix}base_link" />
   </joint>
-<!-- ****************************************************** Base Link ****************************************************************  -->
-  <link name="${prefix}base">
+  <!-- Base Link -->
+  <link name="${prefix}base_link">
     <collision>
       <origin xyz="0 0 ${height1/2}" rpy="0 0 0"/>
@@ -62,144 +39,146 @@
         iyy="${mass / 12.0 * (height1*height1 + width*width)}" iyz="0.0"
         izz="${mass / 12.0 * (width*width + width*width)}"/>
-    </inertial>
-  </link>
-<!-- ****************************************************** Joint 1 ******************************************************************  -->
-  <joint name="${prefix}joint1" type="continuous">
-    <parent link="${prefix}base"/>
-    <child link="${prefix}link2"/>
-    <origin xyz="0 ${joint1_y} ${joint1_z}" rpy="0 0 0"/>
-    <axis xyz="0 1 0"/>
-    <dynamics damping="0.7"/>
-  </joint>
-<!-- ****************************************************** Link 2 *******************************************************************  -->
-  <link name="${prefix}link2">
-    <collision>
-      <origin xyz="0 0 ${height2/2 - joint_gap}" rpy="0 0 0"/>
-      <geometry>
-        <box size="${width} ${width} ${height2}"/>
-      </geometry>
-    </collision>
-    <visual>
-      <origin xyz="0 0 ${height2/2 - joint_gap}" rpy="0 0 0"/>
-      <geometry>
-        <box size="${width} ${width} ${height2}"/>
-      </geometry>
-      <material name="yellow"/>
-    </visual>
-    <inertial>
-      <origin xyz="0 0 ${height2/2 - joint_gap}" rpy="0 0 0"/>
-      <mass value="${mass}"/>
-      <inertia
-        ixx="${mass / 12.0 * (width*width + height2*height2)}" ixy="0.0" ixz="0.0"
-        iyy="${mass / 12.0 * (height2*height2 + width*width)}" iyz="0.0"
-        izz="${mass / 12.0 * (width*width + width*width)}"/>
-    </inertial>
-  </link>
-<!-- ****************************************************** Joint 2 ******************************************************************  -->
-  <joint name="${prefix}joint2" type="continuous">
-    <parent link="${prefix}link2"/>
-    <child link="${prefix}link3"/>
-    <origin xyz="0 ${joint2_y} ${joint2_z}" rpy="0 0 0"/>
-    <axis xyz="0 1 0"/>
-    <dynamics damping="0.7"/>
-  </joint>
-<!-- ****************************************************** Link 3 *******************************************************************  -->
-  <link name="${prefix}link3">
-    <collision>
-      <origin xyz="0 0 ${height3/2 - joint_gap}" rpy="0 0 0"/>
-      <geometry>
-        <box size="${width} ${width} ${height3}"/>
-      </geometry>
-    </collision>
-    <visual>
-      <origin xyz="0 0 ${height3/2 - joint_gap}" rpy="0 0 0"/>
-      <geometry>
-        <box size="${width} ${width} ${height3}"/>
-      </geometry>
-      <material name="orange"/>
-    </visual>
-    <inertial>
-      <origin xyz="0 0 ${height3/2 - joint_gap}" rpy="0 0 0"/>
-      <mass value="${mass}"/>
-      <inertia
-        ixx="${mass / 12.0 * (width*width + height3*height3)}" ixy="0.0" ixz="0.0"
-        iyy="${mass / 12.0 * (height3*height3 + width*width)}" iyz="0.0"
-        izz="${mass / 12.0 * (width*width + width*width)}"/>
-    </inertial>
-  </link>
-<!-- ****************************************************** Tool Joint ***************************************************************  -->
-  <joint name="${prefix}tool_joint" type="fixed">
-    <origin xyz="0 0 ${tool_z}" rpy="0 0 0" />
-    <parent link="${prefix}link3"/>
-    <child link="${prefix}tool" />
-  </joint>
-<!-- ****************************************************** Tool Link ****************************************************************  -->
-  <link name="${prefix}tool" />
-<!-- ****************************************************** Camera Joint *************************************************************  -->
-  <joint name="${prefix}camera_joint" type="fixed">
-    <axis xyz="0 1 0" />
-    <origin xyz="${camera_x} 0 ${camera_z}" rpy="0 0 0"/>
-    <parent link="${prefix}link3"/>
-    <child link="${prefix}camera"/>
-  </joint>
-<!-- ****************************************************** Camera Link **************************************************************  -->
-<link name="${prefix}camera">
-  <inertial>
-    <mass value="${camera_mass}"/>
-    <origin xyz="0 0 0" rpy=" 0 0 0"/>
-    <inertia ixx="1e-6" ixy="0" ixz="0" iyy="1e-6" iyz="0" izz="1e-6" />
-  </inertial>
-  <visual name="camera_visual">
-    <origin xyz="0 0 0" rpy="0 0 0" />
-    <geometry>
-      <box size="${camera_length} ${camera_width} ${camera_height}"/>
-    </geometry>
-    <material name="green"/>
-  </visual>
-  <collision name="camera_colision">
-    <origin xyz="0 0 0" rpy="0 0 0" />
-    <geometry>
-      <box size="${camera_length} ${camera_width} ${camera_height}"/>
-    </geometry>
-  </collision>
-</link>
-<!-- ****************************************************** Camera Optical Joint *****************************************************  -->
-<!-- generate an optical frame http://www.ros.org/reps/rep-0103.html#suffix-frames so that ros and opencv can operate on the camera     -->
-<!-- frame correctly. these values have to be these values otherwise the gazebo camera image won't be aligned properly with the frame   -->
-<!-- it is supposedly originating from                                                                                                  -->
-  <joint name="${prefix}camera_optical_joint" type="fixed">
-    <origin xyz="0 0 0" rpy="${-radians(90)} 0 ${-radians(90)}"/>
-    <parent link="${prefix}camera"/>
-    <child link="${prefix}camera_optical"/>
-  </joint>
-<!-- ****************************************************** Camera Optical Link ******************************************************  -->
-  <link name="${prefix}camera_optical"/>
-<!-- ****************************************************** Hokuyo Joint *************************************************************  -->
-  <joint name="${prefix}hokuyo_joint" type="fixed">
-    <axis xyz="0 1 0" />
-    <origin xyz="0 0 ${hokuyo_z}" rpy="0 0 0"/>
-    <parent link="${prefix}link3"/>
-    <child link="${prefix}hokuyo"/>
-  </joint>
-<!-- ****************************************************** Hokuyo Link **************************************************************  -->
-  <link name="${prefix}hokuyo">
-    <collision>
-      <origin xyz="0 0 0" rpy="0 0 0"/>
-      <geometry>
-        <mesh filename="${mesh_path}hokuyo.dae"/> <!--  <box size="${hokuyo_length} ${hokuyo_width} ${hokuyo_height}"/> -->
-      </geometry>
-    </collision>
-    <visual>
-      <origin xyz="0 0 0" rpy="0 0 0"/>
-      <geometry>
-        <mesh filename="${mesh_path}hokuyo.dae"/> <!--  <box size="${hokuyo_length} ${hokuyo_width} ${hokuyo_height}"/> -->
-      </geometry>
-    </visual>
-    <inertial>
-      <mass value="${hokuyo_mass}" />
-      <origin xyz="0 0 0" rpy="0 0 0"/>
-      <inertia ixx="1e-6" ixy="0" ixz="0" iyy="1e-6" iyz="0" izz="1e-6" />
-    </inertial>
-  </link>
-<!-- ****************************************************** END **********************************************************************  -->
+      </inertial>
+    </link>
+    <joint name="${prefix}joint1" type="continuous">
+      <parent link="${prefix}base_link"/>
+      <child link="${prefix}link1"/>
+      <origin xyz="0 ${width} ${height1 - axel_offset}" rpy="0 0 0"/>
+      <axis xyz="0 1 0"/>
+      <dynamics damping="0.7"/>
+    </joint>
+    <!-- Middle Link -->
+    <link name="${prefix}link1">
+      <collision>
+        <origin xyz="0 0 ${height2/2 - axel_offset}" rpy="0 0 0"/>
+        <geometry>
+          <box size="${width} ${width} ${height2}"/>
+        </geometry>
+      </collision>
+      <visual>
+        <origin xyz="0 0 ${height2/2 - axel_offset}" rpy="0 0 0"/>
+        <geometry>
+          <box size="${width} ${width} ${height2}"/>
+        </geometry>
+        <material name="yellow"/>
+      </visual>
+      <inertial>
+        <origin xyz="0 0 ${height2/2 - axel_offset}" rpy="0 0 0"/>
+        <mass value="${mass}"/>
+        <inertia
+          ixx="${mass / 12.0 * (width*width + height2*height2)}" ixy="0.0" ixz="0.0"
+          iyy="${mass / 12.0 * (height2*height2 + width*width)}" iyz="0.0"
+          izz="${mass / 12.0 * (width*width + width*width)}"/>
+        </inertial>
+      </link>
+      <joint name="${prefix}joint2" type="continuous">
+        <parent link="${prefix}link1"/>
+        <child link="${prefix}link2"/>
+        <origin xyz="0 ${width} ${height2 - axel_offset*2}" rpy="0 0 0"/>
+        <axis xyz="0 1 0"/>
+        <dynamics damping="0.7"/>
+      </joint>
+      <!-- Top Link -->
+      <link name="${prefix}link2">
+        <collision>
+          <origin xyz="0 0 ${height3/2 - axel_offset}" rpy="0 0 0"/>
+          <geometry>
+            <box size="${width} ${width} ${height3}"/>
+          </geometry>
+        </collision>
+        <visual>
+          <origin xyz="0 0 ${height3/2 - axel_offset}" rpy="0 0 0"/>
+          <geometry>
+            <box size="${width} ${width} ${height3}"/>
+          </geometry>
+          <material name="orange"/>
+        </visual>
+        <inertial>
+          <origin xyz="0 0 ${height3/2 - axel_offset}" rpy="0 0 0"/>
+          <mass value="${mass}"/>
+          <inertia
+            ixx="${mass / 12.0 * (width*width + height3*height3)}" ixy="0.0" ixz="0.0"
+            iyy="${mass / 12.0 * (height3*height3 + width*width)}" iyz="0.0"
+            izz="${mass / 12.0 * (width*width + width*width)}"/>
+          </inertial>
+        </link>
+        <joint name="${prefix}tool_joint" type="fixed">
+          <origin xyz="0 0 1" rpy="0 0 0" />
+          <parent link="${prefix}link2"/>
+          <child link="${prefix}tool_link" />
+        </joint>
+        <!-- Tool Link -->
+        <link name="${prefix}tool_link">
+        </link>
+        <joint name="${prefix}hokuyo_joint" type="fixed">
+          <axis xyz="0 1 0" />
+          <origin xyz="0 0 ${height3 - axel_offset/2}" rpy="0 0 0"/>
+          <parent link="${prefix}link2"/>
+          <child link="${prefix}hokuyo_link"/>
+        </joint>
+        <!-- Hokuyo Laser -->
+        <link name="${prefix}hokuyo_link">
+          <collision>
+            <origin xyz="0 0 0" rpy="0 0 0"/>
+            <geometry>
+              <box size="0.1 0.1 0.1"/>
+            </geometry>
+          </collision>
+          <visual>
+            <origin xyz="0 0 0" rpy="0 0 0"/>
+            <geometry>
+              <box size="${camera_link} ${camera_link} ${camera_link}"/> <!--<mesh filename="${mesh_path}hokuyo.dae"/>-->
+            </geometry>
+          </visual>
+          <inertial>
+            <mass value="1e-5" />
+            <origin xyz="0 0 0" rpy="0 0 0"/>
+            <inertia ixx="1e-6" ixy="0" ixz="0" iyy="1e-6" iyz="0" izz="1e-6" />
+          </inertial>
+        </link>
+        <joint name="${prefix}camera_joint" type="fixed">
+          <axis xyz="0 1 0" />
+          <origin xyz="${camera_link} 0 ${height3 - axel_offset*2}" rpy="0 0 0"/>
+          <parent link="${prefix}link2"/>
+          <child link="${prefix}camera_link"/>
+        </joint>
+        <!-- Camera -->
+        <link name="${prefix}camera_link">
+          <collision>
+            <origin xyz="0 0 0" rpy="0 0 0"/>
+            <geometry>
+              <box size="${camera_link} ${camera_link} ${camera_link}"/>
+            </geometry>
+          </collision>
+          <visual>
+            <origin xyz="0 0 0" rpy="0 0 0"/>
+            <geometry>
+              <box size="${camera_link} ${camera_link} ${camera_link}"/>
+            </geometry>
+            <material name="red"/>
+          </visual>
+          <inertial>
+            <mass value="1e-5" />
+            <origin xyz="0 0 0" rpy="0 0 0"/>
+            <inertia ixx="1e-6" ixy="0" ixz="0" iyy="1e-6" iyz="0" izz="1e-6" />
+          </inertial>
+        </link>
+        <!-- generate an optical frame http://www.ros.org/reps/rep-0103.html#suffix-frames
+        so that ros and opencv can operate on the camera frame correctly -->
+        <joint name="${prefix}camera_optical_joint" type="fixed">
+          <!-- these values have to be these values otherwise the gazebo camera image
+          won't be aligned properly with the frame it is supposedly originating from -->
+          <origin xyz="0 0 0" rpy="${-pi/2} 0 ${-pi/2}"/>
+          <parent link="${prefix}camera_link"/>
+          <child link="${prefix}camera_link_optical"/>
+        </joint>
+        <link name="${prefix}camera_link_optical">
+        </link>
+  </xacro:macro>
+  <!-- Used for fixing robot -->
+  <link name="world"/>
+  <gazebo reference="world">
+    <static>true</static>
+  </gazebo>
+  <xacro:rrbot parent="world" prefix="" />
 </robot>

Commit message: u

File: urdf/rrbot.urdf (robot description, URDF)
Before this commit: robot rrbot, 8 links, 7 joints
Links:
- removed link base_link
- removed link camera_link
- removed link camera_link_optical
- removed link hokuyo_link
- removed link link1
- removed link tool_link
- added link base, mass 1; collision box size=0.1 0.1 2; visual box size=0.1 0.1 2
- added link camera, mass 1e-05; collision box size=0.05 0.05 0.05; visual box size=0.05 0.05 0.05
- added link camera_optical
- added link hokuyo, mass 1e-05; collision mesh filename=package://robot_gazebo/meshes/rrbot/hokuyo.dae; visual mesh filename=package://robot_gazebo/meshes/rrbot/hokuyo.dae
- added link link3, mass 1; collision box size=0.1 0.1 1; visual box size=0.1 0.1 1
- added link tool
Joints:
- joint base_joint: child base_link -> base
- joint camera_joint: child camera_link -> camera; origin xyz=0.05 0 0.9 rpy=0 0 0 -> xyz=0.07500000000000001 0 0.9 rpy=0 0 0; parent link2 -> link3
- joint camera_optical_joint: child camera_link_optical -> camera_optical; parent camera_link -> camera
- joint hokuyo_joint: child hokuyo_link -> hokuyo; parent link2 -> link3
- joint joint1: child link1 -> link2; parent base_link -> base
- joint joint2: child link2 -> link3; parent link1 -> link2
- joint tool_joint: child tool_link -> tool; parent link2 -> link3
