Commit message: update

File: urdf/golem.urdf (robot description, URDF)
Before this commit: robot Golem, 42 links, 41 joints
Links:
- link body_link: geometry collision mesh filename=package://robot_gazebo/meshes/golem/body.stl scale=0.001 0.001 0.001; visual mesh filename=package://robot_gazebo/meshes/golem/body.stl scale=0.001 0.001 0.001
- link coxa_LF: geometry collision mesh filename=package://robot_gazebo/meshes/golem/coxa.stl scale=0.001 0.001 0.001; visual mesh filename=package://robot_gazebo/meshes/golem/coxa.stl scale=0.001 0.001 0.001
- link coxa_LM: geometry collision mesh filename=package://robot_gazebo/meshes/golem/coxa.stl scale=0.001 0.001 0.001; visual mesh filename=package://robot_gazebo/meshes/golem/coxa.stl scale=0.001 0.001 0.001
- link coxa_LR: geometry collision mesh filename=package://robot_gazebo/meshes/golem/coxa.stl scale=0.001 0.001 0.001; visual mesh filename=package://robot_gazebo/meshes/golem/coxa.stl scale=0.001 0.001 0.001
- link coxa_RF: geometry collision mesh filename=package://robot_gazebo/meshes/golem/coxa.stl scale=0.001 0.001 0.001; visual mesh filename=package://robot_gazebo/meshes/golem/coxa.stl scale=0.001 0.001 0.001
- link coxa_RM: geometry collision mesh filename=package://robot_gazebo/meshes/golem/coxa.stl scale=0.001 0.001 0.001; visual mesh filename=package://robot_gazebo/meshes/golem/coxa.stl scale=0.001 0.001 0.001
- link coxa_RR: geometry collision mesh filename=package://robot_gazebo/meshes/golem/coxa.stl scale=0.001 0.001 0.001; visual mesh filename=package://robot_gazebo/meshes/golem/coxa.stl scale=0.001 0.001 0.001
- link femur_LF: geometry collision mesh filename=package://robot_gazebo/meshes/golem/femur.stl scale=0.001 0.001 0.001; visual mesh filename=package://robot_gazebo/meshes/golem/femur.stl scale=0.001 0.001 0.001
- link femur_LM: geometry collision mesh filename=package://robot_gazebo/meshes/golem/femur.stl scale=0.001 0.001 0.001; visual mesh filename=package://robot_gazebo/meshes/golem/femur.stl scale=0.001 0.001 0.001
- link femur_LR: geometry collision mesh filename=package://robot_gazebo/meshes/golem/femur.stl scale=0.001 0.001 0.001; visual mesh filename=package://robot_gazebo/meshes/golem/femur.stl scale=0.001 0.001 0.001
- link femur_RF: geometry collision mesh filename=package://robot_gazebo/meshes/golem/femur.stl scale=0.001 0.001 0.001; visual mesh filename=package://robot_gazebo/meshes/golem/femur.stl scale=0.001 0.001 0.001
- link femur_RM: geometry collision mesh filename=package://robot_gazebo/meshes/golem/femur.stl scale=0.001 0.001 0.001; visual mesh filename=package://robot_gazebo/meshes/golem/femur.stl scale=0.001 0.001 0.001
- link femur_RR: geometry collision mesh filename=package://robot_gazebo/meshes/golem/femur.stl scale=0.001 0.001 0.001; visual mesh filename=package://robot_gazebo/meshes/golem/femur.stl scale=0.001 0.001 0.001
- link tarsus_LF: geometry collision mesh filename=package://robot_gazebo/meshes/golem/tarsus.stl scale=0.001 0.001 0.001; visual mesh filename=package://robot_gazebo/meshes/golem/tarsus.stl scale=0.001 0.001 0.001
- link tarsus_LM: geometry collision mesh filename=package://robot_gazebo/meshes/golem/tarsus.stl scale=0.001 0.001 0.001; visual mesh filename=package://robot_gazebo/meshes/golem/tarsus.stl scale=0.001 0.001 0.001
- link tarsus_LR: geometry collision mesh filename=package://robot_gazebo/meshes/golem/tarsus.stl scale=0.001 0.001 0.001; visual mesh filename=package://robot_gazebo/meshes/golem/tarsus.stl scale=0.001 0.001 0.001
- link tarsus_RF: geometry collision mesh filename=package://robot_gazebo/meshes/golem/tarsus.stl scale=0.001 0.001 0.001; visual mesh filename=package://robot_gazebo/meshes/golem/tarsus.stl scale=0.001 0.001 0.001
- link tarsus_RM: geometry collision mesh filename=package://robot_gazebo/meshes/golem/tarsus.stl scale=0.001 0.001 0.001; visual mesh filename=package://robot_gazebo/meshes/golem/tarsus.stl scale=0.001 0.001 0.001
- link tarsus_RR: geometry collision mesh filename=package://robot_gazebo/meshes/golem/tarsus.stl scale=0.001 0.001 0.001; visual mesh filename=package://robot_gazebo/meshes/golem/tarsus.stl scale=0.001 0.001 0.001
- link tibia_LF: geometry collision mesh filename=package://robot_gazebo/meshes/golem/tibia.stl scale=0.001 0.001 0.001; visual mesh filename=package://robot_gazebo/meshes/golem/tibia.stl scale=0.001 0.001 0.001
- link tibia_LM: geometry collision mesh filename=package://robot_gazebo/meshes/golem/tibia.stl scale=0.001 0.001 0.001; visual mesh filename=package://robot_gazebo/meshes/golem/tibia.stl scale=0.001 0.001 0.001
- link tibia_LR: geometry collision mesh filename=package://robot_gazebo/meshes/golem/tibia.stl scale=0.001 0.001 0.001; visual mesh filename=package://robot_gazebo/meshes/golem/tibia.stl scale=0.001 0.001 0.001
- link tibia_RF: geometry collision mesh filename=package://robot_gazebo/meshes/golem/tibia.stl scale=0.001 0.001 0.001; visual mesh filename=package://robot_gazebo/meshes/golem/tibia.stl scale=0.001 0.001 0.001
- link tibia_RM: geometry collision mesh filename=package://robot_gazebo/meshes/golem/tibia.stl scale=0.001 0.001 0.001; visual mesh filename=package://robot_gazebo/meshes/golem/tibia.stl scale=0.001 0.001 0.001
- link tibia_RR: geometry collision mesh filename=package://robot_gazebo/meshes/golem/tibia.stl scale=0.001 0.001 0.001; visual mesh filename=package://robot_gazebo/meshes/golem/tibia.stl scale=0.001 0.001 0.001

File: urdf/pxm3.urdf (robot description, URDF)
Before this commit: robot pxm3, 26 links, 25 joints
Links:
- link MP_BODY: geometry collision mesh filename=package://robot_gazebo/meshes/pxm3/body_coll.STL scale=1 1 1; visual mesh filename=package://robot_gazebo/meshes/pxm3/body.STL scale=1 1 1
- link c1_LF: geometry collision mesh filename=package://robot_gazebo/meshes/pxm3/connect_coll.STL scale=1 1 1; visual mesh filename=package://robot_gazebo/meshes/pxm3/connect.STL scale=1 1 1
- link c1_LM: geometry collision mesh filename=package://robot_gazebo/meshes/pxm3/connect_coll.STL scale=1 1 1; visual mesh filename=package://robot_gazebo/meshes/pxm3/connect.STL scale=1 1 1
- link c1_LR: geometry collision mesh filename=package://robot_gazebo/meshes/pxm3/connect_coll.STL scale=1 1 1; visual mesh filename=package://robot_gazebo/meshes/pxm3/connect.STL scale=1 1 1
- link c1_RF: geometry collision mesh filename=package://robot_gazebo/meshes/pxm3/connect_coll.STL scale=1 1 1; visual mesh filename=package://robot_gazebo/meshes/pxm3/connect.STL scale=1 1 1
- link c1_RM: geometry collision mesh filename=package://robot_gazebo/meshes/pxm3/connect_coll.STL scale=1 1 1; visual mesh filename=package://robot_gazebo/meshes/pxm3/connect.STL scale=1 1 1
- link c1_RR: geometry collision mesh filename=package://robot_gazebo/meshes/pxm3/connect_coll.STL scale=1 1 1; visual mesh filename=package://robot_gazebo/meshes/pxm3/connect.STL scale=1 1 1
- link c2_LF: geometry collision mesh filename=package://robot_gazebo/meshes/pxm3/connect_coll.STL scale=1 1 1; visual mesh filename=package://robot_gazebo/meshes/pxm3/connect.STL scale=1 1 1
- link c2_LM: geometry collision mesh filename=package://robot_gazebo/meshes/pxm3/connect_coll.STL scale=1 1 1; visual mesh filename=package://robot_gazebo/meshes/pxm3/connect.STL scale=1 1 1
- link c2_LR: geometry collision mesh filename=package://robot_gazebo/meshes/pxm3/connect_coll.STL scale=1 1 1; visual mesh filename=package://robot_gazebo/meshes/pxm3/connect.STL scale=1 1 1
- link c2_RF: geometry collision mesh filename=package://robot_gazebo/meshes/pxm3/connect_coll.STL scale=1 1 1; visual mesh filename=package://robot_gazebo/meshes/pxm3/connect.STL scale=1 1 1
- link c2_RM: geometry collision mesh filename=package://robot_gazebo/meshes/pxm3/connect_coll.STL scale=1 1 1; visual mesh filename=package://robot_gazebo/meshes/pxm3/connect.STL scale=1 1 1
- link c2_RR: geometry collision mesh filename=package://robot_gazebo/meshes/pxm3/connect_coll.STL scale=1 1 1; visual mesh filename=package://robot_gazebo/meshes/pxm3/connect.STL scale=1 1 1
- link thigh_LF: geometry collision mesh filename=package://robot_gazebo/meshes/pxm3/thigh_l_coll.STL scale=1 1 1; visual mesh filename=package://robot_gazebo/meshes/pxm3/thigh_l.STL scale=1 1 1
- link thigh_LM: geometry collision mesh filename=package://robot_gazebo/meshes/pxm3/thigh_l_coll.STL scale=1 1 1; visual mesh filename=package://robot_gazebo/meshes/pxm3/thigh_l.STL scale=1 1 1
- link thigh_LR: geometry collision mesh filename=package://robot_gazebo/meshes/pxm3/thigh_l_coll.STL scale=1 1 1; visual mesh filename=package://robot_gazebo/meshes/pxm3/thigh_l.STL scale=1 1 1
- link thigh_RF: geometry collision mesh filename=package://robot_gazebo/meshes/pxm3/thigh_l_coll.STL scale=1 1 1; visual mesh filename=package://robot_gazebo/meshes/pxm3/thigh_l.STL scale=1 1 1
- link thigh_RM: geometry collision mesh filename=package://robot_gazebo/meshes/pxm3/thigh_l_coll.STL scale=1 1 1; visual mesh filename=package://robot_gazebo/meshes/pxm3/thigh_l.STL scale=1 1 1
- link thigh_RR: geometry collision mesh filename=package://robot_gazebo/meshes/pxm3/thigh_l_coll.STL scale=1 1 1; visual mesh filename=package://robot_gazebo/meshes/pxm3/thigh_l.STL scale=1 1 1
- link tibia_LF: geometry collision mesh filename=package://robot_gazebo/meshes/pxm3/tibia_l_coll.STL scale=1 1 1; visual mesh filename=package://robot_gazebo/meshes/pxm3/tibia_l.STL scale=1 1 1
- link tibia_LM: geometry collision mesh filename=package://robot_gazebo/meshes/pxm3/tibia_l_coll.STL scale=1 1 1; visual mesh filename=package://robot_gazebo/meshes/pxm3/tibia_l.STL scale=1 1 1
- link tibia_LR: geometry collision mesh filename=package://robot_gazebo/meshes/pxm3/tibia_l_coll.STL scale=1 1 1; visual mesh filename=package://robot_gazebo/meshes/pxm3/tibia_l.STL scale=1 1 1
- link tibia_RF: geometry collision mesh filename=package://robot_gazebo/meshes/pxm3/tibia_l_coll.STL scale=1 1 1; visual mesh filename=package://robot_gazebo/meshes/pxm3/tibia_l.STL scale=1 1 1
- link tibia_RM: geometry collision mesh filename=package://robot_gazebo/meshes/pxm3/tibia_l_coll.STL scale=1 1 1; visual mesh filename=package://robot_gazebo/meshes/pxm3/tibia_l.STL scale=1 1 1
- link tibia_RR: geometry collision mesh filename=package://robot_gazebo/meshes/pxm3/tibia_l_coll.STL scale=1 1 1; visual mesh filename=package://robot_gazebo/meshes/pxm3/tibia_l.STL scale=1 1 1

File: urdf/razbot.urdf (robot description, URDF)
Before this commit: robot razbot, 27 links, 26 joints
Links:
- link body_link: geometry collision mesh filename=package://robot_gazebo/meshes/razbot/body.stl scale=0.001 0.001 0.001; visual mesh filename=package://robot_gazebo/meshes/razbot/body.stl scale=0.001 0.001 0.001
- link coxa_LF: geometry collision mesh filename=package://robot_gazebo/meshes/razbot/coxa.stl scale=0.001 0.001 0.001; visual mesh filename=package://robot_gazebo/meshes/razbot/coxa.stl scale=0.001 0.001 0.001
- link coxa_LM: geometry collision mesh filename=package://robot_gazebo/meshes/razbot/coxa.stl scale=0.001 0.001 0.001; visual mesh filename=package://robot_gazebo/meshes/razbot/coxa.stl scale=0.001 0.001 0.001
- link coxa_LR: geometry collision mesh filename=package://robot_gazebo/meshes/razbot/coxa.stl scale=0.001 0.001 0.001; visual mesh filename=package://robot_gazebo/meshes/razbot/coxa.stl scale=0.001 0.001 0.001
- link coxa_RF: geometry collision mesh filename=package://robot_gazebo/meshes/razbot/coxa.stl scale=0.001 0.001 0.001; visual mesh filename=package://robot_gazebo/meshes/razbot/coxa.stl scale=0.001 0.001 0.001
- link coxa_RM: geometry collision mesh filename=package://robot_gazebo/meshes/razbot/coxa.stl scale=0.001 0.001 0.001; visual mesh filename=package://robot_gazebo/meshes/razbot/coxa.stl scale=0.001 0.001 0.001
- link coxa_RR: geometry collision mesh filename=package://robot_gazebo/meshes/razbot/coxa.stl scale=0.001 0.001 0.001; visual mesh filename=package://robot_gazebo/meshes/razbot/coxa.stl scale=0.001 0.001 0.001
- link femur_LF: geometry collision mesh filename=package://robot_gazebo/meshes/razbot/femur.stl scale=0.001 0.001 0.001; visual mesh filename=package://robot_gazebo/meshes/razbot/femur.stl scale=0.001 0.001 0.001
- link femur_LM: geometry collision mesh filename=package://robot_gazebo/meshes/razbot/femur.stl scale=0.001 0.001 0.001; visual mesh filename=package://robot_gazebo/meshes/razbot/femur.stl scale=0.001 0.001 0.001
- link femur_LR: geometry collision mesh filename=package://robot_gazebo/meshes/razbot/femur.stl scale=0.001 0.001 0.001; visual mesh filename=package://robot_gazebo/meshes/razbot/femur.stl scale=0.001 0.001 0.001
- link femur_RF: geometry collision mesh filename=package://robot_gazebo/meshes/razbot/femur.stl scale=0.001 0.001 0.001; visual mesh filename=package://robot_gazebo/meshes/razbot/femur.stl scale=0.001 0.001 0.001
- link femur_RM: geometry collision mesh filename=package://robot_gazebo/meshes/razbot/femur.stl scale=0.001 0.001 0.001; visual mesh filename=package://robot_gazebo/meshes/razbot/femur.stl scale=0.001 0.001 0.001
- link femur_RR: geometry collision mesh filename=package://robot_gazebo/meshes/razbot/femur.stl scale=0.001 0.001 0.001; visual mesh filename=package://robot_gazebo/meshes/razbot/femur.stl scale=0.001 0.001 0.001
- link tibia_LF: geometry collision mesh filename=package://robot_gazebo/meshes/razbot/tibia.stl scale=0.001 0.001 0.001; visual mesh filename=package://robot_gazebo/meshes/razbot/tibia.stl scale=0.001 0.001 0.001
- link tibia_LM: geometry collision mesh filename=package://robot_gazebo/meshes/razbot/tibia.stl scale=0.001 0.001 0.001; visual mesh filename=package://robot_gazebo/meshes/razbot/tibia.stl scale=0.001 0.001 0.001
- link tibia_LR: geometry collision mesh filename=package://robot_gazebo/meshes/razbot/tibia.stl scale=0.001 0.001 0.001; visual mesh filename=package://robot_gazebo/meshes/razbot/tibia.stl scale=0.001 0.001 0.001
- link tibia_RF: geometry collision mesh filename=package://robot_gazebo/meshes/razbot/tibia.stl scale=0.001 0.001 0.001; visual mesh filename=package://robot_gazebo/meshes/razbot/tibia.stl scale=0.001 0.001 0.001
- link tibia_RM: geometry collision mesh filename=package://robot_gazebo/meshes/razbot/tibia.stl scale=0.001 0.001 0.001; visual mesh filename=package://robot_gazebo/meshes/razbot/tibia.stl scale=0.001 0.001 0.001
- link tibia_RR: geometry collision mesh filename=package://robot_gazebo/meshes/razbot/tibia.stl scale=0.001 0.001 0.001; visual mesh filename=package://robot_gazebo/meshes/razbot/tibia.stl scale=0.001 0.001 0.001

File: urdf/tb3_burger.urdf (robot description, URDF)
Before this commit: robot tb3_burger, 7 links, 6 joints
Links:
- link base_link: geometry collision box size=0.140 0.140 0.143; visual mesh filename=package://robot_gazebo/meshes/tb3/burger_base.stl scale=0.001 0.001 0.001
- link base_scan: geometry collision cylinder length=0.0315 radius=0.055; visual mesh filename=package://robot_gazebo/meshes/tb3/lds.stl scale=0.001 0.001 0.001
- link wheel_left_link: geometry collision cylinder length=0.018 radius=0.033; visual mesh filename=package://robot_gazebo/meshes/tb3/left_tire.stl scale=0.001 0.001 0.001
- link wheel_right_link: geometry collision cylinder length=0.018 radius=0.033; visual mesh filename=package://robot_gazebo/meshes/tb3/right_tire.stl scale=0.001 0.001 0.001

File: urdf/tb3_waffle.urdf (robot description, URDF)
Before this commit: robot tb3_waffle, 13 links, 12 joints
Links:
- link base_link: geometry collision box size=0.266 0.266 0.094; visual mesh filename=package://robot_gazebo/meshes/tb3/waffle_base.stl scale=0.001 0.001 0.001
- link base_scan: geometry collision cylinder length=0.0315 radius=0.055; visual mesh filename=package://robot_gazebo/meshes/tb3/lds.stl scale=0.001 0.001 0.001
- link camera_link: geometry collision box size=0.012 0.132 0.020; visual mesh filename=package://robot_gazebo/meshes/tb3/r200.dae
- link wheel_left_link: geometry collision cylinder length=0.018 radius=0.033; visual mesh filename=package://robot_gazebo/meshes/tb3/left_tire.stl scale=0.001 0.001 0.001
- link wheel_right_link: geometry collision cylinder length=0.018 radius=0.033; visual mesh filename=package://robot_gazebo/meshes/tb3/right_tire.stl scale=0.001 0.001 0.001

File: urdf/tb3_waffle_pi.urdf (robot description, URDF)
Before this commit: robot tb3_waffle_pi, 11 links, 10 joints
Links:
- link base_link: geometry collision box size=0.266 0.266 0.094; visual mesh filename=package://robot_gazebo/meshes/tb3/waffle_pi_base.stl scale=0.001 0.001 0.001
- link base_scan: geometry collision cylinder length=0.0315 radius=0.055; visual mesh filename=package://robot_gazebo/meshes/tb3/lds.stl scale=0.001 0.001 0.001
- link wheel_left_link: geometry collision cylinder length=0.018 radius=0.033; visual mesh filename=package://robot_gazebo/meshes/tb3/left_tire.stl scale=0.001 0.001 0.001
- link wheel_right_link: geometry collision cylinder length=0.018 radius=0.033; visual mesh filename=package://robot_gazebo/meshes/tb3/right_tire.stl scale=0.001 0.001 0.001

File: urdf/twr.urdf (robot description, URDF)
Before this commit: robot twr, 7 links, 6 joints
Links:
- link base_link: geometry collision box size=0.7 0.39 0.2; visual mesh filename=package://robot_gazebo/meshes/twr/robot_base.stl
