Commit message: u

File: urdf/golem.urdf (robot description, URDF)
Before this commit: robot Golem, 42 links, 41 joints
Links:
- removed link body_link
- added link base_footprint
- link base_link: mass None -> 0.00001; geometry collision mesh filename=package://robot_gazebo/meshes/golem/body.stl scale=0.001 0.001 0.001; visual mesh filename=package://robot_gazebo/meshes/golem/body.stl scale=0.001 0.001 0.001
Joints:
- joint base_joint: child body_link -> base_link; parent base_link -> base_footprint
- joint camera_depth_joint: parent body_link -> base_link
- joint camera_rgb_joint: parent body_link -> base_link
- joint imu_joint: parent body_link -> base_link
- joint leg_center_joint_LF: parent body_link -> base_link
- joint leg_center_joint_LM: parent body_link -> base_link
- joint leg_center_joint_LR: parent body_link -> base_link
- joint leg_center_joint_RF: parent body_link -> base_link
- joint leg_center_joint_RM: parent body_link -> base_link
- joint leg_center_joint_RR: parent body_link -> base_link
- joint pan_joint: parent body_link -> base_link

File: xacro/golem.xacro (robot description, xacro)
@@ -33,14 +33,14 @@
         <color rgba="1.0 1.0 1.0 1.0"/>
     </material>
-<!-- ****************************************************** Base Link ****************************************************************  -->
-    <link name="base_link"/>
+<!-- ****************************************************** Base Footprint ***********************************************************  -->
+    <link name="base_footprint"/>
 <!-- ****************************************************** Base Joint ***************************************************************  -->
     <joint name="base_joint" type="fixed">
-        <parent link="base_link"/>
-        <child link="body_link"/>
+        <parent link="base_footprint"/>
+        <child link="base_link"/>
         <origin xyz="0.0 0.0 0.064" rpy="0.0 0.0 0.0"/>
     </joint>
-<!-- ****************************************************** Body Link ****************************************************************  -->
-    <link name="body_link">
+<!-- ****************************************************** Base Link ****************************************************************  -->
+    <link name="base_link">
         <visual>
             <origin xyz="0.0 0.0 0.0" rpy="0.0 0.0 0.0"/>
@@ -53,5 +53,5 @@
             <origin xyz="0.0 0.0 0.0" rpy="0.0 0.0 0.0"/>
             <geometry>
-                <mesh filename="package://robot_gazebo/meshes/golem/body.stl" scale="0.001 0.001 0.001"/>
+                <mesh filename="${mesh_path}body.stl" scale="0.001 0.001 0.001"/>
             </geometry>
             <material name="blue"/>
@@ -68,5 +68,5 @@
 <!-- ****************************************************** Camera RGB Joint *********************************************************  -->
     <joint name="camera_rgb_joint" type="fixed">
-        <parent link="body_link"/>
+        <parent link="base_link"/>
         <child link="camera_rgb_optical_frame"/>
         <origin xyz="0.150 0.0255 0.034" rpy="${pi/2} ${pi} ${pi/2}"/>
@@ -85,5 +85,5 @@
 <!-- ****************************************************** Camera Depth Joint *******************************************************  -->
     <joint name="camera_depth_joint" type="fixed">
-        <parent link="body_link"/>
+        <parent link="base_link"/>
         <child link="camera_depth_optical_frame"/>
         <origin xyz="0.150 -0.0225 0.034" rpy="${pi/2} ${pi} ${pi/2}"/>
@@ -102,5 +102,5 @@
 <!-- ****************************************************** IMU Joint ****************************************************************  -->
     <joint name="imu_joint" type="fixed">
-        <parent link="body_link"/>
+        <parent link="base_link"/>
         <child link="imu_link"/>
         <origin xyz="0.0 0.0 0.034" rpy="0.0 0.0 0.0"/>
@@ -119,5 +119,5 @@
 <!-- ****************************************************** Pan Joint ****************************************************************  -->
     <joint name="pan_joint" type="revolute">
-        <parent link="body_link"/>
+        <parent link="base_link"/>
         <child link="pan_link"/>
         <origin xyz="0.1 0.0 0.034" rpy="0.0 0.0 0.0"/>
@@ -141,5 +141,5 @@
     <joint name="leg_center_joint_${side}${position}" type="fixed">
         <origin xyz="${x} ${y} 0.0" rpy="0.0 0.0 0.0"/>
-        <parent link="body_link"/>
+        <parent link="base_link"/>
         <child link="leg_center_${side}${position}"/>
     </joint>
@@ -179,5 +179,5 @@
             <origin xyz="0.0 0.0 0.0" rpy="0.0 0.0 0.0"/>
             <geometry>
-                <mesh filename="package://robot_gazebo/meshes/golem/coxa.stl" scale="0.001 0.001 0.001"/>
+                <mesh filename="${mesh_path}coxa.stl" scale="0.001 0.001 0.001"/>
             </geometry>
             <material name="green"/>
@@ -186,5 +186,5 @@
             <origin xyz="0.0 0.0 0.0" rpy="0.0 0.0 0.0" />
             <geometry>
-                <mesh filename="package://robot_gazebo/meshes/golem/coxa.stl" scale="0.001 0.001 0.001"/>
+                <mesh filename="${mesh_path}coxa.stl" scale="0.001 0.001 0.001"/>
             </geometry>
             <material name="green"/>
@@ -223,5 +223,5 @@
             <origin xyz="0.0 0.0 0.0" rpy="0.0 0.0 0.0"/>
             <geometry>
-                <mesh filename="package://robot_gazebo/meshes/golem/femur.stl" scale="0.001 0.001 0.001"/>
+                <mesh filename="${mesh_path}femur.stl" scale="0.001 0.001 0.001"/>
             </geometry>
             <material name="red"/>
@@ -230,5 +230,5 @@
             <origin xyz="0.0 0.0 0.0" rpy="0.0 0.0 0.0" />
             <geometry>
-                <mesh filename="package://robot_gazebo/meshes/golem/femur.stl" scale="0.001 0.001 0.001"/>
+                <mesh filename="${mesh_path}femur.stl" scale="0.001 0.001 0.001"/>
             </geometry>
             <material name="read"/>
@@ -267,5 +267,5 @@
             <origin xyz="0.0 0.0 0.0" rpy="0.0 0.0 0.0"/>
             <geometry>
-                <mesh filename="package://robot_gazebo/meshes/golem/tibia.stl" scale="0.001 0.001 0.001"/>
+                <mesh filename="${mesh_path}tibia.stl" scale="0.001 0.001 0.001"/>
             </geometry>
             <material name="green"/>
@@ -274,5 +274,5 @@
             <origin xyz="0.0 0.0 0.0" rpy="0.0 0.0 0.0" />
             <geometry>
-                <mesh filename="package://robot_gazebo/meshes/golem/tibia.stl" scale="0.001 0.001 0.001"/>
+                <mesh filename="${mesh_path}tibia.stl" scale="0.001 0.001 0.001"/>
             </geometry>
             <material name="green"/>
@@ -311,5 +311,5 @@
             <origin xyz="0.0 0.0 0.0" rpy="0.0 0.0 0.0"/>
             <geometry>
-                <mesh filename="package://robot_gazebo/meshes/golem/tarsus.stl" scale="0.001 0.001 0.001"/>
+                <mesh filename="${mesh_path}tarsus.stl" scale="0.001 0.001 0.001"/>
             </geometry>
             <material name="red"/>
@@ -318,5 +318,5 @@
             <origin xyz="0.0 0.0 0.0" rpy="0.0 0.0 0.0" />
             <geometry>
-                <mesh filename="package://robot_gazebo/meshes/golem/tarsus.stl" scale="0.001 0.001 0.001"/>
+                <mesh filename="${mesh_path}tarsus.stl" scale="0.001 0.001 0.001"/>
             </geometry>
             <material name="red"/>
@@ -349,5 +349,5 @@
     </link>
 <!-- ****************************************************** Gazebo Colors*************************************************************  -->
-    <gazebo reference="body_link">
+    <gazebo reference="base_link">
         <material>Gazebo/Blue</material>
     </gazebo>

File: xacro/twr.xacro (robot description, xacro)
@@ -6,11 +6,11 @@
 <!-- *********************************************************************************************************************************  -->
 <!-- ****************************************************** Parameters ***************************************************************  -->
+  <xacro:property name="mesh_path"    value="package://robot_gazebo/meshes/twr/"/>
 <!-- Define the size of the robot's main chassis in meters                                                                              -->
-  <xacro:property name="base_width" value="0.39"/>
-  <xacro:property name="base_length" value="0.70"/>
-  <xacro:property name="base_height" value="0.20"/>
-<!-- Define the shape of the robot's two back wheels in meters                                                                          -->
+  <xacro:property name="base_width"   value="0.39"/>
+  <xacro:property name="base_length"  value="0.70"/>
+  <xacro:property name="base_height"  value="0.20"/>
   <xacro:property name="wheel_radius" value="0.14"/>
-  <xacro:property name="wheel_width" value="0.06"/>
+  <xacro:property name="wheel_width"  value="0.06"/>
 <!-- x-axis points forward, y-axis points to left, z-axis points upwards                                                                -->
 <!-- Define the gap between the wheel and chassis along y-axis in meters                                                                -->
@@ -75,5 +75,5 @@
       <origin xyz="0 0 -0.05" rpy="1.5707963267949 0 3.141592654"/>
       <geometry>
-        <mesh filename="package://robot_gazebo/meshes/twr/robot_base.stl" />
+        <mesh filename="${mesh_path}robot_base.stl" />
       </geometry>
       <material name="red"/>
@@ -161,16 +161,16 @@
 <!-- ****************************************************** LIDAR Link ***************************************************************  -->
   <link name="lidar_link">
-    <collision>
-     <origin xyz="0 0 0" rpy="0 0 0"/>
-     <geometry>
-      <cylinder radius="0.0508" length="0.18"/>
-     </geometry>
-    </collision>
+      <collision>
+      <origin xyz="0 0 0" rpy="0 0 0"/>
+      <geometry>
+        <cylinder radius="0.0508" length="0.18"/>
+      </geometry>
+      </collision>
     <visual>
-     <origin xyz="0 0 0" rpy="0 0 0"/>
-     <geometry>
-      <cylinder radius="0.0508" length="0.18"/>
-     </geometry>
-     <material name="green"/>
+      <origin xyz="0 0 0" rpy="0 0 0"/>
+      <geometry>
+        <cylinder radius="0.0508" length="0.18"/>
+      </geometry>
+      <material name="green"/>
     </visual>
     <inertial>

Commit message: u

File: urdf/golem.urdf (robot description, URDF)
Before this commit: robot Golem, 42 links, 41 joints
Joints:
- joint coxa_joint_LF: limit lower=-3.14 upper=3.14 effort=6.0 velocity=0.524 -> lower=-3.141592653589793 upper=3.141592653589793 effort=6.0 velocity=0.524
- joint coxa_joint_LM: limit lower=-3.14 upper=3.14 effort=6.0 velocity=0.524 -> lower=-3.141592653589793 upper=3.141592653589793 effort=6.0 velocity=0.524
- joint coxa_joint_LR: limit lower=-3.14 upper=3.14 effort=6.0 velocity=0.524 -> lower=-3.141592653589793 upper=3.141592653589793 effort=6.0 velocity=0.524
- joint coxa_joint_RF: limit lower=-3.14 upper=3.14 effort=6.0 velocity=0.524 -> lower=-3.141592653589793 upper=3.141592653589793 effort=6.0 velocity=0.524
- joint coxa_joint_RM: limit lower=-3.14 upper=3.14 effort=6.0 velocity=0.524 -> lower=-3.141592653589793 upper=3.141592653589793 effort=6.0 velocity=0.524
- joint coxa_joint_RR: limit lower=-3.14 upper=3.14 effort=6.0 velocity=0.524 -> lower=-3.141592653589793 upper=3.141592653589793 effort=6.0 velocity=0.524
- joint femur_joint_LF: limit lower=-3.14 upper=3.14 effort=6.0 velocity=0.524 -> lower=-3.141592653589793 upper=3.141592653589793 effort=6.0 velocity=0.524
- joint femur_joint_LM: limit lower=-3.14 upper=3.14 effort=6.0 velocity=0.524 -> lower=-3.141592653589793 upper=3.141592653589793 effort=6.0 velocity=0.524
- joint femur_joint_LR: limit lower=-3.14 upper=3.14 effort=6.0 velocity=0.524 -> lower=-3.141592653589793 upper=3.141592653589793 effort=6.0 velocity=0.524
- joint femur_joint_RF: limit lower=-3.14 upper=3.14 effort=6.0 velocity=0.524 -> lower=-3.141592653589793 upper=3.141592653589793 effort=6.0 velocity=0.524
- joint femur_joint_RM: limit lower=-3.14 upper=3.14 effort=6.0 velocity=0.524 -> lower=-3.141592653589793 upper=3.141592653589793 effort=6.0 velocity=0.524
- joint femur_joint_RR: limit lower=-3.14 upper=3.14 effort=6.0 velocity=0.524 -> lower=-3.141592653589793 upper=3.141592653589793 effort=6.0 velocity=0.524
- joint pan_joint: limit lower=-3.14 upper=3.14 effort=6.0 velocity=0.524 -> lower=-3.141592653589793 upper=3.141592653589793 effort=6.0 velocity=0.524
- joint tarsus_joint_LF: limit lower=-3.14 upper=3.14 effort=6.0 velocity=0.524 -> lower=-3.141592653589793 upper=3.141592653589793 effort=6.0 velocity=0.524
- joint tarsus_joint_LM: limit lower=-3.14 upper=3.14 effort=6.0 velocity=0.524 -> lower=-3.141592653589793 upper=3.141592653589793 effort=6.0 velocity=0.524
- joint tarsus_joint_LR: limit lower=-3.14 upper=3.14 effort=6.0 velocity=0.524 -> lower=-3.141592653589793 upper=3.141592653589793 effort=6.0 velocity=0.524
- joint tarsus_joint_RF: limit lower=-3.14 upper=3.14 effort=6.0 velocity=0.524 -> lower=-3.141592653589793 upper=3.141592653589793 effort=6.0 velocity=0.524
- joint tarsus_joint_RM: limit lower=-3.14 upper=3.14 effort=6.0 velocity=0.524 -> lower=-3.141592653589793 upper=3.141592653589793 effort=6.0 velocity=0.524
- joint tarsus_joint_RR: limit lower=-3.14 upper=3.14 effort=6.0 velocity=0.524 -> lower=-3.141592653589793 upper=3.141592653589793 effort=6.0 velocity=0.524
- joint tibia_joint_LF: limit lower=-3.14 upper=3.14 effort=6.0 velocity=0.524 -> lower=-3.141592653589793 upper=3.141592653589793 effort=6.0 velocity=0.524
- joint tibia_joint_LM: limit lower=-3.14 upper=3.14 effort=6.0 velocity=0.524 -> lower=-3.141592653589793 upper=3.141592653589793 effort=6.0 velocity=0.524
- joint tibia_joint_LR: limit lower=-3.14 upper=3.14 effort=6.0 velocity=0.524 -> lower=-3.141592653589793 upper=3.141592653589793 effort=6.0 velocity=0.524
- joint tibia_joint_RF: limit lower=-3.14 upper=3.14 effort=6.0 velocity=0.524 -> lower=-3.141592653589793 upper=3.141592653589793 effort=6.0 velocity=0.524
- joint tibia_joint_RM: limit lower=-3.14 upper=3.14 effort=6.0 velocity=0.524 -> lower=-3.141592653589793 upper=3.141592653589793 effort=6.0 velocity=0.524
- joint tibia_joint_RR: limit lower=-3.14 upper=3.14 effort=6.0 velocity=0.524 -> lower=-3.141592653589793 upper=3.141592653589793 effort=6.0 velocity=0.524

File: urdf/pxm3.urdf (robot description, URDF)
Before this commit: robot pxm3, 26 links, 25 joints
Joints:
- joint j_c1_LF: origin xyz=0.1248    0.06164   0.001116 rpy=0 4.7123 2.356194490192345 -> xyz= 0.1248   0.06164  0.001116 rpy=0 4.7123  2.356194490192345
- joint j_c1_LM: origin xyz=0         0.1034    0.001116 rpy=0 4.7123 3.14159 -> xyz= 0        0.1034   0.001116 rpy=0 4.7123  3.14159
- joint j_c1_LR: origin xyz=-0.1248   0.06164   0.001116 rpy=0 4.7123 3.9269908169872414 -> xyz=-0.1248   0.06164  0.001116 rpy=0 4.7123  3.9269908169872414
- joint j_c1_RF: origin xyz=0.1248    -0.06164  0.001116 rpy=0 4.7123 0.7853981633974483 -> xyz= 0.1248  -0.06164  0.001116 rpy=0 4.7123  0.7853981633974483
- joint j_c1_RM: origin xyz=0         -0.1034   0.001116 rpy=0 4.7123 0 -> xyz= 0       -0.1034   0.001116 rpy=0 4.7123  0
- joint j_c1_RR: origin xyz=-0.1248   -0.06164  0.001116 rpy=0 4.7123 -0.7853981633974483 -> xyz=-0.1248  -0.06164  0.001116 rpy=0 4.7123 -0.7853981633974483
