Commit message: u

File: urdf/golem.urdf (robot description, URDF)
Before this commit: robot Golem, 42 links, 41 joints
Joints:
- joint coxa_joint_LF: limit lower=-3.141592653589793 upper=3.141592653589793 effort=6.0 velocity=0.524 -> lower=-3.141592653589793 upper=3.141592653589793 effort=6.0 velocity=5.235987755982989
- joint coxa_joint_LM: limit lower=-3.141592653589793 upper=3.141592653589793 effort=6.0 velocity=0.524 -> lower=-3.141592653589793 upper=3.141592653589793 effort=6.0 velocity=5.235987755982989
- joint coxa_joint_LR: limit lower=-3.141592653589793 upper=3.141592653589793 effort=6.0 velocity=0.524 -> lower=-3.141592653589793 upper=3.141592653589793 effort=6.0 velocity=5.235987755982989
- joint coxa_joint_RF: limit lower=-3.141592653589793 upper=3.141592653589793 effort=6.0 velocity=0.524 -> lower=-3.141592653589793 upper=3.141592653589793 effort=6.0 velocity=5.235987755982989
- joint coxa_joint_RM: limit lower=-3.141592653589793 upper=3.141592653589793 effort=6.0 velocity=0.524 -> lower=-3.141592653589793 upper=3.141592653589793 effort=6.0 velocity=5.235987755982989
- joint coxa_joint_RR: limit lower=-3.141592653589793 upper=3.141592653589793 effort=6.0 velocity=0.524 -> lower=-3.141592653589793 upper=3.141592653589793 effort=6.0 velocity=5.235987755982989
- joint femur_joint_LF: limit lower=-3.141592653589793 upper=3.141592653589793 effort=6.0 velocity=0.524 -> lower=-3.141592653589793 upper=3.141592653589793 effort=6.0 velocity=5.235987755982989
- joint femur_joint_LM: limit lower=-3.141592653589793 upper=3.141592653589793 effort=6.0 velocity=0.524 -> lower=-3.141592653589793 upper=3.141592653589793 effort=6.0 velocity=5.235987755982989
- joint femur_joint_LR: limit lower=-3.141592653589793 upper=3.141592653589793 effort=6.0 velocity=0.524 -> lower=-3.141592653589793 upper=3.141592653589793 effort=6.0 velocity=5.235987755982989
- joint femur_joint_RF: limit lower=-3.141592653589793 upper=3.141592653589793 effort=6.0 velocity=0.524 -> lower=-3.141592653589793 upper=3.141592653589793 effort=6.0 velocity=5.235987755982989
- joint femur_joint_RM: limit lower=-3.141592653589793 upper=3.141592653589793 effort=6.0 velocity=0.524 -> lower=-3.141592653589793 upper=3.141592653589793 effort=6.0 velocity=5.235987755982989
- joint femur_joint_RR: limit lower=-3.141592653589793 upper=3.141592653589793 effort=6.0 velocity=0.524 -> lower=-3.141592653589793 upper=3.141592653589793 effort=6.0 velocity=5.235987755982989
- joint pan_joint: limit lower=-3.141592653589793 upper=3.141592653589793 effort=6.0 velocity=0.524 -> lower=-3.141592653589793 upper=3.141592653589793 effort=6.0 velocity=5.235987755982989
- joint tarsus_joint_LF: limit lower=-3.141592653589793 upper=3.141592653589793 effort=6.0 velocity=0.524 -> lower=-3.141592653589793 upper=3.141592653589793 effort=6.0 velocity=5.235987755982989
- joint tarsus_joint_LM: limit lower=-3.141592653589793 upper=3.141592653589793 effort=6.0 velocity=0.524 -> lower=-3.141592653589793 upper=3.141592653589793 effort=6.0 velocity=5.235987755982989
- joint tarsus_joint_LR: limit lower=-3.141592653589793 upper=3.141592653589793 effort=6.0 velocity=0.524 -> lower=-3.141592653589793 upper=3.141592653589793 effort=6.0 velocity=5.235987755982989
- joint tarsus_joint_RF: limit lower=-3.141592653589793 upper=3.141592653589793 effort=6.0 velocity=0.524 -> lower=-3.141592653589793 upper=3.141592653589793 effort=6.0 velocity=5.235987755982989
- joint tarsus_joint_RM: limit lower=-3.141592653589793 upper=3.141592653589793 effort=6.0 velocity=0.524 -> lower=-3.141592653589793 upper=3.141592653589793 effort=6.0 velocity=5.235987755982989
- joint tarsus_joint_RR: limit lower=-3.141592653589793 upper=3.141592653589793 effort=6.0 velocity=0.524 -> lower=-3.141592653589793 upper=3.141592653589793 effort=6.0 velocity=5.235987755982989
- joint tibia_joint_LF: limit lower=-3.141592653589793 upper=3.141592653589793 effort=6.0 velocity=0.524 -> lower=-3.141592653589793 upper=3.141592653589793 effort=6.0 velocity=5.235987755982989
- joint tibia_joint_LM: limit lower=-3.141592653589793 upper=3.141592653589793 effort=6.0 velocity=0.524 -> lower=-3.141592653589793 upper=3.141592653589793 effort=6.0 velocity=5.235987755982989
- joint tibia_joint_LR: limit lower=-3.141592653589793 upper=3.141592653589793 effort=6.0 velocity=0.524 -> lower=-3.141592653589793 upper=3.141592653589793 effort=6.0 velocity=5.235987755982989
- joint tibia_joint_RF: limit lower=-3.141592653589793 upper=3.141592653589793 effort=6.0 velocity=0.524 -> lower=-3.141592653589793 upper=3.141592653589793 effort=6.0 velocity=5.235987755982989
- joint tibia_joint_RM: limit lower=-3.141592653589793 upper=3.141592653589793 effort=6.0 velocity=0.524 -> lower=-3.141592653589793 upper=3.141592653589793 effort=6.0 velocity=5.235987755982989
- joint tibia_joint_RR: limit lower=-3.141592653589793 upper=3.141592653589793 effort=6.0 velocity=0.524 -> lower=-3.141592653589793 upper=3.141592653589793 effort=6.0 velocity=5.235987755982989

File: urdf/pxm3.urdf (robot description, URDF)
Before this commit: robot pxm3, 26 links, 25 joints
Joints:
- joint j_c1_LF: limit lower=-2.6179939 upper=2.6179939 effort=2.8 velocity=5.6548668 -> lower=-2.6179938779914944 upper=2.6179938779914944 effort=2.8 velocity=5.654866776461628
- joint j_c1_LM: limit lower=-2.6179939 upper=2.6179939 effort=2.8 velocity=5.6548668 -> lower=-2.6179938779914944 upper=2.6179938779914944 effort=2.8 velocity=5.654866776461628
- joint j_c1_LR: limit lower=-2.6179939 upper=2.6179939 effort=2.8 velocity=5.6548668 -> lower=-2.6179938779914944 upper=2.6179938779914944 effort=2.8 velocity=5.654866776461628
- joint j_c1_RF: limit lower=-2.6179939 upper=2.6179939 effort=2.8 velocity=5.6548668 -> lower=-2.6179938779914944 upper=2.6179938779914944 effort=2.8 velocity=5.654866776461628
- joint j_c1_RM: limit lower=-2.6179939 upper=2.6179939 effort=2.8 velocity=5.6548668 -> lower=-2.6179938779914944 upper=2.6179938779914944 effort=2.8 velocity=5.654866776461628
- joint j_c1_RR: limit lower=-2.6179939 upper=2.6179939 effort=2.8 velocity=5.6548668 -> lower=-2.6179938779914944 upper=2.6179938779914944 effort=2.8 velocity=5.654866776461628
- joint j_thigh_LF: limit lower=-2.6179939 upper=2.6179939 effort=2.8 velocity=5.6548668 -> lower=-2.6179938779914944 upper=2.6179938779914944 effort=2.8 velocity=5.654866776461628
- joint j_thigh_LM: limit lower=-2.6179939 upper=2.6179939 effort=2.8 velocity=5.6548668 -> lower=-2.6179938779914944 upper=2.6179938779914944 effort=2.8 velocity=5.654866776461628
- joint j_thigh_LR: limit lower=-2.6179939 upper=2.6179939 effort=2.8 velocity=5.6548668 -> lower=-2.6179938779914944 upper=2.6179938779914944 effort=2.8 velocity=5.654866776461628
- joint j_thigh_RF: limit lower=-2.6179939 upper=2.6179939 effort=2.8 velocity=5.6548668 -> lower=-2.6179938779914944 upper=2.6179938779914944 effort=2.8 velocity=5.654866776461628
- joint j_thigh_RM: limit lower=-2.6179939 upper=2.6179939 effort=2.8 velocity=5.6548668 -> lower=-2.6179938779914944 upper=2.6179938779914944 effort=2.8 velocity=5.654866776461628
- joint j_thigh_RR: limit lower=-2.6179939 upper=2.6179939 effort=2.8 velocity=5.6548668 -> lower=-2.6179938779914944 upper=2.6179938779914944 effort=2.8 velocity=5.654866776461628
- joint j_tibia_LF: limit lower=-2.6179939 upper=2.6179939 effort=2.8 velocity=5.6548668 -> lower=-2.6179938779914944 upper=2.6179938779914944 effort=2.8 velocity=5.654866776461628
- joint j_tibia_LM: limit lower=-2.6179939 upper=2.6179939 effort=2.8 velocity=5.6548668 -> lower=-2.6179938779914944 upper=2.6179938779914944 effort=2.8 velocity=5.654866776461628
- joint j_tibia_LR: limit lower=-2.6179939 upper=2.6179939 effort=2.8 velocity=5.6548668 -> lower=-2.6179938779914944 upper=2.6179938779914944 effort=2.8 velocity=5.654866776461628
- joint j_tibia_RF: limit lower=-2.6179939 upper=2.6179939 effort=2.8 velocity=5.6548668 -> lower=-2.6179938779914944 upper=2.6179938779914944 effort=2.8 velocity=5.654866776461628
- joint j_tibia_RM: limit lower=-2.6179939 upper=2.6179939 effort=2.8 velocity=5.6548668 -> lower=-2.6179938779914944 upper=2.6179938779914944 effort=2.8 velocity=5.654866776461628
- joint j_tibia_RR: limit lower=-2.6179939 upper=2.6179939 effort=2.8 velocity=5.6548668 -> lower=-2.6179938779914944 upper=2.6179938779914944 effort=2.8 velocity=5.654866776461628
