Commit message: u

File: urdf/golem.urdf (robot description, URDF)
Before this commit: robot Golem, 42 links, 41 joints
Links:
- link base_link: geometry collision mesh filename=package://bots/meshes/golem/body.stl scale=0.001 0.001 0.001; visual mesh filename=package://bots/meshes/golem/body.stl scale=0.001 0.001 0.001
- link coxa_LF: geometry collision mesh filename=package://bots/meshes/golem/coxa.stl scale=0.001 0.001 0.001; visual mesh filename=package://bots/meshes/golem/coxa.stl scale=0.001 0.001 0.001
- link coxa_LM: geometry collision mesh filename=package://bots/meshes/golem/coxa.stl scale=0.001 0.001 0.001; visual mesh filename=package://bots/meshes/golem/coxa.stl scale=0.001 0.001 0.001
- link coxa_LR: geometry collision mesh filename=package://bots/meshes/golem/coxa.stl scale=0.001 0.001 0.001; visual mesh filename=package://bots/meshes/golem/coxa.stl scale=0.001 0.001 0.001
- link coxa_RF: geometry collision mesh filename=package://bots/meshes/golem/coxa.stl scale=0.001 0.001 0.001; visual mesh filename=package://bots/meshes/golem/coxa.stl scale=0.001 0.001 0.001
- link coxa_RM: geometry collision mesh filename=package://bots/meshes/golem/coxa.stl scale=0.001 0.001 0.001; visual mesh filename=package://bots/meshes/golem/coxa.stl scale=0.001 0.001 0.001
- link coxa_RR: geometry collision mesh filename=package://bots/meshes/golem/coxa.stl scale=0.001 0.001 0.001; visual mesh filename=package://bots/meshes/golem/coxa.stl scale=0.001 0.001 0.001
- link femur_LF: geometry collision mesh filename=package://bots/meshes/golem/femur.stl scale=0.001 0.001 0.001; visual mesh filename=package://bots/meshes/golem/femur.stl scale=0.001 0.001 0.001
- link femur_LM: geometry collision mesh filename=package://bots/meshes/golem/femur.stl scale=0.001 0.001 0.001; visual mesh filename=package://bots/meshes/golem/femur.stl scale=0.001 0.001 0.001
- link femur_LR: geometry collision mesh filename=package://bots/meshes/golem/femur.stl scale=0.001 0.001 0.001; visual mesh filename=package://bots/meshes/golem/femur.stl scale=0.001 0.001 0.001
- link femur_RF: geometry collision mesh filename=package://bots/meshes/golem/femur.stl scale=0.001 0.001 0.001; visual mesh filename=package://bots/meshes/golem/femur.stl scale=0.001 0.001 0.001
- link femur_RM: geometry collision mesh filename=package://bots/meshes/golem/femur.stl scale=0.001 0.001 0.001; visual mesh filename=package://bots/meshes/golem/femur.stl scale=0.001 0.001 0.001
- link femur_RR: geometry collision mesh filename=package://bots/meshes/golem/femur.stl scale=0.001 0.001 0.001; visual mesh filename=package://bots/meshes/golem/femur.stl scale=0.001 0.001 0.001
- link tarsus_LF: geometry collision mesh filename=package://bots/meshes/golem/tarsus.stl scale=0.001 0.001 0.001; visual mesh filename=package://bots/meshes/golem/tarsus.stl scale=0.001 0.001 0.001
- link tarsus_LM: geometry collision mesh filename=package://bots/meshes/golem/tarsus.stl scale=0.001 0.001 0.001; visual mesh filename=package://bots/meshes/golem/tarsus.stl scale=0.001 0.001 0.001
- link tarsus_LR: geometry collision mesh filename=package://bots/meshes/golem/tarsus.stl scale=0.001 0.001 0.001; visual mesh filename=package://bots/meshes/golem/tarsus.stl scale=0.001 0.001 0.001
- link tarsus_RF: geometry collision mesh filename=package://bots/meshes/golem/tarsus.stl scale=0.001 0.001 0.001; visual mesh filename=package://bots/meshes/golem/tarsus.stl scale=0.001 0.001 0.001
- link tarsus_RM: geometry collision mesh filename=package://bots/meshes/golem/tarsus.stl scale=0.001 0.001 0.001; visual mesh filename=package://bots/meshes/golem/tarsus.stl scale=0.001 0.001 0.001
- link tarsus_RR: geometry collision mesh filename=package://bots/meshes/golem/tarsus.stl scale=0.001 0.001 0.001; visual mesh filename=package://bots/meshes/golem/tarsus.stl scale=0.001 0.001 0.001
- link tibia_LF: geometry collision mesh filename=package://bots/meshes/golem/tibia.stl scale=0.001 0.001 0.001; visual mesh filename=package://bots/meshes/golem/tibia.stl scale=0.001 0.001 0.001
- link tibia_LM: geometry collision mesh filename=package://bots/meshes/golem/tibia.stl scale=0.001 0.001 0.001; visual mesh filename=package://bots/meshes/golem/tibia.stl scale=0.001 0.001 0.001
- link tibia_LR: geometry collision mesh filename=package://bots/meshes/golem/tibia.stl scale=0.001 0.001 0.001; visual mesh filename=package://bots/meshes/golem/tibia.stl scale=0.001 0.001 0.001
- link tibia_RF: geometry collision mesh filename=package://bots/meshes/golem/tibia.stl scale=0.001 0.001 0.001; visual mesh filename=package://bots/meshes/golem/tibia.stl scale=0.001 0.001 0.001
- link tibia_RM: geometry collision mesh filename=package://bots/meshes/golem/tibia.stl scale=0.001 0.001 0.001; visual mesh filename=package://bots/meshes/golem/tibia.stl scale=0.001 0.001 0.001
- link tibia_RR: geometry collision mesh filename=package://bots/meshes/golem/tibia.stl scale=0.001 0.001 0.001; visual mesh filename=package://bots/meshes/golem/tibia.stl scale=0.001 0.001 0.001

File: urdf/kr120r2500pro.urdf (robot description, URDF)
Before this commit: robot kr120r2500pro, 11 links, 10 joints
Links:
- link base_link: geometry collision mesh filename=package://bots/meshes/kr120r2500pro/collision/base_link.stl; visual mesh filename=package://bots/meshes/kr120r2500pro/visual/base_link.dae
- link link_1: geometry collision mesh filename=package://bots/meshes/kr120r2500pro/collision/link_1.stl; visual mesh filename=package://bots/meshes/kr120r2500pro/visual/link_1.dae
- link link_2: geometry collision mesh filename=package://bots/meshes/kr120r2500pro/collision/link_2.stl; visual mesh filename=package://bots/meshes/kr120r2500pro/visual/link_2.dae
- link link_3: geometry collision mesh filename=package://bots/meshes/kr120r2500pro/collision/link_3.stl; visual mesh filename=package://bots/meshes/kr120r2500pro/visual/link_3.dae
- link link_4: geometry collision mesh filename=package://bots/meshes/kr120r2500pro/collision/link_4.stl; visual mesh filename=package://bots/meshes/kr120r2500pro/visual/link_4.dae
- link link_5: geometry collision mesh filename=package://bots/meshes/kr120r2500pro/collision/link_5.stl; visual mesh filename=package://bots/meshes/kr120r2500pro/visual/link_5.dae
- link link_6: geometry collision mesh filename=package://bots/meshes/kr120r2500pro/collision/link_6.stl; visual mesh filename=package://bots/meshes/kr120r2500pro/visual/link_6.dae

File: urdf/kr16_2.urdf (robot description, URDF)
Before this commit: robot kr16_2, 11 links, 10 joints
Links:
- link base_link: geometry collision mesh filename=package://bots/meshes/kr16_2/collision/base_link.stl; visual mesh filename=package://bots/meshes/kr16_2/visual/base_link.dae
- link link_1: geometry collision mesh filename=package://bots/meshes/kr16_2/collision/link_1.stl; visual mesh filename=package://bots/meshes/kr16_2/visual/link_1.dae
- link link_2: geometry collision mesh filename=package://bots/meshes/kr16_2/collision/link_2.stl; visual mesh filename=package://bots/meshes/kr16_2/visual/link_2.dae
- link link_3: geometry collision mesh filename=package://bots/meshes/kr16_2/collision/link_3.stl; visual mesh filename=package://bots/meshes/kr16_2/visual/link_3.dae
- link link_4: geometry collision mesh filename=package://bots/meshes/kr16_2/collision/link_4.stl; visual mesh filename=package://bots/meshes/kr16_2/visual/link_4.dae
- link link_5: geometry collision mesh filename=package://bots/meshes/kr16_2/collision/link_5.stl; visual mesh filename=package://bots/meshes/kr16_2/visual/link_5.dae
- link link_6: geometry collision mesh filename=package://bots/meshes/kr16_2/collision/link_6.stl; visual mesh filename=package://bots/meshes/kr16_2/visual/link_6.dae

File: urdf/kr3r540.urdf (robot description, URDF)
Before this commit: robot kr3r540, 11 links, 10 joints
Links:
- link base_link: geometry collision mesh filename=package://bots/meshes/kr3r540/collision/base_link.stl; visual mesh filename=package://bots/meshes/kr3r540/visual/base_link.stl
- link link_1: geometry collision mesh filename=package://bots/meshes/kr3r540/collision/link_1.stl; visual mesh filename=package://bots/meshes/kr3r540/visual/link_1.stl
- link link_2: geometry collision mesh filename=package://bots/meshes/kr3r540/collision/link_2.stl; visual mesh filename=package://bots/meshes/kr3r540/visual/link_2.stl
- link link_3: geometry collision mesh filename=package://bots/meshes/kr3r540/collision/link_3.stl; visual mesh filename=package://bots/meshes/kr3r540/visual/link_3.stl
- link link_4: geometry collision mesh filename=package://bots/meshes/kr3r540/collision/link_4.stl; visual mesh filename=package://bots/meshes/kr3r540/visual/link_4.stl
- link link_5: geometry collision mesh filename=package://bots/meshes/kr3r540/collision/link_5.stl; visual mesh filename=package://bots/meshes/kr3r540/visual/link_5.stl
- link link_6: geometry collision mesh filename=package://bots/meshes/kr3r540/collision/link_6.stl; visual mesh filename=package://bots/meshes/kr3r540/visual/link_6.stl

File: urdf/kr5_arc.urdf (robot description, URDF)
Before this commit: robot kr5_arc, 11 links, 10 joints
Links:
- link base_link: geometry collision mesh filename=package://bots/meshes/kr5_arc/collision/base_link.stl; visual mesh filename=package://bots/meshes/kr5_arc/visual/base_link.dae
- link link_1: geometry collision mesh filename=package://bots/meshes/kr5_arc/collision/link_1.stl; visual mesh filename=package://bots/meshes/kr5_arc/visual/link_1.dae
- link link_2: geometry collision mesh filename=package://bots/meshes/kr5_arc/collision/link_2.stl; visual mesh filename=package://bots/meshes/kr5_arc/visual/link_2.dae
- link link_3: geometry collision mesh filename=package://bots/meshes/kr5_arc/collision/link_3.stl; visual mesh filename=package://bots/meshes/kr5_arc/visual/link_3.dae
- link link_4: geometry collision mesh filename=package://bots/meshes/kr5_arc/collision/link_4.stl; visual mesh filename=package://bots/meshes/kr5_arc/visual/link_4.dae
- link link_5: geometry collision mesh filename=package://bots/meshes/kr5_arc/collision/link_5.stl; visual mesh filename=package://bots/meshes/kr5_arc/visual/link_5.dae
- link link_6: geometry collision mesh filename=package://bots/meshes/kr5_arc/collision/link_6.stl; visual mesh filename=package://bots/meshes/kr5_arc/visual/link_6.dae

File: urdf/lbr_iiwa_14_r820.urdf (robot description, URDF)
Before this commit: robot lbr_iiwa_14_r820, 11 links, 10 joints
Links:
- link base_link: geometry collision mesh filename=package://bots/meshes/lbr_iiwa_14_r820/collision/base_link.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; visual mesh filename=package://bots/meshes/lbr_iiwa_14_r820/visual/base_link.dae
- link link_1: geometry collision mesh filename=package://bots/meshes/lbr_iiwa_14_r820/collision/link_1.stl; visual mesh filename=package://bots/meshes/lbr_iiwa_14_r820/visual/link_1.dae
- link link_2: geometry collision mesh filename=package://bots/meshes/lbr_iiwa_14_r820/collision/link_2.stl; visual mesh filename=package://bots/meshes/lbr_iiwa_14_r820/visual/link_2.dae
- link link_3: geometry collision mesh filename=package://bots/meshes/lbr_iiwa_14_r820/collision/link_3.stl; visual mesh filename=package://bots/meshes/lbr_iiwa_14_r820/visual/link_3.dae
- link link_4: geometry collision mesh filename=package://bots/meshes/lbr_iiwa_14_r820/collision/link_4.stl; visual mesh filename=package://bots/meshes/lbr_iiwa_14_r820/visual/link_4.dae
- link link_5: geometry collision mesh filename=package://bots/meshes/lbr_iiwa_14_r820/collision/link_5.stl; visual mesh filename=package://bots/meshes/lbr_iiwa_14_r820/visual/link_5.dae
- link link_6: geometry collision mesh filename=package://bots/meshes/lbr_iiwa_14_r820/collision/link_6.stl; visual mesh filename=package://bots/meshes/lbr_iiwa_14_r820/visual/link_6.dae
- link link_7: geometry collision mesh filename=package://bots/meshes/lbr_iiwa_14_r820/collision/link_7.stl; visual mesh filename=package://bots/meshes/lbr_iiwa_14_r820/visual/link_7.dae

File: urdf/pxm3.urdf (robot description, URDF)
Before this commit: robot pxm3, 26 links, 25 joints
Links:
- link base_link: geometry collision mesh filename=package://bots/meshes/pxm3/body_coll.STL scale=1 1 1; visual mesh filename=package://bots/meshes/pxm3/body.STL scale=1 1 1
- link c1_LF: geometry collision mesh filename=package://bots/meshes/pxm3/connect_coll.STL scale=1 1 1; visual mesh filename=package://bots/meshes/pxm3/connect.STL scale=1 1 1
- link c1_LM: geometry collision mesh filename=package://bots/meshes/pxm3/connect_coll.STL scale=1 1 1; visual mesh filename=package://bots/meshes/pxm3/connect.STL scale=1 1 1
- link c1_LR: geometry collision mesh filename=package://bots/meshes/pxm3/connect_coll.STL scale=1 1 1; visual mesh filename=package://bots/meshes/pxm3/connect.STL scale=1 1 1
- link c1_RF: geometry collision mesh filename=package://bots/meshes/pxm3/connect_coll.STL scale=1 1 1; visual mesh filename=package://bots/meshes/pxm3/connect.STL scale=1 1 1
- link c1_RM: geometry collision mesh filename=package://bots/meshes/pxm3/connect_coll.STL scale=1 1 1; visual mesh filename=package://bots/meshes/pxm3/connect.STL scale=1 1 1
- link c1_RR: geometry collision mesh filename=package://bots/meshes/pxm3/connect_coll.STL scale=1 1 1; visual mesh filename=package://bots/meshes/pxm3/connect.STL scale=1 1 1
- link c2_LF: geometry collision mesh filename=package://bots/meshes/pxm3/connect_coll.STL scale=1 1 1; visual mesh filename=package://bots/meshes/pxm3/connect.STL scale=1 1 1
- link c2_LM: geometry collision mesh filename=package://bots/meshes/pxm3/connect_coll.STL scale=1 1 1; visual mesh filename=package://bots/meshes/pxm3/connect.STL scale=1 1 1
- link c2_LR: geometry collision mesh filename=package://bots/meshes/pxm3/connect_coll.STL scale=1 1 1; visual mesh filename=package://bots/meshes/pxm3/connect.STL scale=1 1 1
- link c2_RF: geometry collision mesh filename=package://bots/meshes/pxm3/connect_coll.STL scale=1 1 1; visual mesh filename=package://bots/meshes/pxm3/connect.STL scale=1 1 1
- link c2_RM: geometry collision mesh filename=package://bots/meshes/pxm3/connect_coll.STL scale=1 1 1; visual mesh filename=package://bots/meshes/pxm3/connect.STL scale=1 1 1
- link c2_RR: geometry collision mesh filename=package://bots/meshes/pxm3/connect_coll.STL scale=1 1 1; visual mesh filename=package://bots/meshes/pxm3/connect.STL scale=1 1 1
- link thigh_LF: geometry collision mesh filename=package://bots/meshes/pxm3/thigh_l_coll.STL scale=1 1 1; visual mesh filename=package://bots/meshes/pxm3/thigh_l.STL scale=1 1 1
- link thigh_LM: geometry collision mesh filename=package://bots/meshes/pxm3/thigh_l_coll.STL scale=1 1 1; visual mesh filename=package://bots/meshes/pxm3/thigh_l.STL scale=1 1 1
- link thigh_LR: geometry collision mesh filename=package://bots/meshes/pxm3/thigh_l_coll.STL scale=1 1 1; visual mesh filename=package://bots/meshes/pxm3/thigh_l.STL scale=1 1 1
- link thigh_RF: geometry collision mesh filename=package://bots/meshes/pxm3/thigh_l_coll.STL scale=1 1 1; visual mesh filename=package://bots/meshes/pxm3/thigh_l.STL scale=1 1 1
- link thigh_RM: geometry collision mesh filename=package://bots/meshes/pxm3/thigh_l_coll.STL scale=1 1 1; visual mesh filename=package://bots/meshes/pxm3/thigh_l.STL scale=1 1 1
- link thigh_RR: geometry collision mesh filename=package://bots/meshes/pxm3/thigh_l_coll.STL scale=1 1 1; visual mesh filename=package://bots/meshes/pxm3/thigh_l.STL scale=1 1 1
- link tibia_LF: geometry collision mesh filename=package://bots/meshes/pxm3/tibia_l_coll.STL scale=1 1 1; visual mesh filename=package://bots/meshes/pxm3/tibia_l.STL scale=1 1 1
- link tibia_LM: geometry collision mesh filename=package://bots/meshes/pxm3/tibia_l_coll.STL scale=1 1 1; visual mesh filename=package://bots/meshes/pxm3/tibia_l.STL scale=1 1 1
- link tibia_LR: geometry collision mesh filename=package://bots/meshes/pxm3/tibia_l_coll.STL scale=1 1 1; visual mesh filename=package://bots/meshes/pxm3/tibia_l.STL scale=1 1 1
- link tibia_RF: geometry collision mesh filename=package://bots/meshes/pxm3/tibia_l_coll.STL scale=1 1 1; visual mesh filename=package://bots/meshes/pxm3/tibia_l.STL scale=1 1 1
- link tibia_RM: geometry collision mesh filename=package://bots/meshes/pxm3/tibia_l_coll.STL scale=1 1 1; visual mesh filename=package://bots/meshes/pxm3/tibia_l.STL scale=1 1 1
- link tibia_RR: geometry collision mesh filename=package://bots/meshes/pxm3/tibia_l_coll.STL scale=1 1 1; visual mesh filename=package://bots/meshes/pxm3/tibia_l.STL scale=1 1 1

File: urdf/razbot.urdf (robot description, URDF)
Before this commit: robot razbot, 27 links, 26 joints
Links:
- link base_link: geometry collision mesh filename=package://bots/meshes/razbot/body.stl scale=0.001 0.001 0.001; visual mesh filename=package://bots/meshes/razbot/body.stl scale=0.001 0.001 0.001
- link coxa_LF: geometry collision mesh filename=package://bots/meshes/razbot/coxa.stl scale=0.001 0.001 0.001; visual mesh filename=package://bots/meshes/razbot/coxa.stl scale=0.001 0.001 0.001
- link coxa_LM: geometry collision mesh filename=package://bots/meshes/razbot/coxa.stl scale=0.001 0.001 0.001; visual mesh filename=package://bots/meshes/razbot/coxa.stl scale=0.001 0.001 0.001
- link coxa_LR: geometry collision mesh filename=package://bots/meshes/razbot/coxa.stl scale=0.001 0.001 0.001; visual mesh filename=package://bots/meshes/razbot/coxa.stl scale=0.001 0.001 0.001
- link coxa_RF: geometry collision mesh filename=package://bots/meshes/razbot/coxa.stl scale=0.001 0.001 0.001; visual mesh filename=package://bots/meshes/razbot/coxa.stl scale=0.001 0.001 0.001
- link coxa_RM: geometry collision mesh filename=package://bots/meshes/razbot/coxa.stl scale=0.001 0.001 0.001; visual mesh filename=package://bots/meshes/razbot/coxa.stl scale=0.001 0.001 0.001
- link coxa_RR: geometry collision mesh filename=package://bots/meshes/razbot/coxa.stl scale=0.001 0.001 0.001; visual mesh filename=package://bots/meshes/razbot/coxa.stl scale=0.001 0.001 0.001
- link femur_LF: geometry collision mesh filename=package://bots/meshes/razbot/femur.stl scale=0.001 0.001 0.001; visual mesh filename=package://bots/meshes/razbot/femur.stl scale=0.001 0.001 0.001
- link femur_LM: geometry collision mesh filename=package://bots/meshes/razbot/femur.stl scale=0.001 0.001 0.001; visual mesh filename=package://bots/meshes/razbot/femur.stl scale=0.001 0.001 0.001
- link femur_LR: geometry collision mesh filename=package://bots/meshes/razbot/femur.stl scale=0.001 0.001 0.001; visual mesh filename=package://bots/meshes/razbot/femur.stl scale=0.001 0.001 0.001
- link femur_RF: geometry collision mesh filename=package://bots/meshes/razbot/femur.stl scale=0.001 0.001 0.001; visual mesh filename=package://bots/meshes/razbot/femur.stl scale=0.001 0.001 0.001
- link femur_RM: geometry collision mesh filename=package://bots/meshes/razbot/femur.stl scale=0.001 0.001 0.001; visual mesh filename=package://bots/meshes/razbot/femur.stl scale=0.001 0.001 0.001
- link femur_RR: geometry collision mesh filename=package://bots/meshes/razbot/femur.stl scale=0.001 0.001 0.001; visual mesh filename=package://bots/meshes/razbot/femur.stl scale=0.001 0.001 0.001
- link tibia_LF: geometry collision mesh filename=package://bots/meshes/razbot/tibia.stl scale=0.001 0.001 0.001; visual mesh filename=package://bots/meshes/razbot/tibia.stl scale=0.001 0.001 0.001
- link tibia_LM: geometry collision mesh filename=package://bots/meshes/razbot/tibia.stl scale=0.001 0.001 0.001; visual mesh filename=package://bots/meshes/razbot/tibia.stl scale=0.001 0.001 0.001
- link tibia_LR: geometry collision mesh filename=package://bots/meshes/razbot/tibia.stl scale=0.001 0.001 0.001; visual mesh filename=package://bots/meshes/razbot/tibia.stl scale=0.001 0.001 0.001
- link tibia_RF: geometry collision mesh filename=package://bots/meshes/razbot/tibia.stl scale=0.001 0.001 0.001; visual mesh filename=package://bots/meshes/razbot/tibia.stl scale=0.001 0.001 0.001
- link tibia_RM: geometry collision mesh filename=package://bots/meshes/razbot/tibia.stl scale=0.001 0.001 0.001; visual mesh filename=package://bots/meshes/razbot/tibia.stl scale=0.001 0.001 0.001
- link tibia_RR: geometry collision mesh filename=package://bots/meshes/razbot/tibia.stl scale=0.001 0.001 0.001; visual mesh filename=package://bots/meshes/razbot/tibia.stl scale=0.001 0.001 0.001

File: urdf/skidbot.urdf (robot description, URDF)
Before this commit: robot skidbot, 9 links, 8 joints
Links:
- link back_left_wheel: geometry collision mesh filename=package://bots/meshes/skidbot/wheel.dae; visual mesh filename=package://bots/meshes/skidbot/wheel.dae
- link back_right_wheel: geometry collision mesh filename=package://bots/meshes/skidbot/wheel.dae; visual mesh filename=package://bots/meshes/skidbot/wheel.dae
- link base: geometry collision mesh filename=package://bots/meshes/skidbot/base.stl scale=1 1 1; visual mesh filename=package://bots/meshes/skidbot/base.stl scale=1 1 1
- link front_left_wheel: geometry collision mesh filename=package://bots/meshes/skidbot/wheel.dae; visual mesh filename=package://bots/meshes/skidbot/wheel.dae
- link front_right_wheel: geometry collision mesh filename=package://bots/meshes/skidbot/wheel.dae; visual mesh filename=package://bots/meshes/skidbot/wheel.dae
- link hokuyo: geometry collision mesh filename=package://bots/meshes/skidbot/hokuyo.dae; visual mesh filename=package://bots/meshes/skidbot/hokuyo.dae

File: urdf/tb3_burger.urdf (robot description, URDF)
Before this commit: robot tb3_burger, 7 links, 6 joints
Links:
- link base_link: geometry collision box size=0.140 0.140 0.143; visual mesh filename=package://bots/meshes/tb3/burger_base.stl scale=0.001 0.001 0.001
- link base_scan: geometry collision cylinder length=0.0315 radius=0.055; visual mesh filename=package://bots/meshes/tb3/lds.stl scale=0.001 0.001 0.001
- link wheel_left_link: geometry collision cylinder length=0.018 radius=0.033; visual mesh filename=package://bots/meshes/tb3/left_tire.stl scale=0.001 0.001 0.001
- link wheel_right_link: geometry collision cylinder length=0.018 radius=0.033; visual mesh filename=package://bots/meshes/tb3/right_tire.stl scale=0.001 0.001 0.001

File: urdf/tb3_waffle.urdf (robot description, URDF)
Before this commit: robot tb3_waffle, 13 links, 12 joints
Links:
- link base_link: geometry collision box size=0.266 0.266 0.094; visual mesh filename=package://bots/meshes/tb3/waffle_base.stl scale=0.001 0.001 0.001
- link base_scan: geometry collision cylinder length=0.0315 radius=0.055; visual mesh filename=package://bots/meshes/tb3/lds.stl scale=0.001 0.001 0.001
- link camera_link: geometry collision box size=0.012 0.132 0.020; visual mesh filename=package://bots/meshes/tb3/r200.dae
- link wheel_left_link: geometry collision cylinder length=0.018 radius=0.033; visual mesh filename=package://bots/meshes/tb3/left_tire.stl scale=0.001 0.001 0.001
- link wheel_right_link: geometry collision cylinder length=0.018 radius=0.033; visual mesh filename=package://bots/meshes/tb3/right_tire.stl scale=0.001 0.001 0.001
