Commit message: u

File: urdf/tb3_waffle_pi.urdf (robot description, URDF)
Before this commit: robot tb3_waffle_pi, 11 links, 10 joints
Links:
- link base_link: geometry collision box size=0.266 0.266 0.094; visual mesh filename=package://bots/meshes/tb3/waffle_pi_base.stl scale=0.001 0.001 0.001
- link base_scan: geometry collision cylinder length=0.0315 radius=0.055; visual mesh filename=package://bots/meshes/tb3/lds.stl scale=0.001 0.001 0.001
- link wheel_left_link: geometry collision cylinder length=0.018 radius=0.033; visual mesh filename=package://bots/meshes/tb3/left_tire.stl scale=0.001 0.001 0.001
- link wheel_right_link: geometry collision cylinder length=0.018 radius=0.033; visual mesh filename=package://bots/meshes/tb3/right_tire.stl scale=0.001 0.001 0.001

File: urdf/twr.urdf (robot description, URDF)
Before this commit: robot twr, 7 links, 6 joints
Links:
- link base_link: geometry collision box size=0.7 0.39 0.2; visual mesh filename=package://bots/meshes/twr/robot_base.stl

File: xacro/common_kuka_materials.xacro (robot description, xacro)
@@ -1,5 +1,5 @@
 <?xml version="1.0"?>
 <robot xmlns:xacro="http://wiki.ros.org/xacro">
-  <xacro:include filename="$(find robot_gazebo)/xacro/common_kuka_colours.xacro"/>
+  <xacro:include filename="$(find bots)/xacro/common_kuka_colours.xacro"/>
   <xacro:macro name="material_kuka_orange">
     <material name="">

File: xacro/golem.xacro (robot description, xacro)
@@ -6,5 +6,5 @@
 <!-- *********************************************************************************************************************************  -->
 <!-- ****************************************************** Parameters ***************************************************************  -->
-    <xacro:property name="mesh_path"            value="package://robot_gazebo/meshes/golem/"/>
+    <xacro:property name="mesh_path"            value="package://bots/meshes/golem/"/>
     <xacro:property name="body_length_x"        value="0.3556"/>
     <xacro:property name="body_length_y"        value="0.165"/>
@@ -18,6 +18,6 @@
     <xacro:property name="joint_velocity"       value=" ${radians(300)}"/>
 <!-- ****************************************************** Includes *****************************************************************  -->
-  <xacro:include filename="$(find robot_gazebo)/xacro/common_rviz_materials.xacro" />   <!-- RVIZ Colors                                -->
-  <xacro:include filename="$(find robot_gazebo)/gazebo/gz_golem.xacro" />               <!-- Gazebo                                     -->
+  <xacro:include filename="$(find bots)/xacro/common_rviz_materials.xacro" />   <!-- RVIZ Colors                                -->
+  <xacro:include filename="$(find bots)/gazebo/gz_golem.xacro" />               <!-- Gazebo                                     -->
 <!-- ****************************************************** Base Footprint ***********************************************************  -->
     <link name="base_footprint"/>

File: xacro/kr120r2500pro.xacro (robot description, xacro)
@@ -2,8 +2,8 @@
 <robot name="kr120r2500pro" xmlns:xacro="http://wiki.ros.org/xacro">
 <!-- ****************************************************** Properties**************************************************************** -->
-  <xacro:property name="mesh_path"        value="package://robot_gazebo/meshes/kr120r2500pro/"/>
+  <xacro:property name="mesh_path"        value="package://bots/meshes/kr120r2500pro/"/>
 <!-- ****************************************************** Includes *****************************************************************  -->
-  <xacro:include filename="$(find robot_gazebo)/xacro/common_kuka_materials.xacro" />   <!-- RVIZ Colors                                -->
-  <xacro:include filename="$(find robot_gazebo)/gazebo/gz_kr120r2500pro.xacro" />       <!-- Gazebo                                     -->
+  <xacro:include filename="$(find bots)/xacro/common_kuka_materials.xacro" />   <!-- RVIZ Colors                                -->
+  <xacro:include filename="$(find bots)/gazebo/gz_kr120r2500pro.xacro" />       <!-- Gazebo                                     -->
 <!-- ****************************************************** Macro ******************************************************************** -->
   <xacro:macro name="kuka_kr120r2500pro" params="parent prefix">

File: xacro/kr16_2.xacro (robot description, xacro)
@@ -2,8 +2,8 @@
 <robot name="kr16_2" xmlns:xacro="http://wiki.ros.org/xacro">
 <!-- ****************************************************** Properties**************************************************************** -->
-  <xacro:property name="mesh_path"        value="package://robot_gazebo/meshes/kr16_2/"/>
+  <xacro:property name="mesh_path"        value="package://bots/meshes/kr16_2/"/>
 <!-- ****************************************************** Includes *****************************************************************  -->
-  <xacro:include filename="$(find robot_gazebo)/xacro/common_kuka_materials.xacro" />   <!-- RVIZ Colors                                -->
-  <xacro:include filename="$(find robot_gazebo)/gazebo/gz_kr16_2.xacro" />              <!-- Gazebo                                     -->
+  <xacro:include filename="$(find bots)/xacro/common_kuka_materials.xacro" />   <!-- RVIZ Colors                                -->
+  <xacro:include filename="$(find bots)/gazebo/gz_kr16_2.xacro" />              <!-- Gazebo                                     -->
 <!-- ****************************************************** Macro ******************************************************************** -->
   <xacro:macro name="kuka_kr16_2" params="parent prefix">

File: xacro/kr3r540.xacro (robot description, xacro)
@@ -2,8 +2,8 @@
 <robot name="kr3r540" xmlns:xacro="http://wiki.ros.org/xacro">
 <!-- ****************************************************** Parameters ***************************************************************  -->
-  <xacro:property name="mesh_path" value="package://robot_gazebo/meshes/kr3r540/"/>
+  <xacro:property name="mesh_path" value="package://bots/meshes/kr3r540/"/>
 <!-- ****************************************************** Includes *****************************************************************  -->
-  <xacro:include filename="$(find robot_gazebo)/xacro/common_kuka_materials.xacro" />   <!-- RVIZ Colors                                -->
-  <xacro:include filename="$(find robot_gazebo)/gazebo/gz_kr3r540.xacro" />             <!-- Gazebo                                     -->
+  <xacro:include filename="$(find bots)/xacro/common_kuka_materials.xacro" />   <!-- RVIZ Colors                                -->
+  <xacro:include filename="$(find bots)/gazebo/gz_kr3r540.xacro" />             <!-- Gazebo                                     -->
 <!-- ****************************************************** Macro ******************************************************************** -->
   <xacro:macro name="kuka_kr3r540" params="parent prefix">

File: xacro/kr5_arc.xacro (robot description, xacro)
@@ -2,8 +2,8 @@
 <robot name="kr5_arc" xmlns:xacro="http://wiki.ros.org/xacro">
 <!-- ****************************************************** Properties**************************************************************** -->
-  <xacro:property name="mesh_path"        value="package://robot_gazebo/meshes/kr5_arc/"/>
+  <xacro:property name="mesh_path"        value="package://bots/meshes/kr5_arc/"/>
 <!-- ****************************************************** Includes *****************************************************************  -->
-  <xacro:include filename="$(find robot_gazebo)/xacro/common_kuka_materials.xacro" />   <!-- RVIZ Colors                                -->
-  <xacro:include filename="$(find robot_gazebo)/gazebo/gz_kr5_arc.xacro" />             <!-- Gazebo                                     -->
+  <xacro:include filename="$(find bots)/xacro/common_kuka_materials.xacro" />   <!-- RVIZ Colors                                -->
+  <xacro:include filename="$(find bots)/gazebo/gz_kr5_arc.xacro" />             <!-- Gazebo                                     -->
 <!-- ****************************************************** Macro ******************************************************************** -->
   <xacro:macro name="kuka_kr5_arc" params="parent prefix">

File: xacro/lbr_iiwa_14_r820.xacro (robot description, xacro)
@@ -2,8 +2,8 @@
 <robot name="lbr_iiwa_14_r820" xmlns:xacro="http://wiki.ros.org/xacro">
 <!-- ****************************************************** Properties**************************************************************** -->
-  <xacro:property name="mesh_path"        value="package://robot_gazebo/meshes/lbr_iiwa_14_r820/"/>
+  <xacro:property name="mesh_path"        value="package://bots/meshes/lbr_iiwa_14_r820/"/>
 <!-- ****************************************************** Includes *****************************************************************  -->
-  <xacro:include filename="$(find robot_gazebo)/xacro/common_kuka_materials.xacro" />   <!-- RVIZ Colors                                -->
-  <xacro:include filename="$(find robot_gazebo)/gazebo/gz_lbr_iiwa_14_r820.xacro" />    <!-- Gazebo                                     -->
+  <xacro:include filename="$(find bots)/xacro/common_kuka_materials.xacro" />   <!-- RVIZ Colors                                -->
+  <xacro:include filename="$(find bots)/gazebo/gz_lbr_iiwa_14_r820.xacro" />    <!-- Gazebo                                     -->
 <!-- ****************************************************** Macro ******************************************************************** -->
   <xacro:macro name="kuka_lbr_iiwa_14_r820" params="parent prefix">
