Commit message: u

File: urdf/cart.urdf (robot description, URDF)
Before this commit: robot cart, 3 links, 2 joints
Links:
- link cart: geometry visual mesh filename=/home/mkhuthir/ws/install/bots/share/bots/meshes/cart/cart.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 scale=1 1 1

File: urdf/diffbot.urdf (robot description, URDF)
Before this commit: robot diffbot, 8 links, 7 joints
Links:
- link base: geometry collision mesh filename=/home/mkhuthir/ws/install/bots/share/bots/meshes/diffbot/ba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 scale=1 1 1; visual mesh filename=/home/mkhuthir/ws/install/bots/share/bots/meshes/diffbot/ba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 scale=1 1 1
- link hokuyo: geometry collision box size=0.05 0.05 0.0706; visual mesh filename=/home/mkhuthir/ws/install/bots/share/bots/meshes/diffbot/ho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
- link left_wheel: geometry collision mesh filename=/home/mkhuthir/ws/install/bots/share/bots/meshes/diffbot/wh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 scale=1 1 1; visual mesh filename=/home/mkhuthir/ws/install/bots/share/bots/meshes/diffbot/wh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 scale=1 1 1
- link right_wheel: geometry collision mesh filename=/home/mkhuthir/ws/install/bots/share/bots/meshes/diffbot/wh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 scale=1 1 1; visual mesh filename=/home/mkhuthir/ws/install/bots/share/bots/meshes/diffbot/wh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 scale=1 1 1
