Commit message: u

File: urdf/skidbot.urdf (robot description, URDF)
Before this commit: robot skidbot, 8 links, 7 joints
Links:
- link back_left_wheel: geometry collision cylinder length=0.05 radius=0.08; visual cylinder length=0.05 radius=0.08
- link back_right_wheel: geometry collision cylinder length=0.05 radius=0.08; visual cylinder length=0.05 radius=0.08
- link front_left_wheel: geometry collision cylinder length=0.05 radius=0.08; visual cylinder length=0.05 radius=0.08
- link front_right_wheel: geometry collision cylinder length=0.05 radius=0.08; visual cylinder length=0.05 radius=0.08
Joints:
- joint back_left_wheel_joint: origin xyz=-0.12 0.15 0 rpy=0 0 0 -> xyz=-0.125 0.15 0 rpy=0 0 0
- joint back_right_wheel_joint: origin xyz=-0.12 -0.15 0 rpy=0 0 0 -> xyz=-0.125 -0.15 0 rpy=0 0 0
- joint front_left_wheel_joint: origin xyz=0.12 0.15 0 rpy=0 0 0 -> xyz=0.125 0.15 0 rpy=0 0 0
- joint front_right_wheel_joint: origin xyz=0.12 -0.15 0 rpy=0 0 0 -> xyz=0.125 -0.15 0 rpy=0 0 0
- joint hokuyo_joint: origin xyz=0.15 0 0.1 rpy=0 0 0 -> xyz=0.11 0 0.0853 rpy=0 0 0

File: xacro/skidbot.xacro (robot description, xacro)
@@ -13,6 +13,7 @@
   <xacro:property name="wheel_mass"     value="5.0"      />
   <xacro:property name="wheel_width"    value="0.05"     />
-  <xacro:property name="wheel_radius"   value="0.10"     />
-  <xacro:property name="wheel_x"        value="0.12"     />
+  <xacro:property name="wheel_radius"   value="0.08"     />
+  <xacro:property name="wheel_gap"      value="0.0"      />
+  <xacro:property name="wheel_x"        value="${(base_width+wheel_width)/2+wheel_gap}" />
   <xacro:property name="wheel_y"        value="0.15"     />
   <xacro:property name="camera_mass"    value="0.1"      />
@@ -24,7 +25,7 @@
   <xacro:property name="hokuyo_width"   value="0.05"     />
   <xacro:property name="hokuyo_length"  value="0.05"     />
-  <xacro:property name="hokuyo_height"  value="0.080165" />
-  <xacro:property name="hokuyo_x"       value="0.15"     />
-  <xacro:property name="hokuyo_z"       value="0.05"     />
+  <xacro:property name="hokuyo_height"  value="0.0706"   />
+  <xacro:property name="hokuyo_x"       value="0.11"     />
+  <xacro:property name="hokuyo_z"       value="${(hokuyo_height+base_height)/2}" />
 <!-- ****************************************************** Includes *****************************************************************  -->
   <xacro:include filename="$(find robot_gazebo)/xacro/common_rviz_materials.xacro" />   <!-- RVIZ Colors                                -->
@@ -40,5 +41,5 @@
 <!-- ****************************************************** Base Link ****************************************************************  -->
   <link name='base'>
-    <pose>0 0 0.1 0 0 0</pose>
+    <pose>0 0 0 0 0 0</pose>
     <inertial>
       <mass value="${base_mass}"/>
@@ -150,5 +151,5 @@
 <!-- ****************************************************** Hokuyo Joint *************************************************************  -->
   <joint type="fixed" name="hokuyo_joint">
-    <origin xyz="${hokuyo_x} 0 ${hokuyo_Z}" rpy="0 0 0"/>
+    <origin xyz="${hokuyo_x} 0 ${hokuyo_z}" rpy="0 0 0"/>
     <child link="hokuyo"/>
     <parent link="base"/>

Commit message: u

File: urdf/skidbot.urdf (robot description, URDF)
Before this commit: robot skidbot, 8 links, 7 joints
Joints:
- joint back_left_wheel_joint: origin xyz=-0.125 0.15 0 rpy=0 0 0 -> xyz=-0.12 0.225 0 rpy=0 0 0
- joint back_right_wheel_joint: origin xyz=-0.125 -0.15 0 rpy=0 0 0 -> xyz=-0.12 -0.225 0 rpy=0 0 0
- joint front_left_wheel_joint: origin xyz=0.125 0.15 0 rpy=0 0 0 -> xyz=0.12 0.225 0 rpy=0 0 0
- joint front_right_wheel_joint: origin xyz=0.125 -0.15 0 rpy=0 0 0 -> xyz=0.12 -0.225 0 rpy=0 0 0

File: xacro/skidbot.xacro (robot description, xacro)
@@ -14,7 +14,7 @@
   <xacro:property name="wheel_width"    value="0.05"     />
   <xacro:property name="wheel_radius"   value="0.08"     />
-  <xacro:property name="wheel_gap"      value="0.0"      />
-  <xacro:property name="wheel_x"        value="${(base_width+wheel_width)/2+wheel_gap}" />
-  <xacro:property name="wheel_y"        value="0.15"     />
+  <xacro:property name="wheel_gap"      value="0.01"     />
+  <xacro:property name="wheel_x"        value="0.12"     />
+  <xacro:property name="wheel_y"        value="${(base_width+wheel_width)/2+wheel_gap}" />
   <xacro:property name="camera_mass"    value="0.1"      />
   <xacro:property name="camera_width"   value="0.05"     />
@@ -30,5 +30,5 @@
 <!-- ****************************************************** Includes *****************************************************************  -->
   <xacro:include filename="$(find robot_gazebo)/xacro/common_rviz_materials.xacro" />   <!-- RVIZ Colors                                -->
-  <xacro:include filename="$(find robot_gazebo)/gazebo/gz_skidbot.xacro" />              <!-- Gazebo                                     -->
+  <xacro:include filename="$(find robot_gazebo)/gazebo/gz_skidbot.xacro" />             <!-- Gazebo                                     -->
 <!-- ****************************************************** Base Footprint ***********************************************************  -->
   <link name="footprint"></link>

Commit message: u

File: urdf/skidbot.urdf (robot description, URDF)
Before this commit: robot skidbot, 8 links, 7 joints
Joints:
- joint back_left_wheel_joint: origin xyz=-0.12 0.225 0 rpy=0 0 0 -> xyz=-0.12 0.135 0 rpy=0 0 0
- joint back_right_wheel_joint: origin xyz=-0.12 -0.225 0 rpy=0 0 0 -> xyz=-0.12 -0.135 0 rpy=0 0 0
- joint front_left_wheel_joint: origin xyz=0.12 0.225 0 rpy=0 0 0 -> xyz=0.12 0.135 0 rpy=0 0 0
- joint front_right_wheel_joint: origin xyz=0.12 -0.225 0 rpy=0 0 0 -> xyz=0.12 -0.135 0 rpy=0 0 0

Commit message: u

File: urdf/skidbot.urdf (robot description, URDF)
Before this commit: robot skidbot, 8 links, 7 joints
Links:
- link back_left_wheel: geometry collision mesh filename=package://robot_gazebo/meshes/skidbot/wheel.dae; visual mesh filename=package://robot_gazebo/meshes/skidbot/wheel.dae
- link back_right_wheel: geometry collision mesh filename=package://robot_gazebo/meshes/skidbot/wheel.dae; visual mesh filename=package://robot_gazebo/meshes/skidbot/wheel.dae
- link front_left_wheel: geometry collision mesh filename=package://robot_gazebo/meshes/skidbot/wheel.dae; visual mesh filename=package://robot_gazebo/meshes/skidbot/wheel.dae
- link front_right_wheel: geometry collision mesh filename=package://robot_gazebo/meshes/skidbot/wheel.dae; visual mesh filename=package://robot_gazebo/meshes/skidbot/wheel.dae

File: xacro/skidbot.xacro (robot description, xacro)
@@ -74,5 +74,5 @@
         <origin xyz="0 0 0" rpy=" 0 ${radians(90)} ${radians(90)}"/>
         <geometry>
-          <cylinder length="${wheel_width}" radius="${wheel_radius}"/>
+          <mesh filename="${mesh_path}wheel.dae"/> <!--  <cylinder length="${wheel_width}" radius="${wheel_radius}"/> -->
         </geometry>
         <material name="grey"/>
@@ -81,5 +81,5 @@
         <origin xyz="0 0 0" rpy=" 0 ${radians(90)} ${radians(90)}"/>
         <geometry>
-          <cylinder length="${wheel_width}" radius="${wheel_radius}"/>
+          <mesh filename="${mesh_path}wheel.dae"/> <!--  <cylinder length="${wheel_width}" radius="${wheel_radius}"/> -->
         </geometry>
       </collision>

Commit message: u

File: urdf/skidbot.urdf (robot description, URDF)
Before this commit: robot skidbot, 8 links, 7 joints
Links:
- added link camera_optical
Joints:
- added joint camera_optical_joint: type fixed, parent camera, child camera_optical, origin xyz=0 0 0 rpy=-1.5707963267948966 0 -1.5707963267948966

File: xacro/skidbot.xacro (robot description, xacro)
@@ -130,4 +130,15 @@
     <axis xyz="0 1 0" rpy="0 0 0"/>
   </joint>
+<!-- ****************************************************** Camera Optical Joint *****************************************************  -->
+<!-- generate an optical frame http://www.ros.org/reps/rep-0103.html#suffix-frames so that ros and opencv can operate on the camera     -->
+<!-- frame correctly. these values have to be these values otherwise the gazebo camera image won't be aligned properly with the frame   -->
+<!-- it is supposedly originating from                                                                                                  -->                                                                                                                   -->
+  <joint name="${prefix}camera_optical_joint" type="fixed">
+    <origin xyz="0 0 0" rpy="${-radians(90)} 0 ${-radians(90)}"/>
+    <parent link="${prefix}camera"/>
+    <child link="${prefix}camera_optical"/>
+  </joint>
+<!-- ****************************************************** Camera Optical Link ******************************************************  -->
+  <link name="${prefix}camera_optical"/>
 <!-- ****************************************************** Hokuyo Link **************************************************************  -->
   <link name="${prefix}hokuyo">

Commit message: u

File: urdf/skidbot.urdf (robot description, URDF)
Before this commit: robot skidbot, 9 links, 8 joints
Links:
- link hokuyo: geometry collision box size=0.05 0.05 0.0706; visual mesh filename=package://bots/meshes/skidbot/hokuyo.dae

Commit message: u

File: urdf/skidbot.urdf (robot description, URDF)
Before this commit: robot skidbot, 9 links, 8 joints
Links:
- link back_left_wheel: geometry collision mesh filename=/home/mkhuthir/ws/install/bots/share/bots/meshes/skidbot/wh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; visual mesh filename=/home/mkhuthir/ws/install/bots/share/bots/meshes/skidbot/wh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
- link back_right_wheel: geometry collision mesh filename=/home/mkhuthir/ws/install/bots/share/bots/meshes/skidbot/wh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; visual mesh filename=/home/mkhuthir/ws/install/bots/share/bots/meshes/skidbot/wh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
- link base: geometry collision mesh filename=/home/mkhuthir/ws/install/bots/share/bots/meshes/skidbot/ba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 scale=1 1 1; visual mesh filename=/home/mkhuthir/ws/install/bots/share/bots/meshes/skidbot/ba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 scale=1 1 1
- link front_left_wheel: geometry collision mesh filename=/home/mkhuthir/ws/install/bots/share/bots/meshes/skidbot/wh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; visual mesh filename=/home/mkhuthir/ws/install/bots/share/bots/meshes/skidbot/wh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
- link front_right_wheel: geometry collision mesh filename=/home/mkhuthir/ws/install/bots/share/bots/meshes/skidbot/wh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; visual mesh filename=/home/mkhuthir/ws/install/bots/share/bots/meshes/skidbot/wh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
- link hokuyo: geometry collision box size=0.05 0.05 0.0706; visual mesh filename=/home/mkhuthir/ws/install/bots/share/bots/meshes/skidbot/ho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
