Commit message: u

File: xacro/tb3_burger.xacro (robot description, xacro)
@@ -50,4 +50,7 @@
     </inertial>
   </link>
+  <gazebo reference="base_link">
+    <material>Gazebo/Blue</material>
+  </gazebo>
 <!-- ****************************************************** Wheel Left Joint *********************************************************  -->
   <joint name="wheel_left_joint" type="continuous">

File: xacro/tb3_waffle.xacro (robot description, xacro)
@@ -52,4 +52,7 @@
     </inertial>
   </link>
+  <gazebo reference="base_link">
+    <material>Gazebo/Blue</material>
+  </gazebo>
 <!-- ****************************************************** Wheel Left Joint *********************************************************  -->
   <joint name="wheel_left_joint" type="continuous">

File: xacro/tb3_waffle_pi.xacro (robot description, xacro)
@@ -52,4 +52,7 @@
     </inertial>
   </link>
+  <gazebo reference="base_link">
+    <material>Gazebo/Blue</material>
+  </gazebo>
 <!-- ****************************************************** Wheel Left Joint *********************************************************  -->
   <joint name="wheel_left_joint" type="continuous">

Commit message: u

File: xacro/tb3_burger.xacro (robot description, xacro)
@@ -81,4 +81,7 @@
     </inertial>
   </link>
+  <gazebo reference="wheel_left_link">
+    <material>Gazebo/FlatBlack</material>
+  </gazebo>
 <!-- ****************************************************** Wheel Right Joint ********************************************************  -->
   <joint name="wheel_right_joint" type="continuous">
@@ -109,4 +112,7 @@
     </inertial>
   </link>
+  <gazebo reference="wheel_right_link">
+    <material>Gazebo/FlatBlack</material>
+  </gazebo>
 <!-- ****************************************************** Caster Back Joint ********************************************************  -->
   <joint name="caster_back_joint" type="fixed">
@@ -135,4 +141,7 @@
     </inertial>
   </link>
+  <gazebo reference="caster_back_link">
+    <material>Gazebo/White</material>
+  </gazebo>
 <!-- ****************************************************** IMU Joint ****************************************************************  -->
   <joint name="imu_joint" type="fixed">
@@ -170,4 +179,7 @@
     </inertial>
   </link>
+  <gazebo reference="base_scan">
+    <material>Gazebo/Green</material>
+  </gazebo>
 <!-- *********************************************************************************************************************************  -->
 </robot>

Commit message: u

File: xacro/tb3_burger.xacro (robot description, xacro)
@@ -47,5 +47,7 @@
       <origin xyz="0 0 0" rpy="0 0 0"/>
       <mass value="8.2573504e-01"/>
-      <inertia ixx="2.2124416e-03" ixy="-1.2294101e-05" ixz="3.4938785e-05" iyy="2.1193702e-03" iyz="-5.0120904e-06" izz="2.0064271e-03" />
+      <inertia ixx="2.2124416e-03" ixy="-1.2294101e-05" ixz="3.4938785e-05"
+               iyy="2.1193702e-03" iyz="-5.0120904e-06" izz="2.0064271e-03"
+               />
     </inertial>
   </link>
@@ -78,5 +80,7 @@
       <origin xyz="0 0 0" />
       <mass value="2.8498940e-02" />
-      <inertia ixx="1.1175580e-05" ixy="-4.2369783e-11" ixz="-5.9381719e-09" iyy="1.1192413e-05" iyz="-1.4400107e-11" izz="2.0712558e-05" />
+      <inertia ixx="1.1175580e-05" ixy="-4.2369783e-11" ixz="-5.9381719e-09"
+               iyy="1.1192413e-05" iyz="-1.4400107e-11" izz="2.0712558e-05"
+               />
     </inertial>
   </link>
@@ -109,5 +113,7 @@
       <origin xyz="0 0 0" />
       <mass value="2.8498940e-02" />
-      <inertia ixx="1.1175580e-05" ixy="-4.2369783e-11" ixz="-5.9381719e-09" iyy="1.1192413e-05" iyz="-1.4400107e-11" izz="2.0712558e-05" />
+      <inertia ixx="1.1175580e-05" ixy="-4.2369783e-11" ixz="-5.9381719e-09"
+               iyy="1.1192413e-05" iyz="-1.4400107e-11" izz="2.0712558e-05"
+               />
     </inertial>
   </link>
@@ -138,5 +144,7 @@
       <origin xyz="0 0 0" />
       <mass value="0.005" />
-      <inertia ixx="0.001" ixy="0.0" ixz="0.0" iyy="0.001" iyz="0.0" izz="0.001" />
+      <inertia ixx="0.001" ixy="0.0" ixz="0.0"
+               iyy="0.001" iyz="0.0"
+               izz="0.001" />
     </inertial>
   </link>
@@ -176,5 +184,7 @@
       <mass value="0.114" />
       <origin xyz="0 0 0" />
-      <inertia ixx="0.001" ixy="0.0" ixz="0.0" iyy="0.001" iyz="0.0" izz="0.001" />
+      <inertia ixx="0.001" ixy="0.0" ixz="0.0"
+               iyy="0.001" iyz="0.0"
+               izz="0.001" />
     </inertial>
   </link>

File: xacro/tb3_waffle_pi.xacro (robot description, xacro)
@@ -85,4 +85,7 @@
       </inertial>
   </link>
+  <gazebo reference="wheel_left_link">
+    <material>Gazebo/FlatBlack</material>
+  </gazebo>
 <!-- ****************************************************** Wheel Right Joint ********************************************************  -->
   <joint name="wheel_right_joint" type="continuous">
@@ -115,4 +118,7 @@
       </inertial>
   </link>
+  <gazebo reference="wheel_right_link">
+    <material>Gazebo/FlatBlack</material>
+  </gazebo>
 <!-- ****************************************************** Caster Back Right Joint **************************************************  -->
   <joint name="caster_back_right_joint" type="fixed">
@@ -143,4 +149,7 @@
     </inertial>
   </link>
+  <gazebo reference="caster_back_right_link">
+    <material>Gazebo/White</material>
+  </gazebo>
 <!-- ****************************************************** Caster Back Left Joint ***************************************************  -->
   <joint name="caster_back_left_joint" type="fixed">
@@ -171,4 +180,7 @@
     </inertial>
   </link>
+  <gazebo reference="caster_back_left_link">
+    <material>Gazebo/White</material>
+  </gazebo>
 <!-- ****************************************************** IMU Joint ****************************************************************  -->
   <joint name="imu_joint" type="fixed">
@@ -208,4 +220,7 @@
     </inertial>
   </link>
+  <gazebo reference="base_scan">
+    <material>Gazebo/Green</material>
+  </gazebo>
 <!-- ****************************************************** Camera Joint ************************************************************* -->
   <joint name="camera_joint" type="fixed">
