Commit message: u

File: xacro/kr5_arc.xacro (robot description, xacro)
@@ -2,5 +2,5 @@
 <robot name="kuka_kr5_arc" xmlns:xacro="http://wiki.ros.org/xacro">
   <xacro:property name="mesh_path"        value="package://robot_gazebo/meshes/kr5_arc/"/>
-  <xacro:macro name="kr5_arc" params="prefix">
+  <xacro:macro name="kuka_kr5_arc" params="prefix">
     <!-- LINKS -->
     <!-- base link -->
