Commit message: u

File: xacro/kr3r540.xacro (robot description, xacro)
@@ -2,5 +2,5 @@
 <robot name="kr3r540" xmlns:xacro="http://wiki.ros.org/xacro">
   <xacro:include filename="$(find robot_gazebo)/xacro/common_materials.xacro"/>
-  <xacro:property name="mesh_path"        value="package://robot_gazebo/meshes/kr3r540/"/>
+  <xacro:property name="mesh_path" value="package://robot_gazebo/meshes/kr3r540/"/>
 <!-- ****************************************************** Macro ******************************************************************** -->
   <xacro:macro name="kuka_kr3r540" params="prefix">

Commit message: u

File: xacro/kr3r540.xacro (robot description, xacro)
@@ -6,5 +6,5 @@
   <xacro:macro name="kuka_kr3r540" params="prefix">
 <!-- ****************************************************** LINKS ******************************************************************** -->
-<!-- ****************************************************** base link ************************************************************ -->
+<!-- ****************************************************** base link **************************************************************** -->
     <link name="${prefix}base_link">
       <visual>
@@ -22,4 +22,7 @@
       </collision>
     </link>
+    <gazebo reference="${prefix}base_link">
+      <material>Gazebo/Orange</material>
+    </gazebo>
 <!-- ****************************************************** link 1 (A1) **************************************************************** -->
     <link name="${prefix}link_1">
@@ -38,4 +41,7 @@
       </collision>
     </link>
+    <gazebo reference="${prefix}link_1">
+      <material>Gazebo/Orange</material>
+    </gazebo>
 <!-- ****************************************************** link 2 **************************************************************** -->
     <link name="${prefix}link_2">
@@ -54,5 +60,8 @@
       </collision>
     </link>
-<!-- ****************************************************** link 3 **************************************************************** -->
+    <gazebo reference="${prefix}link_2">
+      <material>Gazebo/Orange</material>
+    </gazebo>
+<!-- ****************************************************** link 2 **************************************************************** -->
     <link name="${prefix}link_3">
       <visual>
@@ -70,4 +79,7 @@
       </collision>
     </link>
+    <gazebo reference="${prefix}link_3">
+      <material>Gazebo/Orange</material>
+    </gazebo>
 <!-- ****************************************************** link 4 **************************************************************** -->
     <link name="${prefix}link_4">
@@ -86,4 +98,7 @@
       </collision>
     </link>
+    <gazebo reference="${prefix}link_4">
+      <material>Gazebo/Orange</material>
+    </gazebo>
 <!-- ****************************************************** link 5 **************************************************************** -->
     <link name="${prefix}link_5">
@@ -102,4 +117,7 @@
       </collision>
     </link>
+    <gazebo reference="${prefix}link_5">
+      <material>Gazebo/Orange</material>
+    </gazebo>
 <!-- ****************************************************** link 6 **************************************************************** -->
     <link name="${prefix}link_6">
@@ -118,4 +136,7 @@
       </collision>
     </link>
+    <gazebo reference="${prefix}link_6">
+      <material>Gazebo/Orange</material>
+    </gazebo>
 <!-- ****************************************************** tool 0 ******************************************************************* -->
 <!-- ************************************** Following REP199, this frame shall be use to attach EEF or other equipment *************** -->

File: xacro/kr5_arc.xacro (robot description, xacro)
@@ -2,7 +2,8 @@
 <robot name="kr5_arc" xmlns:xacro="http://wiki.ros.org/xacro">
   <xacro:property name="mesh_path"        value="package://robot_gazebo/meshes/kr5_arc/"/>
+<!-- ****************************************************** Macro ******************************************************************** -->
   <xacro:macro name="kuka_kr5_arc" params="prefix">
-    <!-- LINKS -->
-    <!-- base link -->
+<!-- ****************************************************** LINKS ******************************************************************** -->
+<!-- ****************************************************** base link ************************************************************ -->
     <link name="${prefix}base_link">
       <inertial>
@@ -31,5 +32,8 @@
       </collision>
     </link>
-    <!-- link 1 (A1) -->
+    <gazebo reference="${prefix}base_link">
+      <material>Gazebo/Orange</material>
+    </gazebo>
+<!-- ****************************************************** link 1 (A1) **************************************************************** -->
     <link name="${prefix}link_1">
       <inertial>
@@ -60,5 +64,8 @@
       </collision>
     </link>
-    <!-- link 2 -->
+    <gazebo reference="${prefix}link_1">
+      <material>Gazebo/Orange</material>
+    </gazebo>
+<!-- ****************************************************** link 2 **************************************************************** -->
     <link name="${prefix}link_2">
       <inertial>
@@ -89,5 +96,8 @@
       </collision>
     </link>
-    <!-- link 3 -->
+    <gazebo reference="${prefix}link_2">
+      <material>Gazebo/Orange</material>
+    </gazebo>
+<!-- ****************************************************** link 2 **************************************************************** -->
     <link name="${prefix}link_3">
       <inertial>
@@ -118,5 +128,8 @@
       </collision>
     </link>
-    <!-- link 4 -->
+    <gazebo reference="${prefix}link_3">
+      <material>Gazebo/Orange</material>
+    </gazebo>
+<!-- ****************************************************** link 4 **************************************************************** -->
     <link name="${prefix}link_4">
       <inertial>
@@ -147,5 +160,8 @@
       </collision>
     </link>
-    <!-- link 5 -->
+    <gazebo reference="${prefix}link_4">
+      <material>Gazebo/Orange</material>
+    </gazebo>
+<!-- ****************************************************** link 5 **************************************************************** -->
     <link name="${prefix}link_5">
       <inertial>
@@ -176,5 +192,8 @@
       </collision>
     </link>
-    <!-- link 6 -->
+    <gazebo reference="${prefix}link_5">
+      <material>Gazebo/Orange</material>
+    </gazebo>
+<!-- ****************************************************** link 6 **************************************************************** -->
     <link name="${prefix}link_6">
       <inertial>
@@ -205,10 +224,13 @@
       </collision>
     </link>
-    <!-- tool link -->
-    <!-- Following REP199, this frame shall be use to attach EEF or other equipment -->
+    <gazebo reference="${prefix}link_6">
+      <material>Gazebo/Orange</material>
+    </gazebo>
+<!-- ****************************************************** tool 0 ******************************************************************* -->
+<!-- ************************************** Following REP199, this frame shall be use to attach EEF or other equipment *************** -->
     <link name="${prefix}flange" />
-    <!-- END LINKS -->
-    <!-- JOINTS -->
-    <!-- joint 1 (A1) -->
+<!-- ****************************************************** END LINKS **************************************************************** -->
+<!-- ****************************************************** JOINTS ******************************************************************* -->
+<!-- ****************************************************** joint 1 (A1) ************************************************************* -->
     <joint name="${prefix}joint_a1" type="revolute">
       <origin xyz="0 0 0.4" rpy="${radians(180)} 0 0"/>
@@ -218,5 +240,5 @@
       <limit effort="0" lower="${radians(-155)}" upper="${radians(155)}" velocity="${radians(154)}"/>
     </joint>
-    <!-- joint 2 (A2) -->
+<!-- ****************************************************** joint 2 (A2) **************************************************************** -->
     <joint name="${prefix}joint_a2" type="revolute">
       <origin xyz="0.18 0 0" rpy="${radians(90)} 0 0"/>
@@ -226,5 +248,5 @@
       <limit effort="0" lower="${radians(-180)}" upper="${radians(65)}" velocity="${radians(154)}"/>
     </joint>
-    <!-- joint 3 (A3) -->
+<!-- ****************************************************** joint 3 (A3) **************************************************************** -->
     <joint name="${prefix}joint_a3" type="revolute">
       <origin xyz="0.6 0 0" rpy="0 0 0"/>
@@ -234,5 +256,5 @@
       <limit effort="0" lower="${radians(-15)}" upper="${radians(158)}" velocity="${radians(228)}"/>
     </joint>
-    <!-- joint 4 (A4) -->
+<!-- ****************************************************** joint 4 (A4) **************************************************************** -->
     <joint name="${prefix}joint_a4" type="revolute">
       <origin xyz="0 -0.12 0" rpy="0 ${-radians(90)} 0"/>
@@ -242,5 +264,5 @@
       <limit effort="0" lower="${radians(-350)}" upper="${radians(350)}" velocity="${radians(343)}"/>
     </joint>
-    <!-- joint 5 (A5) -->
+<!-- ****************************************************** joint 5 (A5) **************************************************************** -->
     <joint name="${prefix}joint_a5" type="revolute">
       <origin xyz="0 0 -0.62" rpy="0 ${radians(90)} 0"/>
@@ -250,5 +272,5 @@
       <limit effort="0" lower="${radians(-130)}" upper="${radians(130)}" velocity="${radians(384)}"/>
     </joint>
-    <!-- joint 6 (A6) -->
+<!-- ****************************************************** joint 6 (A6) **************************************************************** -->
     <joint name="${prefix}joint_a6" type="revolute">
       <origin xyz="0 0 0" rpy="0 ${-radians(90)} 0"/>
@@ -258,5 +280,5 @@
       <limit effort="0" lower="${radians(-350)}" upper="${radians(350)}" velocity="${radians(721)}"/>
     </joint>
-    <!-- tool frame - fixed frame -->
+<!-- ****************************************************** tool frame - fixed frame ********************************************* -->
     <joint name="${prefix}joint_a6-flange" type="fixed">
       <parent link="${prefix}link_6"/>
@@ -264,6 +286,6 @@
       <origin xyz="0 0 -0.115" rpy="0 ${radians(90)} ${-radians(90)}"/>
     </joint>
-    <!-- END JOINTS -->
-    <!-- ROS base_link to KUKA $ROBROOT coordinate system transform -->
+<!-- ****************************************************** END JOINTS *********************************************************** -->
+<!-- ****************************** ROS base_link to KUKA $ROBROOT coordinate system transform *********************************** -->
     <link name="${prefix}base" />
     <joint name="${prefix}base_link-base" type="fixed">
@@ -272,5 +294,5 @@
       <child link="${prefix}base"/>
     </joint>
-    <!-- This frame corresponds to the $TOOL coordinate system in KUKA KRC controllers -->
+<!-- ********************** This frame corresponds to the $TOOL coordinate system in KUKA KRC controllers **************************** -->
     <link name="${prefix}tool0" />
     <joint name="${prefix}flange-tool0" type="fixed">
@@ -279,5 +301,8 @@
       <origin xyz="0 0 0" rpy="0 ${radians(90)} 0"/>
     </joint>
+<!-- ****************************************************** End Macro **************************************************************** -->
   </xacro:macro>
+<!-- ****************************************************** Generates a urdf from macro ********************************************** -->
   <xacro:kuka_kr5_arc prefix=""/>
+<!-- ****************************************************** End ********************************************************************** -->
 </robot>
