Commit message: u

File: xacro/kr120r2500pro.xacro (robot description, xacro)
@@ -1,7 +1,10 @@
 <?xml version="1.0"?>
 <robot name="kr120r2500pro" xmlns:xacro="http://wiki.ros.org/xacro">
+<!-- ****************************************************** Properties**************************************************************** -->
+  <xacro:property name="mesh_path"        value="package://robot_gazebo/meshes/kr120r2500pro/"/>
+<!-- ****************************************************** Macro ******************************************************************** -->
   <xacro:macro name="kuka_kr120r2500pro" params="prefix">
-    <!-- LINKS -->
-    <!-- base link -->
+<!-- ****************************************************** LINKS ******************************************************************** -->
+<!-- ****************************************************** base link **************************************************************** -->
     <link name="${prefix}base_link">
       <inertial>
@@ -13,15 +16,15 @@
         <origin xyz="0 0 0" rpy="0 0 0"/>
         <geometry>
-          <mesh filename="package://kuka_kr120_support/meshes/kr120r2500pro/visual/base_link.dae" />
-        </geometry>
-      </visual>
-      <collision>
-        <origin xyz="0 0 0" rpy="0 0 0"/>
-        <geometry>
-          <mesh filename="package://kuka_kr120_support/meshes/kr120r2500pro/collision/base_link.stl" />
-        </geometry>
-      </collision>
-    </link>
-    <!-- link 1 (A1) -->
+          <mesh filename="${mesh_path}visual/base_link.dae" />
+        </geometry>
+      </visual>
+      <collision>
+        <origin xyz="0 0 0" rpy="0 0 0"/>
+        <geometry>
+          <mesh filename="${mesh_path}collision/base_link.stl" />
+        </geometry>
+      </collision>
+    </link>
+<!-- ****************************************************** link 1 (A1) ************************************************************** -->
     <link name="${prefix}link_1">
       <inertial>
@@ -33,15 +36,15 @@
         <origin xyz="0 0 0" rpy="0 0 0"/>
         <geometry>
-          <mesh filename="package://kuka_kr120_support/meshes/kr120r2500pro/visual/link_1.dae" />
-        </geometry>
-      </visual>
-      <collision>
-        <origin xyz="0 0 0" rpy="0 0 0"/>
-        <geometry>
-          <mesh filename="package://kuka_kr120_support/meshes/kr120r2500pro/collision/link_1.stl" />
-        </geometry>
-      </collision>
-    </link>
-    <!-- link 2 -->
+          <mesh filename="${mesh_path}visual/link_1.dae" />
+        </geometry>
+      </visual>
+      <collision>
+        <origin xyz="0 0 0" rpy="0 0 0"/>
+        <geometry>
+          <mesh filename="${mesh_path}collision/link_1.stl" />
+        </geometry>
+      </collision>
+    </link>
+<!-- ****************************************************** link 2 **************************************************************** -->
     <link name="${prefix}link_2">
       <inertial>
@@ -53,15 +56,15 @@
         <origin xyz="0 0 0" rpy="0 0 0"/>
         <geometry>
-          <mesh filename="package://kuka_kr120_support/meshes/kr120r2500pro/visual/link_2.dae"/>
-        </geometry>
-      </visual>
-      <collision>
-        <origin xyz="0 0 0" rpy="0 0 0"/>
-        <geometry>
-          <mesh filename="package://kuka_kr120_support/meshes/kr120r2500pro/collision/link_2.stl" />
-        </geometry>
-      </collision>
-    </link>
-    <!-- link 3 -->
+          <mesh filename="${mesh_path}visual/link_2.dae"/>
+        </geometry>
+      </visual>
+      <collision>
+        <origin xyz="0 0 0" rpy="0 0 0"/>
+        <geometry>
+          <mesh filename="${mesh_path}collision/link_2.stl" />
+        </geometry>
+      </collision>
+    </link>
+<!-- ****************************************************** link 3 **************************************************************** -->
     <link name="${prefix}link_3">
       <inertial>
@@ -73,15 +76,15 @@
         <origin xyz="0 0 0" rpy="0 0 0"/>
         <geometry>
-          <mesh filename="package://kuka_kr120_support/meshes/kr120r2500pro/visual/link_3.dae" />
-        </geometry>
-      </visual>
-      <collision>
-        <origin xyz="0 0 0" rpy="0 0 0"/>
-        <geometry>
-          <mesh filename="package://kuka_kr120_support/meshes/kr120r2500pro/collision/link_3.stl" />
-        </geometry>
-      </collision>
-    </link>
-    <!-- link 4 -->
+          <mesh filename="${mesh_path}visual/link_3.dae" />
+        </geometry>
+      </visual>
+      <collision>
+        <origin xyz="0 0 0" rpy="0 0 0"/>
+        <geometry>
+          <mesh filename="${mesh_path}collision/link_3.stl" />
+        </geometry>
+      </collision>
+    </link>
+<!-- ****************************************************** link 4 **************************************************************** -->
     <link name="${prefix}link_4">
       <inertial>
@@ -93,15 +96,15 @@
         <origin xyz="0 0 0" rpy="0 0 0"/>
         <geometry>
-          <mesh filename="package://kuka_kr120_support/meshes/kr120r2500pro/visual/link_4.dae" />
-        </geometry>
-      </visual>
-      <collision>
-        <origin xyz="0 0 0" rpy="0 0 0"/>
-        <geometry>
-          <mesh filename="package://kuka_kr120_support/meshes/kr120r2500pro/collision/link_4.stl" />
-        </geometry>
-      </collision>
-    </link>
-    <!-- link 5 -->
+          <mesh filename="${mesh_path}visual/link_4.dae" />
+        </geometry>
+      </visual>
+      <collision>
+        <origin xyz="0 0 0" rpy="0 0 0"/>
+        <geometry>
+          <mesh filename="${mesh_path}collision/link_4.stl" />
+        </geometry>
+      </collision>
+    </link>
+<!-- ****************************************************** link 5 **************************************************************** -->
     <link name="${prefix}link_5">
       <inertial>
@@ -113,15 +116,15 @@
         <origin xyz="0 0 0" rpy="0 0 0"/>
         <geometry>
-          <mesh filename="package://kuka_kr120_support/meshes/kr120r2500pro/visual/link_5.dae" />
-        </geometry>
-      </visual>
-      <collision>
-        <origin xyz="0 0 0" rpy="0 0 0"/>
-        <geometry>
-          <mesh filename="package://kuka_kr120_support/meshes/kr120r2500pro/collision/link_5.stl" />
-        </geometry>
-      </collision>
-    </link>
-    <!-- link 6 -->
+          <mesh filename="${mesh_path}visual/link_5.dae" />
+        </geometry>
+      </visual>
+      <collision>
+        <origin xyz="0 0 0" rpy="0 0 0"/>
+        <geometry>
+          <mesh filename="${mesh_path}collision/link_5.stl" />
+        </geometry>
+      </collision>
+    </link>
+<!-- ****************************************************** link 6 **************************************************************** -->
     <link name="${prefix}link_6">
       <inertial>
@@ -133,19 +136,20 @@
         <origin xyz="0 0 0" rpy="0 0 0"/>
         <geometry>
-          <mesh filename="package://kuka_kr120_support/meshes/kr120r2500pro/visual/link_6.dae" />
-        </geometry>
-      </visual>
-      <collision>
-        <origin xyz="0 0 0" rpy="0 0 0"/>
-        <geometry>
-          <mesh filename="package://kuka_kr120_support/meshes/kr120r2500pro/collision/link_6.stl" />
-        </geometry>
-      </collision>
-    </link>
-    <!-- Following REP199, this frame shall be use to attach EEF or other equipment -->
+          <mesh filename="${mesh_path}visual/link_6.dae" />
+        </geometry>
+      </visual>
+      <collision>
+        <origin xyz="0 0 0" rpy="0 0 0"/>
+        <geometry>
+          <mesh filename="${mesh_path}collision/link_6.stl" />
+        </geometry>
+      </collision>
+    </link>
+<!-- ****************************************************** tool 0 ******************************************************************* -->
+<!-- ******************* Following REP199, this frame shall be use to attach EEF or other equipment ********************************** -->
     <link name="${prefix}flange" />
-    <!-- END LINKS -->
-    <!-- JOINTS -->
-    <!-- joint 1 (A1) -->
+ <!-- ****************************************************** END LINKS **************************************************************** -->
+<!-- ****************************************************** JOINTS ******************************************************************* -->
+<!-- ****************************************************** joint 1 (A1) ************************************************************* -->
     <joint name="${prefix}joint_a1" type="revolute">
       <origin xyz="0 0 0.675" rpy="0 0 0"/>
@@ -155,5 +159,5 @@
       <limit effort="0" lower="${-radians(185)}" upper="${radians(185)}" velocity="${radians(156)}"/>
     </joint>
-    <!-- joint 2 (A2) -->
+<!-- ****************************************************** joint 2 (A2) **************************************************************** -->
     <joint name="${prefix}joint_a2" type="revolute">
       <origin xyz="0.35 0 0" rpy="0 0 0"/>
@@ -163,5 +167,5 @@
       <limit effort="0" lower="${-radians(155)}" upper="${radians(35)}" velocity="${radians(156)}"/>
     </joint>
-    <!-- joint 3 (A3) -->
+<!-- ****************************************************** joint 3 (A3) **************************************************************** -->
     <joint name="${prefix}joint_a3" type="revolute">
       <origin xyz="1.150 0 0" rpy="0 0 0"/>
@@ -171,5 +175,5 @@
       <limit effort="0" lower="${-radians(130)}" upper="${radians(154)}" velocity="${radians(156)}"/>
     </joint>
-    <!-- joint 4 (A4) -->
+<!-- ****************************************************** joint 4 (A4) **************************************************************** -->
     <joint name="${prefix}joint_a4" type="revolute">
       <origin xyz="1.0 0 -0.041" rpy="0 0 0"/>
@@ -179,5 +183,5 @@
       <limit effort="0" lower="${-radians(350)}" upper="${radians(350)}" velocity="${radians(330)}"/>
     </joint>
-    <!-- joint 5 (A5) -->
+<!-- ****************************************************** joint 5 (A5) **************************************************************** -->
     <joint name="${prefix}joint_a5" type="revolute">
       <origin xyz="0 0 0" rpy="0 0 0"/>
@@ -187,5 +191,5 @@
       <limit effort="0" lower="${-radians(130)}" upper="${radians(130)}" velocity="${radians(330)}"/>
     </joint>
-    <!-- joint 6 (A6) -->
+<!-- ****************************************************** joint 6 (A6) **************************************************************** -->
     <joint name="${prefix}joint_a6" type="revolute">
       <origin xyz="0 0 0" rpy="0 0 0"/>
@@ -195,5 +199,5 @@
       <limit effort="0" lower="${-radians(350)}" upper="${radians(350)}" velocity="${radians(615)}"/>
     </joint>
-    <!-- tool frame - fixed frame -->
+<!-- ****************************************************** tool frame - fixed frame ********************************************* -->
     <joint name="${prefix}joint_a6-flange" type="fixed">
       <parent link="${prefix}link_6"/>
@@ -201,7 +205,7 @@
       <origin xyz="0.215 0 0" rpy="0 0 0"/>
     </joint>
-    <!-- END JOINTS -->
-    <!-- ROS base_link to KUKA $ROBROOT coordinate system transform -->
-    <link name="${prefix}base" />
+<!-- ****************************************************** END JOINTS *********************************************************** -->
+<!-- ****************************************************** ROS base_link to KUKA $ROBROOT coordinate system transform *********** -->
+   <link name="${prefix}base" />
     <joint name="${prefix}base_link-base" type="fixed">
       <origin xyz="0 0 0" rpy="0 0 0"/>
@@ -209,5 +213,5 @@
       <child link="${prefix}base"/>
     </joint>
-    <!-- This frame corresponds to the $TOOL coordinate system in KUKA KRC controllers -->
+<!-- ***************** This frame corresponds to the $TOOL coordinate system in KUKA KRC controllers ***************************** -->
     <link name="${prefix}tool0" />
     <joint name="${prefix}flange-tool0" type="fixed">
@@ -217,4 +221,6 @@
     </joint>
   </xacro:macro>
+<!-- ****************************************************** Generates a urdf from macro ********************************************** -->
   <xacro:kuka_kr120r2500pro prefix=""/>
+<!-- ****************************************************** End ********************************************************************** -->
 </robot>

File: xacro/kr16_2.xacro (robot description, xacro)
@@ -1,8 +1,10 @@
 <?xml version="1.0"?>
 <robot name="kr16_2" xmlns:xacro="http://wiki.ros.org/xacro">
+<!-- ****************************************************** Properties**************************************************************** -->
   <xacro:property name="mesh_path"        value="package://robot_gazebo/meshes/kr16_2/"/>
+<!-- ****************************************************** Macro ******************************************************************** -->
   <xacro:macro name="kuka_kr16_2" params="prefix">
 <!-- ****************************************************** LINKS ******************************************************************** -->
-<!-- ****************************************************** base link ************************************************************ -->
+<!-- ****************************************************** base link **************************************************************** -->
     <link name="${prefix}base_link">
       <inertial>
@@ -24,5 +26,5 @@
       </collision>
     </link>
-<!-- ****************************************************** link 1 (A1) **************************************************************** -->
+<!-- ****************************************************** link 1 (A1) ************************************************************** -->
     <link name="${prefix}link_1">
       <inertial>

File: xacro/kr3r540.xacro (robot description, xacro)
@@ -1,4 +1,5 @@
 <?xml version="1.0"?>
 <robot name="kr3r540" xmlns:xacro="http://wiki.ros.org/xacro">
+<!-- ****************************************************** Properties**************************************************************** -->
   <xacro:include filename="$(find robot_gazebo)/xacro/common_materials.xacro"/>
   <xacro:property name="mesh_path" value="package://robot_gazebo/meshes/kr3r540/"/>
@@ -33,5 +34,5 @@
       <material>Gazebo/Gray</material>
     </gazebo>
-<!-- ****************************************************** link 1 (A1) **************************************************************** -->
+<!-- ****************************************************** link 1 (A1) ************************************************************** -->
     <link name="${prefix}link_1">
       <inertial>
@@ -60,5 +61,5 @@
       <material>Gazebo/Orange</material>
     </gazebo>
-<!-- ****************************************************** link 2 **************************************************************** -->
+<!-- ****************************************************** link 2 ******************************************************************* -->
     <link name="${prefix}link_2">
       <inertial>
@@ -87,5 +88,5 @@
       <material>Gazebo/Orange</material>
     </gazebo>
-<!-- ****************************************************** link 2 **************************************************************** -->
+<!-- ****************************************************** link 2 ******************************************************************* -->
     <link name="${prefix}link_3">
       <inertial>
@@ -114,5 +115,5 @@
       <material>Gazebo/Orange</material>
     </gazebo>
-<!-- ****************************************************** link 4 **************************************************************** -->
+<!-- ****************************************************** link 4 ******************************************************************* -->
     <link name="${prefix}link_4">
       <inertial>
@@ -141,5 +142,5 @@
       <material>Gazebo/Orange</material>
     </gazebo>
-<!-- ****************************************************** link 5 **************************************************************** -->
+<!-- ****************************************************** link 5 ******************************************************************* -->
     <link name="${prefix}link_5">
       <inertial>
@@ -168,5 +169,5 @@
       <material>Gazebo/Orange</material>
     </gazebo>
-<!-- ****************************************************** link 6 **************************************************************** -->
+<!-- ****************************************************** link 6 ******************************************************************* -->
     <link name="${prefix}link_6">
       <inertial>
@@ -208,5 +209,5 @@
       <limit lower="${radians(-170)}" upper="${radians(170)}" effort="0" velocity="${radians(530)}"/>
     </joint>
-<!-- ****************************************************** joint 2 (A2) **************************************************************** -->
+<!-- ****************************************************** joint 2 (A2) ************************************************************* -->
     <joint name="${prefix}joint_a2" type="revolute">
       <origin xyz="0.020 0 0" rpy="0 0 0"/>
@@ -216,5 +217,5 @@
       <limit lower="${radians(-170)}" upper="${radians(50)}" effort="0" velocity="${radians(529)}"/>
     </joint>
-<!-- ****************************************************** joint 3 (A3) **************************************************************** -->
+<!-- ****************************************************** joint 3 (A3) ************************************************************* -->
     <joint name="${prefix}joint_a3" type="revolute">
       <origin xyz="0.260 0 0" rpy="0 0 0"/>
@@ -224,5 +225,5 @@
       <limit lower="${radians(-110)}" upper="${radians(155)}" effort="0" velocity="${radians(538)}"/>
     </joint>
-<!-- ****************************************************** joint 4 (A4) **************************************************************** -->
+<!-- ****************************************************** joint 4 (A4) ************************************************************* -->
     <joint name="${prefix}joint_a4" type="revolute">
       <origin xyz="0 0 0.020" rpy="0 0 0"/>
@@ -232,5 +233,5 @@
       <limit lower="${radians(-175)}" upper="${radians(175)}" effort="0" velocity="${radians(600)}"/>
     </joint>
-<!-- ****************************************************** joint 5 (A5) **************************************************************** -->
+<!-- ****************************************************** joint 5 (A5) ************************************************************* -->
     <joint name="${prefix}joint_a5" type="revolute">
       <origin xyz="0.260 0 0" rpy="0 0 0"/>
@@ -240,5 +241,5 @@
       <limit lower="${radians(-120)}" upper="${radians(120)}" effort="0" velocity="${radians(600)}"/>
     </joint>
-<!-- ****************************************************** joint 6 (A6) **************************************************************** -->
+<!-- ****************************************************** joint 6 (A6) ************************************************************* -->
     <joint name="${prefix}joint_a6" type="revolute">
       <origin xyz="0.075 0 0" rpy="0 0 0"/>
@@ -248,5 +249,5 @@
       <limit lower="${radians(-350)}" upper="${radians(350)}" effort="0" velocity="${radians(800)}"/>
     </joint>
-<!-- ****************************************************** tool frame - fixed frame ********************************************* -->
+<!-- ****************************************************** tool frame - fixed frame ************************************************* -->
     <joint name="${prefix}joint_a6-tool0" type="fixed">
       <parent link="${prefix}link_6"/>
@@ -254,6 +255,6 @@
       <origin xyz="0 0 0" rpy="0 0 0"/>
     </joint>
-<!-- ****************************************************** END JOINTS *********************************************************** -->
-<!-- ****************************** ROS base_link to KUKA $ROBROOT coordinate system transform *********************************** -->
+<!-- ****************************************************** END JOINTS *************************************************************** -->
+<!-- ****************************** ROS base_link to KUKA $ROBROOT coordinate system transform *************************************** -->
     <link name="${prefix}base" />
     <joint name="${prefix}base_link-base" type="fixed">
@@ -262,5 +263,5 @@
       <child link="${prefix}base"/>
     </joint>
-<!-- ********************** This frame corresponds to the $TOOL coordinate system in KUKA KRC controllers ******************* -->
+<!-- ********************** This frame corresponds to the $TOOL coordinate system in KUKA KRC controllers **************************** -->
     <link name="${prefix}tool0" />
     <joint name="${prefix}flange-tool0" type="fixed">
@@ -269,5 +270,5 @@
       <origin xyz="0 0 0" rpy="0 ${radians(90)} 0"/>
     </joint>
-<!-- ****************************************************** End Macro *********************************************************** -->
+<!-- ****************************************************** End Macro **************************************************************** -->
   </xacro:macro>
 <!-- ****************************************************** Generates a urdf from macro ********************************************** -->
