Commit message: u

File: xacro/kr5_arc.xacro (robot description, xacro)
@@ -1,9 +1,10 @@
 <?xml version="1.0"?>
 <robot name="kr5_arc" xmlns:xacro="http://wiki.ros.org/xacro">
+<!-- ****************************************************** Properties**************************************************************** -->
   <xacro:property name="mesh_path"        value="package://robot_gazebo/meshes/kr5_arc/"/>
 <!-- ****************************************************** Macro ******************************************************************** -->
   <xacro:macro name="kuka_kr5_arc" params="prefix">
 <!-- ****************************************************** LINKS ******************************************************************** -->
-<!-- ****************************************************** base link ************************************************************ -->
+<!-- ****************************************************** base link **************************************************************** -->
     <link name="${prefix}base_link">
       <inertial>
@@ -35,5 +36,5 @@
       <material>Gazebo/Gray</material>
     </gazebo>
-<!-- ****************************************************** link 1 (A1) **************************************************************** -->
+<!-- ****************************************************** link 1 (A1) ************************************************************** -->
     <link name="${prefix}link_1">
       <inertial>
@@ -67,5 +68,5 @@
       <material>Gazebo/Orange</material>
     </gazebo>
-<!-- ****************************************************** link 2 **************************************************************** -->
+<!-- ****************************************************** link 2 ******************************************************************* -->
     <link name="${prefix}link_2">
       <inertial>
@@ -99,5 +100,5 @@
       <material>Gazebo/Orange</material>
     </gazebo>
-<!-- ****************************************************** link 2 **************************************************************** -->
+<!-- ****************************************************** link 2 ******************************************************************* -->
     <link name="${prefix}link_3">
       <inertial>
@@ -131,5 +132,5 @@
       <material>Gazebo/Orange</material>
     </gazebo>
-<!-- ****************************************************** link 4 **************************************************************** -->
+<!-- ****************************************************** link 4 ******************************************************************* -->
     <link name="${prefix}link_4">
       <inertial>
@@ -163,5 +164,5 @@
       <material>Gazebo/Orange</material>
     </gazebo>
-<!-- ****************************************************** link 5 **************************************************************** -->
+<!-- ****************************************************** link 5 ******************************************************************* -->
     <link name="${prefix}link_5">
       <inertial>
@@ -195,5 +196,5 @@
       <material>Gazebo/Orange</material>
     </gazebo>
-<!-- ****************************************************** link 6 **************************************************************** -->
+<!-- ****************************************************** link 6 ******************************************************************* -->
     <link name="${prefix}link_6">
       <inertial>
@@ -240,5 +241,5 @@
       <limit effort="0" lower="${radians(-155)}" upper="${radians(155)}" velocity="${radians(154)}"/>
     </joint>
-<!-- ****************************************************** joint 2 (A2) **************************************************************** -->
+<!-- ****************************************************** joint 2 (A2) ************************************************************* -->
     <joint name="${prefix}joint_a2" type="revolute">
       <origin xyz="0.18 0 0" rpy="${radians(90)} 0 0"/>
@@ -248,5 +249,5 @@
       <limit effort="0" lower="${radians(-180)}" upper="${radians(65)}" velocity="${radians(154)}"/>
     </joint>
-<!-- ****************************************************** joint 3 (A3) **************************************************************** -->
+<!-- ****************************************************** joint 3 (A3) ************************************************************* -->
     <joint name="${prefix}joint_a3" type="revolute">
       <origin xyz="0.6 0 0" rpy="0 0 0"/>
@@ -256,5 +257,5 @@
       <limit effort="0" lower="${radians(-15)}" upper="${radians(158)}" velocity="${radians(228)}"/>
     </joint>
-<!-- ****************************************************** joint 4 (A4) **************************************************************** -->
+<!-- ****************************************************** joint 4 (A4) ************************************************************* -->
     <joint name="${prefix}joint_a4" type="revolute">
       <origin xyz="0 -0.12 0" rpy="0 ${-radians(90)} 0"/>
@@ -264,5 +265,5 @@
       <limit effort="0" lower="${radians(-350)}" upper="${radians(350)}" velocity="${radians(343)}"/>
     </joint>
-<!-- ****************************************************** joint 5 (A5) **************************************************************** -->
+<!-- ****************************************************** joint 5 (A5) ************************************************************* -->
     <joint name="${prefix}joint_a5" type="revolute">
       <origin xyz="0 0 -0.62" rpy="0 ${radians(90)} 0"/>
@@ -272,5 +273,5 @@
       <limit effort="0" lower="${radians(-130)}" upper="${radians(130)}" velocity="${radians(384)}"/>
     </joint>
-<!-- ****************************************************** joint 6 (A6) **************************************************************** -->
+<!-- ****************************************************** joint 6 (A6) ************************************************************* -->
     <joint name="${prefix}joint_a6" type="revolute">
       <origin xyz="0 0 0" rpy="0 ${-radians(90)} 0"/>
@@ -280,5 +281,5 @@
       <limit effort="0" lower="${radians(-350)}" upper="${radians(350)}" velocity="${radians(721)}"/>
     </joint>
-<!-- ****************************************************** tool frame - fixed frame ********************************************* -->
+<!-- ****************************************************** tool frame - fixed frame ************************************************* -->
     <joint name="${prefix}joint_a6-flange" type="fixed">
       <parent link="${prefix}link_6"/>
@@ -286,6 +287,6 @@
       <origin xyz="0 0 -0.115" rpy="0 ${radians(90)} ${-radians(90)}"/>
     </joint>
-<!-- ****************************************************** END JOINTS *********************************************************** -->
-<!-- ****************************** ROS base_link to KUKA $ROBROOT coordinate system transform *********************************** -->
+<!-- ****************************************************** END JOINTS *************************************************************** -->
+<!-- ****************************** ROS base_link to KUKA $ROBROOT coordinate system transform *************************************** -->
     <link name="${prefix}base" />
     <joint name="${prefix}base_link-base" type="fixed">

File: xacro/lbr_iiwa_14_r820.xacro (robot description, xacro)
@@ -1,4 +1,5 @@
 <?xml version="1.0"?>
 <robot name="lbr_iiwa_14_r820" xmlns:xacro="http://wiki.ros.org/xacro">
+<!-- ****************************************************** Properties**************************************************************** -->
   <xacro:macro name="kuka_lbr_iiwa_14_r820" params="prefix">
     <!-- link list -->
@@ -183,3 +184,4 @@
   </xacro:macro>
   <xacro:kuka_lbr_iiwa_14_r820 prefix=""/>
+<!-- ****************************************************** End ********************************************************************** -->
 </robot>
