Commit message: u

File: xacro/kr120r2500pro.xacro (robot description, xacro)
@@ -149,5 +149,5 @@
 <!-- ******************* Following REP199, this frame shall be use to attach EEF or other equipment ********************************** -->
     <link name="${prefix}flange" />
- <!-- ****************************************************** END LINKS **************************************************************** -->
+<!-- ****************************************************** END LINKS **************************************************************** -->
 <!-- ****************************************************** JOINTS ******************************************************************* -->
 <!-- ****************************************************** joint 1 (A1) ************************************************************* -->
@@ -220,4 +220,5 @@
       <origin xyz="0 0 0" rpy="0 ${radians(90)} 0"/>
     </joint>
+<!-- ****************************************************** End Macro **************************************************************** -->
   </xacro:macro>
 <!-- ****************************************************** Generates a urdf from macro ********************************************** -->

File: xacro/kr16_2.xacro (robot description, xacro)
@@ -159,5 +159,5 @@
       <limit effort="0" lower="${radians(-185)}" upper="${radians(185)}" velocity="${radians(156)}"/>
     </joint>
-<!-- ****************************************************** joint 2 (A2) **************************************************************** -->
+<!-- ****************************************************** joint 2 (A2) ************************************************************* -->
     <joint name="${prefix}joint_a2" type="revolute">
       <origin xyz="0.26 0 0" rpy="0 0 0"/>
@@ -167,5 +167,5 @@
       <limit effort="0" lower="${radians(-155)}" upper="${radians(35)}" velocity="${radians(156)}"/>
     </joint>
-<!-- ****************************************************** joint 3 (A3) **************************************************************** -->
+<!-- ****************************************************** joint 3 (A3) ************************************************************* -->
     <joint name="${prefix}joint_a3" type="revolute">
       <origin xyz="0.68 0 0" rpy="0 0 0"/>
@@ -175,5 +175,5 @@
       <limit effort="0" lower="${radians(-130)}" upper="${radians(154)}" velocity="${radians(156)}"/>
     </joint>
-<!-- ****************************************************** joint 4 (A4) **************************************************************** -->
+<!-- ****************************************************** joint 4 (A4) ************************************************************* -->
     <joint name="${prefix}joint_a4" type="revolute">
       <origin xyz="0.67 0 -0.035" rpy="0 0 0"/>
@@ -183,5 +183,5 @@
       <limit effort="0" lower="${radians(-350)}" upper="${radians(350)}" velocity="${radians(330)}"/>
     </joint>
-<!-- ****************************************************** joint 5 (A5) **************************************************************** -->
+<!-- ****************************************************** joint 5 (A5) ************************************************************* -->
     <joint name="${prefix}joint_a5" type="revolute">
       <origin xyz="0 0 0" rpy="0 0 0"/>
@@ -191,5 +191,5 @@
       <limit effort="0" lower="${radians(-130)}" upper="${radians(130)}" velocity="${radians(330)}"/>
     </joint>
-<!-- ****************************************************** joint 6 (A6) **************************************************************** -->
+<!-- ****************************************************** joint 6 (A6) ************************************************************* -->
     <joint name="${prefix}joint_a6" type="revolute">
       <origin xyz="0 0 0" rpy="0 0 0"/>
@@ -199,5 +199,5 @@
       <limit effort="0" lower="${radians(-350)}" upper="${radians(350)}" velocity="${radians(615)}"/>
     </joint>
-<!-- ****************************************************** tool frame - fixed frame ********************************************* -->
+<!-- ****************************************************** tool frame - fixed frame ************************************************* -->
     <joint name="${prefix}joint_a6-flange" type="fixed">
       <parent link="${prefix}link_6"/>
@@ -205,6 +205,6 @@
       <origin xyz="0.158 0 0" rpy="0 0 0"/>
     </joint>
-<!-- ****************************************************** END JOINTS *********************************************************** -->
-<!-- ****************************************************** ROS base_link to KUKA $ROBROOT coordinate system transform *********** -->
+<!-- ****************************************************** END JOINTS *************************************************************** -->
+<!-- ****************************************************** ROS base_link to KUKA $ROBROOT coordinate system transform *************** -->
     <link name="${prefix}base" />
     <joint name="${prefix}base_link-base" type="fixed">
@@ -213,5 +213,5 @@
       <child link="${prefix}base"/>
     </joint>
-<!-- ***************** This frame corresponds to the $TOOL coordinate system in KUKA KRC controllers ***************************** -->
+<!-- ***************** This frame corresponds to the $TOOL coordinate system in KUKA KRC controllers ********************************* -->
     <link name="${prefix}tool0" />
     <joint name="${prefix}flange-tool0" type="fixed">
@@ -220,4 +220,5 @@
       <origin xyz="0 0 0" rpy="0 ${radians(90)} 0"/>
     </joint>
+<!-- ****************************************************** End Macro **************************************************************** -->
   </xacro:macro>
 <!-- ****************************************************** Generates a urdf from macro ********************************************** -->

File: xacro/lbr_iiwa_14_r820.xacro (robot description, xacro)
@@ -2,121 +2,134 @@
 <robot name="lbr_iiwa_14_r820" xmlns:xacro="http://wiki.ros.org/xacro">
 <!-- ****************************************************** Properties**************************************************************** -->
+  <xacro:property name="mesh_path"        value="package://robot_gazebo/meshes/lbr_iiwa_14_r820/"/>
+<!-- ****************************************************** Macro ******************************************************************** -->
   <xacro:macro name="kuka_lbr_iiwa_14_r820" params="prefix">
-    <!-- link list -->
+<!-- ****************************************************** LINKS ******************************************************************** -->
+<!-- ****************************************************** base link **************************************************************** -->
     <link name="${prefix}base_link">
       <visual>
         <origin xyz="0 0 0" rpy="0 0 0" />
         <geometry>
-          <mesh filename="package://kuka_lbr_iiwa_support/meshes/lbr_iiwa_14_r820/visual/base_link.dae" />
-        </geometry>
-      </visual>
-      <collision>
-        <origin xyz="0 0 0" rpy="0 0 0" />
-        <geometry>
-          <mesh filename="package://kuka_lbr_iiwa_support/meshes/lbr_iiwa_14_r820/collision/base_link.stl" />
-        </geometry>
-      </collision>
-    </link>
+          <mesh filename="${mesh_path}visual/base_link.dae" />
+        </geometry>
+      </visual>
+      <collision>
+        <origin xyz="0 0 0" rpy="0 0 0" />
+        <geometry>
+          <mesh filename="${mesh_path}collision/base_link.stl" />
+        </geometry>
+      </collision>
+    </link>
+<!-- ****************************************************** link 1 (A1) ************************************************************** -->
     <link name="${prefix}link_1">
       <visual>
         <origin xyz="0 0 0" rpy="0 0 0" />
         <geometry>
-          <mesh filename="package://kuka_lbr_iiwa_support/meshes/lbr_iiwa_14_r820/visual/link_1.dae" />
-        </geometry>
-      </visual>
-      <collision>
-        <origin xyz="0 0 0" rpy="0 0 0" />
-        <geometry>
-          <mesh filename="package://kuka_lbr_iiwa_support/meshes/lbr_iiwa_14_r820/collision/link_1.stl" />
-        </geometry>
-      </collision>
-    </link>
+          <mesh filename="${mesh_path}visual/link_1.dae" />
+        </geometry>
+      </visual>
+      <collision>
+        <origin xyz="0 0 0" rpy="0 0 0" />
+        <geometry>
+          <mesh filename="${mesh_path}collision/link_1.stl" />
+        </geometry>
+      </collision>
+    </link>
+<!-- ****************************************************** link 2 **************************************************************** -->
     <link name="${prefix}link_2">
       <visual>
         <origin xyz="0 0 0" rpy="0 0 0" />
         <geometry>
-          <mesh filename="package://kuka_lbr_iiwa_support/meshes/lbr_iiwa_14_r820/visual/link_2.dae" />
-        </geometry>
-      </visual>
-      <collision>
-        <origin xyz="0 0 0" rpy="0 0 0" />
-        <geometry>
-          <mesh filename="package://kuka_lbr_iiwa_support/meshes/lbr_iiwa_14_r820/collision/link_2.stl" />
-        </geometry>
-      </collision>
-    </link>
+          <mesh filename="${mesh_path}visual/link_2.dae" />
+        </geometry>
+      </visual>
+      <collision>
+        <origin xyz="0 0 0" rpy="0 0 0" />
+        <geometry>
+          <mesh filename="${mesh_path}collision/link_2.stl" />
+        </geometry>
+      </collision>
+    </link>
+<!-- ****************************************************** link 3 **************************************************************** -->
     <link name="${prefix}link_3">
       <visual>
         <origin xyz="0 0 0" rpy="0 0 0" />
         <geometry>
-          <mesh filename="package://kuka_lbr_iiwa_support/meshes/lbr_iiwa_14_r820/visual/link_3.dae" />
-        </geometry>
-      </visual>
-      <collision>
-        <origin xyz="0 0 0" rpy="0 0 0" />
-        <geometry>
-          <mesh filename="package://kuka_lbr_iiwa_support/meshes/lbr_iiwa_14_r820/collision/link_3.stl" />
-        </geometry>
-      </collision>
-    </link>
+          <mesh filename="${mesh_path}visual/link_3.dae" />
+        </geometry>
+      </visual>
+      <collision>
+        <origin xyz="0 0 0" rpy="0 0 0" />
+        <geometry>
+          <mesh filename="${mesh_path}collision/link_3.stl" />
+        </geometry>
+      </collision>
+    </link>
+<!-- ****************************************************** link 4 **************************************************************** -->
     <link name="${prefix}link_4">
       <visual>
         <origin xyz="0 0 0" rpy="0 0 0" />
         <geometry>
-          <mesh filename="package://kuka_lbr_iiwa_support/meshes/lbr_iiwa_14_r820/visual/link_4.dae" />
-        </geometry>
-      </visual>
-      <collision>
-        <origin xyz="0 0 0" rpy="0 0 0" />
-        <geometry>
-          <mesh filename="package://kuka_lbr_iiwa_support/meshes/lbr_iiwa_14_r820/collision/link_4.stl" />
-        </geometry>
-      </collision>
-    </link>
+          <mesh filename="${mesh_path}visual/link_4.dae" />
+        </geometry>
+      </visual>
+      <collision>
+        <origin xyz="0 0 0" rpy="0 0 0" />
+        <geometry>
+          <mesh filename="${mesh_path}collision/link_4.stl" />
+        </geometry>
+      </collision>
+    </link>
+<!-- ****************************************************** link 5 **************************************************************** -->
     <link name="${prefix}link_5">
       <visual>
         <origin xyz="0 0 0" rpy="0 0 0" />
         <geometry>
-          <mesh filename="package://kuka_lbr_iiwa_support/meshes/lbr_iiwa_14_r820/visual/link_5.dae" />
-        </geometry>
-      </visual>
-      <collision>
-        <origin xyz="0 0 0" rpy="0 0 0" />
-        <geometry>
-          <mesh filename="package://kuka_lbr_iiwa_support/meshes/lbr_iiwa_14_r820/collision/link_5.stl" />
-        </geometry>
-      </collision>
-    </link>
+          <mesh filename="${mesh_path}visual/link_5.dae" />
+        </geometry>
+      </visual>
+      <collision>
+        <origin xyz="0 0 0" rpy="0 0 0" />
+        <geometry>
+          <mesh filename="${mesh_path}collision/link_5.stl" />
+        </geometry>
+      </collision>
+    </link>
+<!-- ****************************************************** link 6 **************************************************************** -->
     <link name="${prefix}link_6">
       <visual>
         <origin xyz="0 0 0" rpy="0 0 0" />
         <geometry>
-          <mesh filename="package://kuka_lbr_iiwa_support/meshes/lbr_iiwa_14_r820/visual/link_6.dae" />
-        </geometry>
-      </visual>
-      <collision>
-        <origin xyz="0 0 0" rpy="0 0 0" />
-        <geometry>
-          <mesh filename="package://kuka_lbr_iiwa_support/meshes/lbr_iiwa_14_r820/collision/link_6.stl" />
-        </geometry>
-      </collision>
-    </link>
+          <mesh filename="${mesh_path}visual/link_6.dae" />
+        </geometry>
+      </visual>
+      <collision>
+        <origin xyz="0 0 0" rpy="0 0 0" />
+        <geometry>
+          <mesh filename="${mesh_path}collision/link_6.stl" />
+        </geometry>
+      </collision>
+    </link>
+<!-- ****************************************************** link 7 **************************************************************** -->
     <link name="${prefix}link_7">
       <visual>
         <origin xyz="0 0 0" rpy="0 0 0" />
         <geometry>
-          <mesh filename="package://kuka_lbr_iiwa_support/meshes/lbr_iiwa_14_r820/visual/link_7.dae" />
-        </geometry>
-      </visual>
-      <collision>
-        <origin xyz="0 0 0" rpy="0 0 0" />
-        <geometry>
-          <mesh filename="package://kuka_lbr_iiwa_support/meshes/lbr_iiwa_14_r820/collision/link_7.stl" />
-        </geometry>
-      </collision>
-    </link>
+          <mesh filename="${mesh_path}visual/link_7.dae" />
+        </geometry>
+      </visual>
+      <collision>
+        <origin xyz="0 0 0" rpy="0 0 0" />
+        <geometry>
+          <mesh filename="${mesh_path}collision/link_7.stl" />
+        </geometry>
+      </collision>
+    </link>
+<!-- ****************************************************** tool 0 ******************************************************************* -->
+<!-- ******************* Following REP199, this frame shall be use to attach EEF or other equipment ********************************** -->
     <link name="${prefix}tool0" />
-    <!-- end of link list -->
-    <!-- joint list -->
+<!-- ****************************************************** END LINKS **************************************************************** -->
+<!-- ****************************************************** JOINTS ******************************************************************* -->
+<!-- ****************************************************** joint 1 (A1) ************************************************************* -->
     <joint name="${prefix}joint_a1" type="revolute">
       <origin xyz="0 0 0" rpy="0 0 0" />
@@ -126,4 +139,5 @@
       <limit lower="-2.9668" upper="2.9668" effort="0" velocity="1.4834" />
     </joint>
+<!-- ****************************************************** joint 2 (A2) **************************************************************** -->
     <joint name="${prefix}joint_a2" type="revolute">
       <origin xyz="-0.00043624 0 0.36" rpy="0 0 0" />
@@ -133,4 +147,5 @@
       <limit lower="-2.0942" upper="2.0942" effort="0" velocity="1.4834" />
     </joint>
+<!-- ****************************************************** joint 3 (A3) **************************************************************** -->
     <joint name="${prefix}joint_a3" type="revolute">
       <origin xyz="0 0 0" rpy="0 0 0" />
@@ -140,4 +155,5 @@
       <limit lower="-2.9668" upper="2.9668" effort="0" velocity="1.7452" />
     </joint>
+<!-- ****************************************************** joint 4 (A4) **************************************************************** -->
     <joint name="${prefix}joint_a4" type="revolute">
       <origin xyz="0.00043624 0 0.42" rpy="0 0 0" />
@@ -147,4 +163,5 @@
       <limit lower="-2.0942" upper="2.0942" effort="0" velocity="1.3089" />
     </joint>
+<!-- ****************************************************** joint 5 (A5) **************************************************************** -->
     <joint name="${prefix}joint_a5" type="revolute">
       <origin xyz="0 0 0" rpy="0 0 0" />
@@ -154,4 +171,5 @@
       <limit lower="-2.9668" upper="2.9668" effort="0" velocity="2.2688" />
     </joint>
+<!-- ****************************************************** joint 6 (A6) **************************************************************** -->
     <joint name="${prefix}joint_a6" type="revolute">
       <origin xyz="0 0 0.4" rpy="0 0 0" />
@@ -161,4 +179,5 @@
       <limit lower="-2.0942" upper="2.0942" effort="0" velocity="2.356" />
     </joint>
+<!-- ****************************************************** joint 7 (A7) **************************************************************** -->
     <joint name="${prefix}joint_a7" type="revolute">
       <origin xyz="0 0 0" rpy="0 0 0" />
@@ -168,4 +187,5 @@
       <limit lower="-3.0541" upper="3.0541" effort="0" velocity="2.356" />
     </joint>
+<!-- ***************** This frame corresponds to the $TOOL coordinate system in KUKA KRC controllers ********************************* -->
     <joint name="${prefix}joint_a7-tool0" type="fixed">
       <origin xyz="0 0 0.126" rpy="0 0 0" />
@@ -174,6 +194,6 @@
       <axis xyz="0 0 0" />
     </joint>
-    <!-- end of joint list -->
-    <!-- ROS base_link to KUKA $ROBROOT coordinate system transform -->
+<!-- ****************************************************** END JOINTS *********************************************************** -->
+<!-- ****************************************************** ROS base_link to KUKA $ROBROOT coordinate system transform *********** -->
     <link name="${prefix}base" />
     <joint name="${prefix}base_link-base" type="fixed">
@@ -182,5 +202,7 @@
       <child link="${prefix}base"/>
     </joint>
+<!-- ****************************************************** End Macro **************************************************************** -->
   </xacro:macro>
+<!-- ****************************************************** Generates a urdf from macro ********************************************** -->
   <xacro:kuka_lbr_iiwa_14_r820 prefix=""/>
 <!-- ****************************************************** End ********************************************************************** -->
