Commit message: u

File: xacro/razbot.xacro (robot description, xacro)
@@ -12,4 +12,9 @@
 	<xacro:property name="femur_length"     value="0.065" />
 	<xacro:property name="tibia_length"     value="0.133" />
+	<!-- Joint properties -->
+	<xacro:property name="joint_lower_limit" value="-${3.14}" />
+	<xacro:property name="joint_upper_limit" value="${3.14}" />
+	<xacro:property name="joint_effort" value="6.0" />
+	<xacro:property name="joint_velocity" value="0.524" />
 <!-- ****************************************************** Colors *******************************************************************  -->
     <material name="red">
@@ -80,10 +85,4 @@
     </link>
 <!-- ******************************************************  *************************************************************************  -->
-	<!-- Joint properties -->
-	<xacro:property name="joint_lower_limit" value="-${3.14}" />
-	<xacro:property name="joint_upper_limit" value="${3.14}" />
-	<xacro:property name="joint_effort" value="6.0" />
-	<xacro:property name="joint_velocity" value="0.524" />
-<!-- ******************************************************  *************************************************************************  -->
 	<!-- Leg macro -->
 	<xacro:macro name="leg" params="side position x y angle axis">

Commit message: u

File: xacro/razbot.xacro (robot description, xacro)
@@ -7,14 +7,13 @@
 <!-- *********************************************************************************************************************************  -->
 <!-- ****************************************************** Parameters ***************************************************************  -->
-	<xacro:property name="body_length_x"    value="0.294" />
-	<xacro:property name="body_length_y"    value="0.340" />
-	<xacro:property name="coxa_length"      value="0.052" />
-	<xacro:property name="femur_length"     value="0.065" />
-	<xacro:property name="tibia_length"     value="0.133" />
-	<!-- Joint properties -->
-	<xacro:property name="joint_lower_limit" value="-${3.14}" />
-	<xacro:property name="joint_upper_limit" value="${3.14}" />
-	<xacro:property name="joint_effort" value="6.0" />
-	<xacro:property name="joint_velocity" value="0.524" />
+	<xacro:property name="body_length_x"        value="0.294" />
+	<xacro:property name="body_length_y"        value="0.340" />
+	<xacro:property name="coxa_length"          value="0.052" />
+	<xacro:property name="femur_length"         value="0.065" />
+	<xacro:property name="tibia_length"         value="0.133" />
+	<xacro:property name="joint_lower_limit"    value="-${3.14}" />
+	<xacro:property name="joint_upper_limit"    value="${3.14}" />
+	<xacro:property name="joint_effort"         value="6.0" />
+	<xacro:property name="joint_velocity"       value="0.524" />
 <!-- ****************************************************** Colors *******************************************************************  -->
     <material name="red">

Commit message: u

File: xacro/razbot.xacro (robot description, xacro)
@@ -7,4 +7,5 @@
 <!-- *********************************************************************************************************************************  -->
 <!-- ****************************************************** Parameters ***************************************************************  -->
+    <xacro:property name="mesh_path"          value="package://robot_gazebo/meshes/razbot/"/>
 	<xacro:property name="body_length_x"        value="0.294" />
 	<xacro:property name="body_length_y"        value="0.340" />
@@ -33,17 +34,17 @@
     </material>
 <!-- ******************************************************  *************************************************************************  -->
-    <link name="base_link"/>
+    <link name="base_footprint"/>
 <!-- ******************************************************  *************************************************************************  -->
     <joint name="base_joint" type="fixed">
-        <parent link="base_link" />
-        <child link="body_link" />
+        <parent link="base_footprint" />
+        <child link="base_link" />
         <origin xyz="0.0 0.0 0.0" rpy="0.0 0.0 0.0" />
     </joint>
 <!-- ******************************************************  *************************************************************************  -->
-	<link name="body_link">
+	<link name="base_link">
         <visual>
             <origin	xyz="0.0 0.0 0.0" rpy="0.0 0.0 0.0" />
             <geometry>
-                <mesh filename="package://robot_gazebo/meshes/razbot/body.stl" scale="0.001 0.001 0.001"/>
+                <mesh filename="${mesh_path}body.stl" scale="0.001 0.001 0.001"/>
             </geometry>
             <material name="blue"/>
@@ -52,5 +53,5 @@
             <origin xyz="0.0 0.0 0.0" rpy="0.0 0.0 0.0"/>
             <geometry>
-                <mesh filename="package://robot_gazebo/meshes/razbot/body.stl" scale="0.001 0.001 0.001"/>
+                <mesh filename="${mesh_path}body.stl" scale="0.001 0.001 0.001"/>
             </geometry>
             <material name="blue"/>
@@ -90,5 +91,5 @@
 		<joint name="leg_center_joint_${side}${position}" type="fixed">
 			<origin xyz="${x} ${y} 0.0" rpy="0.0 0.0 0.0" />
-			<parent link="body_link" />
+			<parent link="base_link" />
 			<child link="leg_center_${side}${position}" />
 		</joint>
@@ -129,5 +130,5 @@
                 <origin xyz="0.0 0.0 0.0" rpy="0.0 0.0 0.0"/>
                 <geometry>
-                    <mesh filename="package://robot_gazebo/meshes/razbot/coxa.stl" scale="0.001 0.001 0.001"/>
+                    <mesh filename="${mesh_path}coxa.stl" scale="0.001 0.001 0.001"/>
                 </geometry>
                 <material name="green"/>
@@ -136,5 +137,5 @@
                 <origin xyz="0.0 0.0 0.0" rpy="0.0 0.0 0.0" />
                 <geometry>
-                    <mesh filename="package://robot_gazebo/meshes/razbot/coxa.stl" scale="0.001 0.001 0.001"/>
+                    <mesh filename="${mesh_path}coxa.stl" scale="0.001 0.001 0.001"/>
                 </geometry>
                 <material name="green"/>
@@ -174,5 +175,5 @@
                 <origin xyz="0.0 0.0 0.0" rpy="0.0 0.0 0.0"/>
                 <geometry>
-                    <mesh filename="package://robot_gazebo/meshes/razbot/femur.stl" scale="0.001 0.001 0.001"/>
+                    <mesh filename="${mesh_path}femur.stl" scale="0.001 0.001 0.001"/>
                 </geometry>
                 <material name="red"/>
@@ -181,5 +182,5 @@
                 <origin xyz="0.0 0.0 0.0" rpy="0.0 0.0 0.0" />
                 <geometry>
-                    <mesh filename="package://robot_gazebo/meshes/razbot/femur.stl" scale="0.001 0.001 0.001"/>
+                    <mesh filename="${mesh_path}femur.stl" scale="0.001 0.001 0.001"/>
                 </geometry>
                 <material name="red"/>
@@ -219,5 +220,5 @@
                 <origin xyz="0.0 0.0 0.0" rpy="0.0 0.0 0.0"/>
                 <geometry>
-                    <mesh filename="package://robot_gazebo/meshes/razbot/tibia.stl" scale="0.001 0.001 0.001"/>
+                    <mesh filename="${mesh_path}tibia.stl" scale="0.001 0.001 0.001"/>
                 </geometry>
                 <material name="green"/>
@@ -226,5 +227,5 @@
                 <origin xyz="0.0 0.0 0.0" rpy="0.0 0.0 0.0" />
                 <geometry>
-                    <mesh filename="package://robot_gazebo/meshes/razbot/tibia.stl" scale="0.001 0.001 0.001"/>
+                    <mesh filename="${mesh_path}tibia.stl" scale="0.001 0.001 0.001"/>
                 </geometry>
                 <material name="green"/>
@@ -239,5 +240,21 @@
             </inertial>
         </link>
-<!-- ******************************************************  *************************************************************************  -->
+<!-- ****************************************************** Gazebo Colors*************************************************************  -->
+    <gazebo reference="base_link">
+        <material>Gazebo/Blue</material>
+    </gazebo>
+    <gazebo reference="leg_center_${side}${position}">
+        <material>Gazebo/Green</material>
+    </gazebo>
+    <gazebo reference="coxa_${side}${position}">
+        <material>Gazebo/Red</material>
+    </gazebo>
+    <gazebo reference="femur_${side}${position}">
+        <material>Gazebo/Green</material>
+    </gazebo>
+    <gazebo reference="tibia_${side}${position}">
+            <material>Gazebo/Red</material>
+    </gazebo>
+<!-- ****************************************************** end of Macro *************************************************************  -->
 	</xacro:macro>
 <!-- ******************************************************  *************************************************************************  -->
