Commit message: u

File: xacro/razbot.xacro (robot description, xacro)
@@ -33,7 +33,7 @@
         <color rgba="1.0 1.0 1.0 1.0"/>
     </material>
-<!-- ******************************************************  *************************************************************************  -->
+<!-- ****************************************************** Base Footprint ***********************************************************  -->
     <link name="base_footprint"/>
-<!-- ******************************************************  *************************************************************************  -->
+<!-- ****************************************************** Base Joint ***************************************************************  -->
     <joint name="base_joint" type="fixed">
         <parent link="base_footprint" />
@@ -41,5 +41,5 @@
         <origin xyz="0.0 0.0 0.0" rpy="0.0 0.0 0.0" />
     </joint>
-<!-- ******************************************************  *************************************************************************  -->
+<!-- ****************************************************** Base Link ****************************************************************  -->
 	<link name="base_link">
         <visual>
@@ -66,6 +66,8 @@
         </inertial>
     </link>
-<!-- ******************************************************  *************************************************************************  -->
-	<!-- IMU properties -->
+    <gazebo reference="base_link">
+        <material>Gazebo/Blue</material>
+    </gazebo>
+<!-- ****************************************************** IMU Joint ****************************************************************  -->
 	<joint name="imu_joint" type="fixed">
 		<parent link="base_link" />
@@ -73,5 +75,5 @@
 		<origin xyz="0.0 0.0 0.0" rpy="0.0 0.0 0.0" />
 	</joint>
-<!-- ******************************************************  *************************************************************************  -->
+<!-- ****************************************************** IMU Link *****************************************************************  -->
 	<link name="imu_link">
         <inertial>
@@ -84,9 +86,7 @@
         </inertial>
     </link>
-<!-- ******************************************************  *************************************************************************  -->
-	<!-- Leg macro -->
+<!-- ****************************************************** Leg Macro ****************************************************************  -->
 	<xacro:macro name="leg" params="side position x y angle axis">
-<!-- ******************************************************  *************************************************************************  -->
-		<!-- leg position -->
+<!-- ****************************************************** Leg Center Joint *********************************************************  -->
 		<joint name="leg_center_joint_${side}${position}" type="fixed">
 			<origin xyz="${x} ${y} 0.0" rpy="0.0 0.0 0.0" />
@@ -94,5 +94,5 @@
 			<child link="leg_center_${side}${position}" />
 		</joint>
-<!-- ******************************************************  *************************************************************************  -->
+<!-- ****************************************************** Leg Center Link **********************************************************  -->
 		<link name="leg_center_${side}${position}" >
             <inertial>
@@ -105,6 +105,5 @@
             </inertial>
         </link>
-<!-- ******************************************************  *************************************************************************  -->
-		<!-- coxa -->
+<!-- ****************************************************** Coxa Joint **************************************************************  -->
 		<joint name="coxa_joint_${side}${position}" type="revolute">
 			<origin xyz="0.0 0.0 0.0" rpy="0.0 0.0 ${angle}" />
@@ -114,5 +113,33 @@
 			<limit lower="${joint_lower_limit}" upper="${joint_upper_limit}" effort="${joint_effort}" velocity="${joint_velocity}" />
 		</joint>
-<!-- ******************************************************  *************************************************************************  -->
+<!-- ****************************************************** Coxa Link *****************************************************************  -->
+        <link name="coxa_${side}${position}">
+            <visual>
+                <origin xyz="0.0 0.0 0.0" rpy="0.0 0.0 0.0"/>
+                <geometry>
+                    <mesh filename="${mesh_path}coxa.stl" scale="0.001 0.001 0.001"/>
+                </geometry>
+                <material name="green"/>
+            </visual>
+            <collision>
+                <origin xyz="0.0 0.0 0.0" rpy="0.0 0.0 0.0" />
+                <geometry>
+                    <mesh filename="${mesh_path}coxa.stl" scale="0.001 0.001 0.001"/>
+                </geometry>
+                <material name="green"/>
+            </collision>
+            <inertial>
+                <origin xyz="0.0 0.0 0.0" rpy="0.0 0.0 0.0" />
+                <mass value="0.00001"/>
+                <inertia
+                    ixx="1.0" ixy="0.0"  ixz="0.0"
+                    iyy="1.0" iyz="0.0"
+                    izz="1.0" />
+            </inertial>
+        </link>
+        <gazebo reference="coxa_${side}${position}">
+            <material>Gazebo/Red</material>
+        </gazebo>
+<!-- ****************************************************** Coxa Transmission ********************************************************  -->
 		<transmission name="coxa_transmission_${side}${position}">
             <type>transmission_interface/SimpleTransmission</type>
@@ -125,31 +152,5 @@
             </actuator>
         </transmission>
-<!-- ******************************************************  *************************************************************************  -->
-        <link name="coxa_${side}${position}">
-            <visual>
-                <origin xyz="0.0 0.0 0.0" rpy="0.0 0.0 0.0"/>
-                <geometry>
-                    <mesh filename="${mesh_path}coxa.stl" scale="0.001 0.001 0.001"/>
-                </geometry>
-                <material name="green"/>
-            </visual>
-            <collision>
-                <origin xyz="0.0 0.0 0.0" rpy="0.0 0.0 0.0" />
-                <geometry>
-                    <mesh filename="${mesh_path}coxa.stl" scale="0.001 0.001 0.001"/>
-                </geometry>
-                <material name="green"/>
-            </collision>
-            <inertial>
-                <origin xyz="0.0 0.0 0.0" rpy="0.0 0.0 0.0" />
-                <mass value="0.00001"/>
-                <inertia
-                    ixx="1.0" ixy="0.0"  ixz="0.0"
-                    iyy="1.0" iyz="0.0"
-                    izz="1.0" />
-            </inertial>
-        </link>
-<!-- ******************************************************  *************************************************************************  -->
-		<!-- femur -->
+<!-- ****************************************************** Femur Joint **************************************************************  -->
 		<joint name="femur_joint_${side}${position}" type="revolute">
 			<origin xyz="${coxa_length} 0.0 0.0" rpy="-${pi/2} ${pi/2} 0.0" />
@@ -159,5 +160,33 @@
 			<limit lower="${joint_lower_limit}" upper="${joint_upper_limit}" effort="${joint_effort}" velocity="${joint_velocity}" />
 		</joint>
-<!-- ******************************************************  *************************************************************************  -->
+<!-- ****************************************************** Femur Link ***************************************************************  -->
+        <link name="femur_${side}${position}">
+            <visual>
+                <origin xyz="0.0 0.0 0.0" rpy="0.0 0.0 0.0"/>
+                <geometry>
+                    <mesh filename="${mesh_path}femur.stl" scale="0.001 0.001 0.001"/>
+                </geometry>
+                <material name="red"/>
+            </visual>
+            <collision>
+                <origin xyz="0.0 0.0 0.0" rpy="0.0 0.0 0.0" />
+                <geometry>
+                    <mesh filename="${mesh_path}femur.stl" scale="0.001 0.001 0.001"/>
+                </geometry>
+                <material name="red"/>
+            </collision>
+            <inertial>
+                <origin xyz="0.0 0.0 0.0" rpy="0.0 0.0 0.0" />
+                <mass value="0.00001"/>
+                <inertia
+                    ixx="1.0" ixy="0.0"  ixz="0.0"
+                    iyy="1.0" iyz="0.0"
+                    izz="1.0" />
+            </inertial>
+        </link>
+        <gazebo reference="femur_${side}${position}">
+            <material>Gazebo/Green</material>
+        </gazebo>
+<!-- ****************************************************** Femur Transmission *******************************************************  -->
 		<transmission name="femur_transmission_${side}${position}">
             <type>transmission_interface/SimpleTransmission</type>
@@ -170,31 +199,5 @@
             </actuator>
         </transmission>
-<!-- ******************************************************  *************************************************************************  -->
-        <link name="femur_${side}${position}">
-            <visual>
-                <origin xyz="0.0 0.0 0.0" rpy="0.0 0.0 0.0"/>
-                <geometry>
-                    <mesh filename="${mesh_path}femur.stl" scale="0.001 0.001 0.001"/>
-                </geometry>
-                <material name="red"/>
-            </visual>
-            <collision>
-                <origin xyz="0.0 0.0 0.0" rpy="0.0 0.0 0.0" />
-                <geometry>
-                    <mesh filename="${mesh_path}femur.stl" scale="0.001 0.001 0.001"/>
-                </geometry>
-                <material name="red"/>
-            </collision>
-            <inertial>
-                <origin xyz="0.0 0.0 0.0" rpy="0.0 0.0 0.0" />
-                <mass value="0.00001"/>
-                <inertia
-                    ixx="1.0" ixy="0.0"  ixz="0.0"
-                    iyy="1.0" iyz="0.0"
-                    izz="1.0" />
-            </inertial>
-        </link>
-<!-- ******************************************************  *************************************************************************  -->
-		<!-- tibia -->
+<!-- ****************************************************** Tibia Joint *************************************************************  -->
 		<joint name="tibia_joint_${side}${position}" type="revolute">
 			<origin xyz="0.0 -${femur_length} 0.0" rpy="${pi} 0.0 0.0" />
@@ -204,5 +207,33 @@
 			<limit lower="${joint_lower_limit}" upper="${joint_upper_limit}" effort="${joint_effort}" velocity="${joint_velocity}" />
 		</joint>
-<!-- ******************************************************  *************************************************************************  -->
+<!-- ****************************************************** Tibia Link **************************************************************  -->
+        <link name="tibia_${side}${position}">
+            <visual>
+                <origin xyz="0.0 0.0 0.0" rpy="0.0 0.0 0.0"/>
+                <geometry>
+                    <mesh filename="${mesh_path}tibia.stl" scale="0.001 0.001 0.001"/>
+                </geometry>
+                <material name="green"/>
+            </visual>
+            <collision>
+                <origin xyz="0.0 0.0 0.0" rpy="0.0 0.0 0.0" />
+                <geometry>
+                    <mesh filename="${mesh_path}tibia.stl" scale="0.001 0.001 0.001"/>
+                </geometry>
+                <material name="green"/>
+            </collision>
+            <inertial>
+                <origin xyz="0.0 0.0 0.0" rpy="0.0 0.0 0.0" />
+                <mass value="0.00001"/>
+                <inertia
+                    ixx="1.0" ixy="0.0"  ixz="0.0"
+                    iyy="1.0" iyz="0.0"
+                    izz="1.0" />
+            </inertial>
+        </link>
+        <gazebo reference="tibia_${side}${position}">
+            <material>Gazebo/Red</material>
+        </gazebo>
+<!-- ****************************************************** Tibia Transmission *****************************************************  -->
 		<transmission name="tibia_transmission_${side}${position}">
             <type>transmission_interface/SimpleTransmission</type>
@@ -215,55 +246,13 @@
             </actuator>
         </transmission>
-<!-- ******************************************************  *************************************************************************  -->
-        <link name="tibia_${side}${position}">
-            <visual>
-                <origin xyz="0.0 0.0 0.0" rpy="0.0 0.0 0.0"/>
-                <geometry>
-                    <mesh filename="${mesh_path}tibia.stl" scale="0.001 0.001 0.001"/>
-                </geometry>
-                <material name="green"/>
-            </visual>
-            <collision>
-                <origin xyz="0.0 0.0 0.0" rpy="0.0 0.0 0.0" />
-                <geometry>
-                    <mesh filename="${mesh_path}tibia.stl" scale="0.001 0.001 0.001"/>
-                </geometry>
-                <material name="green"/>
-            </collision>
-            <inertial>
-                <origin xyz="0.0 0.0 0.0" rpy="0.0 0.0 0.0" />
-                <mass value="0.00001"/>
-                <inertia
-                    ixx="1.0" ixy="0.0"  ixz="0.0"
-                    iyy="1.0" iyz="0.0"
-                    izz="1.0" />
-            </inertial>
-        </link>
-<!-- ****************************************************** Gazebo Colors*************************************************************  -->
-    <gazebo reference="base_link">
-        <material>Gazebo/Blue</material>
-    </gazebo>
-    <gazebo reference="leg_center_${side}${position}">
-        <material>Gazebo/Green</material>
-    </gazebo>
-    <gazebo reference="coxa_${side}${position}">
-        <material>Gazebo/Red</material>
-    </gazebo>
-    <gazebo reference="femur_${side}${position}">
-        <material>Gazebo/Green</material>
-    </gazebo>
-    <gazebo reference="tibia_${side}${position}">
-            <material>Gazebo/Red</material>
-    </gazebo>
 <!-- ****************************************************** end of Macro *************************************************************  -->
 	</xacro:macro>
-<!-- ******************************************************  *************************************************************************  -->
-<!-- Build robot model -->
-	<xacro:leg side="R" position="R" x="-${body_length_x/2}" y="-${0.1695/2}" angle="-${5*pi/6}" axis="1" />
-	<xacro:leg side="R" position="M" x="0.0" y="-${body_length_y/2}" angle="-${pi/2}" axis="1" />
-	<xacro:leg side="R" position="F" x="${body_length_x/2}" y="-${0.1695/2}" angle="-${pi/6}" axis="1" />
-	<xacro:leg side="L" position="R" x="-${body_length_x/2}" y="${0.1695/2}" angle="${5*pi/6}" axis="-1" />
-	<xacro:leg side="L" position="M" x="0.0" y="${body_length_y/2}" angle="${pi/2}" axis="-1" />
-	<xacro:leg side="L" position="F" x="${body_length_x/2}" y="${0.1695/2}" angle="${pi/6}" axis="-1" />
+<!-- ****************************************************** Build Robot **************************************************************  -->
+	<xacro:leg side="R" position="R" x="-${body_length_x/2}"    y="-${0.1695/2}"        angle="-${5*pi/6}"   axis=" 1" />
+	<xacro:leg side="R" position="M" x=" 0.0"                   y="-${body_length_y/2}" angle="-${pi/2}"     axis=" 1" />
+	<xacro:leg side="R" position="F" x=" ${body_length_x/2}"    y="-${0.1695/2}"        angle="-${pi/6}"     axis=" 1" />
+	<xacro:leg side="L" position="R" x="-${body_length_x/2}"    y=" ${0.1695/2}"        angle=" ${5*pi/6}"   axis="-1" />
+	<xacro:leg side="L" position="M" x=" 0.0"                   y=" ${body_length_y/2}" angle=" ${pi/2}"     axis="-1" />
+	<xacro:leg side="L" position="F" x=" ${body_length_x/2}"    y=" ${0.1695/2}"        angle=" ${pi/6}"     axis="-1" />
 <!-- ******************************************************  *************************************************************************  -->
 </robot>

Commit message: u

File: xacro/razbot.xacro (robot description, xacro)
@@ -154,5 +154,5 @@
 <!-- ****************************************************** Femur Joint **************************************************************  -->
 		<joint name="femur_joint_${side}${position}" type="revolute">
-			<origin xyz="${coxa_length} 0.0 0.0" rpy="$(radians(-90)} $(radians(90)} 0.0" />
+			<origin xyz="${coxa_length} 0.0 0.0" rpy="${radians(-90)} ${radians(90)} 0.0" />
 			<parent link="coxa_${side}${position}" />
 			<child link="femur_${side}${position}" />
