Commit message: u

File: xacro/pxm3.xacro (robot description, xacro)
@@ -6,7 +6,11 @@
 <!-- *********************************************************************************************************************************  -->
 <!-- ****************************************************** Parameters ***************************************************************  -->
-  <xacro:property name="connect_offset" value="0.02633" />
-  <xacro:property name="thigh_offset_y" value="-0.0645" />
-  <xacro:property name="thigh_offset_z" value="-0.0145" />
+  <xacro:property name="connect_offset"     value="0.02633" />
+  <xacro:property name="thigh_offset_y"     value="-0.0645" />
+  <xacro:property name="thigh_offset_z"     value="-0.0145" />
+  <xacro:property name="joint_lower_limit"  value="-2.6179939"/>
+  <xacro:property name="joint_upper_limit"  value="2.6179939"/>
+  <xacro:property name="joint_effort"       value="2.8"/>
+  <xacro:property name="joint_velocity"     value="5.6548668"/>
 <!-- ****************************************************** Colors *******************************************************************  -->
   <material name="red">
@@ -72,5 +76,5 @@
         <origin xyz="0 -${connect_offset} 0" rpy="0 0 0"  />
         <mass value="0.024357719"/>
-      <inertia ixx="0.0051411124"  ixy="-0.00057530255"  ixz="-0.000024729049" iyy="0.0081915737" iyz="-0.000019223094" izz="0.0011379812" />
+        <inertia ixx="0.0051411124"  ixy="-0.00057530255"  ixz="-0.000024729049" iyy="0.0081915737" iyz="-0.000019223094" izz="0.0011379812" />
       </inertial>
       <visual>
@@ -94,5 +98,5 @@
         <origin xyz="0 -${connect_offset} 0" rpy="0 0 0"  />
         <mass value="0.024357719"/>
-      <inertia ixx="0.0051411124"  ixy="-0.00057530255"  ixz="-0.000024729049" iyy="0.0081915737" iyz="-0.000019223094" izz="0.0011379812" />
+        <inertia ixx="0.0051411124"  ixy="-0.00057530255"  ixz="-0.000024729049" iyy="0.0081915737" iyz="-0.000019223094" izz="0.0011379812" />
       </inertial>
       <visual>
@@ -116,5 +120,5 @@
         <origin xyz="0 0 0" rpy="0 0 0"  />
         <mass value="0.024357719"/>
-      <inertia ixx="0.0051411124"  ixy="-0.00057530255"  ixz="-0.000024729049" iyy="0.0081915737" iyz="-0.000019223094" izz="0.0011379812" />
+        <inertia ixx="0.0051411124"  ixy="-0.00057530255"  ixz="-0.000024729049" iyy="0.0081915737" iyz="-0.000019223094" izz="0.0011379812" />
       </inertial>
       <visual>
@@ -138,5 +142,5 @@
         <origin xyz="0 0 0" rpy="0 0 0"  />
         <mass value="0.024357719"/>
-      <inertia ixx="0.0051411124"  ixy="-0.00057530255"  ixz="-0.000024729049" iyy="0.0081915737" iyz="-0.000019223094" izz="0.0011379812" />
+        <inertia ixx="0.0051411124"  ixy="-0.00057530255"  ixz="-0.000024729049" iyy="0.0081915737" iyz="-0.000019223094" izz="0.0011379812" />
       </inertial>
       <visual>
@@ -161,5 +165,5 @@
       <origin xyz="${xyz}" rpy="${rpy}" />
       <axis xyz="1 0 0" />
-      <limit effort="2.8" velocity="5.6548668" lower="-2.6179939" upper="2.6179939" />
+      <limit lower="${joint_lower_limit}" upper="${joint_upper_limit}" effort="${joint_effort}" velocity="${joint_velocity}"/>
     </joint>
 <!-- ****************************************************** C2 Joint *****************************************************************  -->
@@ -175,5 +179,5 @@
       <origin xyz="0 0 0" rpy=" 0 3.14159 3.14159" />
       <axis xyz="1 0 0" />
-      <limit effort="2.8" velocity="5.6548668" lower="-2.6179939" upper="2.6179939" />
+      <limit lower="${joint_lower_limit}" upper="${joint_upper_limit}" effort="${joint_effort}" velocity="${joint_velocity}"/>
     </joint>
 <!-- ****************************************************** Tibia Joint **************************************************************  -->
@@ -183,5 +187,5 @@
       <origin xyz="0 ${thigh_offset_y} ${thigh_offset_z}" rpy="-1.5707 0 3.14159" />
       <axis xyz="1 0 0" />
-      <limit effort="2.8" velocity="5.6548668" lower="-2.6179939" upper="2.6179939" />
+      <limit lower="${joint_lower_limit}" upper="${joint_upper_limit}" effort="${joint_effort}" velocity="${joint_velocity}"/>
     </joint>
 <!-- ****************************************************** C1 Transmission **********************************************************  -->

Commit message: u

File: xacro/pxm3.xacro (robot description, xacro)
@@ -6,4 +6,5 @@
 <!-- *********************************************************************************************************************************  -->
 <!-- ****************************************************** Parameters ***************************************************************  -->
+  <xacro:property name="mesh_path"          value="package://robot_gazebo/meshes/pxm3/"/>
   <xacro:property name="connect_offset"     value="0.02633" />
   <xacro:property name="thigh_offset_y"     value="-0.0645" />
@@ -32,11 +33,11 @@
   <xacro:macro name="pxm3" params="parent *origin">
 <!-- ****************************************************** Attachment Joint *********************************************************  -->
-        <joint name="j_pxm3_attachment" type="fixed">
+        <joint name="j_base_${parent}" type="fixed">
           <parent link="${parent}"/>
-          <child link="MP_BODY"/>
+          <child link="base_link"/>
           <xacro:insert_block name="origin" />
         </joint>
-<!-- ****************************************************** MP_Body Link *************************************************************  -->
-        <link name="MP_BODY">
+<!-- ****************************************************** base_link Link *************************************************************  -->
+        <link name="base_link">
           <inertial>
             <origin xyz="0 0 0" />
@@ -49,5 +50,5 @@
             <geometry>
               <!--box size="0.102 0.109 0.106" /-->
-              <mesh filename="package://robot_gazebo/meshes/pxm3/body.STL"  scale="1 1 1"/>
+              <mesh filename="${mesh_path}body.STL"  scale="1 1 1"/>
             </geometry>
             <material name="blue"/>
@@ -56,5 +57,5 @@
             <origin xyz="0 0 0" rpy="0 0 0" />
             <geometry>
-              <mesh filename="package://robot_gazebo/meshes/pxm3/body_coll.STL"  scale="1 1 1"/>
+              <mesh filename="${mesh_path}body_coll.STL"  scale="1 1 1"/>
             </geometry>
           </collision>
@@ -82,5 +83,5 @@
         <geometry>
           <!--box size="0.045 0.022 0.0325" /-->
-          <mesh filename="package://robot_gazebo/meshes/pxm3/connect.STL"  scale="1 1 1"/>
+          <mesh filename="${mesh_path}connect.STL"  scale="1 1 1"/>
         </geometry>
         <material name="red"/>
@@ -89,5 +90,5 @@
         <origin xyz="0 -${connect_offset} 0" rpy="0 0 0"  />
         <geometry>
-          <mesh filename="package://robot_gazebo/meshes/pxm3/connect_coll.STL"  scale="1 1 1"/>
+          <mesh filename="${mesh_path}connect_coll.STL"  scale="1 1 1"/>
         </geometry>
       </collision>
@@ -104,5 +105,5 @@
         <geometry>
           <!--box size="0.045 0.022 0.0325" /-->
-          <mesh filename="package://robot_gazebo/meshes/pxm3/connect.STL"  scale="1 1 1"/>
+          <mesh filename="${mesh_path}connect.STL"  scale="1 1 1"/>
         </geometry>
         <material name="green"/>
@@ -111,5 +112,5 @@
         <origin xyz="0 -${connect_offset} 0" rpy="0 0 0"  />
         <geometry>
-          <mesh filename="package://robot_gazebo/meshes/pxm3/connect_coll.STL"  scale="1 1 1"/>
+          <mesh filename="${mesh_path}connect_coll.STL"  scale="1 1 1"/>
         </geometry>
       </collision>
@@ -126,5 +127,5 @@
         <geometry>
           <!--box size="0.045 0.022 0.0325" /-->
-          <mesh filename="package://robot_gazebo/meshes/pxm3/thigh_l.STL"  scale="1 1 1"/>
+          <mesh filename="${mesh_path}thigh_l.STL"  scale="1 1 1"/>
         </geometry>
         <material name="red"/>
@@ -133,5 +134,5 @@
         <origin xyz="0 0 0" rpy="0 0 0"  />
         <geometry>
-          <mesh filename="package://robot_gazebo/meshes/pxm3/thigh_l_coll.STL"  scale="1 1 1"/>
+          <mesh filename="${mesh_path}thigh_l_coll.STL"  scale="1 1 1"/>
         </geometry>
       </collision>
@@ -148,5 +149,5 @@
         <geometry>
           <!--box size="0.045 0.022 0.0325" /-->
-          <mesh filename="package://robot_gazebo/meshes/pxm3/tibia_l.STL"  scale="1 1 1"/>
+          <mesh filename="${mesh_path}tibia_l.STL"  scale="1 1 1"/>
         </geometry>
         <material name="green"/>
@@ -155,5 +156,5 @@
         <origin xyz="0 0 0" rpy="0 0 0"  />
         <geometry>
-          <mesh filename="package://robot_gazebo/meshes/pxm3/tibia_l_coll.STL"  scale="1 1 1"/>
+          <mesh filename="${mesh_path}tibia_l_coll.STL"  scale="1 1 1"/>
         </geometry>
       </collision>
@@ -161,5 +162,5 @@
 <!-- ****************************************************** C1 Joint *****************************************************************  -->
     <joint name="j_c1_${suffix}" type="revolute">
-      <parent link="MP_BODY"/>
+      <parent link="base_link"/>
       <child link="c1_${suffix}"/>
       <origin xyz="${xyz}" rpy="${rpy}" />
@@ -224,8 +225,8 @@
 <!-- ****************************************************** end of Macro *************************************************************  -->
   </xacro:macro>
-<!-- ****************************************************** Base link ****************************************************************  -->
-  <link name="base_link"/>
+<!-- ****************************************************** Base footprint ***********************************************************  -->
+  <link name="base_footprint"/>
 <!-- ****************************************************** Main Macro ***************************************************************  -->
-  <xacro:pxm3 parent="base_link">
+  <xacro:pxm3 parent="base_footprint">
       <origin xyz="0 0 0" rpy="0 0 0" />
   </xacro:pxm3>

Commit message: u

File: xacro/pxm3.xacro (robot description, xacro)
@@ -223,4 +223,20 @@
       </actuator>
     </transmission>
+<!-- ****************************************************** Gazebo Colors*************************************************************  -->
+    <gazebo reference="base_link">
+        <material>Gazebo/Blue</material>
+    </gazebo>
+    <gazebo reference="c1_${suffix}">
+        <material>Gazebo/Green</material>
+    </gazebo>
+    <gazebo reference="c2_${suffix}">
+        <material>Gazebo/Red</material>
+    </gazebo>
+    <gazebo reference="thigh_${suffix}">
+        <material>Gazebo/Green</material>
+    </gazebo>
+    <gazebo reference="tibia_${suffix}">
+            <material>Gazebo/Red</material>
+    </gazebo>
 <!-- ****************************************************** end of Macro *************************************************************  -->
   </xacro:macro>
