Commit message: u

File: xacro/pxm3.xacro (robot description, xacro)
@@ -46,5 +46,4 @@
           </inertial>
           <visual>
-            <!--origin xyz="-0.0235 0 -0.03525" rpy="0 0 0" /-->
             <origin xyz="0 0 0" rpy="0 0 0" />
             <geometry>
@@ -61,103 +60,18 @@
           </collision>
         </link>
+        <gazebo reference="base_link">
+          <material>Gazebo/Blue</material>
+        </gazebo>
 <!-- ****************************************************** Create Legs using Legs Macro **********************************************  -->
-      <xacro:legs xyz="0.1248    -0.06164  0.001116" rpy="0 4.7123 0.7853981633974483"   suffix="RF"/> <!-- Right Front  -->
-      <xacro:legs xyz="0         -0.1034   0.001116" rpy="0 4.7123 0"                    suffix="RM"/> <!-- Right Middle -->
-      <xacro:legs xyz="-0.1248   -0.06164  0.001116" rpy="0 4.7123 -0.7853981633974483"  suffix="RR"/> <!-- Right Rear   -->
-      <xacro:legs xyz="0.1248    0.06164   0.001116" rpy="0 4.7123 2.356194490192345"    suffix="LF"/> <!-- Left Front   -->
-      <xacro:legs xyz="0         0.1034    0.001116" rpy="0 4.7123 3.14159"              suffix="LM"/> <!-- Left Middle  -->
-      <xacro:legs xyz="-0.1248   0.06164   0.001116" rpy="0 4.7123 3.9269908169872414"   suffix="LR"/> <!-- Left Rear    -->
+      <xacro:legs xyz=" 0.1248  -0.06164  0.001116" rpy="0 4.7123  0.7853981633974483"   suffix="RF"/> <!-- Right Front  -->
+      <xacro:legs xyz=" 0       -0.1034   0.001116" rpy="0 4.7123  0"                    suffix="RM"/> <!-- Right Middle -->
+      <xacro:legs xyz="-0.1248  -0.06164  0.001116" rpy="0 4.7123 -0.7853981633974483"   suffix="RR"/> <!-- Right Rear   -->
+      <xacro:legs xyz=" 0.1248   0.06164  0.001116" rpy="0 4.7123  2.356194490192345"    suffix="LF"/> <!-- Left Front   -->
+      <xacro:legs xyz=" 0        0.1034   0.001116" rpy="0 4.7123  3.14159"              suffix="LM"/> <!-- Left Middle  -->
+      <xacro:legs xyz="-0.1248   0.06164  0.001116" rpy="0 4.7123  3.9269908169872414"   suffix="LR"/> <!-- Left Rear    -->
 <!-- ****************************************************** End of Main Macro ********************************************************  -->
   </xacro:macro>
 <!-- ****************************************************** Legs Macro ***************************************************************  -->
   <xacro:macro name="legs" params="xyz rpy suffix">
-<!-- ****************************************************** C1 Link ******************************************************************  -->
-    <link name="c1_${suffix}">
-      <inertial>
-        <origin xyz="0 -${connect_offset} 0" rpy="0 0 0"  />
-        <mass value="0.024357719"/>
-        <inertia ixx="0.0051411124"  ixy="-0.00057530255"  ixz="-0.000024729049" iyy="0.0081915737" iyz="-0.000019223094" izz="0.0011379812" />
-      </inertial>
-      <visual>
-        <origin xyz="0 -0.0252 0" rpy="0 0 0"  />
-        <geometry>
-          <!--box size="0.045 0.022 0.0325" /-->
-          <mesh filename="${mesh_path}connect.STL"  scale="1 1 1"/>
-        </geometry>
-        <material name="red"/>
-      </visual>
-      <collision>
-        <origin xyz="0 -${connect_offset} 0" rpy="0 0 0"  />
-        <geometry>
-          <mesh filename="${mesh_path}connect_coll.STL"  scale="1 1 1"/>
-        </geometry>
-      </collision>
-    </link>
-<!-- ****************************************************** C2 Link ******************************************************************  -->
-    <link name="c2_${suffix}">
-      <inertial>
-        <origin xyz="0 -${connect_offset} 0" rpy="0 0 0"  />
-        <mass value="0.024357719"/>
-        <inertia ixx="0.0051411124"  ixy="-0.00057530255"  ixz="-0.000024729049" iyy="0.0081915737" iyz="-0.000019223094" izz="0.0011379812" />
-      </inertial>
-      <visual>
-        <origin xyz="0 -0.0252 0" rpy="0 0 0"  />
-        <geometry>
-          <!--box size="0.045 0.022 0.0325" /-->
-          <mesh filename="${mesh_path}connect.STL"  scale="1 1 1"/>
-        </geometry>
-        <material name="green"/>
-      </visual>
-      <collision>
-        <origin xyz="0 -${connect_offset} 0" rpy="0 0 0"  />
-        <geometry>
-          <mesh filename="${mesh_path}connect_coll.STL"  scale="1 1 1"/>
-        </geometry>
-      </collision>
-    </link>
-<!-- ****************************************************** Thigh Link ***************************************************************  -->
-    <link name="thigh_${suffix}">
-      <inertial>
-        <origin xyz="0 0 0" rpy="0 0 0"  />
-        <mass value="0.024357719"/>
-        <inertia ixx="0.0051411124"  ixy="-0.00057530255"  ixz="-0.000024729049" iyy="0.0081915737" iyz="-0.000019223094" izz="0.0011379812" />
-      </inertial>
-      <visual>
-        <origin xyz="0 0 0" rpy="0 0 0"  />
-        <geometry>
-          <!--box size="0.045 0.022 0.0325" /-->
-          <mesh filename="${mesh_path}thigh_l.STL"  scale="1 1 1"/>
-        </geometry>
-        <material name="red"/>
-      </visual>
-      <collision>
-        <origin xyz="0 0 0" rpy="0 0 0"  />
-        <geometry>
-          <mesh filename="${mesh_path}thigh_l_coll.STL"  scale="1 1 1"/>
-        </geometry>
-      </collision>
-    </link>
-<!-- ****************************************************** Tibia Link ***************************************************************  -->
-    <link name="tibia_${suffix}">
-      <inertial>
-        <origin xyz="0 0 0" rpy="0 0 0"  />
-        <mass value="0.024357719"/>
-        <inertia ixx="0.0051411124"  ixy="-0.00057530255"  ixz="-0.000024729049" iyy="0.0081915737" iyz="-0.000019223094" izz="0.0011379812" />
-      </inertial>
-      <visual>
-        <origin xyz="0 0 0" rpy="0 0 0"  />
-        <geometry>
-          <!--box size="0.045 0.022 0.0325" /-->
-          <mesh filename="${mesh_path}tibia_l.STL"  scale="1 1 1"/>
-        </geometry>
-        <material name="green"/>
-      </visual>
-      <collision>
-        <origin xyz="0 0 0" rpy="0 0 0"  />
-        <geometry>
-          <mesh filename="${mesh_path}tibia_l_coll.STL"  scale="1 1 1"/>
-        </geometry>
-      </collision>
-    </link>
 <!-- ****************************************************** C1 Joint *****************************************************************  -->
     <joint name="j_c1_${suffix}" type="revolute">
@@ -168,4 +82,40 @@
       <limit lower="${joint_lower_limit}" upper="${joint_upper_limit}" effort="${joint_effort}" velocity="${joint_velocity}"/>
     </joint>
+<!-- ****************************************************** C1 Link ******************************************************************  -->
+    <link name="c1_${suffix}">
+      <inertial>
+        <origin xyz="0 -${connect_offset} 0" rpy="0 0 0"  />
+        <mass value="0.024357719"/>
+        <inertia ixx="0.0051411124"  ixy="-0.00057530255"  ixz="-0.000024729049" iyy="0.0081915737" iyz="-0.000019223094" izz="0.0011379812" />
+      </inertial>
+      <visual>
+        <origin xyz="0 -0.0252 0" rpy="0 0 0"  />
+        <geometry>
+          <!--box size="0.045 0.022 0.0325" /-->
+          <mesh filename="${mesh_path}connect.STL"  scale="1 1 1"/>
+        </geometry>
+        <material name="red"/>
+      </visual>
+      <collision>
+        <origin xyz="0 -${connect_offset} 0" rpy="0 0 0"  />
+        <geometry>
+          <mesh filename="${mesh_path}connect_coll.STL"  scale="1 1 1"/>
+        </geometry>
+      </collision>
+    </link>
+    <gazebo reference="c1_${suffix}">
+      <material>Gazebo/Green</material>
+    </gazebo>
+<!-- ****************************************************** C1 Transmission **********************************************************  -->
+    <transmission name="t_c1_${suffix}">
+      <type>transmission_interface/SimpleTransmission</type>
+      <joint name="j_c1_${suffix}">
+        <hardwareInterface>EffortJointInterface</hardwareInterface>
+      </joint>
+      <actuator name="m_c1_${suffix}">
+        <hardwareInterface>EffortJointInterface</hardwareInterface>
+        <mechanicalReduction>1</mechanicalReduction>
+      </actuator>
+    </transmission>
 <!-- ****************************************************** C2 Joint *****************************************************************  -->
     <joint name="j_c2_${suffix}" type="fixed">
@@ -174,4 +124,29 @@
       <origin xyz="0 -0.054 0" rpy="0 1.5704 3.14159" />
     </joint>
+<!-- ****************************************************** C2 Link ******************************************************************  -->
+    <link name="c2_${suffix}">
+      <inertial>
+        <origin xyz="0 -${connect_offset} 0" rpy="0 0 0"  />
+        <mass value="0.024357719"/>
+        <inertia ixx="0.0051411124"  ixy="-0.00057530255"  ixz="-0.000024729049" iyy="0.0081915737" iyz="-0.000019223094" izz="0.0011379812" />
+      </inertial>
+      <visual>
+        <origin xyz="0 -0.0252 0" rpy="0 0 0"  />
+        <geometry>
+          <!--box size="0.045 0.022 0.0325" /-->
+          <mesh filename="${mesh_path}connect.STL"  scale="1 1 1"/>
+        </geometry>
+        <material name="green"/>
+      </visual>
+      <collision>
+        <origin xyz="0 -${connect_offset} 0" rpy="0 0 0"  />
+        <geometry>
+          <mesh filename="${mesh_path}connect_coll.STL"  scale="1 1 1"/>
+        </geometry>
+      </collision>
+    </link>
+    <gazebo reference="c2_${suffix}">
+      <material>Gazebo/Red</material>
+    </gazebo>
 <!-- ****************************************************** Thigh Joint **************************************************************  -->
     <joint name="j_thigh_${suffix}" type="revolute">
@@ -182,4 +157,40 @@
       <limit lower="${joint_lower_limit}" upper="${joint_upper_limit}" effort="${joint_effort}" velocity="${joint_velocity}"/>
     </joint>
+<!-- ****************************************************** Thigh Link ***************************************************************  -->
+    <link name="thigh_${suffix}">
+      <inertial>
+        <origin xyz="0 0 0" rpy="0 0 0"  />
+        <mass value="0.024357719"/>
+        <inertia ixx="0.0051411124"  ixy="-0.00057530255"  ixz="-0.000024729049" iyy="0.0081915737" iyz="-0.000019223094" izz="0.0011379812" />
+      </inertial>
+      <visual>
+        <origin xyz="0 0 0" rpy="0 0 0"  />
+        <geometry>
+          <!--box size="0.045 0.022 0.0325" /-->
+          <mesh filename="${mesh_path}thigh_l.STL"  scale="1 1 1"/>
+        </geometry>
+        <material name="red"/>
+      </visual>
+      <collision>
+        <origin xyz="0 0 0" rpy="0 0 0"  />
+        <geometry>
+          <mesh filename="${mesh_path}thigh_l_coll.STL"  scale="1 1 1"/>
+        </geometry>
+      </collision>
+    </link>
+    <gazebo reference="thigh_${suffix}">
+      <material>Gazebo/Green</material>
+    </gazebo>
+<!-- ****************************************************** Thigh Transmission *******************************************************  -->
+    <transmission name="t_thigh_${suffix}">
+      <type>transmission_interface/SimpleTransmission</type>
+      <joint name="j_thigh_${suffix}">
+        <hardwareInterface>EffortJointInterface</hardwareInterface>
+      </joint>
+      <actuator name="m_thigh_${suffix}">
+        <hardwareInterface>EffortJointInterface</hardwareInterface>
+        <mechanicalReduction>1</mechanicalReduction>
+      </actuator>
+    </transmission>
 <!-- ****************************************************** Tibia Joint **************************************************************  -->
     <joint name="j_tibia_${suffix}" type="revolute">
@@ -190,26 +201,29 @@
       <limit lower="${joint_lower_limit}" upper="${joint_upper_limit}" effort="${joint_effort}" velocity="${joint_velocity}"/>
     </joint>
-<!-- ****************************************************** C1 Transmission **********************************************************  -->
-    <transmission name="t_c1_${suffix}">
-      <type>transmission_interface/SimpleTransmission</type>
-      <joint name="j_c1_${suffix}">
-        <hardwareInterface>EffortJointInterface</hardwareInterface>
-      </joint>
-      <actuator name="m_c1_${suffix}">
-        <hardwareInterface>EffortJointInterface</hardwareInterface>
-        <mechanicalReduction>1</mechanicalReduction>
-      </actuator>
-    </transmission>
-<!-- ****************************************************** Thigh Transmission *******************************************************  -->
-    <transmission name="t_thigh_${suffix}">
-      <type>transmission_interface/SimpleTransmission</type>
-      <joint name="j_thigh_${suffix}">
-        <hardwareInterface>EffortJointInterface</hardwareInterface>
-      </joint>
-      <actuator name="m_thigh_${suffix}">
-        <hardwareInterface>EffortJointInterface</hardwareInterface>
-        <mechanicalReduction>1</mechanicalReduction>
-      </actuator>
-    </transmission>
+<!-- ****************************************************** Tibia Link ***************************************************************  -->
+    <link name="tibia_${suffix}">
+      <inertial>
+        <origin xyz="0 0 0" rpy="0 0 0"  />
+        <mass value="0.024357719"/>
+        <inertia ixx="0.0051411124"  ixy="-0.00057530255"  ixz="-0.000024729049" iyy="0.0081915737" iyz="-0.000019223094" izz="0.0011379812" />
+      </inertial>
+      <visual>
+        <origin xyz="0 0 0" rpy="0 0 0"  />
+        <geometry>
+          <!--box size="0.045 0.022 0.0325" /-->
+          <mesh filename="${mesh_path}tibia_l.STL"  scale="1 1 1"/>
+        </geometry>
+        <material name="green"/>
+      </visual>
+      <collision>
+        <origin xyz="0 0 0" rpy="0 0 0"  />
+        <geometry>
+          <mesh filename="${mesh_path}tibia_l_coll.STL"  scale="1 1 1"/>
+        </geometry>
+      </collision>
+    </link>
+    <gazebo reference="tibia_${suffix}">
+      <material>Gazebo/Red</material>
+    </gazebo>
 <!-- ****************************************************** Tibia Transmission *******************************************************  -->
     <transmission name="t_tibia_${suffix}">
@@ -223,20 +237,4 @@
       </actuator>
     </transmission>
-<!-- ****************************************************** Gazebo Colors*************************************************************  -->
-    <gazebo reference="base_link">
-        <material>Gazebo/Blue</material>
-    </gazebo>
-    <gazebo reference="c1_${suffix}">
-        <material>Gazebo/Green</material>
-    </gazebo>
-    <gazebo reference="c2_${suffix}">
-        <material>Gazebo/Red</material>
-    </gazebo>
-    <gazebo reference="thigh_${suffix}">
-        <material>Gazebo/Green</material>
-    </gazebo>
-    <gazebo reference="tibia_${suffix}">
-            <material>Gazebo/Red</material>
-    </gazebo>
 <!-- ****************************************************** end of Macro *************************************************************  -->
   </xacro:macro>

Commit message: u

File: xacro/pxm3.xacro (robot description, xacro)
@@ -10,8 +10,8 @@
   <xacro:property name="thigh_offset_y"     value="-0.0645" />
   <xacro:property name="thigh_offset_z"     value="-0.0145" />
-  <xacro:property name="joint_lower_limit"  value="-${radians(150)}"/>
-  <xacro:property name="joint_upper_limit"  value=" ${radians(150)}"/>
-  <xacro:property name="joint_effort"       value=" 2.8"/>
-  <xacro:property name="joint_velocity"     value=" ${radians(324)}"/>
+  <xacro:property name="joint_lower_limit"  value="${radians(-150)}"/>
+  <xacro:property name="joint_upper_limit"  value="${radians(150)}"/>
+  <xacro:property name="joint_effort"       value="2.8"/>
+  <xacro:property name="joint_velocity"     value="${radians(324)}"/>
 <!-- ****************************************************** Colors *******************************************************************  -->
   <material name="red">

File: xacro/razbot.xacro (robot description, xacro)
@@ -13,8 +13,8 @@
 	<xacro:property name="femur_length"         value="0.065" />
 	<xacro:property name="tibia_length"         value="0.133" />
-	<xacro:property name="joint_lower_limit"    value="-${3.14}" />
-	<xacro:property name="joint_upper_limit"    value="${3.14}" />
+	<xacro:property name="joint_lower_limit"    value="${radians(-180)}" />
+	<xacro:property name="joint_upper_limit"    value="${radians( 180)}" />
 	<xacro:property name="joint_effort"         value="6.0" />
-	<xacro:property name="joint_velocity"       value="0.524" />
+	<xacro:property name="joint_velocity"       value="${radians( 300)}" />
 <!-- ****************************************************** Colors *******************************************************************  -->
     <material name="red">

Commit message: u

File: xacro/pxm3.xacro (robot description, xacro)
@@ -43,5 +43,7 @@
             <origin xyz="0 0 0" />
             <mass value="0.97559947"/>
-            <inertia ixx="3.1081800"  ixy="-0.25460189"  ixz="2.0318174" iyy="6.3787776" iyz="0.16417863" izz="5.3316425" />
+            <inertia  ixx="3.1081800" ixy="-0.25460189" ixz="2.0318174"
+                      iyy="6.3787776" iyz="0.16417863"
+                      izz="5.3316425" />
           </inertial>
           <visual>
@@ -87,5 +89,7 @@
         <origin xyz="0 -${connect_offset} 0" rpy="0 0 0"  />
         <mass value="0.024357719"/>
-        <inertia ixx="0.0051411124"  ixy="-0.00057530255"  ixz="-0.000024729049" iyy="0.0081915737" iyz="-0.000019223094" izz="0.0011379812" />
+        <inertia  ixx="0.0051411124" ixy="-0.00057530255" ixz="-0.000024729049"
+                  iyy="0.0081915737" iyz="-0.000019223094"
+                  izz="0.0011379812" />
       </inertial>
       <visual>
@@ -122,5 +126,5 @@
       <parent link="c1_${suffix}"/>
       <child link="c2_${suffix}"/>
-      <origin xyz="0 -0.054 0" rpy="0 1.5704 3.14159" />
+      <origin xyz="0 -0.054 0" rpy="0 ${radians(90)} ${radians(180)}" />
     </joint>
 <!-- ****************************************************** C2 Link ******************************************************************  -->
@@ -129,5 +133,7 @@
         <origin xyz="0 -${connect_offset} 0" rpy="0 0 0"  />
         <mass value="0.024357719"/>
-        <inertia ixx="0.0051411124"  ixy="-0.00057530255"  ixz="-0.000024729049" iyy="0.0081915737" iyz="-0.000019223094" izz="0.0011379812" />
+        <inertia  ixx="0.0051411124" ixy="-0.00057530255" ixz="-0.000024729049"
+                  iyy="0.0081915737" iyz="-0.000019223094"
+                  izz="0.0011379812" />
       </inertial>
       <visual>
@@ -153,5 +159,5 @@
       <parent link="c2_${suffix}"/>
       <child link="thigh_${suffix}"/>
-      <origin xyz="0 0 0" rpy=" 0 3.14159 3.14159" />
+      <origin xyz="0 0 0" rpy=" 0 ${radians(180)} ${radians(180)}" />
       <axis xyz="1 0 0" />
       <limit lower="${joint_lower_limit}" upper="${joint_upper_limit}" effort="${joint_effort}" velocity="${joint_velocity}"/>
@@ -162,5 +168,7 @@
         <origin xyz="0 0 0" rpy="0 0 0"  />
         <mass value="0.024357719"/>
-        <inertia ixx="0.0051411124"  ixy="-0.00057530255"  ixz="-0.000024729049" iyy="0.0081915737" iyz="-0.000019223094" izz="0.0011379812" />
+        <inertia  ixx="0.0051411124" ixy="-0.00057530255" ixz="-0.000024729049"
+                  iyy="0.0081915737" iyz="-0.000019223094"
+                  izz="0.0011379812" />
       </inertial>
       <visual>
@@ -197,5 +205,5 @@
       <parent link="thigh_${suffix}"/>
       <child link="tibia_${suffix}"/>
-      <origin xyz="0 ${thigh_offset_y} ${thigh_offset_z}" rpy="-1.5707 0 3.14159" />
+      <origin xyz="0 ${thigh_offset_y} ${thigh_offset_z}" rpy="${radians(-90)} 0 ${radians(180)}" />
       <axis xyz="1 0 0" />
       <limit lower="${joint_lower_limit}" upper="${joint_upper_limit}" effort="${joint_effort}" velocity="${joint_velocity}"/>
@@ -206,5 +214,7 @@
         <origin xyz="0 0 0" rpy="0 0 0"  />
         <mass value="0.024357719"/>
-        <inertia ixx="0.0051411124"  ixy="-0.00057530255"  ixz="-0.000024729049" iyy="0.0081915737" iyz="-0.000019223094" izz="0.0011379812" />
+        <inertia  ixx="0.0051411124" ixy="-0.00057530255"  ixz="-0.000024729049"
+                  iyy="0.0081915737" iyz="-0.000019223094"
+                  izz="0.0011379812" />
       </inertial>
       <visual>
@@ -242,7 +252,5 @@
   <link name="base_footprint"/>
 <!-- ****************************************************** Main Macro ***************************************************************  -->
-  <xacro:pxm3 parent="base_footprint">
-      <origin xyz="0 0 0" rpy="0 0 0" />
-  </xacro:pxm3>
+  <xacro:pxm3 parent="base_footprint" />
 <!-- ****************************************************** Gazebo Control ***********************************************************  -->
 <!-- *********************************************************************************************************************************  -->

Commit message: u

File: xacro/pxm3.xacro (robot description, xacro)
@@ -31,10 +31,10 @@
   </material>
 <!-- ****************************************************** Main Macro ***************************************************************  -->
-  <xacro:macro name="pxm3" params="parent *origin">
+  <xacro:macro name="pxm3" params="parent">
 <!-- ****************************************************** Attachment Joint *********************************************************  -->
         <joint name="j_base_${parent}" type="fixed">
           <parent link="${parent}"/>
           <child link="base_link"/>
-          <xacro:insert_block name="origin" />
+          <origin rpy="0 0 0" xyz="0 0 0"/>
         </joint>
 <!-- ****************************************************** base_link Link *************************************************************  -->
@@ -252,7 +252,5 @@
   <link name="base_footprint"/>
 <!-- ****************************************************** Main Macro ***************************************************************  -->
-  <xacro:pxm3 parent="base_footprint">
-    <origin xyz="0 0 0" rpy="0 0 0" />
-  </xacro:pxm3>
+  <xacro:pxm3 parent="base_footprint" />
 <!-- ****************************************************** Gazebo Control ***********************************************************  -->
 <!-- *********************************************************************************************************************************  -->
