Commit message: u

File: xacro/common_rviz_materials.xacro (robot description, xacro)
@@ -1,12 +1,22 @@
 <?xml version="1.0"?>
+<!-- ****************************************************** RVIZ Colors **************************************************************  -->
+<!-- Muthanna Alwahash                                                                                                                  -->
+<!-- March 2022                                                                                                                         -->
+<!-- *********************************************************************************************************************************  -->
 <robot>
-  <material name="black">
-    <color rgba="0.0 0.0 0.0 1.0"/>
+  <material name="red">
+    <color rgba="1.0 0.0 0.0 1.0"/>
+  </material>
+  <material name="green">
+    <color rgba="0.0 1.0 0.0 1.0"/>
   </material>
   <material name="blue">
-    <color rgba="0.0 0.0 0.8 1.0"/>
+    <color rgba="0.0 0.0 1.0 1.0"/>
   </material>
-  <material name="green">
-    <color rgba="0.0 0.8 0.0 1.0"/>
+  <material name="black">
+    <color rgba="0.3 0.3 0.3 1.0"/>
+  </material>
+  <material name="white">
+    <color rgba="1.0 1.0 1.0 1.0"/>
   </material>
   <material name="grey">
@@ -19,12 +29,6 @@
     <color rgba="${222/255} ${207/255} ${195/255} 1.0"/>
   </material>
-  <material name="red">
-    <color rgba="0.8 0.0 0.0 1.0"/>
-  </material>
   <material name="yellow">
     <color rgba="1.0 1.0 0.0 1.0"/>
   </material>
-  <material name="white">
-    <color rgba="1.0 1.0 1.0 1.0"/>
-  </material>
 </robot>

File: xacro/golem.xacro (robot description, xacro)
@@ -17,20 +17,6 @@
     <xacro:property name="joint_effort"         value=" 6.0"/>
     <xacro:property name="joint_velocity"       value=" ${radians(300)}"/>
-<!-- ****************************************************** Colors *******************************************************************  -->
-    <material name="red">
-        <color rgba="1.0 0.0 0.0 1.0"/>
-    </material>
-    <material name="green">
-        <color rgba="0.0 1.0 0.0 1.0"/>
-    </material>
-    <material name="blue">
-        <color rgba="0.0 0.0 1.0 1.0"/>
-    </material>
-    <material name="black">
-        <color rgba="0.3 0.3 0.3 1.0"/>
-    </material>
-    <material name="white">
-        <color rgba="1.0 1.0 1.0 1.0"/>
-    </material>
+<!-- ****************************************************** Import RVIZ Materials*****************************************************  -->
+  <xacro:include filename="$(find robot_gazebo)/xacro/common_rviz_materials.xacro" />
 <!-- ****************************************************** Base Footprint ***********************************************************  -->
     <link name="base_footprint"/>

File: xacro/pxm3.xacro (robot description, xacro)
@@ -14,20 +14,6 @@
   <xacro:property name="joint_effort"       value="2.8"/>
   <xacro:property name="joint_velocity"     value="${radians(324)}"/>
-<!-- ****************************************************** Colors *******************************************************************  -->
-  <material name="red">
-    <color rgba="1.0 0.0 0.0 1.0"/>
-  </material>
-  <material name="green">
-    <color rgba="0.0 1.0 0.0 1.0"/>
-  </material>
-  <material name="blue">
-    <color rgba="0.0 0.0 1.0 1.0"/>
-  </material>
-  <material name="black">
-    <color rgba="0.3 0.3 0.3 1.0"/>
-  </material>
-  <material name="white">
-    <color rgba="1.0 1.0 1.0 1.0"/>
-  </material>
+<!-- ****************************************************** Import RVIZ Materials*****************************************************  -->
+  <xacro:include filename="$(find robot_gazebo)/xacro/common_rviz_materials.xacro" />
 <!-- ****************************************************** Main Macro ***************************************************************  -->
   <xacro:macro name="pxm3" params="parent">

File: xacro/razbot.xacro (robot description, xacro)
@@ -17,20 +17,6 @@
 	<xacro:property name="joint_effort"         value="6.0" />
 	<xacro:property name="joint_velocity"       value="${radians( 300)}" />
-<!-- ****************************************************** Colors *******************************************************************  -->
-    <material name="red">
-        <color rgba="1.0 0.0 0.0 1.0"/>
-    </material>
-    <material name="green">
-        <color rgba="0.0 1.0 0.0 1.0"/>
-    </material>
-    <material name="blue">
-        <color rgba="0.0 0.0 1.0 1.0"/>
-    </material>
-    <material name="black">
-        <color rgba="0.3 0.3 0.3 1.0"/>
-    </material>
-    <material name="white">
-        <color rgba="1.0 1.0 1.0 1.0"/>
-    </material>
+<!-- ****************************************************** Import RVIZ Materials*****************************************************  -->
+  <xacro:include filename="$(find robot_gazebo)/xacro/common_rviz_materials.xacro" />
 <!-- ****************************************************** Base Footprint ***********************************************************  -->
     <link name="base_footprint"/>

File: xacro/rrbot.xacro (robot description, xacro)
@@ -5,8 +5,4 @@
 <!-- March 2022                                                                                                                         -->
 <!-- *********************************************************************************************************************************  -->
-<!-- ****************************************************** Import RVIZ Materials*****************************************************  -->
-  <xacro:include filename="$(find robot_gazebo)/xacro/common_rviz_materials.xacro" />
-<!-- ****************************************************** Macro ********************************************************************  -->
-  <xacro:macro name="rrbot" params="parent prefix">
 <!-- ****************************************************** Parameters ***************************************************************  -->
     <xacro:property name="mesh_path"    value="package://robot_gazebo/meshes/rrbot/" />
@@ -18,4 +14,8 @@
     <xacro:property name="camera_link"  value="0.05"  /> <!-- Size of square 'camera' box -->
     <xacro:property name="axel_offset"  value="0.05"  /> <!-- Space btw top of beam and the each joint -->
+<!-- ****************************************************** Import RVIZ Materials*****************************************************  -->
+  <xacro:include filename="$(find robot_gazebo)/xacro/common_rviz_materials.xacro" />
+<!-- ****************************************************** Macro ********************************************************************  -->
+  <xacro:macro name="rrbot" params="parent prefix">
 <!-- ****************************************************** Base Joint ***************************************************************  -->
     <joint name="${prefix}base_joint" type="fixed">

File: xacro/tb3_burger.xacro (robot description, xacro)
@@ -5,20 +5,6 @@
 <!-- March 2022                                                                                                                         -->
 <!-- *********************************************************************************************************************************  -->
-<!-- ****************************************************** Colors *******************************************************************  -->
-  <material name="red">
-    <color rgba="1.0 0.0 0.0 1.0"/>
-  </material>
-  <material name="green">
-    <color rgba="0.0 1.0 0.0 1.0"/>
-  </material>
-  <material name="blue">
-    <color rgba="0.0 0.0 1.0 1.0"/>
-  </material>
-  <material name="black">
-    <color rgba="0.3 0.3 0.3 1.0"/>
-  </material>
-  <material name="white">
-    <color rgba="1.0 1.0 1.0 1.0"/>
-  </material>
+<!-- ****************************************************** Import RVIZ Materials*****************************************************  -->
+  <xacro:include filename="$(find robot_gazebo)/xacro/common_rviz_materials.xacro" />
 <!-- ****************************************************** Base Footprint Link ******************************************************  -->
   <link name="base_footprint"/>

File: xacro/tb3_waffle.xacro (robot description, xacro)
@@ -5,20 +5,6 @@
 <!-- March 2022                                                                                                                         -->
 <!-- *********************************************************************************************************************************  -->
-<!-- ****************************************************** Colors *******************************************************************  -->
-  <material name="red">
-    <color rgba="1.0 0.0 0.0 1.0"/>
-  </material>
-  <material name="green">
-    <color rgba="0.0 1.0 0.0 1.0"/>
-  </material>
-  <material name="blue">
-    <color rgba="0.0 0.0 1.0 1.0"/>
-  </material>
-  <material name="black">
-    <color rgba="0.3 0.3 0.3 1.0"/>
-  </material>
-  <material name="white">
-    <color rgba="1.0 1.0 1.0 1.0"/>
-  </material>
+<!-- ****************************************************** Import RVIZ Materials*****************************************************  -->
+  <xacro:include filename="$(find robot_gazebo)/xacro/common_rviz_materials.xacro" />
 <!-- ****************************************************** Base Footprint Link ******************************************************  -->
   <link name="base_footprint"/>

File: xacro/tb3_waffle_pi.xacro (robot description, xacro)
@@ -5,20 +5,6 @@
 <!-- March 2022                                                                                                                         -->
 <!-- *********************************************************************************************************************************  -->
-<!-- ****************************************************** Colors *******************************************************************  -->
-  <material name="red">
-    <color rgba="1.0 0.0 0.0 1.0"/>
-  </material>
-  <material name="green">
-    <color rgba="0.0 1.0 0.0 1.0"/>
-  </material>
-  <material name="blue">
-    <color rgba="0.0 0.0 1.0 1.0"/>
-  </material>
-  <material name="black">
-    <color rgba="0.3 0.3 0.3 1.0"/>
-  </material>
-  <material name="white">
-    <color rgba="1.0 1.0 1.0 1.0"/>
-  </material>
+<!-- ****************************************************** Import RVIZ Materials*****************************************************  -->
+  <xacro:include filename="$(find robot_gazebo)/xacro/common_rviz_materials.xacro" />
 <!-- ****************************************************** Base Footprint Link ******************************************************  -->
   <link name="base_footprint"/>
