Commit message: merge

File: xacro/golem.xacro (robot description, xacro)
@@ -45,5 +45,5 @@
             <origin xyz="0.0 0.0 0.0" rpy="0.0 0.0 0.0"/>
             <geometry>
-                <mesh filename="package://robot_description/meshes/golem/body.stl" scale="0.001 0.001 0.001"/>
+                <mesh filename="package://robot_gazebo/meshes/golem/body.stl" scale="0.001 0.001 0.001"/>
             </geometry>
             <material name="blue"/>
@@ -52,5 +52,5 @@
             <origin xyz="0.0 0.0 0.0" rpy="0.0 0.0 0.0"/>
             <geometry>
-                <mesh filename="package://robot_description/meshes/golem/body.stl" scale="0.001 0.001 0.001"/>
+                <mesh filename="package://robot_gazebo/meshes/golem/body.stl" scale="0.001 0.001 0.001"/>
             </geometry>
             <material name="blue"/>
@@ -178,5 +178,5 @@
             <origin xyz="0.0 0.0 0.0" rpy="0.0 0.0 0.0"/>
             <geometry>
-                <mesh filename="package://robot_description/meshes/golem/coxa.stl" scale="0.001 0.001 0.001"/>
+                <mesh filename="package://robot_gazebo/meshes/golem/coxa.stl" scale="0.001 0.001 0.001"/>
             </geometry>
             <material name="green"/>
@@ -185,5 +185,5 @@
             <origin xyz="0.0 0.0 0.0" rpy="0.0 0.0 0.0" />
             <geometry>
-                <mesh filename="package://robot_description/meshes/golem/coxa.stl" scale="0.001 0.001 0.001"/>
+                <mesh filename="package://robot_gazebo/meshes/golem/coxa.stl" scale="0.001 0.001 0.001"/>
             </geometry>
             <material name="green"/>
@@ -222,5 +222,5 @@
             <origin xyz="0.0 0.0 0.0" rpy="0.0 0.0 0.0"/>
             <geometry>
-                <mesh filename="package://robot_description/meshes/golem/femur.stl" scale="0.001 0.001 0.001"/>
+                <mesh filename="package://robot_gazebo/meshes/golem/femur.stl" scale="0.001 0.001 0.001"/>
             </geometry>
             <material name="red"/>
@@ -229,5 +229,5 @@
             <origin xyz="0.0 0.0 0.0" rpy="0.0 0.0 0.0" />
             <geometry>
-                <mesh filename="package://robot_description/meshes/golem/femur.stl" scale="0.001 0.001 0.001"/>
+                <mesh filename="package://robot_gazebo/meshes/golem/femur.stl" scale="0.001 0.001 0.001"/>
             </geometry>
             <material name="read"/>
@@ -266,5 +266,5 @@
             <origin xyz="0.0 0.0 0.0" rpy="0.0 0.0 0.0"/>
             <geometry>
-                <mesh filename="package://robot_description/meshes/golem/tibia.stl" scale="0.001 0.001 0.001"/>
+                <mesh filename="package://robot_gazebo/meshes/golem/tibia.stl" scale="0.001 0.001 0.001"/>
             </geometry>
             <material name="green"/>
@@ -273,5 +273,5 @@
             <origin xyz="0.0 0.0 0.0" rpy="0.0 0.0 0.0" />
             <geometry>
-                <mesh filename="package://robot_description/meshes/golem/tibia.stl" scale="0.001 0.001 0.001"/>
+                <mesh filename="package://robot_gazebo/meshes/golem/tibia.stl" scale="0.001 0.001 0.001"/>
             </geometry>
             <material name="green"/>
@@ -310,5 +310,5 @@
             <origin xyz="0.0 0.0 0.0" rpy="0.0 0.0 0.0"/>
             <geometry>
-                <mesh filename="package://robot_description/meshes/golem/tarsus.stl" scale="0.001 0.001 0.001"/>
+                <mesh filename="package://robot_gazebo/meshes/golem/tarsus.stl" scale="0.001 0.001 0.001"/>
             </geometry>
             <material name="red"/>
@@ -317,5 +317,5 @@
             <origin xyz="0.0 0.0 0.0" rpy="0.0 0.0 0.0" />
             <geometry>
-                <mesh filename="package://robot_description/meshes/golem/tarsus.stl" scale="0.001 0.001 0.001"/>
+                <mesh filename="package://robot_gazebo/meshes/golem/tarsus.stl" scale="0.001 0.001 0.001"/>
             </geometry>
             <material name="red"/>

File: xacro/pxm3.xacro (robot description, xacro)
@@ -45,5 +45,5 @@
             <geometry>
               <!--box size="0.102 0.109 0.106" /-->
-              <mesh filename="package://robot_description/meshes/pxm3/body.STL"  scale="1 1 1"/>
+              <mesh filename="package://robot_gazebo/meshes/pxm3/body.STL"  scale="1 1 1"/>
             </geometry>
             <material name="blue"/>
@@ -52,5 +52,5 @@
             <origin xyz="0 0 0" rpy="0 0 0" />
             <geometry>
-              <mesh filename="package://robot_description/meshes/pxm3/body_coll.STL"  scale="1 1 1"/>
+              <mesh filename="package://robot_gazebo/meshes/pxm3/body_coll.STL"  scale="1 1 1"/>
             </geometry>
           </collision>
@@ -78,5 +78,5 @@
         <geometry>
           <!--box size="0.045 0.022 0.0325" /-->
-          <mesh filename="package://robot_description/meshes/pxm3/connect.STL"  scale="1 1 1"/>
+          <mesh filename="package://robot_gazebo/meshes/pxm3/connect.STL"  scale="1 1 1"/>
         </geometry>
         <material name="red"/>
@@ -85,5 +85,5 @@
         <origin xyz="0 -${connect_offset} 0" rpy="0 0 0"  />
         <geometry>
-          <mesh filename="package://robot_description/meshes/pxm3/connect_coll.STL"  scale="1 1 1"/>
+          <mesh filename="package://robot_gazebo/meshes/pxm3/connect_coll.STL"  scale="1 1 1"/>
         </geometry>
       </collision>
@@ -100,5 +100,5 @@
         <geometry>
           <!--box size="0.045 0.022 0.0325" /-->
-          <mesh filename="package://robot_description/meshes/pxm3/connect.STL"  scale="1 1 1"/>
+          <mesh filename="package://robot_gazebo/meshes/pxm3/connect.STL"  scale="1 1 1"/>
         </geometry>
         <material name="green"/>
@@ -107,5 +107,5 @@
         <origin xyz="0 -${connect_offset} 0" rpy="0 0 0"  />
         <geometry>
-          <mesh filename="package://robot_description/meshes/pxm3/connect_coll.STL"  scale="1 1 1"/>
+          <mesh filename="package://robot_gazebo/meshes/pxm3/connect_coll.STL"  scale="1 1 1"/>
         </geometry>
       </collision>
@@ -122,5 +122,5 @@
         <geometry>
           <!--box size="0.045 0.022 0.0325" /-->
-          <mesh filename="package://robot_description/meshes/pxm3/thigh_l.STL"  scale="1 1 1"/>
+          <mesh filename="package://robot_gazebo/meshes/pxm3/thigh_l.STL"  scale="1 1 1"/>
         </geometry>
         <material name="red"/>
@@ -129,5 +129,5 @@
         <origin xyz="0 0 0" rpy="0 0 0"  />
         <geometry>
-          <mesh filename="package://robot_description/meshes/pxm3/thigh_l_coll.STL"  scale="1 1 1"/>
+          <mesh filename="package://robot_gazebo/meshes/pxm3/thigh_l_coll.STL"  scale="1 1 1"/>
         </geometry>
       </collision>
@@ -144,5 +144,5 @@
         <geometry>
           <!--box size="0.045 0.022 0.0325" /-->
-          <mesh filename="package://robot_description/meshes/pxm3/tibia_l.STL"  scale="1 1 1"/>
+          <mesh filename="package://robot_gazebo/meshes/pxm3/tibia_l.STL"  scale="1 1 1"/>
         </geometry>
         <material name="green"/>
@@ -151,5 +151,5 @@
         <origin xyz="0 0 0" rpy="0 0 0"  />
         <geometry>
-          <mesh filename="package://robot_description/meshes/pxm3/tibia_l_coll.STL"  scale="1 1 1"/>
+          <mesh filename="package://robot_gazebo/meshes/pxm3/tibia_l_coll.STL"  scale="1 1 1"/>
         </geometry>
       </collision>

File: xacro/razbot.xacro (robot description, xacro)
@@ -41,5 +41,5 @@
             <origin	xyz="0.0 0.0 0.0" rpy="0.0 0.0 0.0" />
             <geometry>
-                <mesh filename="package://robot_description/meshes/razbot/body.stl" scale="0.001 0.001 0.001"/>
+                <mesh filename="package://robot_gazebo/meshes/razbot/body.stl" scale="0.001 0.001 0.001"/>
             </geometry>
             <material name="blue"/>
@@ -48,5 +48,5 @@
             <origin xyz="0.0 0.0 0.0" rpy="0.0 0.0 0.0"/>
             <geometry>
-                <mesh filename="package://robot_description/meshes/razbot/body.stl" scale="0.001 0.001 0.001"/>
+                <mesh filename="package://robot_gazebo/meshes/razbot/body.stl" scale="0.001 0.001 0.001"/>
             </geometry>
             <material name="blue"/>
@@ -131,5 +131,5 @@
                 <origin xyz="0.0 0.0 0.0" rpy="0.0 0.0 0.0"/>
                 <geometry>
-                    <mesh filename="package://robot_description/meshes/razbot/coxa.stl" scale="0.001 0.001 0.001"/>
+                    <mesh filename="package://robot_gazebo/meshes/razbot/coxa.stl" scale="0.001 0.001 0.001"/>
                 </geometry>
                 <material name="green"/>
@@ -138,5 +138,5 @@
                 <origin xyz="0.0 0.0 0.0" rpy="0.0 0.0 0.0" />
                 <geometry>
-                    <mesh filename="package://robot_description/meshes/razbot/coxa.stl" scale="0.001 0.001 0.001"/>
+                    <mesh filename="package://robot_gazebo/meshes/razbot/coxa.stl" scale="0.001 0.001 0.001"/>
                 </geometry>
                 <material name="green"/>
@@ -176,5 +176,5 @@
                 <origin xyz="0.0 0.0 0.0" rpy="0.0 0.0 0.0"/>
                 <geometry>
-                    <mesh filename="package://robot_description/meshes/razbot/femur.stl" scale="0.001 0.001 0.001"/>
+                    <mesh filename="package://robot_gazebo/meshes/razbot/femur.stl" scale="0.001 0.001 0.001"/>
                 </geometry>
                 <material name="red"/>
@@ -183,5 +183,5 @@
                 <origin xyz="0.0 0.0 0.0" rpy="0.0 0.0 0.0" />
                 <geometry>
-                    <mesh filename="package://robot_description/meshes/razbot/femur.stl" scale="0.001 0.001 0.001"/>
+                    <mesh filename="package://robot_gazebo/meshes/razbot/femur.stl" scale="0.001 0.001 0.001"/>
                 </geometry>
                 <material name="red"/>
@@ -221,5 +221,5 @@
                 <origin xyz="0.0 0.0 0.0" rpy="0.0 0.0 0.0"/>
                 <geometry>
-                    <mesh filename="package://robot_description/meshes/razbot/tibia.stl" scale="0.001 0.001 0.001"/>
+                    <mesh filename="package://robot_gazebo/meshes/razbot/tibia.stl" scale="0.001 0.001 0.001"/>
                 </geometry>
                 <material name="green"/>
@@ -228,5 +228,5 @@
                 <origin xyz="0.0 0.0 0.0" rpy="0.0 0.0 0.0" />
                 <geometry>
-                    <mesh filename="package://robot_description/meshes/razbot/tibia.stl" scale="0.001 0.001 0.001"/>
+                    <mesh filename="package://robot_gazebo/meshes/razbot/tibia.stl" scale="0.001 0.001 0.001"/>
                 </geometry>
                 <material name="green"/>

File: xacro/tb3_burger.xacro (robot description, xacro)
@@ -34,5 +34,5 @@
       <origin xyz="-0.032 0 0.0" rpy="0 0 0"/>
       <geometry>
-        <mesh filename="package://robot_description/meshes/tb3/burger_base.stl" scale="0.001 0.001 0.001"/>
+        <mesh filename="package://robot_gazebo/meshes/tb3/burger_base.stl" scale="0.001 0.001 0.001"/>
       </geometry>
       <material name="blue"/>
@@ -62,5 +62,5 @@
       <origin xyz="0 0 0" rpy="1.57 0 0"/>
       <geometry>
-        <mesh filename="package://robot_description/meshes/tb3/left_tire.stl" scale="0.001 0.001 0.001"/>
+        <mesh filename="package://robot_gazebo/meshes/tb3/left_tire.stl" scale="0.001 0.001 0.001"/>
       </geometry>
       <material name="black"/>
@@ -90,5 +90,5 @@
       <origin xyz="0 0 0" rpy="1.57 0 0"/>
       <geometry>
-        <mesh filename="package://robot_description/meshes/tb3/right_tire.stl" scale="0.001 0.001 0.001"/>
+        <mesh filename="package://robot_gazebo/meshes/tb3/right_tire.stl" scale="0.001 0.001 0.001"/>
       </geometry>
       <material name="black"/>
@@ -151,5 +151,5 @@
       <origin xyz="0 0 0.0" rpy="0 0 0"/>
       <geometry>
-        <mesh filename="package://robot_description/meshes/tb3/lds.stl" scale="0.001 0.001 0.001"/>
+        <mesh filename="package://robot_gazebo/meshes/tb3/lds.stl" scale="0.001 0.001 0.001"/>
       </geometry>
       <material name="green"/>

File: xacro/tb3_waffle.xacro (robot description, xacro)
@@ -34,5 +34,5 @@
       <origin xyz="-0.064 0 0.0" rpy="0 0 0"/>
       <geometry>
-        <mesh filename="package://robot_description/meshes/tb3/waffle_base.stl" scale="0.001 0.001 0.001"/>
+        <mesh filename="package://robot_gazebo/meshes/tb3/waffle_base.stl" scale="0.001 0.001 0.001"/>
       </geometry>
       <material name="blue"/>
@@ -64,5 +64,5 @@
       <origin xyz="0 0 0" rpy="1.57 0 0"/>
       <geometry>
-        <mesh filename="package://robot_description/meshes/tb3/left_tire.stl" scale="0.001 0.001 0.001"/>
+        <mesh filename="package://robot_gazebo/meshes/tb3/left_tire.stl" scale="0.001 0.001 0.001"/>
       </geometry>
       <material name="black"/>
@@ -94,5 +94,5 @@
       <origin xyz="0 0 0" rpy="1.57 0 0"/>
       <geometry>
-        <mesh filename="package://robot_description/meshes/tb3/right_tire.stl" scale="0.001 0.001 0.001"/>
+        <mesh filename="package://robot_gazebo/meshes/tb3/right_tire.stl" scale="0.001 0.001 0.001"/>
       </geometry>
       <material name="black"/>
@@ -187,5 +187,5 @@
       <origin xyz="0 0 0" rpy="0 0 0"/>
       <geometry>
-        <mesh filename="package://robot_description/meshes/tb3/lds.stl" scale="0.001 0.001 0.001"/>
+        <mesh filename="package://robot_gazebo/meshes/tb3/lds.stl" scale="0.001 0.001 0.001"/>
       </geometry>
       <material name="green"/>
@@ -216,5 +216,5 @@
      <origin xyz="0 0 0" rpy="1.57 0 1.57"/>
       <geometry>
-       <mesh filename="package://robot_description/meshes/tb3/r200.dae" />
+       <mesh filename="package://robot_gazebo/meshes/tb3/r200.dae" />
       </geometry>
       <material name="green"/>

File: xacro/tb3_waffle_pi.xacro (robot description, xacro)
@@ -34,5 +34,5 @@
       <origin xyz="-0.064 0 0.0" rpy="0 0 0"/>
       <geometry>
-        <mesh filename="package://robot_description/meshes/tb3/waffle_pi_base.stl" scale="0.001 0.001 0.001"/>
+        <mesh filename="package://robot_gazebo/meshes/tb3/waffle_pi_base.stl" scale="0.001 0.001 0.001"/>
       </geometry>
       <material name="blue"/>
@@ -64,5 +64,5 @@
       <origin xyz="0 0 0" rpy="1.57 0 0"/>
       <geometry>
-        <mesh filename="package://robot_description/meshes/tb3/left_tire.stl" scale="0.001 0.001 0.001"/>
+        <mesh filename="package://robot_gazebo/meshes/tb3/left_tire.stl" scale="0.001 0.001 0.001"/>
       </geometry>
       <material name="black"/>
@@ -94,5 +94,5 @@
       <origin xyz="0 0 0" rpy="1.57 0 0"/>
       <geometry>
-        <mesh filename="package://robot_description/meshes/tb3/right_tire.stl" scale="0.001 0.001 0.001"/>
+        <mesh filename="package://robot_gazebo/meshes/tb3/right_tire.stl" scale="0.001 0.001 0.001"/>
       </geometry>
       <material name="black"/>
@@ -187,5 +187,5 @@
       <origin xyz="0 0 0.0" rpy="0 0 0"/>
       <geometry>
-        <mesh filename="package://robot_description/meshes/tb3/lds.stl" scale="0.001 0.001 0.001"/>
+        <mesh filename="package://robot_gazebo/meshes/tb3/lds.stl" scale="0.001 0.001 0.001"/>
       </geometry>
       <material name="green"/>

File: xacro/twr.xacro (robot description, xacro)
@@ -75,5 +75,5 @@
       <origin xyz="0 0 -0.05" rpy="1.5707963267949 0 3.141592654"/>
       <geometry>
-        <mesh filename="package://robot_description/meshes/twr/robot_base.stl" />
+        <mesh filename="package://robot_gazebo/meshes/twr/robot_base.stl" />
       </geometry>
       <material name="red"/>

Commit message: update

File: xacro/golem.xacro (robot description, xacro)
@@ -65,4 +65,7 @@
         </inertial>
     </link>
+    <gazebo reference="body_link">
+        <material>Gazebo/Blue</material>
+    </gazebo>
 <!-- ****************************************************** Camera RGB Joint *********************************************************  -->
     <joint name="camera_rgb_joint" type="fixed">
@@ -198,4 +201,7 @@
         </inertial>
     </link>
+    <gazebo reference="coxa_${side}${position}">
+        <material>Gazebo/Green</material>
+    </gazebo>
 <!-- ****************************************************** Femur Joint **************************************************************  -->
     <joint name="femur_joint_${side}${position}" type="revolute">
@@ -242,4 +248,7 @@
         </inertial>
     </link>
+    <gazebo reference="femur_${side}${position}">
+        <material>Gazebo/Red</material>
+    </gazebo>
 <!-- ****************************************************** Tibia Joint **************************************************************  -->
     <joint name="tibia_joint_${side}${position}" type="revolute">
@@ -286,4 +295,7 @@
         </inertial>
     </link>
+     <gazebo reference="tibia_${side}${position}">
+        <material>Gazebo/Green</material>
+    </gazebo>
 <!-- ****************************************************** Tarsus Joint *************************************************************  -->
     <joint name="tarsus_joint_${side}${position}" type="revolute">
@@ -330,4 +342,7 @@
         </inertial>
     </link>
+    <gazebo reference="tarsus_${side}${position}">
+        <material>Gazebo/Red</material>
+    </gazebo>
 <!-- ****************************************************** Foot Joint ***************************************************************  -->
     <joint name="foot_joint_${side}${position}" type="fixed">

Commit message: update

File: xacro/golem.xacro (robot description, xacro)
@@ -65,7 +65,4 @@
         </inertial>
     </link>
-    <gazebo reference="body_link">
-        <material>Gazebo/Blue</material>
-    </gazebo>
 <!-- ****************************************************** Camera RGB Joint *********************************************************  -->
     <joint name="camera_rgb_joint" type="fixed">
@@ -201,7 +198,4 @@
         </inertial>
     </link>
-    <gazebo reference="coxa_${side}${position}">
-        <material>Gazebo/Green</material>
-    </gazebo>
 <!-- ****************************************************** Femur Joint **************************************************************  -->
     <joint name="femur_joint_${side}${position}" type="revolute">
@@ -248,7 +242,4 @@
         </inertial>
     </link>
-    <gazebo reference="femur_${side}${position}">
-        <material>Gazebo/Red</material>
-    </gazebo>
 <!-- ****************************************************** Tibia Joint **************************************************************  -->
     <joint name="tibia_joint_${side}${position}" type="revolute">
@@ -295,7 +286,4 @@
         </inertial>
     </link>
-     <gazebo reference="tibia_${side}${position}">
-        <material>Gazebo/Green</material>
-    </gazebo>
 <!-- ****************************************************** Tarsus Joint *************************************************************  -->
     <joint name="tarsus_joint_${side}${position}" type="revolute">
@@ -342,7 +330,4 @@
         </inertial>
     </link>
-    <gazebo reference="tarsus_${side}${position}">
-        <material>Gazebo/Red</material>
-    </gazebo>
 <!-- ****************************************************** Foot Joint ***************************************************************  -->
     <joint name="foot_joint_${side}${position}" type="fixed">
@@ -362,4 +347,20 @@
         </inertial>
     </link>
+<!-- ****************************************************** Gazebo Colors*************************************************************  -->
+    <gazebo reference="body_link">
+        <material>Gazebo/Blue</material>
+    </gazebo>
+    <gazebo reference="coxa_${side}${position}">
+        <material>Gazebo/Green</material>
+    </gazebo>
+    <gazebo reference="femur_${side}${position}">
+        <material>Gazebo/Red</material>
+    </gazebo>
+    <gazebo reference="tibia_${side}${position}">
+        <material>Gazebo/Green</material>
+    </gazebo>
+    <gazebo reference="tarsus_${side}${position}">
+            <material>Gazebo/Red</material>
+    </gazebo>
 <!-- ******************************************************  End of Macro ************************************************************  -->
     </xacro:macro>

Commit message: u

File: xacro/golem.xacro (robot description, xacro)
@@ -6,4 +6,5 @@
 <!-- *********************************************************************************************************************************  -->
 <!-- ****************************************************** Parameters ***************************************************************  -->
+    <xacro:property name="mesh_path"        value="package://robot_gazebo/meshes/golem/"/>
     <xacro:property name="body_length_x"    value="0.3556"/>
     <xacro:property name="body_length_y"    value="0.165"/>
@@ -45,5 +46,5 @@
             <origin xyz="0.0 0.0 0.0" rpy="0.0 0.0 0.0"/>
             <geometry>
-                <mesh filename="package://robot_gazebo/meshes/golem/body.stl" scale="0.001 0.001 0.001"/>
+                <mesh filename="${mesh_path}body.stl" scale="0.001 0.001 0.001"/>
             </geometry>
             <material name="blue"/>
