Commit message: u

File: xacro/golem.xacro (robot description, xacro)
@@ -13,6 +13,6 @@
     <xacro:property name="tibia_length"     value="0.08774"/>
     <xacro:property name="tarsus_length"    value="0.12065"/>
-    <xacro:property name="joint_lower_limit"    value="-${3.14}"/>
-    <xacro:property name="joint_upper_limit"    value="${3.14}"/>
+    <xacro:property name="joint_lower_limit"    value="-${pi}"/>
+    <xacro:property name="joint_upper_limit"    value="${pi}"/>
     <xacro:property name="joint_effort"         value="6.0"/>
     <xacro:property name="joint_velocity"       value="0.524"/>
@@ -66,4 +66,7 @@
         </inertial>
     </link>
+    <gazebo reference="base_link">
+        <material>Gazebo/Blue</material>
+    </gazebo>
 <!-- ****************************************************** Camera RGB Joint *********************************************************  -->
     <joint name="camera_rgb_joint" type="fixed">
@@ -199,4 +202,7 @@
         </inertial>
     </link>
+    <gazebo reference="coxa_${side}${position}">
+        <material>Gazebo/Green</material>
+    </gazebo>
 <!-- ****************************************************** Femur Joint **************************************************************  -->
     <joint name="femur_joint_${side}${position}" type="revolute">
@@ -243,4 +249,7 @@
         </inertial>
     </link>
+    <gazebo reference="femur_${side}${position}">
+        <material>Gazebo/Red</material>
+    </gazebo>
 <!-- ****************************************************** Tibia Joint **************************************************************  -->
     <joint name="tibia_joint_${side}${position}" type="revolute">
@@ -287,4 +296,7 @@
         </inertial>
     </link>
+    <gazebo reference="tibia_${side}${position}">
+        <material>Gazebo/Green</material>
+    </gazebo>
 <!-- ****************************************************** Tarsus Joint *************************************************************  -->
     <joint name="tarsus_joint_${side}${position}" type="revolute">
@@ -331,4 +343,7 @@
         </inertial>
     </link>
+    <gazebo reference="tarsus_${side}${position}">
+            <material>Gazebo/Red</material>
+    </gazebo>
 <!-- ****************************************************** Foot Joint ***************************************************************  -->
     <joint name="foot_joint_${side}${position}" type="fixed">
@@ -348,20 +363,4 @@
         </inertial>
     </link>
-<!-- ****************************************************** Gazebo Colors*************************************************************  -->
-    <gazebo reference="base_link">
-        <material>Gazebo/Blue</material>
-    </gazebo>
-    <gazebo reference="coxa_${side}${position}">
-        <material>Gazebo/Green</material>
-    </gazebo>
-    <gazebo reference="femur_${side}${position}">
-        <material>Gazebo/Red</material>
-    </gazebo>
-    <gazebo reference="tibia_${side}${position}">
-        <material>Gazebo/Green</material>
-    </gazebo>
-    <gazebo reference="tarsus_${side}${position}">
-            <material>Gazebo/Red</material>
-    </gazebo>
 <!-- ******************************************************  End of Macro ************************************************************  -->
     </xacro:macro>

Commit message: u

File: xacro/golem.xacro (robot description, xacro)
@@ -13,8 +13,8 @@
     <xacro:property name="tibia_length"     value="0.08774"/>
     <xacro:property name="tarsus_length"    value="0.12065"/>
-    <xacro:property name="joint_lower_limit"    value="-${pi}"/>
-    <xacro:property name="joint_upper_limit"    value="${pi}"/>
+    <xacro:property name="joint_lower_limit"    value="-${radians(180)}"/>
+    <xacro:property name="joint_upper_limit"    value=" ${radians(180)}"/>
     <xacro:property name="joint_effort"         value="6.0"/>
-    <xacro:property name="joint_velocity"       value="0.524"/>
+    <xacro:property name="joint_velocity"       value=" ${radians(300)}"/>
 <!-- ****************************************************** Colors *******************************************************************  -->
     <material name="red">

File: xacro/pxm3.xacro (robot description, xacro)
@@ -7,11 +7,11 @@
 <!-- ****************************************************** Parameters ***************************************************************  -->
   <xacro:property name="mesh_path"          value="package://robot_gazebo/meshes/pxm3/"/>
-  <xacro:property name="connect_offset"     value="0.02633" />
+  <xacro:property name="connect_offset"     value=" 0.02633" />
   <xacro:property name="thigh_offset_y"     value="-0.0645" />
   <xacro:property name="thigh_offset_z"     value="-0.0145" />
-  <xacro:property name="joint_lower_limit"  value="-2.6179939"/>
-  <xacro:property name="joint_upper_limit"  value="2.6179939"/>
-  <xacro:property name="joint_effort"       value="2.8"/>
-  <xacro:property name="joint_velocity"     value="5.6548668"/>
+  <xacro:property name="joint_lower_limit"  value="-${radians(150)}"/>
+  <xacro:property name="joint_upper_limit"  value=" ${radians(150)}"/>
+  <xacro:property name="joint_effort"       value=" 2.8"/>
+  <xacro:property name="joint_velocity"     value=" ${radians(324)}"/>
 <!-- ****************************************************** Colors *******************************************************************  -->
   <material name="red">

Commit message: u

File: xacro/golem.xacro (robot description, xacro)
@@ -15,5 +15,5 @@
     <xacro:property name="joint_lower_limit"    value="-${radians(180)}"/>
     <xacro:property name="joint_upper_limit"    value=" ${radians(180)}"/>
-    <xacro:property name="joint_effort"         value="6.0"/>
+    <xacro:property name="joint_effort"         value=" 6.0"/>
     <xacro:property name="joint_velocity"       value=" ${radians(300)}"/>
 <!-- ****************************************************** Colors *******************************************************************  -->

Commit message: u

File: xacro/golem.xacro (robot description, xacro)
@@ -6,11 +6,11 @@
 <!-- *********************************************************************************************************************************  -->
 <!-- ****************************************************** Parameters ***************************************************************  -->
-    <xacro:property name="mesh_path"        value="package://robot_gazebo/meshes/golem/"/>
-    <xacro:property name="body_length_x"    value="0.3556"/>
-    <xacro:property name="body_length_y"    value="0.165"/>
-    <xacro:property name="coxa_length"      value="0.05893"/>
-    <xacro:property name="femur_length"     value="0.10798"/>
-    <xacro:property name="tibia_length"     value="0.08774"/>
-    <xacro:property name="tarsus_length"    value="0.12065"/>
+    <xacro:property name="mesh_path"            value="package://robot_gazebo/meshes/golem/"/>
+    <xacro:property name="body_length_x"        value="0.3556"/>
+    <xacro:property name="body_length_y"        value="0.165"/>
+    <xacro:property name="coxa_length"          value="0.05893"/>
+    <xacro:property name="femur_length"         value="0.10798"/>
+    <xacro:property name="tibia_length"         value="0.08774"/>
+    <xacro:property name="tarsus_length"        value="0.12065"/>
     <xacro:property name="joint_lower_limit"    value="-${radians(180)}"/>
     <xacro:property name="joint_upper_limit"    value=" ${radians(180)}"/>

File: xacro/razbot.xacro (robot description, xacro)
@@ -39,10 +39,10 @@
         <parent link="base_footprint" />
         <child link="base_link" />
-        <origin xyz="0.0 0.0 0.0" rpy="0.0 0.0 0.0" />
+        <origin xyz="0 0 0" rpy="0 0 0" />
     </joint>
 <!-- ****************************************************** Base Link ****************************************************************  -->
 	<link name="base_link">
         <visual>
-            <origin	xyz="0.0 0.0 0.0" rpy="0.0 0.0 0.0" />
+            <origin	xyz="0 0 0" rpy="0 0 0" />
             <geometry>
                 <mesh filename="${mesh_path}body.stl" scale="0.001 0.001 0.001"/>
@@ -51,5 +51,5 @@
         </visual>
         <collision>
-            <origin xyz="0.0 0.0 0.0" rpy="0.0 0.0 0.0"/>
+            <origin xyz="0 0 0" rpy="0 0 0"/>
             <geometry>
                 <mesh filename="${mesh_path}body.stl" scale="0.001 0.001 0.001"/>
@@ -58,5 +58,5 @@
         </collision>
         <inertial>
-            <origin xyz="0.0 0.0 0.0" rpy="0.0 0.0 0.0" />
+            <origin xyz="0 0 0" rpy="0 0 0" />
             <mass value="0.00001"/>
             <inertia
@@ -73,10 +73,10 @@
 		<parent link="base_link" />
 		<child link="imu_link" />
-		<origin xyz="0.0 0.0 0.0" rpy="0.0 0.0 0.0" />
+		<origin xyz="0 0 0" rpy="0 0 0" />
 	</joint>
 <!-- ****************************************************** IMU Link *****************************************************************  -->
 	<link name="imu_link">
         <inertial>
-            <origin xyz="0.0 0.0 0.0" rpy="0.0 0.0 0.0" />
+            <origin xyz="0 0 0" rpy="0 0 0" />
             <mass value="0.00001"/>
             <inertia
@@ -90,5 +90,5 @@
 <!-- ****************************************************** Leg Center Joint *********************************************************  -->
 		<joint name="leg_center_joint_${side}${position}" type="fixed">
-			<origin xyz="${x} ${y} 0.0" rpy="0.0 0.0 0.0" />
+			<origin xyz="${x} ${y} 0.0" rpy="0 0 0" />
 			<parent link="base_link" />
 			<child link="leg_center_${side}${position}" />
@@ -97,5 +97,5 @@
 		<link name="leg_center_${side}${position}" >
             <inertial>
-                <origin xyz="0.0 0.0 0.0" rpy="0.0 0.0 0.0" />
+                <origin xyz="0 0 0" rpy="0 0 0" />
                 <mass value="0.00001"/>
                 <inertia
@@ -107,5 +107,5 @@
 <!-- ****************************************************** Coxa Joint **************************************************************  -->
 		<joint name="coxa_joint_${side}${position}" type="revolute">
-			<origin xyz="0.0 0.0 0.0" rpy="0.0 0.0 ${angle}" />
+			<origin xyz="0 0 0" rpy="0.0 0.0 ${angle}" />
 			<parent link="leg_center_${side}${position}" />
 			<child link="coxa_${side}${position}" />
@@ -116,5 +116,5 @@
         <link name="coxa_${side}${position}">
             <visual>
-                <origin xyz="0.0 0.0 0.0" rpy="0.0 0.0 0.0"/>
+                <origin xyz="0 0 0" rpy="0 0 0"/>
                 <geometry>
                     <mesh filename="${mesh_path}coxa.stl" scale="0.001 0.001 0.001"/>
@@ -123,5 +123,5 @@
             </visual>
             <collision>
-                <origin xyz="0.0 0.0 0.0" rpy="0.0 0.0 0.0" />
+                <origin xyz="0 0 0" rpy="0 0 0" />
                 <geometry>
                     <mesh filename="${mesh_path}coxa.stl" scale="0.001 0.001 0.001"/>
@@ -130,5 +130,5 @@
             </collision>
             <inertial>
-                <origin xyz="0.0 0.0 0.0" rpy="0.0 0.0 0.0" />
+                <origin xyz="0 0 0" rpy="0 0 0" />
                 <mass value="0.00001"/>
                 <inertia
@@ -154,5 +154,5 @@
 <!-- ****************************************************** Femur Joint **************************************************************  -->
 		<joint name="femur_joint_${side}${position}" type="revolute">
-			<origin xyz="${coxa_length} 0.0 0.0" rpy="-${pi/2} ${pi/2} 0.0" />
+			<origin xyz="${coxa_length} 0.0 0.0" rpy="$(radians(-90)} $(radians(90)} 0.0" />
 			<parent link="coxa_${side}${position}" />
 			<child link="femur_${side}${position}" />
@@ -163,5 +163,5 @@
         <link name="femur_${side}${position}">
             <visual>
-                <origin xyz="0.0 0.0 0.0" rpy="0.0 0.0 0.0"/>
+                <origin xyz="0 0 0" rpy="0 0 0"/>
                 <geometry>
                     <mesh filename="${mesh_path}femur.stl" scale="0.001 0.001 0.001"/>
@@ -170,5 +170,5 @@
             </visual>
             <collision>
-                <origin xyz="0.0 0.0 0.0" rpy="0.0 0.0 0.0" />
+                <origin xyz="0 0 0" rpy="0 0 0" />
                 <geometry>
                     <mesh filename="${mesh_path}femur.stl" scale="0.001 0.001 0.001"/>
@@ -177,5 +177,5 @@
             </collision>
             <inertial>
-                <origin xyz="0.0 0.0 0.0" rpy="0.0 0.0 0.0" />
+                <origin xyz="0 0 0" rpy="0 0 0" />
                 <mass value="0.00001"/>
                 <inertia
@@ -201,5 +201,5 @@
 <!-- ****************************************************** Tibia Joint *************************************************************  -->
 		<joint name="tibia_joint_${side}${position}" type="revolute">
-			<origin xyz="0.0 -${femur_length} 0.0" rpy="${pi} 0.0 0.0" />
+			<origin xyz="0.0 -${femur_length} 0.0" rpy="${radians(180)} 0 0" />
 			<parent link="femur_${side}${position}" />
 			<child link="tibia_${side}${position}" />
@@ -210,5 +210,5 @@
         <link name="tibia_${side}${position}">
             <visual>
-                <origin xyz="0.0 0.0 0.0" rpy="0.0 0.0 0.0"/>
+                <origin xyz="0 0 0" rpy="0 0 0"/>
                 <geometry>
                     <mesh filename="${mesh_path}tibia.stl" scale="0.001 0.001 0.001"/>
@@ -217,5 +217,5 @@
             </visual>
             <collision>
-                <origin xyz="0.0 0.0 0.0" rpy="0.0 0.0 0.0" />
+                <origin xyz="0 0.0 0.0" rpy="0 0 0" />
                 <geometry>
                     <mesh filename="${mesh_path}tibia.stl" scale="0.001 0.001 0.001"/>
@@ -224,5 +224,5 @@
             </collision>
             <inertial>
-                <origin xyz="0.0 0.0 0.0" rpy="0.0 0.0 0.0" />
+                <origin xyz="0 0.0 0.0" rpy="0 0 0" />
                 <mass value="0.00001"/>
                 <inertia
@@ -249,10 +249,10 @@
 	</xacro:macro>
 <!-- ****************************************************** Build Robot **************************************************************  -->
-	<xacro:leg side="R" position="R" x="-${body_length_x/2}"    y="-${0.1695/2}"        angle="-${5*pi/6}"   axis=" 1" />
-	<xacro:leg side="R" position="M" x=" 0.0"                   y="-${body_length_y/2}" angle="-${pi/2}"     axis=" 1" />
-	<xacro:leg side="R" position="F" x=" ${body_length_x/2}"    y="-${0.1695/2}"        angle="-${pi/6}"     axis=" 1" />
-	<xacro:leg side="L" position="R" x="-${body_length_x/2}"    y=" ${0.1695/2}"        angle=" ${5*pi/6}"   axis="-1" />
-	<xacro:leg side="L" position="M" x=" 0.0"                   y=" ${body_length_y/2}" angle=" ${pi/2}"     axis="-1" />
-	<xacro:leg side="L" position="F" x=" ${body_length_x/2}"    y=" ${0.1695/2}"        angle=" ${pi/6}"     axis="-1" />
+	<xacro:leg side="R" position="R" x="-${body_length_x/2}"    y="-${0.1695/2}"        angle="${radians(-150)}"    axis=" 1" />
+	<xacro:leg side="R" position="M" x=" 0.0"                   y="-${body_length_y/2}" angle="${radians(-90)}"     axis=" 1" />
+	<xacro:leg side="R" position="F" x=" ${body_length_x/2}"    y="-${0.1695/2}"        angle="${radians(-30)}"     axis=" 1" />
+	<xacro:leg side="L" position="R" x="-${body_length_x/2}"    y=" ${0.1695/2}"        angle="${radians(150)}"     axis="-1" />
+	<xacro:leg side="L" position="M" x=" 0.0"                   y=" ${body_length_y/2}" angle="${radians(90)}"      axis="-1" />
+	<xacro:leg side="L" position="F" x=" ${body_length_x/2}"    y=" ${0.1695/2}"        angle="${radians(30)}"      axis="-1" />
 <!-- ******************************************************  *************************************************************************  -->
 </robot>

Commit message: u

File: xacro/golem.xacro (robot description, xacro)
@@ -17,6 +17,7 @@
     <xacro:property name="joint_effort"         value=" 6.0"/>
     <xacro:property name="joint_velocity"       value=" ${radians(300)}"/>
-<!-- ****************************************************** Import RVIZ Materials*****************************************************  -->
-  <xacro:include filename="$(find robot_gazebo)/xacro/common_rviz_materials.xacro" />
+<!-- ****************************************************** Includes *****************************************************************  -->
+  <xacro:include filename="$(find robot_gazebo)/xacro/common_rviz_materials.xacro" />   <!-- RVIZ Colors                                -->
+  <xacro:include filename="$(find robot_gazebo)/gazebo/golem_gz.xacro" />               <!-- Gazebo                                     -->
 <!-- ****************************************************** Base Footprint ***********************************************************  -->
     <link name="base_footprint"/>
@@ -52,7 +53,4 @@
         </inertial>
     </link>
-    <gazebo reference="base_link">
-        <material>Gazebo/Blue</material>
-    </gazebo>
 <!-- ****************************************************** Camera RGB Joint *********************************************************  -->
     <joint name="camera_rgb_joint" type="fixed">
@@ -188,7 +186,4 @@
         </inertial>
     </link>
-    <gazebo reference="coxa_${side}${position}">
-        <material>Gazebo/Green</material>
-    </gazebo>
 <!-- ****************************************************** Femur Joint **************************************************************  -->
     <joint name="femur_joint_${side}${position}" type="revolute">
@@ -235,7 +230,4 @@
         </inertial>
     </link>
-    <gazebo reference="femur_${side}${position}">
-        <material>Gazebo/Red</material>
-    </gazebo>
 <!-- ****************************************************** Tibia Joint **************************************************************  -->
     <joint name="tibia_joint_${side}${position}" type="revolute">
@@ -282,7 +274,4 @@
         </inertial>
     </link>
-    <gazebo reference="tibia_${side}${position}">
-        <material>Gazebo/Green</material>
-    </gazebo>
 <!-- ****************************************************** Tarsus Joint *************************************************************  -->
     <joint name="tarsus_joint_${side}${position}" type="revolute">
@@ -329,7 +318,4 @@
         </inertial>
     </link>
-    <gazebo reference="tarsus_${side}${position}">
-            <material>Gazebo/Red</material>
-    </gazebo>
 <!-- ****************************************************** Foot Joint ***************************************************************  -->
     <joint name="foot_joint_${side}${position}" type="fixed">
