Commit message: u

File: xacro/tb3_waffle.xacro (robot description, xacro)
@@ -85,4 +85,7 @@
       </inertial>
   </link>
+  <gazebo reference="wheel_left_link">
+    <material>Gazebo/FlatBlack</material>
+  </gazebo>
 <!-- ****************************************************** Wheel Right Joint ********************************************************  -->
   <joint name="wheel_right_joint" type="continuous">
@@ -115,4 +118,7 @@
       </inertial>
   </link>
+  <gazebo reference="wheel_right_link">
+    <material>Gazebo/FlatBlack</material>
+  </gazebo>
 <!-- ****************************************************** Caster Back Right Joint **************************************************  -->
   <joint name="caster_back_right_joint" type="fixed">
@@ -143,4 +149,7 @@
     </inertial>
   </link>
+  <gazebo reference="caster_back_link">
+    <material>Gazebo/White</material>
+  </gazebo>
 <!-- ****************************************************** Caster Back Left Joint ***************************************************  -->
   <joint name="caster_back_left_joint" type="fixed">
@@ -208,4 +217,7 @@
     </inertial>
   </link>
+  <gazebo reference="base_scan">
+    <material>Gazebo/Green</material>
+  </gazebo>
 <!-- ****************************************************** Camera Joint ************************************************************* -->
   <joint name="camera_joint" type="fixed">

Commit message: u

File: xacro/tb3_waffle.xacro (robot description, xacro)
@@ -39,7 +39,4 @@
     </inertial>
   </link>
-  <gazebo reference="base_link">
-    <material>Gazebo/Blue</material>
-  </gazebo>
 <!-- ****************************************************** Wheel Left Joint *********************************************************  -->
   <joint name="wheel_left_joint" type="continuous">
@@ -72,7 +69,4 @@
       </inertial>
   </link>
-  <gazebo reference="wheel_left_link">
-    <material>Gazebo/FlatBlack</material>
-  </gazebo>
 <!-- ****************************************************** Wheel Right Joint ********************************************************  -->
   <joint name="wheel_right_joint" type="continuous">
@@ -105,7 +99,4 @@
       </inertial>
   </link>
-  <gazebo reference="wheel_right_link">
-    <material>Gazebo/FlatBlack</material>
-  </gazebo>
 <!-- ****************************************************** Caster Back Right Joint **************************************************  -->
   <joint name="caster_back_right_joint" type="fixed">
@@ -136,7 +127,4 @@
     </inertial>
   </link>
-  <gazebo reference="caster_back_link">
-    <material>Gazebo/White</material>
-  </gazebo>
 <!-- ****************************************************** Caster Back Left Joint ***************************************************  -->
   <joint name="caster_back_left_joint" type="fixed">
@@ -204,7 +192,4 @@
     </inertial>
   </link>
-  <gazebo reference="base_scan">
-    <material>Gazebo/Green</material>
-  </gazebo>
 <!-- ****************************************************** Camera Joint ************************************************************* -->
   <joint name="camera_joint" type="fixed">

File: xacro/tb3_waffle_pi.xacro (robot description, xacro)
@@ -221,4 +221,5 @@
     <child link="camera_rgb_optical_frame"/>
   </joint>
+<!-- ****************************************************** RGB Camera Optical Link **************************************************  -->
   <link name="camera_rgb_optical_frame"/>
 <!-- *********************************************************************************************************************************  -->
