Commit message: u

File: xacro/twr.xacro (robot description, xacro)
@@ -180,4 +180,17 @@
     </inertial>
   </link>
+<!-- ****************************************************** Gazebo Colors*************************************************************  -->
+    <gazebo reference="base_link">
+        <material>Gazebo/Red</material>
+    </gazebo>
+    <gazebo reference="${prefix}_link">
+        <material>Gazebo/Gray</material>
+    </gazebo>
+    <gazebo reference="front_caster">
+        <material>Gazebo/White</material>
+    </gazebo>
+    <gazebo reference="lidar_link">
+        <material>Gazebo/Green</material>
+    </gazebo>
 <!-- *********************************************************************************************************************************  -->
 </robot>

Commit message: u

File: xacro/twr.xacro (robot description, xacro)
@@ -184,5 +184,8 @@
         <material>Gazebo/Red</material>
     </gazebo>
-    <gazebo reference="${prefix}_link">
+    <gazebo reference="drivewhl_l_link">
+        <material>Gazebo/Gray</material>
+    </gazebo>
+    <gazebo reference="drivewhl_r_link">
         <material>Gazebo/Gray</material>
     </gazebo>

Commit message: u

File: xacro/twr.xacro (robot description, xacro)
@@ -86,4 +86,7 @@
     <xacro:box_inertia m="40.0" w="${base_width}" d="${base_length}" h="${base_height}"/>
   </link>
+  <gazebo reference="base_link">
+      <material>Gazebo/Red</material>
+  </gazebo>
 <!-- ****************************************************** Drive Wheels Link Macro **************************************************  -->
   <xacro:macro name="wheel" params="prefix x_reflect y_reflect">
@@ -104,4 +107,7 @@
       <xacro:cylinder_inertia m="110.5" r="${wheel_radius}" h="${wheel_width}"/>
     </link>
+    <gazebo reference="${prefix}_link">
+        <material>Gazebo/Flatblack</material>
+    </gazebo>
 <!-- ****************************************************** Drive Wheels Joint Macro *************************************************  -->
 <!-- Connect the wheels to the base_link at the appropriate location, and define a continuous joint to allow the wheels to freely       -->
@@ -138,4 +144,7 @@
     <xacro:sphere_inertia m="10.05" r="${(wheel_radius+wheel_zoff-(base_height/2))}"/>
   </link>
+  <gazebo reference="front_caster">
+      <material>Gazebo/White</material>
+  </gazebo>
 <!-- **************************************************** Front Caster Joint *********************************************************  -->
   <joint name="caster_joint" type="fixed">
@@ -180,20 +189,7 @@
     </inertial>
   </link>
-<!-- ****************************************************** Gazebo Colors*************************************************************  -->
-    <gazebo reference="base_link">
-        <material>Gazebo/Red</material>
-    </gazebo>
-    <gazebo reference="drivewhl_l_link">
-        <material>Gazebo/Gray</material>
-    </gazebo>
-    <gazebo reference="drivewhl_r_link">
-        <material>Gazebo/Gray</material>
-    </gazebo>
-    <gazebo reference="front_caster">
-        <material>Gazebo/White</material>
-    </gazebo>
-    <gazebo reference="lidar_link">
-        <material>Gazebo/Green</material>
-    </gazebo>
+  <gazebo reference="lidar_link">
+    <material>Gazebo/Green</material>
+  </gazebo>
 <!-- *********************************************************************************************************************************  -->
 </robot>

Commit message: finshed Gazebo Colors

File: xacro/twr.xacro (robot description, xacro)
@@ -108,5 +108,5 @@
     </link>
     <gazebo reference="${prefix}_link">
-        <material>Gazebo/Flatblack</material>
+        <material>Gazebo/FlatBlack</material>
     </gazebo>
 <!-- ****************************************************** Drive Wheels Joint Macro *************************************************  -->

Commit message: u

File: xacro/twr.xacro (robot description, xacro)
@@ -14,28 +14,10 @@
   <xacro:property name="wheel_width"  value="0.06"/>
 <!-- x-axis points forward, y-axis points to left, z-axis points upwards                                                                -->
-<!-- Define the gap between the wheel and chassis along y-axis in meters                                                                -->
-  <xacro:property name="wheel_ygap" value="0.035"/>
-<!-- Position the wheels along the z-axis                                                                                               -->
-  <xacro:property name="wheel_zoff" value="0.05"/>
-<!-- Position the wheels along the x-axis                                                                                               -->
-  <xacro:property name="wheel_xoff" value="0.221"/>
-<!-- Position the caster wheel along the x-axis                                                                                         -->
-  <xacro:property name="caster_xoff" value="0.217"/>
-<!-- ****************************************************** Colors *******************************************************************  -->
-  <material name="red">
-    <color rgba="1.0 0.0 0.0 1.0"/>
-  </material>
-  <material name="green">
-    <color rgba="0.0 1.0 0.0 1.0"/>
-  </material>
-  <material name="blue">
-    <color rgba="0.0 0.0 1.0 1.0"/>
-  </material>
-  <material name="black">
-    <color rgba="0.3 0.3 0.3 1.0"/>
-  </material>
-  <material name="white">
-    <color rgba="1.0 1.0 1.0 1.0"/>
-  </material>
+  <xacro:property name="wheel_ygap"   value="0.035"/> <!-- gap between the wheel and chassis along y-axis in meters                     -->
+  <xacro:property name="wheel_zoff"   value="0.05" /> <!-- Position the wheels along the z-axis                                         -->
+  <xacro:property name="wheel_xoff"   value="0.221"/> <!-- Position the wheels along the x-axis                                         -->
+  <xacro:property name="caster_xoff"  value="0.217"/> <!-- Position the caster wheel along the x-axis                                   -->
+<!-- ****************************************************** Import RVIZ Materials*****************************************************  -->
+  <xacro:include filename="$(find robot_gazebo)/xacro/common_rviz_materials.xacro" />
 <!-- ****************************************************** Macros *******************************************************************  -->
 <!-- Define intertial property macros                                                                                                   -->

Commit message: u

File: xacro/twr.xacro (robot description, xacro)
@@ -55,5 +55,5 @@
   <link name="base_link">
     <visual>
-      <origin xyz="0 0 -0.05" rpy="${radians(90)} 0 ${radians(180)}"/>
+      <origin xyz="0 0 0" rpy="0 0 0"/>
       <geometry>
         <mesh filename="${mesh_path}robot_base.stl" />
