Commit message: u

File: xacro/cart_effort.xacro (robot description, xacro)
@@ -1,80 +1,18 @@
-<?xml version="1.0" ?>
-<robot name="cart" xmlns:xacro="http://ros.org/wiki/xacro">
-<!-- ****************************************************** World Link *************************************************************** -->
-  <link name="world"/>
-<!-- ****************************************************** slideBar Link ************************************************************ -->
-  <link name="slideBar">
-    <visual>
-      <geometry>
-        <box size="30 0.05 0.05"/>
-      </geometry>
-      <origin xyz="0 0 0"/>
-      <material name="green">
-        <color rgba="0 0.8 .8 1"/>
-      </material>
-    </visual>
-    <inertial>
-      <mass value="100"/>
-      <inertia ixx="1.0" ixy="0.0" ixz="0.0" iyy="1.0" iyz="0.0" izz="1.0"/>
-    </inertial>
-  </link>
-  <gazebo reference="slideBar">
-    <material>Gazebo/Orange</material>
-  </gazebo>
-<!-- ****************************************************** cart Link **************************************************************** -->
-  <link name="cart">
-    <visual>
-      <geometry>
-        <box size="0.5 0.5 0.2"/>
-      </geometry>
-      <origin xyz="0 0 0"/>
-      <material name="blue">
-        <color rgba="0 0 .8 1"/>
-      </material>
-    </visual>
-    <inertial>
-      <mass value="1"/>
-      <inertia ixx="1.0" ixy="0.0" ixz="0.0" iyy="1.0" iyz="0.0" izz="1.0"/>
-    </inertial>
-  </link>
-  <gazebo reference="cart">
-    <material>Gazebo/Red</material>
-  </gazebo>
-<!-- ****************************************************** world to slideBar Joint ************************************************** -->
-  <joint name="world_to_base" type="fixed">
-    <origin rpy="0 0 0" xyz="0 0 1"/>
-    <parent link="world"/>
-    <child link="slideBar"/>
-  </joint>
-<!-- ****************************************************** slideBar to cart Joint *************************************************** -->
-  <joint name="slider_to_cart" type="prismatic">
-    <axis xyz="1 0 0"/>
-    <origin xyz="0.0 0.0 0.0"/>
-    <parent link="slideBar"/>
-    <child link="cart"/>
-    <limit effort="1000.0" lower="-15" upper="15" velocity="30"/>
-    <dynamics damping="0.0" friction="0.0"/>
-  </joint>
-<!-- ****************************************************** Gazebo ROS2 Control ****************************************************** -->
-  <ros2_control name="GazeboSystem" type="system">
-    <hardware>
-      <plugin>gazebo_ros2_control/GazeboSystem</plugin>
-    </hardware>
-    <joint name="slider_to_cart">
-      <command_interface name="effort">
-        <param name="min">-1000</param>
-        <param name="max">1000</param>
-      </command_interface>
-      <state_interface name="position"/>
-      <state_interface name="velocity"/>
-      <state_interface name="effort"/>
-    </joint>
-  </ros2_control>
-<!-- ****************************************************** Gazebo ROS2 Plugin ******************************************************* -->
-  <gazebo>
-    <plugin filename="libgazebo_ros2_control.so" name="gazebo_ros2_control">
-      <parameters>$(find cart)/config/cartpole_controller_effort.yaml</parameters>
-    </plugin>
-  </gazebo>
-<!-- ****************************************************** End ********************************************************************** -->
+<?xml version="1.0"?>
+<robot name="cart" xmlns:xacro="http://www.ros.org/wiki/xacro">
+<!-- ****************************************************** Cart Robot ***************************************************************  -->
+<!-- Muthanna Alwahash                                                                                                                  -->
+<!-- March 2022                                                                                                                         -->
+<!-- *********************************************************************************************************************************  -->
+<!-- ****************************************************** Parameters ***************************************************************  -->
+    <xacro:property name="pkg_path"     value="$(find bots)"                />
+    <xacro:property name="mesh_path"    value="${pkg_path}/meshes/cart/"    />
+    <xacro:property name="name_space"   value="cart" />
+    <xacro:property name="prefix"       value=""      />
+<!-- ****************************************************** Includes *****************************************************************  -->
+    <xacro:include filename="${pkg_path}/xacro/common_rviz_materials.xacro" />  <!--  RVIZ Colors  -->
+    <xacro:include filename="${pkg_path}/xacro/urdf_cart_effort.xacro" />             <!--  Robot URDF   -->
+    <xacro:include filename="${pkg_path}/gazebo/gz_cart_effort.xacro" />              <!--  Gazebo Sim   -->
+    <xacro:include filename="${pkg_path}/r2c/r2c_cart_effort.xacro" />                <!--  ROS2_Control -->
+<!-- ****************************************************** END **********************************************************************  -->
 </robot>

File: xacro/cart_position.xacro (robot description, xacro)
@@ -1,82 +1,18 @@
-<?xml version="1.0" ?>
-<robot name="cart" xmlns:xacro="http://ros.org/wiki/xacro">
-<!-- ****************************************************** World Link *************************************************************** -->
-  <link name="world"/>
-<!-- ****************************************************** slideBar Link ************************************************************ -->
-  <link name="slideBar">
-    <visual>
-      <geometry>
-        <box size="30 0.05 0.05"/>
-      </geometry>
-      <origin xyz="0 0 0"/>
-      <material name="green">
-        <color rgba="0 0.8 .8 1"/>
-      </material>
-    </visual>
-    <inertial>
-      <mass value="100"/>
-      <inertia ixx="1.0" ixy="0.0" ixz="0.0" iyy="1.0" iyz="0.0" izz="1.0"/>
-    </inertial>
-  </link>
-  <gazebo reference="slideBar">
-    <material>Gazebo/Orange</material>
-  </gazebo>
-<!-- ****************************************************** cart Link **************************************************************** -->
-  <link name="cart">
-    <visual>
-      <geometry>
-        <box size="0.5 0.5 0.2"/>
-      </geometry>
-      <origin xyz="0 0 0"/>
-      <material name="blue">
-        <color rgba="0 0 .8 1"/>
-      </material>
-    </visual>
-    <inertial>
-      <mass value="1"/>
-      <inertia ixx="1.0" ixy="0.0" ixz="0.0" iyy="1.0" iyz="0.0" izz="1.0"/>
-    </inertial>
-  </link>
-  <gazebo reference="cart">
-    <material>Gazebo/Red</material>
-  </gazebo>
-<!-- ****************************************************** world to slideBar Joint ************************************************** -->
-  <joint name="world_to_base" type="fixed">
-    <origin rpy="0 0 0" xyz="0 0 1"/>
-    <parent link="world"/>
-    <child link="slideBar"/>
-  </joint>
-<!-- ****************************************************** slideBar to cart Joint *************************************************** -->
-  <joint name="slider_to_cart" type="prismatic">
-    <axis xyz="1 0 0"/>
-    <origin xyz="0.0 0.0 0.0"/>
-    <parent link="slideBar"/>
-    <child link="cart"/>
-    <limit effort="1000.0" lower="-15" upper="15" velocity="30"/>
-    <dynamics damping="0.0" friction="0.0"/>
-  </joint>
-<!-- ****************************************************** Gazebo ROS2 Control ****************************************************** -->
-  <ros2_control name="GazeboSystem" type="system">
-    <hardware>
-      <plugin>gazebo_ros2_control/GazeboSystem</plugin>
-    </hardware>
-    <joint name="slider_to_cart">
-      <command_interface name="position">
-        <param name="min">-15</param>
-        <param name="max">15</param>
-      </command_interface>
-      <state_interface name="position">
-        <param name="initial_value">1.0</param>
-      </state_interface>
-      <state_interface name="velocity"/>
-      <state_interface name="effort"/>
-    </joint>
-  </ros2_control>
-<!-- ****************************************************** Gazebo ROS2 Plugin ******************************************************* -->
-  <gazebo>
-    <plugin filename="libgazebo_ros2_control.so" name="gazebo_ros2_control">
-      <parameters>$(find cart)/config/cartpole_controller.yaml</parameters>
-    </plugin>
-  </gazebo>
-<!-- ****************************************************** End ********************************************************************** -->
+<?xml version="1.0"?>
+<robot name="cart" xmlns:xacro="http://www.ros.org/wiki/xacro">
+<!-- ****************************************************** Cart Robot ***************************************************************  -->
+<!-- Muthanna Alwahash                                                                                                                  -->
+<!-- March 2022                                                                                                                         -->
+<!-- *********************************************************************************************************************************  -->
+<!-- ****************************************************** Parameters ***************************************************************  -->
+    <xacro:property name="pkg_path"     value="$(find bots)"                />
+    <xacro:property name="mesh_path"    value="${pkg_path}/meshes/cart/"    />
+    <xacro:property name="name_space"   value="cart" />
+    <xacro:property name="prefix"       value=""      />
+<!-- ****************************************************** Includes *****************************************************************  -->
+    <xacro:include filename="${pkg_path}/xacro/common_rviz_materials.xacro" />  <!--  RVIZ Colors  -->
+    <xacro:include filename="${pkg_path}/xacro/urdf_cart.xacro" />             <!--  Robot URDF   -->
+    <xacro:include filename="${pkg_path}/gazebo/gz_cart_position.xacro" />              <!--  Gazebo Sim   -->
+    <xacro:include filename="${pkg_path}/r2c/r2c_cart_position.xacro" />                <!--  ROS2_Control -->
+<!-- ****************************************************** END **********************************************************************  -->
 </robot>

File: xacro/cart_velocity.xacro (robot description, xacro)
@@ -1,113 +1,18 @@
-<?xml version="1.0" ?>
-<robot name="cart" xmlns:xacro="http://ros.org/wiki/xacro">
-<!-- ****************************************************** World Link *************************************************************** -->
-  <link name="world"/>
-<!-- ****************************************************** slideBar Link ************************************************************ -->
-  <link name="slideBar">
-    <visual>
-      <geometry>
-        <box size="30 0.05 0.05"/>
-      </geometry>
-      <origin xyz="0 0 0"/>
-      <material name="green">
-        <color rgba="0 0.8 .8 1"/>
-      </material>
-    </visual>
-    <inertial>
-      <mass value="100"/>
-      <inertia ixx="1.0" ixy="0.0" ixz="0.0" iyy="1.0" iyz="0.0" izz="1.0"/>
-    </inertial>
-  </link>
-  <gazebo reference="slideBar">
-    <material>Gazebo/Orange</material>
-  </gazebo>
-<!-- ****************************************************** cart Link **************************************************************** -->
-  <link name="cart">
-    <visual>
-      <geometry>
-        <box size="0.5 0.5 0.2"/>
-      </geometry>
-      <origin xyz="0 0 0"/>
-      <material name="blue">
-        <color rgba="0 0 .8 1"/>
-      </material>
-    </visual>
-    <inertial>
-      <mass value="1"/>
-      <inertia ixx="1.0" ixy="0.0" ixz="0.0" iyy="1.0" iyz="0.0" izz="1.0"/>
-    </inertial>
-  </link>
-  <gazebo reference="cart">
-    <material>Gazebo/Red</material>
-  </gazebo>
-  <!-- ****************************************************** world to slideBar Joint ************************************************** -->
-  <joint name="world_to_base" type="fixed">
-    <origin rpy="0 0 0" xyz="0 0 1"/>
-    <parent link="world"/>
-    <child link="slideBar"/>
-  </joint>
-<!-- ****************************************************** slideBar to cart Joint *************************************************** -->
-  <joint name="slider_to_cart" type="prismatic">
-    <axis xyz="1 0 0"/>
-    <origin xyz="0.0 0.0 0.0"/>
-    <parent link="slideBar"/>
-    <child link="cart"/>
-    <limit effort="1000.0" lower="-15" upper="15" velocity="30"/>
-    <dynamics damping="0.0" friction="0.0"/>
-  </joint>
-<!-- ****************************************************** IMU Link ***************************************************************** -->
-  <link name="imu">
-    <inertial>
-      <mass value="0.1"/>
-      <inertia ixx="1.0" ixy="0" ixz="0" iyy="1.0" iyz="0" izz="1.0"/>
-    </inertial>
-  </link>
-<!-- ****************************************************** cart to IMU joint ******************************************************** -->
-  <joint name="cart_to_imu" type="fixed">
-    <origin xyz="0.0 0.0 0.0"/>
-    <parent link="cart"/>
-    <child link="imu"/>
-    <dynamics damping="0.0" friction="0.0"/>
-  </joint>
-<!-- ****************************************************** imu Gazebo *************************************************************** -->
-  <gazebo reference="imu">
-    <sensor name="cart_imu_sensor" type="imu">
-      <always_on>1</always_on>
-      <update_rate>10.0</update_rate>
-    </sensor>
-  </gazebo>
-<!-- ****************************************************** Gazebo ROS2 Control ****************************************************** -->
-  <ros2_control name="GazeboSystem" type="system">
-    <hardware>
-      <plugin>gazebo_ros2_control/GazeboSystem</plugin>
-    </hardware>
-    <joint name="slider_to_cart">
-      <command_interface name="velocity">
-        <param name="min">-10</param>
-        <param name="max">10</param>
-      </command_interface>
-      <state_interface name="position"/>
-      <state_interface name="velocity"/>
-      <state_interface name="effort"/>
-    </joint>
-    <sensor name="cart_imu_sensor">
-      <state_interface name="orientation.x"/>
-      <state_interface name="orientation.y"/>
-      <state_interface name="orientation.z"/>
-      <state_interface name="orientation.w"/>
-      <state_interface name="angular_velocity.x"/>
-      <state_interface name="angular_velocity.y"/>
-      <state_interface name="angular_velocity.z"/>
-      <state_interface name="linear_acceleration.x"/>
-      <state_interface name="linear_acceleration.y"/>
-      <state_interface name="linear_acceleration.z"/>
-    </sensor>
-  </ros2_control>
-<!-- ****************************************************** Gazebo ROS2 Plugin ******************************************************* -->
-  <gazebo>
-    <plugin filename="libgazebo_ros2_control.so" name="gazebo_ros2_control">
-      <parameters>$(find cart)/config/cartpole_controller_velocity.yaml</parameters>
-    </plugin>
-  </gazebo>
-<!-- ****************************************************** End ********************************************************************** -->
+<?xml version="1.0"?>
+<robot name="cart" xmlns:xacro="http://www.ros.org/wiki/xacro">
+<!-- ****************************************************** Cart Robot ***************************************************************  -->
+<!-- Muthanna Alwahash                                                                                                                  -->
+<!-- March 2022                                                                                                                         -->
+<!-- *********************************************************************************************************************************  -->
+<!-- ****************************************************** Parameters ***************************************************************  -->
+    <xacro:property name="pkg_path"     value="$(find bots)"                />
+    <xacro:property name="mesh_path"    value="${pkg_path}/meshes/cart/"    />
+    <xacro:property name="name_space"   value="cart" />
+    <xacro:property name="prefix"       value=""      />
+<!-- ****************************************************** Includes *****************************************************************  -->
+    <xacro:include filename="${pkg_path}/xacro/common_rviz_materials.xacro" />  <!--  RVIZ Colors  -->
+    <xacro:include filename="${pkg_path}/xacro/urdf_cart.xacro" />             <!--  Robot URDF   -->
+    <xacro:include filename="${pkg_path}/gazebo/gz_cart_velocity.xacro" />              <!--  Gazebo Sim   -->
+    <xacro:include filename="${pkg_path}/r2c/r2c_cart_velocity.xacro" />                <!--  ROS2_Control -->
+<!-- ****************************************************** END **********************************************************************  -->
 </robot>
