Commit message: u

File: xacro/urdf_cart.xacro (robot description, xacro)
@@ -23,5 +23,5 @@
     <visual>
       <geometry>
-        <box size="0.5 0.5 0.2"/>
+        <mesh filename="${mesh_path}cart.stl" scale="1 1 1"/> <!-- <box size="0.5 0.5 0.2"/> -->
       </geometry>
       <origin xyz="0 0 0"/>
