Commit message: u

File: xacro/gripper.xacro (robot description, xacro)
@@ -1,116 +1,18 @@
-<?xml version="1.0" ?>
-<robot name="gripper"  xmlns:xacro="http://ros.org/wiki/xacro">
-<!-- ****************************************************** World Link *************************************************************** -->
-  <link name="world"/>
-<!-- ****************************************************** Base Link **************************************************************** -->
-  <link name="base">
-    <visual>
-      <geometry>
-        <box size="0.5 1 1"/>
-      </geometry>
-      <origin xyz="0 0 0.5"/>
-      <material name="violet">
-        <color rgba="0.4 0.18 0.57 1.0" />
-      </material>
-    </visual>
-    <inertial>
-      <mass value="50"/>
-      <inertia ixx="1.0" ixy="0.0" ixz="0.0" iyy="1.0" iyz="0.0" izz="1.0"/>
-    </inertial>
-  </link>
-  <gazebo reference="base">
-    <material>Gazebo/Orange</material>
-  </gazebo>
-<!-- ****************************************************** finger_right Link ******************************************************** -->
-  <link name="finger_right">
-    <visual>
-      <geometry>
-        <box size="0.4 0.1 1"/>
-      </geometry>
-      <origin xyz="0 0.05 0.5"/>
-      <material name="grey">
-        <color rgba="0.2 0.2 0.2 1"/>
-      </material>
-    </visual>
-    <inertial>
-      <mass value="5"/>
-      <inertia ixx="1.0" ixy="0.0" ixz="0.0" iyy="1.0" iyz="0.0" izz="1.0"/>
-    </inertial>
-  </link>
-  <gazebo reference="finger_right">
-    <material>Gazebo/Red</material>
-  </gazebo>
-<!-- ****************************************************** finger_left Link ********************************************************* -->
-  <link name="finger_left">
-    <visual>
-      <geometry>
-        <box size="0.4 0.1 1"/>
-      </geometry>
-      <origin xyz="0 0.05 0.5"/>
-      <material name="grey">
-        <color rgba="0.2 0.2 0.2 1"/>
-      </material>
-    </visual>
-    <inertial>
-      <mass value="5"/>
-      <inertia ixx="1.0" ixy="0.0" ixz="0.0" iyy="1.0" iyz="0.0" izz="1.0"/>
-    </inertial>
-  </link>
-  <gazebo reference="finger_left">
-    <material>Gazebo/Red</material>
-  </gazebo>
-<!-- ****************************************************** world to base Joint ****************************************************** -->
-  <joint name="world_to_base" type="fixed">
-    <origin rpy="0 0 0" xyz="0 0 0"/>
-    <parent link="world"/>
-    <child link="base"/>
-  </joint>
-<!-- ****************************************************** right_finger Joint ******************************************************* -->
-  <joint name="right_finger_joint" type="prismatic">
-    <axis xyz="0 1 0"/>
-    <origin xyz="0.0 -0.48 1" rpy="0.0 0.0 0.0"/>
-    <parent link="base"/>
-    <child link="finger_right"/>
-    <limit effort="1000.0" lower="0" upper="0.38" velocity="10"/>
-  </joint>
-<!-- ****************************************************** left_finger Joint ******************************************************** -->
-  <joint name="left_finger_joint" type="prismatic">
-    <mimic joint="right_finger_joint"/>
-    <axis xyz="0 1 0"/>
-    <origin xyz="0.0 0.48 1" rpy="0.0 0.0 3.1415926535"/>
-    <parent link="base"/>
-    <child link="finger_left"/>
-    <limit effort="1000.0" lower="0" upper="0.38" velocity="10"/>
-  </joint>
-<!-- ****************************************************** Gazebo ROS2 Control ****************************************************** -->
-  <ros2_control name="GazeboSystem" type="system">
-    <hardware>
-      <plugin>gazebo_ros2_control/GazeboSystem</plugin>
-    </hardware>
-    <joint name="right_finger_joint">
-      <command_interface name="position"/>
-      <state_interface name="position">
-        <param name="initial_value">0.15</param>
-      </state_interface>
-      <state_interface name="velocity"/>
-      <state_interface name="effort"/>
-    </joint>
-    <joint name="left_finger_joint">
-      <param name="mimic">right_finger_joint</param>
-      <param name="multiplier">1</param>
-      <command_interface name="position"/>
-      <state_interface name="position"/>
-      <state_interface name="velocity"/>
-      <state_interface name="effort"/>
-    </joint>
-  </ros2_control>
-<!-- ****************************************************** Gazebo ROS2 Plugin ******************************************************* -->
-  <gazebo>
-    <plugin filename="libgazebo_ros2_control.so" name="gazebo_ros2_control">
-      <robot_param>robot_description</robot_param>
-      <robot_param_node>robot_state_publisher</robot_param_node>
-      <parameters>$(find bots)/config/gripper.yaml</parameters>
-    </plugin>
-  </gazebo>
-<!-- ****************************************************** End ********************************************************************** -->
+<?xml version="1.0"?>
+<robot name="gripper" xmlns:xacro="http://www.ros.org/wiki/xacro">
+<!-- ****************************************************** Gripper Robot ************************************************************  -->
+<!-- Muthanna Alwahash                                                                                                                  -->
+<!-- March 2022                                                                                                                         -->
+<!-- *********************************************************************************************************************************  -->
+<!-- ****************************************************** Parameters ***************************************************************  -->
+    <xacro:property name="pkg_path"     value="$(find bots)"                />
+    <xacro:property name="mesh_path"    value="${pkg_path}/meshes/gripper/"    />
+    <xacro:property name="name_space"   value="cart" />
+    <xacro:property name="prefix"       value=""      />
+<!-- ****************************************************** Includes *****************************************************************  -->
+    <xacro:include filename="${pkg_path}/xacro/common_rviz_materials.xacro" />  <!--  RVIZ Colors  -->
+    <xacro:include filename="${pkg_path}/xacro/urdf_gripper.xacro" />           <!--  Robot URDF   -->
+    <xacro:include filename="${pkg_path}/gazebo/gz_gripper.xacro" />            <!--  Gazebo Sim   -->
+    <xacro:include filename="${pkg_path}/r2c/r2c_gripper.xacro" />              <!--  ROS2_Control -->
+<!-- ****************************************************** END **********************************************************************  -->
 </robot>
