Commit message: u

File: xacro/cart.xacro (robot description, xacro)
@@ -56,27 +56,4 @@
     <dynamics damping="0.0" friction="0.0"/>
   </joint>
-<!-- ****************************************************** Gazebo ROS2 Control ****************************************************** -->
-  <ros2_control name="GazeboSystem" type="system">
-    <hardware>
-      <plugin>gazebo_ros2_control/GazeboSystem</plugin>
-    </hardware>
-    <joint name="slider_to_cart">
-      <command_interface name="position">
-        <param name="min">-15</param>
-        <param name="max">15</param>
-      </command_interface>
-      <state_interface name="position">
-        <param name="initial_value">1.0</param>
-      </state_interface>
-      <state_interface name="velocity"/>
-      <state_interface name="effort"/>
-    </joint>
-  </ros2_control>
-<!-- ****************************************************** Gazebo ROS2 Plugin ******************************************************* -->
-  <gazebo>
-    <plugin filename="libgazebo_ros2_control.so" name="gazebo_ros2_control">
-      <parameters>$(find cart)/config/cartpole_controller.yaml</parameters>
-    </plugin>
-  </gazebo>
 <!-- ****************************************************** End ********************************************************************** -->
 </robot>

File: xacro/cart_effort.xacro (robot description, xacro)
@@ -1,4 +1,4 @@
 <?xml version="1.0" ?>
-<robot name="cartopole" xmlns:xacro="http://ros.org/wiki/xacro">
+<robot name="cart" xmlns:xacro="http://ros.org/wiki/xacro">
 <!-- ****************************************************** World Link *************************************************************** -->
   <link name="world"/>

File: xacro/cart_velocity.xacro (robot description, xacro)
@@ -1,4 +1,4 @@
 <?xml version="1.0" ?>
-<robot name="cartopole" xmlns:xacro="http://ros.org/wiki/xacro">
+<robot name="cart" xmlns:xacro="http://ros.org/wiki/xacro">
 <!-- ****************************************************** World Link *************************************************************** -->
   <link name="world"/>

Commit message: u

File: xacro/cart.xacro (robot description, xacro)
@@ -1,53 +1,16 @@
-<?xml version="1.0" ?>
-<robot name="cart" xmlns:xacro="http://ros.org/wiki/xacro">
-<!-- ****************************************************** World Link *************************************************************** -->
-  <link name="world"/>
-<!-- ****************************************************** slideBar Link ************************************************************ -->
-  <link name="slideBar">
-    <visual>
-      <geometry>
-        <box size="30 0.05 0.05"/>
-      </geometry>
-      <origin xyz="0 0 0"/>
-      <material name="green">
-        <color rgba="0 0.8 .8 1"/>
-      </material>
-    </visual>
-    <inertial>
-      <mass value="100"/>
-      <inertia ixx="1.0" ixy="0.0" ixz="0.0" iyy="1.0" iyz="0.0" izz="1.0"/>
-    </inertial>
-  </link>
-<!-- ****************************************************** cart Link **************************************************************** -->
-  <link name="cart">
-    <visual>
-      <geometry>
-        <box size="0.5 0.5 0.2"/>
-      </geometry>
-      <origin xyz="0 0 0"/>
-      <material name="blue">
-        <color rgba="0 0 .8 1"/>
-      </material>
-    </visual>
-    <inertial>
-      <mass value="1"/>
-      <inertia ixx="1.0" ixy="0.0" ixz="0.0" iyy="1.0" iyz="0.0" izz="1.0"/>
-    </inertial>
-  </link>
-<!-- ****************************************************** world to slideBar Joint ************************************************** -->
-  <joint name="world_to_base" type="fixed">
-    <origin rpy="0 0 0" xyz="0 0 1"/>
-    <parent link="world"/>
-    <child link="slideBar"/>
-  </joint>
-<!-- ****************************************************** slideBar to cart Joint *************************************************** -->
-  <joint name="slider_to_cart" type="prismatic">
-    <axis xyz="1 0 0"/>
-    <origin xyz="0.0 0.0 0.0"/>
-    <parent link="slideBar"/>
-    <child link="cart"/>
-    <limit effort="1000.0" lower="-15" upper="15" velocity="30"/>
-    <dynamics damping="0.0" friction="0.0"/>
-  </joint>
-<!-- ****************************************************** End ********************************************************************** -->
+<?xml version="1.0"?>
+<robot name="cart" xmlns:xacro="http://www.ros.org/wiki/xacro">
+<!-- ****************************************************** Cart Robot ***************************************************************  -->
+<!-- Muthanna Alwahash                                                                                                                  -->
+<!-- March 2022                                                                                                                         -->
+<!-- *********************************************************************************************************************************  -->
+<!-- ****************************************************** Parameters ***************************************************************  -->
+    <xacro:property name="pkg_path"     value="$(find bots)"                />
+    <xacro:property name="mesh_path"    value="${pkg_path}/meshes/cart/"    />
+    <xacro:property name="name_space"   value="cart" />
+    <xacro:property name="prefix"       value=""      />
+<!-- ****************************************************** Includes *****************************************************************  -->
+    <xacro:include filename="${pkg_path}/xacro/common_rviz_materials.xacro" />  <!--  RVIZ Colors  -->
+    <xacro:include filename="${pkg_path}/xacro/urdf_cart.xacro" />              <!--  Robot URDF   -->
+<!-- ****************************************************** END **********************************************************************  -->
 </robot>
