Commit message: u

File: xacro/diffbot.xacro (robot description, xacro)
@@ -1,17 +1,16 @@
 <?xml version="1.0"?>
-<robot xmlns:xacro="http://www.ros.org/wiki/xacro">
+<robot name="diffbot" xmlns:xacro="http://www.ros.org/wiki/xacro">
   <xacro:macro name="diffbot" params="prefix">
   <!-- Constants for robot dimensions -->
-  <xacro:property name="PI" value="3.1415926535897931"/>
-  <xacro:property name="base_mass" value="0.3" /> <!-- arbitrary value for base mass -->
-  <xacro:property name="base_width" value="0.1" />
-  <xacro:property name="base_length" value="0.1" />
-  <xacro:property name="base_height" value="0.05" />
-  <xacro:property name="wheel_mass" value="0.3" /> <!-- arbitrary value for wheel mass -->
-  <xacro:property name="wheel_len" value="0.020" />
-  <xacro:property name="wheel_radius" value="0.015" />
-  <xacro:property name="caster_wheel_mass" value="0.1" /> <!-- arbitrary value for caster wheel mass -->
-  <xacro:property name="caster_wheel_radius" value="0.015" />
-  <xacro:property name="z_offset" value="-${base_height/2}" /> <!-- Space btw top of beam and the each joint -->
+  <xacro:property name="base_mass"            value="0.3"               /> <!-- arbitrary value for base mass             -->
+  <xacro:property name="base_width"           value="0.1"               />
+  <xacro:property name="base_length"          value="0.1"               />
+  <xacro:property name="base_height"          value="0.05"              />
+  <xacro:property name="wheel_mass"           value="0.3"               /> <!-- arbitrary value for wheel mass            -->
+  <xacro:property name="wheel_len"            value="0.020"             />
+  <xacro:property name="wheel_radius"         value="0.015"             />
+  <xacro:property name="caster_wheel_mass"    value="0.1"               /> <!-- arbitrary value for caster wheel mass     -->
+  <xacro:property name="caster_wheel_radius"  value="0.015"             />
+  <xacro:property name="z_offset"             value="-${base_height/2}" /> <!-- Space btw top of beam and the each joint  -->
   <!-- Base Link -->
   <link name="${prefix}base_link">
@@ -36,6 +35,6 @@
         iyy="${base_mass / 12.0 * (base_height*base_height + base_width*base_width)}" iyz="0.0"
         izz="${base_mass / 12.0 * (base_width*base_width + base_length*base_length)}"/>
-      </inertial>
-    </link>
+    </inertial>
+  </link>
     <joint name="${prefix}left_wheel_joint" type="continuous">
       <parent link="${prefix}base_link"/>
@@ -48,5 +47,5 @@
     <link name="${prefix}left_wheel">
       <collision>
-        <origin xyz="0 0 0" rpy="${PI/2} 0 0"/>
+        <origin xyz="0 0 0" rpy="${pi/2} 0 0"/>
         <geometry>
           <cylinder length="${wheel_len}" radius="${wheel_radius}"/>
@@ -54,5 +53,5 @@
       </collision>
       <visual>
-        <origin xyz="0 0 0" rpy="${PI/2} 0 0"/>
+        <origin xyz="0 0 0" rpy="${pi/2} 0 0"/>
         <geometry>
           <cylinder length="${wheel_len}" radius="${wheel_radius}"/>
@@ -61,5 +60,5 @@
       </visual>
       <inertial>
-        <origin xyz="0 0 0" rpy="${PI/2} 0 0"/>
+        <origin xyz="0 0 0" rpy="${pi/2} 0 0"/>
         <mass value="${wheel_mass}"/>
         <inertia
@@ -67,6 +66,6 @@
           iyy="${wheel_mass / 12.0 * wheel_radius*wheel_radius}" iyz="0.0"
           izz="${wheel_mass / 12.0 * wheel_radius*wheel_radius}"/>
-        </inertial>
-      </link>
+      </inertial>
+    </link>
     <joint name="${prefix}right_wheel_joint" type="continuous">
       <parent link="${prefix}base_link"/>
@@ -79,5 +78,5 @@
     <link name="${prefix}right_wheel">
       <collision>
-        <origin xyz="0 0 0" rpy="${PI/2} 0 0"/>
+        <origin xyz="0 0 0" rpy="${pi/2} 0 0"/>
         <geometry>
           <cylinder length="${wheel_len}" radius="${wheel_radius}"/>
@@ -85,5 +84,5 @@
       </collision>
       <visual>
-        <origin xyz="0 0 0" rpy="${PI/2} 0 0"/>
+        <origin xyz="0 0 0" rpy="${pi/2} 0 0"/>
         <geometry>
           <cylinder length="${wheel_len}" radius="${wheel_radius}"/>
@@ -92,5 +91,5 @@
       </visual>
       <inertial>
-        <origin xyz="0 0 0" rpy="${PI/2} 0 0"/>
+        <origin xyz="0 0 0" rpy="${pi/2} 0 0"/>
         <mass value="${wheel_mass}"/>
         <inertia
@@ -98,6 +97,6 @@
           iyy="${wheel_mass / 12.0 * wheel_radius*wheel_radius}" iyz="0.0"
           izz="${wheel_mass / 12.0 * wheel_radius*wheel_radius}"/>
-        </inertial>
-      </link>
+      </inertial>
+    </link>
     <joint name="${prefix}caster_frontal_wheel_joint" type="fixed">
       <parent link="${prefix}base_link"/>
@@ -127,6 +126,6 @@
           iyy="${caster_wheel_mass * 0.4 * (caster_wheel_radius * caster_wheel_radius)}" iyz="0.0"
           izz="${caster_wheel_mass * 0.4 * (caster_wheel_radius * caster_wheel_radius)}"/>
-        </inertial>
-      </link>
+      </inertial>
+    </link>
     <joint name="${prefix}caster_rear_wheel_joint" type="fixed">
       <parent link="${prefix}base_link"/>
@@ -156,6 +155,6 @@
           iyy="${caster_wheel_mass * 0.4 * (caster_wheel_radius * caster_wheel_radius)}" iyz="0.0"
           izz="${caster_wheel_mass * 0.4 * (caster_wheel_radius * caster_wheel_radius)}"/>
-        </inertial>
-      </link>
+      </inertial>
+    </link>
   </xacro:macro>
 </robot>

Commit message: u

File: xacro/diffbot.xacro (robot description, xacro)
@@ -1,6 +1,9 @@
 <?xml version="1.0"?>
 <robot name="diffbot" xmlns:xacro="http://www.ros.org/wiki/xacro">
-  <xacro:macro name="diffbot" params="prefix">
-  <!-- Constants for robot dimensions -->
+<!-- ****************************************************** RRBot Robot **************************************************************  -->
+<!-- Muthanna Alwahash                                                                                                                  -->
+<!-- March 2022                                                                                                                         -->
+<!-- *********************************************************************************************************************************  -->
+<!-- ****************************************************** Parameters ***************************************************************  -->
   <xacro:property name="base_mass"            value="0.3"               /> <!-- arbitrary value for base mass             -->
   <xacro:property name="base_width"           value="0.1"               />
@@ -13,5 +16,9 @@
   <xacro:property name="caster_wheel_radius"  value="0.015"             />
   <xacro:property name="z_offset"             value="-${base_height/2}" /> <!-- Space btw top of beam and the each joint  -->
-  <!-- Base Link -->
+<!-- ****************************************************** Import RVIZ Materials*****************************************************  -->
+  <xacro:include filename="$(find robot_gazebo)/xacro/common_rviz_materials.xacro" />
+<!-- ****************************************************** Macro ********************************************************************  -->
+  <xacro:macro name="diffbot" params="prefix">
+<!-- ****************************************************** Base Link ****************************************************************  -->
   <link name="${prefix}base_link">
     <collision>
@@ -37,4 +44,5 @@
     </inertial>
   </link>
+<!-- ****************************************************** Left Wheel Joint *********************************************************  -->
     <joint name="${prefix}left_wheel_joint" type="continuous">
       <parent link="${prefix}base_link"/>
@@ -44,5 +52,5 @@
       <dynamics damping="0.2"/>
     </joint>
-    <!-- left wheel Link -->
+<!-- ****************************************************** Left Wheel Link **********************************************************  -->
     <link name="${prefix}left_wheel">
       <collision>
@@ -68,4 +76,5 @@
       </inertial>
     </link>
+<!-- ****************************************************** Right Wheel Joint ********************************************************  -->
     <joint name="${prefix}right_wheel_joint" type="continuous">
       <parent link="${prefix}base_link"/>
@@ -75,5 +84,5 @@
       <dynamics damping="0.2"/>
     </joint>
-    <!-- right wheel Link -->
+<!-- ****************************************************** Right Wheel Link ********************************************************  -->
     <link name="${prefix}right_wheel">
       <collision>
@@ -99,4 +108,5 @@
       </inertial>
     </link>
+<!-- ****************************************************** Right Wheel Link ********************************************************  -->
     <joint name="${prefix}caster_frontal_wheel_joint" type="fixed">
       <parent link="${prefix}base_link"/>
@@ -104,5 +114,5 @@
       <origin xyz="${base_width/2 - caster_wheel_radius} 0 ${z_offset}" rpy="0 0 0"/>
     </joint>
-    <!-- caster frontal wheel Link -->
+<!-- ****************************************************** Right Wheel Link ********************************************************  -->
     <link name="${prefix}caster_frontal_wheel">
       <collision>
@@ -128,4 +138,5 @@
       </inertial>
     </link>
+<!-- ****************************************************** Right Wheel Link ********************************************************  -->
     <joint name="${prefix}caster_rear_wheel_joint" type="fixed">
       <parent link="${prefix}base_link"/>
@@ -133,5 +144,5 @@
       <origin xyz="${-base_width/2 + caster_wheel_radius} 0 ${z_offset}" rpy="0 0 0"/>
     </joint>
-    <!-- caster rear wheel Link -->
+<!-- ****************************************************** Right Wheel Link ********************************************************  -->
     <link name="${prefix}caster_rear_wheel">
       <collision>
@@ -157,4 +168,8 @@
       </inertial>
     </link>
+<!-- ****************************************************** End Macro ****************************************************************  -->
   </xacro:macro>
+<!-- ****************************************************** Expand Macro *************************************************************  -->
+  <xacro:diffbot prefix="" />
+<!-- ****************************************************** END **********************************************************************  -->
 </robot>

File: xacro/rrbot.xacro (robot description, xacro)
@@ -195,4 +195,4 @@
 <!-- ****************************************************** Expand Macro *************************************************************  -->
   <xacro:rrbot parent="world" prefix="" />
-<!-- ****************************************************** Expand Macro *************************************************************  -->
+<!-- ****************************************************** END **********************************************************************  -->
 </robot>

Commit message: u

File: xacro/diffbot.xacro (robot description, xacro)
@@ -38,5 +38,5 @@
     </collision>
     <visual>
-      <origin xyz="0 0 ${base_height/2}" rpy="0 0 0"/>
+      <origin xyz="0 0 0" rpy="0 0 0"/>
       <geometry>
         <box size="${base_width} ${base_length} ${base_height}"/>

Commit message: u

File: xacro/diffbot.xacro (robot description, xacro)
@@ -36,5 +36,5 @@
       <origin xyz="0 0 0" rpy="0 0 0"/>
       <geometry>
-        <mesh filename="${mesh_path}base.dae" scale="1 1 1"/>  <!--  <box size="${base_length} ${base_width} ${base_height}"/> -->
+        <mesh filename="${mesh_path}base.stl" scale="1 1 1"/>  <!--  <box size="${base_length} ${base_width} ${base_height}"/> -->
       </geometry>
     </collision>
@@ -42,5 +42,5 @@
       <origin xyz="0 0 0" rpy="0 0 0"/>
       <geometry>
-        <mesh filename="${mesh_path}base.dae" scale="1 1 1"/>  <!--  <box size="${base_length} ${base_width} ${base_height}"/> -->
+        <mesh filename="${mesh_path}base.stl" scale="1 1 1"/>  <!--  <box size="${base_length} ${base_width} ${base_height}"/> -->
       </geometry>
       <material name="orange"/>

Commit message: u

File: xacro/diffbot.xacro (robot description, xacro)
@@ -59,15 +59,15 @@
     </inertial>
   </link>
-<!-- ****************************************************** Left Wheel Joint *********************************************************  -->
-    <joint name="${prefix}left_wheel_joint" type="continuous">
+<!-- ****************************************************** Right Wheel Joint ********************************************************  -->
+    <joint name="${prefix}right_wheel_joint" type="continuous">
       <parent link="${prefix}base_link"/>
-      <child link="${prefix}left_wheel"/>
-      <origin xyz="0 -${wheel_y} -${wheel_z}" rpy="0 0 0"/>
+      <child link="${prefix}right_wheel"/>
+      <origin xyz="0 ${wheel_y} -${wheel_z}" rpy="0 0 0"/>
       <limit upper="${radians(180)}" lower="-${radians(180)}" effort="30" velocity="5.0"/>
       <axis xyz="0 1 0"/>
       <dynamics damping="0.2"/>
     </joint>
-<!-- ****************************************************** Left Wheel Link **********************************************************  -->
-    <link name="${prefix}left_wheel">
+<!-- ****************************************************** Right Wheel Link ********************************************************  -->
+    <link name="${prefix}right_wheel">
       <collision>
         <origin xyz="0 0 0" rpy="${radians(90)} 0 0"/>
@@ -92,15 +92,15 @@
       </inertial>
     </link>
-<!-- ****************************************************** Right Wheel Joint ********************************************************  -->
-    <joint name="${prefix}right_wheel_joint" type="continuous">
+<!-- ****************************************************** Left Wheel Joint *********************************************************  -->
+    <joint name="${prefix}left_wheel_joint" type="continuous">
       <parent link="${prefix}base_link"/>
-      <child link="${prefix}right_wheel"/>
-      <origin xyz="0 ${wheel_y} -${wheel_z}" rpy="0 0 0"/>
+      <child link="${prefix}left_wheel"/>
+      <origin xyz="0 -${wheel_y} -${wheel_z}" rpy="0 0 0"/>
       <limit upper="${radians(180)}" lower="-${radians(180)}" effort="30" velocity="5.0"/>
       <axis xyz="0 1 0"/>
       <dynamics damping="0.2"/>
     </joint>
-<!-- ****************************************************** Right Wheel Link ********************************************************  -->
-    <link name="${prefix}right_wheel">
+<!-- ****************************************************** Left Wheel Link **********************************************************  -->
+    <link name="${prefix}left_wheel">
       <collision>
         <origin xyz="0 0 0" rpy="${radians(90)} 0 0"/>

Commit message: u

File: xacro/diffbot.xacro (robot description, xacro)
@@ -22,4 +22,10 @@
   <xacro:property name="caster_x"       value="${(base_length/2 - caster_radius)*0.95}" />
   <xacro:property name="caster_z"       value="${base_height/2}"/>
+  <xacro:property name="hokuyo_mass"    value="1e-5"     />
+  <xacro:property name="hokuyo_width"   value="0.05"     />
+  <xacro:property name="hokuyo_length"  value="0.05"     />
+  <xacro:property name="hokuyo_height"  value="0.0706"   />
+  <xacro:property name="hokuyo_x"       value="0.11"     /> <!-- x offset from base center -->
+  <xacro:property name="hokuyo_z"       value="${(hokuyo_height+base_height)/2}" />
 <!-- ****************************************************** Includes *****************************************************************  -->
   <xacro:include filename="$(find robot_gazebo)/xacro/common_rviz_materials.xacro" />   <!-- RVIZ Colors                                -->
@@ -185,4 +191,32 @@
       </inertial>
     </link>
+<!-- ****************************************************** Hokuyo Link **************************************************************  -->
+  <link name="${prefix}hokuyo">
+    <inertial>
+      <mass value="${hokuyo_mass}"/>
+      <origin xyz="0 0 0" rpy=" 0 0 0"/>
+      <inertia ixx="1e-6" ixy="0" ixz="0" iyy="1e-6" iyz="0" izz="1e-6" />
+    </inertial>
+    <visual name="hokuyo_visual">
+      <origin xyz="0 0 0" rpy="0 0 0" />
+      <geometry>
+        <mesh filename="${mesh_path}hokuyo.dae"/> <!--  <box size="${hokuyo_length} ${hokuyo_width} ${hokuyo_height}"/> -->
+      </geometry>
+      <!-- <material name="red"/> -->
+    </visual>
+    <collision name="hokuyo_colision">
+      <origin xyz="0 0 0" rpy="0 0 0" />
+      <geometry>
+        <mesh filename="${mesh_path}hokuyo.dae"/> <!--  <box size="${hokuyo_length} ${hokuyo_width} ${hokuyo_height}"/> -->
+      </geometry>
+    </collision>
+  </link>
+<!-- ****************************************************** Hokuyo Joint *************************************************************  -->
+  <joint type="fixed" name="${prefix}hokuyo_joint">
+    <origin xyz="${hokuyo_x} 0 ${hokuyo_z}" rpy="0 0 0"/>
+    <child link="${prefix}hokuyo"/>
+    <parent link="${prefix}base"/>
+    <axis xyz="0 1 0" rpy="0 0 0"/>
+  </joint>
 <!-- ****************************************************** End Macro ****************************************************************  -->
   </xacro:macro>

Commit message: u

File: xacro/diffbot.xacro (robot description, xacro)
@@ -194,4 +194,15 @@
     <axis xyz="0 1 0" rpy="0 0 0"/>
   </joint>
+<!-- ****************************************************** Camera Optical Joint *****************************************************  -->
+<!-- generate an optical frame http://www.ros.org/reps/rep-0103.html#suffix-frames so that ros and opencv can operate on the camera     -->
+<!-- frame correctly. these values have to be these values otherwise the gazebo camera image won't be aligned properly with the frame   -->
+<!-- it is supposedly originating from                                                                                                  -->                                                                                                                   -->
+  <joint name="${prefix}camera_optical_joint" type="fixed">
+    <origin xyz="0 0 0" rpy="${-radians(90)} 0 ${-radians(90)}"/>
+    <parent link="${prefix}camera"/>
+    <child link="${prefix}camera_optical"/>
+  </joint>
+<!-- ****************************************************** Camera Optical Link ******************************************************  -->
+  <link name="${prefix}camera_optical"/>
 <!-- ****************************************************** Hokuyo Link **************************************************************  -->
   <link name="${prefix}hokuyo">

Commit message: u

File: xacro/diffbot.xacro (robot description, xacro)
@@ -6,5 +6,5 @@
 <!-- *********************************************************************************************************************************  -->
 <!-- ****************************************************** Parameters ***************************************************************  -->
-  <xacro:property name="mesh_path"      value="package://diffbot/meshes/diffbot/"/>
+  <xacro:property name="mesh_path"      value="package://bots/meshes/diffbot/"/>
   <xacro:property name="name_space"     value="diffbot"  />
   <xacro:property name="prefix"         value=""  />
@@ -36,6 +36,6 @@
   <xacro:property name="hokuyo_z"       value="${(hokuyo_height+base_height)/2}" />
 <!-- ****************************************************** Includes *****************************************************************  -->
-  <xacro:include filename="$(find diffbot)/xacro/common_rviz_materials.xacro" />   <!-- RVIZ Colors                                -->
-  <xacro:include filename="$(find diffbot)/gazebo/gz_diffbot.xacro" />             <!-- Gazebo                                     -->
+  <xacro:include filename="$(find bots)/xacro/common_rviz_materials.xacro" />   <!-- RVIZ Colors                                -->
+  <xacro:include filename="$(find bots)/gazebo/gz_diffbot.xacro" />             <!-- Gazebo                                     -->
 <!-- ****************************************************** Footprint ****************************************************************  -->
     <link name="${prefix}footprint"/>
