Commit message: u

File: xacro/diffbot.xacro (robot description, xacro)
@@ -1,236 +1,19 @@
 <?xml version="1.0"?>
 <robot name="diffbot" xmlns:xacro="http://www.ros.org/wiki/xacro">
-<!-- ****************************************************** diffbot Robot ************************************************************  -->
+<!-- ****************************************************** Diffbot Robot ***************************************************************  -->
 <!-- Muthanna Alwahash                                                                                                                  -->
 <!-- March 2022                                                                                                                         -->
 <!-- *********************************************************************************************************************************  -->
 <!-- ****************************************************** Parameters ***************************************************************  -->
-  <xacro:property name="mesh_path"      value="package://bots/meshes/diffbot/"/>
-  <xacro:property name="name_space"     value="diffbot"  />
-  <xacro:property name="prefix"         value=""  />
-  <xacro:property name="base_mass"      value="0.6"                               />  <!-- arbitrary value for base mass                -->
-  <xacro:property name="base_width"     value="0.20"                              />
-  <xacro:property name="base_length"    value="0.40"                              />
-  <xacro:property name="base_height"    value="0.10"                              />
-  <xacro:property name="wheel_mass"     value="5.0"                               />
-  <xacro:property name="wheel_width"    value="0.05"                              />
-  <xacro:property name="wheel_radius"   value="0.08"                              />
-  <xacro:property name="wheel_gap"      value="0.01"                              /> <!-- Gap between wheels and base                   -->
-  <xacro:property name="wheel_x"        value="0.12"                              /> <!-- x offset from base center -->
-  <xacro:property name="wheel_y"        value="${(base_width+wheel_width)/2+wheel_gap}" />
-  <xacro:property name="wheel_z"        value="${base_height/4}"                  />  <!-- Space btw top of beam and the each joint     -->
-  <xacro:property name="caster_mass"    value="0.1"                               />  <!-- arbitrary value for caster wheel mass        -->
-  <xacro:property name="caster_radius"  value="${wheel_radius-wheel_z}"           />
-  <xacro:property name="caster_x"       value="${(base_length/2 - caster_radius)}" />
-  <xacro:property name="caster_z"       value="${base_height/2}"/>
-  <xacro:property name="camera_mass"    value="0.1"      />
-  <xacro:property name="camera_width"   value="0.05"     />
-  <xacro:property name="camera_length"  value="0.05"     />
-  <xacro:property name="camera_height"  value="0.05"     />
-  <xacro:property name="camera_x"       value="0.2"      /> <!-- x offset from base center -->
-  <xacro:property name="hokuyo_mass"    value="1e-5"     />
-  <xacro:property name="hokuyo_width"   value="0.05"     />
-  <xacro:property name="hokuyo_length"  value="0.05"     />
-  <xacro:property name="hokuyo_height"  value="0.0706"   />
-  <xacro:property name="hokuyo_x"       value="0.11"     /> <!-- x offset from base center -->
-  <xacro:property name="hokuyo_z"       value="${(hokuyo_height+base_height)/2}" />
+    <xacro:property name="pkg_path"     value="$(find bots)"                />
+    <xacro:property name="mesh_path"    value="${pkg_path}/meshes/diffbot/"    />
+    <xacro:property name="config_path"  value="${pkg_path}/config/"         />
+    <xacro:property name="name_space"   value="diffbot" />
+    <xacro:property name="prefix"       value=""      />
 <!-- ****************************************************** Includes *****************************************************************  -->
-  <xacro:include filename="$(find bots)/xacro/common_rviz_materials.xacro" />   <!-- RVIZ Colors                                -->
-  <xacro:include filename="$(find bots)/gazebo/gz_diffbot.xacro" />             <!-- Gazebo                                     -->
-<!-- ****************************************************** Footprint ****************************************************************  -->
-    <link name="${prefix}footprint"/>
-<!-- ****************************************************** Base Joint ***************************************************************  -->
-    <joint name="footprint_joint" type="fixed">
-        <parent link="footprint"/>
-        <child link="${prefix}base"/>
-        <origin xyz="0.0 0.0 ${(wheel_radius+wheel_z)}" rpy="0.0 0.0 0.0"/>
-    </joint>
-<!-- ****************************************************** Base Link ****************************************************************  -->
-  <link name="${prefix}base">
-    <collision>
-      <origin xyz="0 0 0" rpy="0 0 0"/>
-      <geometry>
-        <mesh filename="${mesh_path}base.stl" scale="1 1 1"/>  <!--  <box size="${base_length} ${base_width} ${base_height}"/> -->
-      </geometry>
-    </collision>
-    <visual>
-      <origin xyz="0 0 0" rpy="0 0 0"/>
-      <geometry>
-        <mesh filename="${mesh_path}base.stl" scale="1 1 1"/>  <!--  <box size="${base_length} ${base_width} ${base_height}"/> -->
-      </geometry>
-      <material name="blue"/>
-    </visual>
-    <inertial>
-      <origin xyz="0 0 0" rpy="0 0 0"/>
-      <mass value="${base_mass}"/>
-      <inertia
-        ixx="${base_mass / 12.0 * (base_length*base_length + base_height*base_height)}" ixy="0.0" ixz="0.0"
-        iyy="${base_mass / 12.0 * (base_height*base_height + base_width*base_width)}" iyz="0.0"
-        izz="${base_mass / 12.0 * (base_width*base_width + base_length*base_length)}"/>
-    </inertial>
-  </link>
-<!-- ****************************************************** Right Wheel Joint ********************************************************  -->
-    <joint name="${prefix}right_wheel_joint" type="continuous">
-      <parent link="${prefix}base"/>
-      <child link="${prefix}right_wheel"/>
-      <origin xyz="-${wheel_x} ${wheel_y} -${wheel_z}" rpy="0 0 0"/>
-      <limit upper="${radians(180)}" lower="-${radians(180)}" effort="30" velocity="5.0"/>
-      <axis xyz="0 1 0"/>
-      <dynamics damping="0.2"/>
-    </joint>
-<!-- ****************************************************** Right Wheel Link ********************************************************  -->
-    <link name="${prefix}right_wheel">
-      <collision>
-        <origin xyz="0 0 0" rpy="${radians(90)} 0 0"/>
-        <geometry>
-          <mesh filename="${mesh_path}wheel.dae" scale="1 1 1"/> <!-- <cylinder length="${wheel_width}" radius="${wheel_radius}"/> -->
-        </geometry>
-      </collision>
-      <visual>
-        <origin xyz="0 0 0" rpy="${radians(90)} 0 0"/>
-        <geometry>
-          <mesh filename="${mesh_path}wheel.dae" scale="1 1 1"/> <!-- <cylinder length="${wheel_width}" radius="${wheel_radius}"/> -->
-        </geometry>
-        <material name="black"/>
-      </visual>
-      <inertial>
-        <origin xyz="0 0 0" rpy="${radians(90)} 0 0"/>
-        <mass value="${wheel_mass}"/>
-        <inertia
-          ixx="${wheel_mass / 12.0 * (3*wheel_radius + wheel_width*wheel_width)}" ixy="0.0" ixz="0.0"
-          iyy="${wheel_mass / 12.0 * wheel_radius*wheel_radius}" iyz="0.0"
-          izz="${wheel_mass / 12.0 * wheel_radius*wheel_radius}"/>
-      </inertial>
-    </link>
-<!-- ****************************************************** Left Wheel Joint *********************************************************  -->
-    <joint name="${prefix}left_wheel_joint" type="continuous">
-      <parent link="${prefix}base"/>
-      <child link="${prefix}left_wheel"/>
-      <origin xyz="-${wheel_x} -${wheel_y} -${wheel_z}" rpy="0 0 0"/>
-      <limit upper="${radians(180)}" lower="-${radians(180)}" effort="30" velocity="5.0"/>
-      <axis xyz="0 1 0"/>
-      <dynamics damping="0.2"/>
-    </joint>
-<!-- ****************************************************** Left Wheel Link **********************************************************  -->
-    <link name="${prefix}left_wheel">
-      <collision>
-        <origin xyz="0 0 0" rpy="${radians(90)} 0 0"/>
-        <geometry>
-          <mesh filename="${mesh_path}wheel.dae" scale="1 1 1"/> <!-- <cylinder length="${wheel_width}" radius="${wheel_radius}"/> -->
-        </geometry>
-      </collision>
-      <visual>
-        <origin xyz="0 0 0" rpy="${radians(90)} 0 0"/>
-        <geometry>
-          <mesh filename="${mesh_path}wheel.dae" scale="1 1 1"/> <!-- <cylinder length="${wheel_width}" radius="${wheel_radius}"/> -->
-        </geometry>
-        <material name="black"/>
-      </visual>
-      <inertial>
-        <origin xyz="0 0 0" rpy="${radians(90)} 0 0"/>
-        <mass value="${wheel_mass}"/>
-        <inertia
-          ixx="${wheel_mass / 12.0 * (3*wheel_radius + wheel_width*wheel_width)}" ixy="0.0" ixz="0.0"
-          iyy="${wheel_mass / 12.0 * wheel_radius*wheel_radius}" iyz="0.0"
-          izz="${wheel_mass / 12.0 * wheel_radius*wheel_radius}"/>
-      </inertial>
-    </link>
-<!-- ****************************************************** Front caster joint *******************************************************  -->
-    <joint name="${prefix}front_caster_joint" type="fixed">
-      <parent link="${prefix}base"/>
-      <child link="${prefix}front_caster"/>
-      <origin xyz="${caster_x} 0 ${-caster_z}" rpy="0 0 0"/>
-    </joint>
-<!-- ****************************************************** Front caster Link ********************************************************  -->
-    <link name="${prefix}front_caster">
-      <collision>
-        <origin xyz="0 0 0" rpy="0 0 0"/>
-        <geometry>
-          <sphere radius="${caster_radius}"/>
-        </geometry>
-      </collision>
-      <visual>
-        <origin xyz="0 0 0" rpy="0 0 0"/>
-        <geometry>
-          <sphere radius="${caster_radius}"/>
-        </geometry>
-        <material name="white"/>
-      </visual>
-      <inertial>
-        <origin xyz="0 0 0" rpy="0 0 0"/>
-        <mass value="${caster_mass}"/>
-        <inertia
-          ixx="${caster_mass * 0.4 * (caster_radius * caster_radius)}" ixy="0.0" ixz="0.0"
-          iyy="${caster_mass * 0.4 * (caster_radius * caster_radius)}" iyz="0.0"
-          izz="${caster_mass * 0.4 * (caster_radius * caster_radius)}"/>
-      </inertial>
-    </link>
-<!-- ****************************************************** Camera Link **************************************************************  -->
-  <link name="${prefix}camera">
-    <inertial>
-      <mass value="${camera_mass}"/>
-      <origin xyz="0 0 0" rpy=" 0 0 0"/>
-      <inertia ixx="1e-6" ixy="0" ixz="0" iyy="1e-6" iyz="0" izz="1e-6" />
-    </inertial>
-    <visual name="camera_visual">
-      <origin xyz="0 0 0" rpy="0 0 0" />
-      <geometry>
-        <box size="${camera_length} ${camera_width} ${camera_height}"/>
-      </geometry>
-      <material name="green"/>
-    </visual>
-    <collision name="camera_colision">
-      <origin xyz="0 0 0" rpy="0 0 0" />
-      <geometry>
-        <box size="${camera_length} ${camera_width} ${camera_height}"/>
-      </geometry>
-    </collision>
-  </link>
-<!-- ****************************************************** Camera Joint *************************************************************  -->
-  <joint type="fixed" name="${prefix}camera_joint">
-    <origin xyz="${camera_x} 0 0" rpy="0 0 0"/>
-    <child link="${prefix}camera"/>
-    <parent link="${prefix}base"/>
-    <axis xyz="0 1 0" rpy="0 0 0"/>
-  </joint>
-<!-- ****************************************************** Camera Optical Joint *****************************************************  -->
-<!-- generate an optical frame http://www.ros.org/reps/rep-0103.html#suffix-frames so that ros and opencv can operate on the camera     -->
-<!-- frame correctly. these values have to be these values otherwise the gazebo camera image won't be aligned properly with the frame   -->
-<!-- it is supposedly originating from                                                                                                  -->                                                                                                                   -->
-  <joint name="${prefix}camera_optical_joint" type="fixed">
-    <origin xyz="0 0 0" rpy="${-radians(90)} 0 ${-radians(90)}"/>
-    <parent link="${prefix}camera"/>
-    <child link="${prefix}camera_optical"/>
-  </joint>
-<!-- ****************************************************** Camera Optical Link ******************************************************  -->
-  <link name="${prefix}camera_optical"/>
-<!-- ****************************************************** Hokuyo Link **************************************************************  -->
-  <link name="${prefix}hokuyo">
-    <inertial>
-      <mass value="${hokuyo_mass}"/>
-      <origin xyz="0 0 0" rpy=" 0 0 0"/>
-      <inertia ixx="1e-6" ixy="0" ixz="0" iyy="1e-6" iyz="0" izz="1e-6" />
-    </inertial>
-    <visual name="hokuyo_visual">
-      <origin xyz="0 0 0" rpy="0 0 0" />
-      <geometry>
-        <mesh filename="${mesh_path}hokuyo.dae"/> <!--  <box size="${hokuyo_length} ${hokuyo_width} ${hokuyo_height}"/> -->
-      </geometry>
-      <!-- <material name="red"/> -->
-    </visual>
-    <collision name="hokuyo_colision">
-      <origin xyz="0 0 0" rpy="0 0 0" />
-      <geometry>
-        <box size="${hokuyo_length} ${hokuyo_width} ${hokuyo_height}"/>
-      </geometry>
-    </collision>
-  </link>
-<!-- ****************************************************** Hokuyo Joint *************************************************************  -->
-  <joint type="fixed" name="${prefix}hokuyo_joint">
-    <origin xyz="${hokuyo_x} 0 ${hokuyo_z}" rpy="0 0 0"/>
-    <child link="${prefix}hokuyo"/>
-    <parent link="${prefix}base"/>
-    <axis xyz="0 1 0" rpy="0 0 0"/>
-  </joint>
+    <xacro:include filename="${pkg_path}/xacro/common_rviz_materials.xacro" />  <!--  RVIZ Colors  -->
+    <xacro:include filename="${pkg_path}/xacro/urdf_diffbot.xacro" />           <!--  Robot URDF   -->
+    <xacro:include filename="${pkg_path}/gazebo/gz_diffbot.xacro" />            <!--  Gazebo Sim   -->
+    <xacro:include filename="${pkg_path}/r2c/r2c_diffbot.xacro" />              <!--  ROS2_Control -->
 <!-- ****************************************************** END **********************************************************************  -->
 </robot>
