Commit message: u

File: xacro/skidbot.xacro (robot description, xacro)
@@ -14,6 +14,6 @@
   <xacro:property name="wheel_width"    value="0.05"     />
   <xacro:property name="wheel_radius"   value="0.08"     />
-  <xacro:property name="wheel_gap"      value="0.01"     />
-  <xacro:property name="wheel_x"        value="0.12"     />
+  <xacro:property name="wheel_gap"      value="0.01"     /> <!-- Gap between wheels and base         -->
+  <xacro:property name="wheel_x"        value="0.12"     /> <!-- x offset from base center -->
   <xacro:property name="wheel_y"        value="${(base_width+wheel_width)/2+wheel_gap}" />
   <xacro:property name="camera_mass"    value="0.1"      />
@@ -21,10 +21,10 @@
   <xacro:property name="camera_length"  value="0.05"     />
   <xacro:property name="camera_height"  value="0.05"     />
-  <xacro:property name="camera_x"       value="0.2"      />
+  <xacro:property name="camera_x"       value="0.2"      /> <!-- x offset from base center -->
   <xacro:property name="hokuyo_mass"    value="1e-5"     />
   <xacro:property name="hokuyo_width"   value="0.05"     />
   <xacro:property name="hokuyo_length"  value="0.05"     />
   <xacro:property name="hokuyo_height"  value="0.0706"   />
-  <xacro:property name="hokuyo_x"       value="0.11"     />
+  <xacro:property name="hokuyo_x"       value="0.11"     /> <!-- x offset from base center -->
   <xacro:property name="hokuyo_z"       value="${(hokuyo_height+base_height)/2}" />
 <!-- ****************************************************** Includes *****************************************************************  -->

Commit message: u

File: xacro/skidbot.xacro (robot description, xacro)
@@ -6,5 +6,5 @@
 <!-- *********************************************************************************************************************************  -->
 <!-- ****************************************************** Parameters ***************************************************************  -->
-  <xacro:property name="mesh_path"      value="package://skidbot/meshes/skidbot/"/>
+  <xacro:property name="mesh_path"      value="package://bots/meshes/skidbot/"/>
   <xacro:property name="name_space"     value="skidbot"  />
   <xacro:property name="prefix"         value=""         />

Commit message: u

File: xacro/skidbot.xacro (robot description, xacro)
@@ -1,172 +1,19 @@
-<?xml version='1.0'?>
+<?xml version="1.0"?>
 <robot name="skidbot" xmlns:xacro="http://www.ros.org/wiki/xacro">
-<!-- ****************************************************** skidbot Robot *************************************************************  -->
+<!-- ****************************************************** Skidbot Robot ***************************************************************  -->
 <!-- Muthanna Alwahash                                                                                                                  -->
 <!-- March 2022                                                                                                                         -->
 <!-- *********************************************************************************************************************************  -->
 <!-- ****************************************************** Parameters ***************************************************************  -->
-  <xacro:property name="mesh_path"      value="package://bots/meshes/skidbot/"/>
-  <xacro:property name="name_space"     value="skidbot"  />
-  <xacro:property name="prefix"         value=""         />
-  <xacro:property name="base_mass"      value="15.0"     /> <!-- arbitrary mass value -->
-  <xacro:property name="base_width"     value="0.20"     />
-  <xacro:property name="base_length"    value="0.40"     />
-  <xacro:property name="base_height"    value="0.10"     />
-  <xacro:property name="wheel_mass"     value="5.0"      />
-  <xacro:property name="wheel_width"    value="0.05"     />
-  <xacro:property name="wheel_radius"   value="0.08"     />
-  <xacro:property name="wheel_gap"      value="0.01"     /> <!-- Gap between wheels and base         -->
-  <xacro:property name="wheel_x"        value="0.12"     /> <!-- x offset from base center -->
-  <xacro:property name="wheel_y"        value="${(base_width+wheel_width)/2+wheel_gap}" />
-  <xacro:property name="camera_mass"    value="1e-5"     />
-  <xacro:property name="camera_width"   value="0.05"     />
-  <xacro:property name="camera_length"  value="0.05"     />
-  <xacro:property name="camera_height"  value="0.05"     />
-  <xacro:property name="camera_x"       value="0.2"      /> <!-- x offset from base center -->
-  <xacro:property name="hokuyo_mass"    value="1e-5"     />
-  <xacro:property name="hokuyo_width"   value="0.05"     />
-  <xacro:property name="hokuyo_length"  value="0.05"     />
-  <xacro:property name="hokuyo_height"  value="0.0706"   />
-  <xacro:property name="hokuyo_x"       value="0.11"     /> <!-- x offset from base center -->
-  <xacro:property name="hokuyo_z"       value="${(hokuyo_height+base_height)/2}" />
+    <xacro:property name="pkg_path"     value="$(find bots)"                />
+    <xacro:property name="mesh_path"    value="${pkg_path}/meshes/skidbot/"    />
+    <xacro:property name="config_path"  value="${pkg_path}/config/"         />
+    <xacro:property name="name_space"   value="skidbot" />
+    <xacro:property name="prefix"       value=""      />
 <!-- ****************************************************** Includes *****************************************************************  -->
-  <xacro:include filename="$(find bots)/xacro/common_rviz_materials.xacro" />   <!-- RVIZ Colors                                     -->
-  <xacro:include filename="$(find bots)/gazebo/gz_skidbot.xacro" />             <!-- Gazebo                                          -->
-<!-- ****************************************************** Base Footprint ***********************************************************  -->
-  <link name="${prefix}footprint"></link>
-<!-- ****************************************************** Footprint Joint **********************************************************  -->
-  <joint type="fixed" name="${prefix}footprint_joint" >
-    <origin xyz="0 0 0" rpy="0 0 0" />
-    <parent link="${prefix}footprint"/>
-    <child link="${prefix}base" />
-  </joint>
-<!-- ****************************************************** Base Link ****************************************************************  -->
-  <link name='${prefix}base'>
-    <pose>0 0 0 0 0 0</pose>
-    <inertial>
-      <mass value="${base_mass}"/>
-      <origin xyz="0 0 0" rpy=" 0 0 0"/>
-      <inertia ixx="0.1" ixy="0" ixz="0" iyy="0.1" iyz="0" izz="0.1" />
-    </inertial>
-    <collision name='collision'>
-      <origin xyz="0 0 0" rpy=" 0 0 0"/>
-      <geometry>
-        <mesh filename="${mesh_path}base.stl" scale="1 1 1"/>  <!--  <box size="${base_length} ${base_width} ${base_height}"/> -->
-      </geometry>
-    </collision>
-    <visual name='base_visual'>
-      <origin xyz="0 0 0" rpy=" 0 0 0"/>
-      <geometry>
-        <mesh filename="${mesh_path}base.stl" scale="1 1 1"/>  <!--  <box size="${base_length} ${base_width} ${base_height}"/> -->
-      </geometry>
-      <material name="blue"/>
-    </visual>
-  </link>
-<!-- ****************************************************** Wheels Macro *************************************************************  -->
-  <xacro:macro name="wheel" params="position side x y">
-<!-- ****************************************************** Wheel Link ***************************************************************  -->
-    <link name="${prefix}${prefix}${position}_${side}_wheel">
-      <inertial>
-        <mass value="${base_mass}"/>
-        <origin xyz="0 0 0" rpy=" 0 ${radians(90)} ${radians(90)}"/>
-        <inertia ixx="0.1" ixy="0" ixz="0" iyy="0.1" iyz="0" izz="0.1" />
-      </inertial>
-      <visual>
-        <origin xyz="0 0 0" rpy=" 0 ${radians(90)} ${radians(90)}"/>
-        <geometry>
-          <mesh filename="${mesh_path}wheel.dae"/> <!--  <cylinder length="${wheel_width}" radius="${wheel_radius}"/> -->
-        </geometry>
-        <material name="grey"/>
-      </visual>
-      <collision>
-        <origin xyz="0 0 0" rpy=" 0 ${radians(90)} ${radians(90)}"/>
-        <geometry>
-          <mesh filename="${mesh_path}wheel.dae"/> <!--  <cylinder length="${wheel_width}" radius="${wheel_radius}"/> -->
-        </geometry>
-      </collision>
-    </link>
-<!-- ****************************************************** Wheel Joint **************************************************************  -->
-    <joint type="continuous" name="${prefix}${position}_${side}_wheel_joint">
-        <origin xyz="${x} ${y} 0" rpy="0 0 0"/>
-        <child link="${position}_${side}_wheel"/>
-        <parent link="base"/>
-        <axis xyz="0 1 0" rpy="0 0 0"/>
-        <limit effort="10000" velocity="1000"/>
-        <dynamics damping="1.0" friction="1.0"/>
-    </joint>
-<!-- ****************************************************** End of Macro *************************************************************  -->
-  </xacro:macro>
-<!-- ****************************************************** Expand Wheels Macro ******************************************************  -->
-<xacro:wheel position="front" side="right" x=" ${wheel_x}" y="-${wheel_y}" />
-<xacro:wheel position="front" side="left"  x=" ${wheel_x}" y=" ${wheel_y}" />
-<xacro:wheel position="back"  side="right" x="-${wheel_x}" y="-${wheel_y}" />
-<xacro:wheel position="back"  side="left"  x="-${wheel_x}" y=" ${wheel_y}" />
-<!-- ****************************************************** Camera Link **************************************************************  -->
-  <link name="${prefix}camera">
-    <inertial>
-      <mass value="${camera_mass}"/>
-      <origin xyz="0 0 0" rpy=" 0 0 0"/>
-      <inertia ixx="1e-6" ixy="0" ixz="0" iyy="1e-6" iyz="0" izz="1e-6" />
-    </inertial>
-    <visual name="camera_visual">
-      <origin xyz="0 0 0" rpy="0 0 0" />
-      <geometry>
-        <box size="${camera_length} ${camera_width} ${camera_height}"/>
-      </geometry>
-      <material name="green"/>
-    </visual>
-    <collision name="camera_colision">
-      <origin xyz="0 0 0" rpy="0 0 0" />
-      <geometry>
-        <box size="${camera_length} ${camera_width} ${camera_height}"/>
-      </geometry>
-    </collision>
-  </link>
-<!-- ****************************************************** Camera Joint *************************************************************  -->
-  <joint type="fixed" name="${prefix}camera_joint">
-    <origin xyz="${camera_x} 0 0" rpy="0 0 0"/>
-    <child link="${prefix}camera"/>
-    <parent link="${prefix}base"/>
-    <axis xyz="0 1 0" rpy="0 0 0"/>
-  </joint>
-<!-- ****************************************************** Camera Optical Joint *****************************************************  -->
-<!-- generate an optical frame http://www.ros.org/reps/rep-0103.html#suffix-frames so that ros and opencv can operate on the camera     -->
-<!-- frame correctly. these values have to be these values otherwise the gazebo camera image won't be aligned properly with the frame   -->
-<!-- it is supposedly originating from                                                                                                  -->                                                                                                                   -->
-  <joint name="${prefix}camera_optical_joint" type="fixed">
-    <origin xyz="0 0 0" rpy="${-radians(90)} 0 ${-radians(90)}"/>
-    <parent link="${prefix}camera"/>
-    <child link="${prefix}camera_optical"/>
-  </joint>
-<!-- ****************************************************** Camera Optical Link ******************************************************  -->
-  <link name="${prefix}camera_optical"/>
-<!-- ****************************************************** Hokuyo Link **************************************************************  -->
-  <link name="${prefix}hokuyo">
-    <inertial>
-      <mass value="${hokuyo_mass}"/>
-      <origin xyz="0 0 0" rpy=" 0 0 0"/>
-      <inertia ixx="1e-6" ixy="0" ixz="0" iyy="1e-6" iyz="0" izz="1e-6" />
-    </inertial>
-    <visual name="hokuyo_visual">
-      <origin xyz="0 0 0" rpy="0 0 0" />
-      <geometry>
-        <mesh filename="${mesh_path}hokuyo.dae"/> <!--  <box size="${hokuyo_length} ${hokuyo_width} ${hokuyo_height}"/> -->
-      </geometry>
-      <!-- <material name="red"/> -->
-    </visual>
-    <collision name="hokuyo_colision">
-      <origin xyz="0 0 0" rpy="0 0 0" />
-      <geometry>
-        <box size="${hokuyo_length} ${hokuyo_width} ${hokuyo_height}"/>
-      </geometry>
-    </collision>
-  </link>
-<!-- ****************************************************** Hokuyo Joint *************************************************************  -->
-  <joint type="fixed" name="${prefix}hokuyo_joint">
-    <origin xyz="${hokuyo_x} 0 ${hokuyo_z}" rpy="0 0 0"/>
-    <child link="${prefix}hokuyo"/>
-    <parent link="${prefix}base"/>
-    <axis xyz="0 1 0" rpy="0 0 0"/>
-  </joint>
-<!-- ****************************************************** end **********************************************************************  -->
+    <xacro:include filename="${pkg_path}/xacro/common_rviz_materials.xacro" />  <!--  RVIZ Colors  -->
+    <xacro:include filename="${pkg_path}/xacro/urdf_skidbot.xacro" />           <!--  Robot URDF   -->
+    <xacro:include filename="${pkg_path}/gazebo/gz_skidbot.xacro" />            <!--  Gazebo Sim   -->
+    <xacro:include filename="${pkg_path}/r2c/r2c_skidbot.xacro" />              <!--  ROS2_Control -->
+<!-- ****************************************************** END **********************************************************************  -->
 </robot>
