Commit message: u

File: xacro/urdf_diffbot.xacro (robot description, xacro)
@@ -6,18 +6,18 @@
 <!-- *********************************************************************************************************************************  -->
 <!-- ****************************************************** Parameters ***************************************************************  -->
-  <xacro:property name="base_mass"      value="0.6"                               />  <!-- arbitrary value for base mass                -->
-  <xacro:property name="base_width"     value="0.20"                              />
-  <xacro:property name="base_length"    value="0.40"                              />
-  <xacro:property name="base_height"    value="0.10"                              />
-  <xacro:property name="wheel_mass"     value="5.0"                               />
-  <xacro:property name="wheel_width"    value="0.05"                              />
-  <xacro:property name="wheel_radius"   value="0.08"                              />
-  <xacro:property name="wheel_gap"      value="0.01"                              /> <!-- Gap between wheels and base                   -->
-  <xacro:property name="wheel_x"        value="0.12"                              /> <!-- x offset from base center -->
+  <xacro:property name="base_mass"      value="0.6"                                     /> <!-- arbitrary value for base mass          -->
+  <xacro:property name="base_width"     value="0.20"                                    />
+  <xacro:property name="base_length"    value="0.40"                                    />
+  <xacro:property name="base_height"    value="0.10"                                    />
+  <xacro:property name="wheel_mass"     value="5.0"                                     />
+  <xacro:property name="wheel_width"    value="0.05"                                    />
+  <xacro:property name="wheel_radius"   value="0.08"                                    />
+  <xacro:property name="wheel_gap"      value="0.01"                                    /> <!-- Gap between wheels and base             -->
+  <xacro:property name="wheel_x"        value="0.12"                                    /> <!-- x offset from base center               -->
   <xacro:property name="wheel_y"        value="${(base_width+wheel_width)/2+wheel_gap}" />
-  <xacro:property name="wheel_z"        value="${base_height/4}"                  />  <!-- Space btw top of beam and the each joint     -->
-  <xacro:property name="caster_mass"    value="0.1"                               />  <!-- arbitrary value for caster wheel mass        -->
-  <xacro:property name="caster_radius"  value="${wheel_radius-wheel_z}"           />
-  <xacro:property name="caster_x"       value="${(base_length/2 - caster_radius)}" />
+  <xacro:property name="wheel_z"        value="${base_height/4}"                        /> <!-- Space btw top of beam and the each joint-->
+  <xacro:property name="caster_mass"    value="0.1"                                     /> <!-- arbitrary value for caster wheel mass   -->
+  <xacro:property name="caster_radius"  value="${wheel_radius-wheel_z}"                 />
+  <xacro:property name="caster_x"       value="${(base_length/2 - caster_radius)}"      />
   <xacro:property name="caster_z"       value="${base_height/2}"/>
   <xacro:property name="camera_mass"    value="0.1"      />
