Commit message: u

File: gazebo/gz_twr.xacro (robot description, xacro)
@@ -6,14 +6,12 @@
 <!-- *********************************************************************************************************************************  -->
 <!-- ****************************************************** Base Link ****************************************************************  -->
-    <gazebo reference="base_link">
-        <material>Gazebo/Red</material>
-    </gazebo>
-<!-- ****************************************************** Macro ********************************************************************  -->
-<xacro:macro name="wheel" params="prefix">
+  <gazebo reference="base_link">
+      <material>Gazebo/Red</material>
+  </gazebo>
 <!-- ****************************************************** Drive Wheels Link Macro **************************************************  -->
-    <gazebo reference="${prefix}_link">
-        <material>Gazebo/FlatBlack</material>
-    </gazebo>
-<!-- ****************************************************** End of Macro *************************************************************  -->
+  <xacro:macro name="wheel" params="prefix">
+      <gazebo reference="${prefix}_link">
+          <material>Gazebo/FlatBlack</material>
+      </gazebo>
   </xacro:macro>
 <!-- ****************************************************** Drive Wheels Link and Joint **********************************************  -->
@@ -26,5 +24,5 @@
 <!-- ****************************************************** LIDAR Link ***************************************************************  -->
   <gazebo reference="lidar_link">
-    <material>Gazebo/Green</material>
+      <material>Gazebo/Green</material>
   </gazebo>
 <!-- *********************************************************************************************************************************  -->

File: xacro/twr.xacro (robot description, xacro)
@@ -18,6 +18,7 @@
   <xacro:property name="wheel_xoff"   value="0.221"/> <!-- Position the wheels along the x-axis                                         -->
   <xacro:property name="caster_xoff"  value="0.217"/> <!-- Position the caster wheel along the x-axis                                   -->
-<!-- ****************************************************** Import RVIZ Materials*****************************************************  -->
-  <xacro:include filename="$(find robot_gazebo)/xacro/common_rviz_materials.xacro" />
+<!-- ****************************************************** Includes *****************************************************************  -->
+  <xacro:include filename="$(find robot_gazebo)/xacro/common_rviz_materials.xacro" />   <!-- RVIZ Colors                                -->
+  <xacro:include filename="$(find robot_gazebo)/gazebo/gz_twr.xacro" />               <!-- Gazebo                                     -->
 <!-- ****************************************************** Macros *******************************************************************  -->
 <!-- Define intertial property macros                                                                                                   -->
@@ -68,7 +69,4 @@
     <xacro:box_inertia m="40.0" w="${base_width}" d="${base_length}" h="${base_height}"/>
   </link>
-  <gazebo reference="base_link">
-      <material>Gazebo/Red</material>
-  </gazebo>
 <!-- ****************************************************** Drive Wheels Link Macro **************************************************  -->
   <xacro:macro name="wheel" params="prefix x_reflect y_reflect">
@@ -89,7 +87,4 @@
       <xacro:cylinder_inertia m="110.5" r="${wheel_radius}" h="${wheel_width}"/>
     </link>
-    <gazebo reference="${prefix}_link">
-        <material>Gazebo/FlatBlack</material>
-    </gazebo>
 <!-- ****************************************************** Drive Wheels Joint Macro *************************************************  -->
 <!-- Connect the wheels to the base_link at the appropriate location, and define a continuous joint to allow the wheels to freely       -->
@@ -126,7 +121,4 @@
     <xacro:sphere_inertia m="10.05" r="${(wheel_radius+wheel_zoff-(base_height/2))}"/>
   </link>
-  <gazebo reference="front_caster">
-      <material>Gazebo/White</material>
-  </gazebo>
 <!-- **************************************************** Front Caster Joint *********************************************************  -->
   <joint name="caster_joint" type="fixed">
@@ -171,7 +163,4 @@
     </inertial>
   </link>
-  <gazebo reference="lidar_link">
-    <material>Gazebo/Green</material>
-  </gazebo>
 <!-- *********************************************************************************************************************************  -->
 </robot>
