Commit message: u

File: gazebo/gz_razbot.xacro (robot description, xacro)
@@ -6,239 +6,31 @@
 <!-- Originally developed by Shubhankar Das a.k.a Razbotics                                                                             -->
 <!-- *********************************************************************************************************************************  -->
-<!-- ****************************************************** Parameters ***************************************************************  -->
-    <xacro:property name="mesh_path"          value="package://robot_gazebo/meshes/razbot/"/>
-	<xacro:property name="body_length_x"        value="0.294" />
-	<xacro:property name="body_length_y"        value="0.340" />
-	<xacro:property name="coxa_length"          value="0.052" />
-	<xacro:property name="femur_length"         value="0.065" />
-	<xacro:property name="tibia_length"         value="0.133" />
-	<xacro:property name="joint_lower_limit"    value="${radians(-180)}" />
-	<xacro:property name="joint_upper_limit"    value="${radians( 180)}" />
-	<xacro:property name="joint_effort"         value="6.0" />
-	<xacro:property name="joint_velocity"       value="${radians( 300)}" />
-<!-- ****************************************************** Import RVIZ Materials*****************************************************  -->
-  <xacro:include filename="$(find robot_gazebo)/xacro/common_rviz_materials.xacro" />
-<!-- ****************************************************** Base Footprint ***********************************************************  -->
-    <link name="base_footprint"/>
-<!-- ****************************************************** Base Joint ***************************************************************  -->
-    <joint name="base_joint" type="fixed">
-        <parent link="base_footprint" />
-        <child link="base_link" />
-        <origin xyz="0 0 0" rpy="0 0 0" />
-    </joint>
 <!-- ****************************************************** Base Link ****************************************************************  -->
-	<link name="base_link">
-        <visual>
-            <origin	xyz="0 0 0" rpy="0 0 0" />
-            <geometry>
-                <mesh filename="${mesh_path}body.stl" scale="0.001 0.001 0.001"/>
-            </geometry>
-            <material name="blue"/>
-        </visual>
-        <collision>
-            <origin xyz="0 0 0" rpy="0 0 0"/>
-            <geometry>
-                <mesh filename="${mesh_path}body.stl" scale="0.001 0.001 0.001"/>
-            </geometry>
-            <material name="blue"/>
-        </collision>
-        <inertial>
-            <origin xyz="0 0 0" rpy="0 0 0" />
-            <mass value="0.00001"/>
-            <inertia
-                ixx="1.0" ixy="0.0"  ixz="0.0"
-                iyy="1.0" iyz="0.0"
-                izz="1.0" />
-        </inertial>
-    </link>
     <gazebo reference="base_link">
         <material>Gazebo/Blue</material>
     </gazebo>
-<!-- ****************************************************** IMU Joint ****************************************************************  -->
-	<joint name="imu_joint" type="fixed">
-		<parent link="base_link" />
-		<child link="imu_link" />
-		<origin xyz="0 0 0" rpy="0 0 0" />
-	</joint>
-<!-- ****************************************************** IMU Link *****************************************************************  -->
-	<link name="imu_link">
-        <inertial>
-            <origin xyz="0 0 0" rpy="0 0 0" />
-            <mass value="0.00001"/>
-            <inertia
-                ixx="1.0" ixy="0.0"  ixz="0.0"
-                iyy="1.0" iyz="0.0"
-                izz="1.0" />
-        </inertial>
-    </link>
 <!-- ****************************************************** Leg Macro ****************************************************************  -->
-	<xacro:macro name="leg" params="side position x y angle axis">
-<!-- ****************************************************** Leg Center Joint *********************************************************  -->
-		<joint name="leg_center_joint_${side}${position}" type="fixed">
-			<origin xyz="${x} ${y} 0.0" rpy="0 0 0" />
-			<parent link="base_link" />
-			<child link="leg_center_${side}${position}" />
-		</joint>
-<!-- ****************************************************** Leg Center Link **********************************************************  -->
-		<link name="leg_center_${side}${position}" >
-            <inertial>
-                <origin xyz="0 0 0" rpy="0 0 0" />
-                <mass value="0.00001"/>
-                <inertia
-                    ixx="1.0" ixy="0.0"  ixz="0.0"
-                    iyy="1.0" iyz="0.0"
-                    izz="1.0" />
-            </inertial>
-        </link>
-<!-- ****************************************************** Coxa Joint **************************************************************  -->
-		<joint name="coxa_joint_${side}${position}" type="revolute">
-			<origin xyz="0 0 0" rpy="0.0 0.0 ${angle}" />
-			<parent link="leg_center_${side}${position}" />
-			<child link="coxa_${side}${position}" />
-			<axis xyz="0.0 0.0 1.0" />
-			<limit lower="${joint_lower_limit}" upper="${joint_upper_limit}" effort="${joint_effort}" velocity="${joint_velocity}" />
-		</joint>
+	<xacro:macro name="leg_gz" params="side position">
 <!-- ****************************************************** Coxa Link *****************************************************************  -->
-        <link name="coxa_${side}${position}">
-            <visual>
-                <origin xyz="0 0 0" rpy="0 0 0"/>
-                <geometry>
-                    <mesh filename="${mesh_path}coxa.stl" scale="0.001 0.001 0.001"/>
-                </geometry>
-                <material name="green"/>
-            </visual>
-            <collision>
-                <origin xyz="0 0 0" rpy="0 0 0" />
-                <geometry>
-                    <mesh filename="${mesh_path}coxa.stl" scale="0.001 0.001 0.001"/>
-                </geometry>
-                <material name="green"/>
-            </collision>
-            <inertial>
-                <origin xyz="0 0 0" rpy="0 0 0" />
-                <mass value="0.00001"/>
-                <inertia
-                    ixx="1.0" ixy="0.0"  ixz="0.0"
-                    iyy="1.0" iyz="0.0"
-                    izz="1.0" />
-            </inertial>
-        </link>
         <gazebo reference="coxa_${side}${position}">
             <material>Gazebo/Red</material>
         </gazebo>
-<!-- ****************************************************** Coxa Transmission ********************************************************  -->
-		<transmission name="coxa_transmission_${side}${position}">
-            <type>transmission_interface/SimpleTransmission</type>
-            <joint name="coxa_joint_${side}${position}">
-                <hardwareInterface>EffortJointInterface</hardwareInterface>
-            </joint>
-            <actuator name="coxa_motor_${side}${position}">
-                <hardwareInterface>EffortJointInterface</hardwareInterface>
-                <mechanicalReduction>1</mechanicalReduction>
-            </actuator>
-        </transmission>
-<!-- ****************************************************** Femur Joint **************************************************************  -->
-		<joint name="femur_joint_${side}${position}" type="revolute">
-			<origin xyz="${coxa_length} 0.0 0.0" rpy="${radians(-90)} ${radians(90)} 0.0" />
-			<parent link="coxa_${side}${position}" />
-			<child link="femur_${side}${position}" />
-			<axis xyz="0.0 0.0 ${-axis}" />
-			<limit lower="${joint_lower_limit}" upper="${joint_upper_limit}" effort="${joint_effort}" velocity="${joint_velocity}" />
-		</joint>
 <!-- ****************************************************** Femur Link ***************************************************************  -->
-        <link name="femur_${side}${position}">
-            <visual>
-                <origin xyz="0 0 0" rpy="0 0 0"/>
-                <geometry>
-                    <mesh filename="${mesh_path}femur.stl" scale="0.001 0.001 0.001"/>
-                </geometry>
-                <material name="red"/>
-            </visual>
-            <collision>
-                <origin xyz="0 0 0" rpy="0 0 0" />
-                <geometry>
-                    <mesh filename="${mesh_path}femur.stl" scale="0.001 0.001 0.001"/>
-                </geometry>
-                <material name="red"/>
-            </collision>
-            <inertial>
-                <origin xyz="0 0 0" rpy="0 0 0" />
-                <mass value="0.00001"/>
-                <inertia
-                    ixx="1.0" ixy="0.0"  ixz="0.0"
-                    iyy="1.0" iyz="0.0"
-                    izz="1.0" />
-            </inertial>
-        </link>
         <gazebo reference="femur_${side}${position}">
             <material>Gazebo/Green</material>
         </gazebo>
-<!-- ****************************************************** Femur Transmission *******************************************************  -->
-		<transmission name="femur_transmission_${side}${position}">
-            <type>transmission_interface/SimpleTransmission</type>
-            <joint name="femur_joint_${side}${position}">
-                <hardwareInterface>EffortJointInterface</hardwareInterface>
-            </joint>
-            <actuator name="femur_motor_${side}${position}">
-                <hardwareInterface>EffortJointInterface</hardwareInterface>
-                <mechanicalReduction>1</mechanicalReduction>
-            </actuator>
-        </transmission>
-<!-- ****************************************************** Tibia Joint *************************************************************  -->
-		<joint name="tibia_joint_${side}${position}" type="revolute">
-			<origin xyz="0.0 -${femur_length} 0.0" rpy="${radians(180)} 0 0" />
-			<parent link="femur_${side}${position}" />
-			<child link="tibia_${side}${position}" />
-			<axis xyz="0.0 0.0 ${axis}" />
-			<limit lower="${joint_lower_limit}" upper="${joint_upper_limit}" effort="${joint_effort}" velocity="${joint_velocity}" />
-		</joint>
 <!-- ****************************************************** Tibia Link **************************************************************  -->
-        <link name="tibia_${side}${position}">
-            <visual>
-                <origin xyz="0 0 0" rpy="0 0 0"/>
-                <geometry>
-                    <mesh filename="${mesh_path}tibia.stl" scale="0.001 0.001 0.001"/>
-                </geometry>
-                <material name="green"/>
-            </visual>
-            <collision>
-                <origin xyz="0 0.0 0.0" rpy="0 0 0" />
-                <geometry>
-                    <mesh filename="${mesh_path}tibia.stl" scale="0.001 0.001 0.001"/>
-                </geometry>
-                <material name="green"/>
-            </collision>
-            <inertial>
-                <origin xyz="0 0.0 0.0" rpy="0 0 0" />
-                <mass value="0.00001"/>
-                <inertia
-                    ixx="1.0" ixy="0.0"  ixz="0.0"
-                    iyy="1.0" iyz="0.0"
-                    izz="1.0" />
-            </inertial>
-        </link>
         <gazebo reference="tibia_${side}${position}">
             <material>Gazebo/Red</material>
         </gazebo>
-<!-- ****************************************************** Tibia Transmission *****************************************************  -->
-		<transmission name="tibia_transmission_${side}${position}">
-            <type>transmission_interface/SimpleTransmission</type>
-            <joint name="tibia_joint_${side}${position}">
-                <hardwareInterface>EffortJointInterface</hardwareInterface>
-            </joint>
-            <actuator name="tibia_motor_${side}${position}">
-                <hardwareInterface>EffortJointInterface</hardwareInterface>
-                <mechanicalReduction>1</mechanicalReduction>
-            </actuator>
-        </transmission>
 <!-- ****************************************************** end of Macro *************************************************************  -->
 	</xacro:macro>
 <!-- ****************************************************** Build Robot **************************************************************  -->
-	<xacro:leg side="R" position="R" x="-${body_length_x/2}"    y="-${0.1695/2}"        angle="${radians(-150)}"    axis=" 1" />
-	<xacro:leg side="R" position="M" x=" 0.0"                   y="-${body_length_y/2}" angle="${radians(-90)}"     axis=" 1" />
-	<xacro:leg side="R" position="F" x=" ${body_length_x/2}"    y="-${0.1695/2}"        angle="${radians(-30)}"     axis=" 1" />
-	<xacro:leg side="L" position="R" x="-${body_length_x/2}"    y=" ${0.1695/2}"        angle="${radians(150)}"     axis="-1" />
-	<xacro:leg side="L" position="M" x=" 0.0"                   y=" ${body_length_y/2}" angle="${radians(90)}"      axis="-1" />
-	<xacro:leg side="L" position="F" x=" ${body_length_x/2}"    y=" ${0.1695/2}"        angle="${radians(30)}"      axis="-1" />
+	<xacro:leg side="R" position="R" />
+	<xacro:leg side="R" position="M" />
+	<xacro:leg side="R" position="F" />
+	<xacro:leg side="L" position="R" />
+	<xacro:leg side="L" position="M" />
+	<xacro:leg side="L" position="F" />
 <!-- ******************************************************  *************************************************************************  -->
 </robot>

File: xacro/razbot.xacro (robot description, xacro)
@@ -17,6 +17,7 @@
 	<xacro:property name="joint_effort"         value="6.0" />
 	<xacro:property name="joint_velocity"       value="${radians( 300)}" />
-<!-- ****************************************************** Import RVIZ Materials*****************************************************  -->
-  <xacro:include filename="$(find robot_gazebo)/xacro/common_rviz_materials.xacro" />
+<!-- ****************************************************** Includes *****************************************************************  -->
+  <xacro:include filename="$(find robot_gazebo)/xacro/common_rviz_materials.xacro" />   <!-- RVIZ Colors                                -->
+  <xacro:include filename="$(find robot_gazebo)/gazebo/gz_razbot.xacro" />              <!-- Gazebo                                     -->
 <!-- ****************************************************** Base Footprint ***********************************************************  -->
     <link name="base_footprint"/>
@@ -52,7 +53,4 @@
         </inertial>
     </link>
-    <gazebo reference="base_link">
-        <material>Gazebo/Blue</material>
-    </gazebo>
 <!-- ****************************************************** IMU Joint ****************************************************************  -->
 	<joint name="imu_joint" type="fixed">
@@ -124,7 +122,4 @@
             </inertial>
         </link>
-        <gazebo reference="coxa_${side}${position}">
-            <material>Gazebo/Red</material>
-        </gazebo>
 <!-- ****************************************************** Coxa Transmission ********************************************************  -->
 		<transmission name="coxa_transmission_${side}${position}">
@@ -171,7 +166,4 @@
             </inertial>
         </link>
-        <gazebo reference="femur_${side}${position}">
-            <material>Gazebo/Green</material>
-        </gazebo>
 <!-- ****************************************************** Femur Transmission *******************************************************  -->
 		<transmission name="femur_transmission_${side}${position}">
@@ -218,7 +210,4 @@
             </inertial>
         </link>
-        <gazebo reference="tibia_${side}${position}">
-            <material>Gazebo/Red</material>
-        </gazebo>
 <!-- ****************************************************** Tibia Transmission *****************************************************  -->
 		<transmission name="tibia_transmission_${side}${position}">
