Commit message: u

File: gazebo/gz_kr120r2500pro.xacro (robot description, xacro)
@@ -9,19 +9,25 @@
 <!-- ****************************************************** link 1 (A1) ************************************************************** -->
     <gazebo reference="${prefix}link_1">
+      <material>Gazebo/Orange</material>
     </gazebo>
-<!-- ****************************************************** link 2 **************************************************************** -->
+<!-- ****************************************************** link 2 (A2) ************************************************************** -->
     <gazebo reference="${prefix}link_2">
+      <material>Gazebo/Orange</material>
     </gazebo>
-<!-- ****************************************************** link 3 **************************************************************** -->
+<!-- ****************************************************** link 3 (A3) ************************************************************** -->
     <gazebo reference="${prefix}link_3">
+      <material>Gazebo/Orange</material>
     </gazebo>
-<!-- ****************************************************** link 4 **************************************************************** -->
+<!-- ****************************************************** link 4 (A4) ************************************************************** -->
     <gazebo reference="${prefix}link_4">
+      <material>Gazebo/Orange</material>
     </gazebo>
-<!-- ****************************************************** link 5 **************************************************************** -->
+<!-- ****************************************************** link 5 (A5) ************************************************************** -->
     <gazebo reference="${prefix}link_5">
+      <material>Gazebo/Orange</material>
     </gazebo>
-<!-- ****************************************************** link 6 **************************************************************** -->
+<!-- ****************************************************** link 6 (A6) ************************************************************** -->
     <gazebo reference="${prefix}link_6">
+      <material>Gazebo/Gray</material>
     </gazebo>
 <!-- ****************************************************** End Macro **************************************************************** -->

File: gazebo/gz_kr16_2.xacro (robot description, xacro)
@@ -9,19 +9,25 @@
 <!-- ****************************************************** link 1 (A1) ************************************************************** -->
     <gazebo reference="${prefix}link_1">
+      <material>Gazebo/Orange</material>
     </gazebo>
-<!-- ****************************************************** link 2 **************************************************************** -->
+<!-- ****************************************************** link 2 (A2) ************************************************************** -->
     <gazebo reference="${prefix}link_2">
+      <material>Gazebo/Orange</material>
     </gazebo>
-<!-- ****************************************************** link 3 **************************************************************** -->
+<!-- ****************************************************** link 3 (A3) ************************************************************** -->
     <gazebo reference="${prefix}link_3">
+      <material>Gazebo/Orange</material>
     </gazebo>
-<!-- ****************************************************** link 4 **************************************************************** -->
+<!-- ****************************************************** link 4 (A4) ************************************************************** -->
     <gazebo reference="${prefix}link_4">
+      <material>Gazebo/Orange</material>
     </gazebo>
-<!-- ****************************************************** link 5 **************************************************************** -->
+<!-- ****************************************************** link 5 (A5) ************************************************************** -->
     <gazebo reference="${prefix}link_5">
+      <material>Gazebo/Orange</material>
     </gazebo>
-<!-- ****************************************************** link 6 **************************************************************** -->
+<!-- ****************************************************** link 6 (A6) ************************************************************** -->
     <gazebo reference="${prefix}link_6">
+      <material>Gazebo/Gray</material>
     </gazebo>
 <!-- ****************************************************** End Macro **************************************************************** -->

File: gazebo/gz_kr3r540.xacro (robot description, xacro)
@@ -12,21 +12,21 @@
       <material>Gazebo/Orange</material>
     </gazebo>
-<!-- ****************************************************** link 2 ******************************************************************* -->
+<!-- ****************************************************** link 2 (A2) ************************************************************** -->
     <gazebo reference="${prefix}link_2">
       <material>Gazebo/Orange</material>
     </gazebo>
-<!-- ****************************************************** link 2 ******************************************************************* -->
+<!-- ****************************************************** link 3 (A3) ************************************************************** -->
     <gazebo reference="${prefix}link_3">
       <material>Gazebo/Orange</material>
     </gazebo>
-<!-- ****************************************************** link 4 ******************************************************************* -->
+<!-- ****************************************************** link 4 (A4) ************************************************************** -->
     <gazebo reference="${prefix}link_4">
       <material>Gazebo/Orange</material>
     </gazebo>
-<!-- ****************************************************** link 5 ******************************************************************* -->
+<!-- ****************************************************** link 5 (A5) ************************************************************** -->
     <gazebo reference="${prefix}link_5">
       <material>Gazebo/Orange</material>
     </gazebo>
-<!-- ****************************************************** link 6 ******************************************************************* -->
+<!-- ****************************************************** link 6 (A6) ************************************************************** -->
     <gazebo reference="${prefix}link_6">
       <material>Gazebo/Gray</material>

File: gazebo/gz_kr5_arc.xacro (robot description, xacro)
@@ -12,21 +12,21 @@
       <material>Gazebo/Orange</material>
     </gazebo>
-<!-- ****************************************************** link 2 ******************************************************************* -->
+<!-- ****************************************************** link 2 (A2) ************************************************************** -->
     <gazebo reference="${prefix}link_2">
       <material>Gazebo/Orange</material>
     </gazebo>
-<!-- ****************************************************** link 2 ******************************************************************* -->
+<!-- ****************************************************** link 3 (A3) ************************************************************** -->
     <gazebo reference="${prefix}link_3">
       <material>Gazebo/Orange</material>
     </gazebo>
-<!-- ****************************************************** link 4 ******************************************************************* -->
+<!-- ****************************************************** link 4 (A4) ************************************************************** -->
     <gazebo reference="${prefix}link_4">
       <material>Gazebo/Orange</material>
     </gazebo>
-<!-- ****************************************************** link 5 ******************************************************************* -->
+<!-- ****************************************************** link 5 (A5) ************************************************************** -->
     <gazebo reference="${prefix}link_5">
       <material>Gazebo/Orange</material>
     </gazebo>
-<!-- ****************************************************** link 6 ******************************************************************* -->
+<!-- ****************************************************** link 6 (A6) ************************************************************** -->
     <gazebo reference="${prefix}link_6">
       <material>Gazebo/Gray</material>

File: gazebo/gz_lbr_iiwa_14_r820.xacro (robot description, xacro)
@@ -9,22 +9,29 @@
 <!-- ****************************************************** link 1 (A1) ************************************************************** -->
     <gazebo reference="${prefix}link_1">
+      <material>Gazebo/Orange</material>
     </gazebo>
-<!-- ****************************************************** link 2 **************************************************************** -->
+<!-- ****************************************************** link 2 (A2) ************************************************************** -->
     <gazebo reference="${prefix}link_2">
+      <material>Gazebo/Orange</material>
     </gazebo>
-<!-- ****************************************************** link 3 **************************************************************** -->
+<!-- ****************************************************** link 3 (A3) ************************************************************** -->
     <gazebo reference="${prefix}link_3">
+      <material>Gazebo/Orange</material>
     </gazebo>
-<!-- ****************************************************** link 4 **************************************************************** -->
+<!-- ****************************************************** link 4 (A4) ************************************************************** -->
     <gazebo reference="${prefix}link_4">
+      <material>Gazebo/Orange</material>
     </gazebo>
-<!-- ****************************************************** link 5 **************************************************************** -->
+<!-- ****************************************************** link 5 (A5) ************************************************************** -->
     <gazebo reference="${prefix}link_5">
+      <material>Gazebo/Orange</material>
     </gazebo>
-<!-- ****************************************************** link 6 **************************************************************** -->
+<!-- ****************************************************** link 6 (A6) ************************************************************** -->
     <gazebo reference="${prefix}link_6">
+      <material>Gazebo/Orange</material>
     </gazebo>
-<!-- ****************************************************** link 7 **************************************************************** -->
+<!-- ****************************************************** link 7 (A7) ************************************************************** -->
     <gazebo reference="${prefix}link_7">
+      <material>Gazebo/Gray</material>
     </gazebo>
 <!-- ****************************************************** End Macro **************************************************************** -->

Commit message: u

File: gazebo/gz_kr120r2500pro.xacro (robot description, xacro)
@@ -6,4 +6,5 @@
 <!-- ****************************************************** base link **************************************************************** -->
     <gazebo reference="${prefix}base_link">
+      <material>Gazebo/Gray</material>
     </gazebo>
 <!-- ****************************************************** link 1 (A1) ************************************************************** -->

File: gazebo/gz_kr16_2.xacro (robot description, xacro)
@@ -6,4 +6,5 @@
 <!-- ****************************************************** base link **************************************************************** -->
     <gazebo reference="${prefix}base_link">
+      <material>Gazebo/Gray</material>
     </gazebo>
 <!-- ****************************************************** link 1 (A1) ************************************************************** -->

File: gazebo/gz_lbr_iiwa_14_r820.xacro (robot description, xacro)
@@ -6,4 +6,5 @@
 <!-- ****************************************************** base link **************************************************************** -->
     <gazebo reference="${prefix}base_link">
+      <material>Gazebo/Gray</material>
     </gazebo>
 <!-- ****************************************************** link 1 (A1) ************************************************************** -->
