Commit message: u

File: gazebo/gz_tb3_burger.xacro (robot description, xacro)
@@ -5,174 +5,21 @@
 <!-- March 2022                                                                                                                         -->
 <!-- *********************************************************************************************************************************  -->
-<!-- ****************************************************** Import RVIZ Materials*****************************************************  -->
-  <xacro:include filename="$(find robot_gazebo)/xacro/common_rviz_materials.xacro" />
-<!-- ****************************************************** Base Footprint Link ******************************************************  -->
-  <link name="base_footprint"/>
-<!-- ****************************************************** Base Joint ***************************************************************  -->
-  <joint name="base_joint" type="fixed">
-    <parent link="base_footprint"/>
-    <child link="base_link"/>
-    <origin xyz="0.0 0.0 0.010" rpy="0 0 0"/>
-  </joint>
 <!-- ****************************************************** Base Link ****************************************************************  -->
-  <link name="base_link">
-    <visual>
-      <origin xyz="-0.032 0 0.0" rpy="0 0 0"/>
-      <geometry>
-        <mesh filename="package://robot_gazebo/meshes/tb3/burger_base.stl" scale="0.001 0.001 0.001"/>
-      </geometry>
-      <material name="blue"/>
-    </visual>
-    <collision>
-      <origin xyz="-0.032 0 0.070" rpy="0 0 0"/>
-      <geometry>
-        <box size="0.140 0.140 0.143"/>
-      </geometry>
-    </collision>
-    <inertial>
-      <origin xyz="0 0 0" rpy="0 0 0"/>
-      <mass value="8.2573504e-01"/>
-      <inertia ixx="2.2124416e-03" ixy="-1.2294101e-05" ixz="3.4938785e-05"
-               iyy="2.1193702e-03" iyz="-5.0120904e-06" izz="2.0064271e-03"
-               />
-    </inertial>
-  </link>
   <gazebo reference="base_link">
     <material>Gazebo/Blue</material>
   </gazebo>
-<!-- ****************************************************** Wheel Left Joint *********************************************************  -->
-  <joint name="wheel_left_joint" type="continuous">
-    <parent link="base_link"/>
-    <child link="wheel_left_link"/>
-    <origin xyz="0.0 0.08 0.023" rpy="-1.57 0 0"/>
-    <axis xyz="0 0 1"/>
-  </joint>
 <!-- ****************************************************** Wheel Left Link **********************************************************  -->
-  <link name="wheel_left_link">
-    <visual>
-      <origin xyz="0 0 0" rpy="1.57 0 0"/>
-      <geometry>
-        <mesh filename="package://robot_gazebo/meshes/tb3/left_tire.stl" scale="0.001 0.001 0.001"/>
-      </geometry>
-      <material name="black"/>
-    </visual>
-    <collision>
-      <origin xyz="0 0 0" rpy="0 0 0"/>
-      <geometry>
-        <cylinder length="0.018" radius="0.033"/>
-      </geometry>
-    </collision>
-    <inertial>
-      <origin xyz="0 0 0" />
-      <mass value="2.8498940e-02" />
-      <inertia ixx="1.1175580e-05" ixy="-4.2369783e-11" ixz="-5.9381719e-09"
-               iyy="1.1192413e-05" iyz="-1.4400107e-11" izz="2.0712558e-05"
-               />
-    </inertial>
-  </link>
   <gazebo reference="wheel_left_link">
     <material>Gazebo/FlatBlack</material>
   </gazebo>
-<!-- ****************************************************** Wheel Right Joint ********************************************************  -->
-  <joint name="wheel_right_joint" type="continuous">
-    <parent link="base_link"/>
-    <child link="wheel_right_link"/>
-    <origin xyz="0.0 -0.080 0.023" rpy="-1.57 0 0"/>
-    <axis xyz="0 0 1"/>
-  </joint>
 <!-- ****************************************************** Wheel Right Link *********************************************************  -->
-  <link name="wheel_right_link">
-    <visual>
-      <origin xyz="0 0 0" rpy="1.57 0 0"/>
-      <geometry>
-        <mesh filename="package://robot_gazebo/meshes/tb3/right_tire.stl" scale="0.001 0.001 0.001"/>
-      </geometry>
-      <material name="black"/>
-    </visual>
-    <collision>
-      <origin xyz="0 0 0" rpy="0 0 0"/>
-      <geometry>
-        <cylinder length="0.018" radius="0.033"/>
-      </geometry>
-    </collision>
-    <inertial>
-      <origin xyz="0 0 0" />
-      <mass value="2.8498940e-02" />
-      <inertia ixx="1.1175580e-05" ixy="-4.2369783e-11" ixz="-5.9381719e-09"
-               iyy="1.1192413e-05" iyz="-1.4400107e-11" izz="2.0712558e-05"
-               />
-    </inertial>
-  </link>
   <gazebo reference="wheel_right_link">
     <material>Gazebo/FlatBlack</material>
   </gazebo>
-<!-- ****************************************************** Caster Back Joint ********************************************************  -->
-  <joint name="caster_back_joint" type="fixed">
-    <parent link="base_link"/>
-    <child link="caster_back_link"/>
-    <origin xyz="-0.081 0 -0.004" rpy="-1.57 0 0"/>
-  </joint>
 <!-- ****************************************************** Caster Back Link *********************************************************  -->
-  <link name="caster_back_link">
-    <visual>
-      <geometry>
-        <sphere radius="0.007"/>
-      </geometry>
-      <material name="white"/>
-    </visual>
-    <collision>
-      <origin xyz="0 0.001 0" rpy="0 0 0"/>
-      <geometry>
-        <box size="0.030 0.009 0.020"/>
-      </geometry>
-    </collision>
-    <inertial>
-      <origin xyz="0 0 0" />
-      <mass value="0.005" />
-      <inertia ixx="0.001" ixy="0.0" ixz="0.0"
-               iyy="0.001" iyz="0.0"
-               izz="0.001" />
-    </inertial>
-  </link>
   <gazebo reference="caster_back_link">
     <material>Gazebo/White</material>
   </gazebo>
-<!-- ****************************************************** IMU Joint ****************************************************************  -->
-  <joint name="imu_joint" type="fixed">
-    <parent link="base_link"/>
-    <child link="imu_link"/>
-    <origin xyz="-0.032 0 0.068" rpy="0 0 0"/>
-  </joint>
-<!-- ****************************************************** IMU Link *****************************************************************  -->
-  <link name="imu_link"/>
-<!-- ****************************************************** Laser Scan Joint *********************************************************  -->
-  <joint name="scan_joint" type="fixed">
-    <parent link="base_link"/>
-    <child link="base_scan"/>
-    <origin xyz="-0.032 0 0.172" rpy="0 0 0"/>
-  </joint>
 <!-- ****************************************************** Laser Scan Link **********************************************************  -->
-  <link name="base_scan">
-    <visual>
-      <origin xyz="0 0 0.0" rpy="0 0 0"/>
-      <geometry>
-        <mesh filename="package://robot_gazebo/meshes/tb3/lds.stl" scale="0.001 0.001 0.001"/>
-      </geometry>
-      <material name="green"/>
-    </visual>
-    <collision>
-      <origin xyz="0.015 0 -0.0065" rpy="0 0 0"/>
-      <geometry>
-        <cylinder length="0.0315" radius="0.055"/>
-      </geometry>
-    </collision>
-    <inertial>
-      <mass value="0.114" />
-      <origin xyz="0 0 0" />
-      <inertia ixx="0.001" ixy="0.0" ixz="0.0"
-               iyy="0.001" iyz="0.0"
-               izz="0.001" />
-    </inertial>
-  </link>
   <gazebo reference="base_scan">
     <material>Gazebo/Green</material>

File: gazebo/gz_tb3_waffle.xacro (robot description, xacro)
@@ -5,259 +5,28 @@
 <!-- March 2022                                                                                                                         -->
 <!-- *********************************************************************************************************************************  -->
-<!-- ****************************************************** Import RVIZ Materials*****************************************************  -->
-  <xacro:include filename="$(find robot_gazebo)/xacro/common_rviz_materials.xacro" />
-<!-- ****************************************************** Base Footprint Link ******************************************************  -->
-  <link name="base_footprint"/>
-<!-- ****************************************************** Base Joint ***************************************************************  -->
-  <joint name="base_joint" type="fixed">
-    <parent link="base_footprint"/>
-    <child link="base_link" />
-    <origin xyz="0 0 0.010" rpy="0 0 0"/>
-  </joint>
 <!-- ****************************************************** Base Link ****************************************************************  -->
-  <link name="base_link">
-    <visual>
-      <origin xyz="-0.064 0 0.0" rpy="0 0 0"/>
-      <geometry>
-        <mesh filename="package://robot_gazebo/meshes/tb3/waffle_base.stl" scale="0.001 0.001 0.001"/>
-      </geometry>
-      <material name="blue"/>
-    </visual>
-    <collision>
-      <origin xyz="-0.064 0 0.047" rpy="0 0 0"/>
-      <geometry>
-        <box size="0.266 0.266 0.094"/>
-      </geometry>
-    </collision>
-    <inertial>
-      <origin xyz="0 0 0" rpy="0 0 0"/>
-      <mass value="1.3729096e+00"/>
-      <inertia ixx="8.7002718e-03" ixy="-4.7576583e-05" ixz="1.1160499e-04"
-               iyy="8.6195418e-03" iyz="-3.5422299e-06"
-               izz="1.4612727e-02" />
-    </inertial>
-  </link>
   <gazebo reference="base_link">
     <material>Gazebo/Blue</material>
   </gazebo>
-<!-- ****************************************************** Wheel Left Joint *********************************************************  -->
-  <joint name="wheel_left_joint" type="continuous">
-    <parent link="base_link"/>
-    <child link="wheel_left_link"/>
-    <origin xyz="0.0 0.144 0.023" rpy="-1.57 0 0"/>
-    <axis xyz="0 0 1"/>
-  </joint>
 <!-- ****************************************************** Wheel Left Link **********************************************************  -->
-  <link name="wheel_left_link">
-    <visual>
-      <origin xyz="0 0 0" rpy="1.57 0 0"/>
-      <geometry>
-        <mesh filename="package://robot_gazebo/meshes/tb3/left_tire.stl" scale="0.001 0.001 0.001"/>
-      </geometry>
-      <material name="black"/>
-    </visual>
-    <collision>
-      <origin xyz="0 0 0" rpy="0 0 0"/>
-      <geometry>
-        <cylinder length="0.018" radius="0.033"/>
-      </geometry>
-    </collision>
-    <inertial>
-      <origin xyz="0 0 0" />
-      <mass value="2.8498940e-02" />
-      <inertia ixx="1.1175580e-05" ixy="-4.2369783e-11" ixz="-5.9381719e-09"
-               iyy="1.1192413e-05" iyz="-1.4400107e-11"
-               izz="2.0712558e-05" />
-      </inertial>
-  </link>
   <gazebo reference="wheel_left_link">
     <material>Gazebo/FlatBlack</material>
   </gazebo>
-<!-- ****************************************************** Wheel Right Joint ********************************************************  -->
-  <joint name="wheel_right_joint" type="continuous">
-    <parent link="base_link"/>
-    <child link="wheel_right_link"/>
-    <origin xyz="0.0 -0.144 0.023" rpy="-1.57 0 0"/>
-    <axis xyz="0 0 1"/>
-  </joint>
 <!-- ****************************************************** Wheel Right Link *********************************************************  -->
-  <link name="wheel_right_link">
-    <visual>
-      <origin xyz="0 0 0" rpy="1.57 0 0"/>
-      <geometry>
-        <mesh filename="package://robot_gazebo/meshes/tb3/right_tire.stl" scale="0.001 0.001 0.001"/>
-      </geometry>
-      <material name="black"/>
-    </visual>
-    <collision>
-      <origin xyz="0 0 0" rpy="0 0 0"/>
-      <geometry>
-        <cylinder length="0.018" radius="0.033"/>
-      </geometry>
-    </collision>
-    <inertial>
-      <origin xyz="0 0 0" />
-      <mass value="2.8498940e-02" />
-      <inertia ixx="1.1175580e-05" ixy="-4.2369783e-11" ixz="-5.9381719e-09"
-               iyy="1.1192413e-05" iyz="-1.4400107e-11"
-               izz="2.0712558e-05" />
-      </inertial>
-  </link>
   <gazebo reference="wheel_right_link">
     <material>Gazebo/FlatBlack</material>
   </gazebo>
-<!-- ****************************************************** Caster Back Right Joint **************************************************  -->
-  <joint name="caster_back_right_joint" type="fixed">
-    <parent link="base_link"/>
-    <child link="caster_back_right_link"/>
-    <origin xyz="-0.177 -0.064 -0.004" rpy="-1.57 0 0"/>
-  </joint>
-<!-- ****************************************************** Caster Back Right Link ***************************************************  -->
-  <link name="caster_back_right_link">
-    <visual>
-      <geometry>
-        <sphere radius="0.007"/>
-      </geometry>
-      <material name="white"/>
-    </visual>
-    <collision>
-      <origin xyz="0 0.001 0" rpy="0 0 0"/>
-      <geometry>
-        <box size="0.030 0.009 0.020"/>
-      </geometry>
-    </collision>
-    <inertial>
-      <origin xyz="0 0 0" />
-      <mass value="0.005" />
-      <inertia ixx="0.001" ixy="0.0" ixz="0.0"
-               iyy="0.001" iyz="0.0"
-               izz="0.001" />
-    </inertial>
-  </link>
+<!-- ****************************************************** Caster Back Left Link ****************************************************  -->
   <gazebo reference="caster_back_link">
     <material>Gazebo/White</material>
   </gazebo>
-<!-- ****************************************************** Caster Back Left Joint ***************************************************  -->
-  <joint name="caster_back_left_joint" type="fixed">
-    <parent link="base_link"/>
-    <child link="caster_back_left_link"/>
-    <origin xyz="-0.177 0.064 -0.004" rpy="-1.57 0 0"/>
-  </joint>
-<!-- ****************************************************** Caster Back Left Link ****************************************************  -->
-  <link name="caster_back_left_link">
-    <visual>
-      <geometry>
-        <sphere radius="0.007"/>
-      </geometry>
-      <material name="white"/>
-    </visual>
-    <collision>
-      <origin xyz="0 0.001 0" rpy="0 0 0"/>
-      <geometry>
-        <box size="0.030 0.009 0.020"/>
-      </geometry>
-    </collision>
-    <inertial>
-      <origin xyz="0 0 0" />
-      <mass value="0.005" />
-      <inertia ixx="0.001" ixy="0.0" ixz="0.0"
-               iyy="0.001" iyz="0.0"
-               izz="0.001" />
-    </inertial>
-  </link>
-<!-- ****************************************************** IMU Joint ****************************************************************  -->
-  <joint name="imu_joint" type="fixed">
-    <parent link="base_link"/>
-    <child link="imu_link"/>
-    <origin xyz="0.0 0 0.068" rpy="0 0 0"/>
-  </joint>
-<!-- ****************************************************** IMU Link *****************************************************************  -->
-  <link name="imu_link"/>
-<!-- ****************************************************** Laser Scan Joint *********************************************************  -->
-  <joint name="scan_joint" type="fixed">
-    <parent link="base_link"/>
-    <child link="base_scan"/>
-    <origin xyz="-0.064 0 0.122" rpy="0 0 0"/>
-  </joint>
 <!-- ****************************************************** Laser Scan Link **********************************************************  -->
-  <link name="base_scan">
-    <visual>
-      <origin xyz="0 0 0" rpy="0 0 0"/>
-      <geometry>
-        <mesh filename="package://robot_gazebo/meshes/tb3/lds.stl" scale="0.001 0.001 0.001"/>
-      </geometry>
-      <material name="green"/>
-    </visual>
-    <collision>
-      <origin xyz="0.015 0 -0.0065" rpy="0 0 0"/>
-      <geometry>
-        <cylinder length="0.0315" radius="0.055"/>
-      </geometry>
-    </collision>
-    <inertial>
-      <mass value="0.114" />
-      <origin xyz="0 0 0" />
-      <inertia ixx="0.001" ixy="0.0" ixz="0.0"
-               iyy="0.001" iyz="0.0"
-               izz="0.001" />
-    </inertial>
-  </link>
   <gazebo reference="base_scan">
     <material>Gazebo/Green</material>
   </gazebo>
-<!-- ****************************************************** Camera Joint ************************************************************* -->
-  <joint name="camera_joint" type="fixed">
-    <origin xyz="0.064 -0.065 0.094" rpy="0 0 0"/>
-    <parent link="base_link"/>
-    <child link="camera_link"/>
-  </joint>
 <!-- ****************************************************** Camera Link **************************************************************  -->
-  <link name="camera_link">
-    <visual>
-     <origin xyz="0 0 0" rpy="1.57 0 1.57"/>
-      <geometry>
-       <mesh filename="package://robot_gazebo/meshes/tb3/r200.dae" />
-      </geometry>
-      <material name="green"/>
-    </visual>
-    <collision>
-      <origin xyz="0.003 0.065 0.007" rpy="0 0 0"/>
-      <geometry>
-        <box size="0.012 0.132 0.020"/>
-      </geometry>
-    </collision>
-  </link>
-<!-- ****************************************************** RGB Camera Joint *********************************************************  -->
-  <joint name="camera_rgb_joint" type="fixed">
-    <origin xyz="0.005 0.018 0.013" rpy="0 0 0"/>
-    <parent link="camera_link"/>
-    <child link="camera_rgb_frame"/>
-  </joint>
-<!-- ****************************************************** RGB Camera Frame Link ****************************************************  -->
-  <link name="camera_rgb_frame"/>
-<!-- ****************************************************** RGB Camera Optical Joint *************************************************  -->
-  <joint name="camera_rgb_optical_joint" type="fixed">
-    <origin xyz="0 0 0" rpy="-1.57 0 -1.57"/>
-    <parent link="camera_rgb_frame"/>
-    <child link="camera_rgb_optical_frame"/>
-  </joint>
-<!-- ****************************************************** RGB Camera Optical Link **************************************************  -->
-  <link name="camera_rgb_optical_frame"/>
-<!-- ****************************************************** Depth Camera Joint *******************************************************  -->
-  <joint name="camera_depth_joint" type="fixed">
-    <origin xyz="0.005 0.028 0.013" rpy="0 0 0"/>
-    <parent link="camera_link"/>
-    <child link="camera_depth_frame"/>
-  </joint>
-<!-- ****************************************************** Depth Camera Frame Link **************************************************  -->
-  <link name="camera_depth_frame"/>
-<!-- ****************************************************** Depth Camera Optical Frame Joint *****************************************  -->
-  <joint name="camera_depth_optical_joint" type="fixed">
-    <origin xyz="0 0 0" rpy="-1.57 0 -1.57"/>
-    <parent link="camera_depth_frame"/>
-    <child link="camera_depth_optical_frame"/>
-  </joint>
-<!-- ****************************************************** Depth Camera Optical Frame Link ******************************************  -->
-  <link name="camera_depth_optical_frame"/>
+  <gazebo reference="base_scan">
+    <material>Gazebo/Green</material>
+  </gazebo>
 <!-- *********************************************************************************************************************************  -->
 </robot>
