Commit message: u

File: gazebo/gz_tb3_waffle_pi.xacro (robot description, xacro)
@@ -5,238 +5,28 @@
 <!-- March 2022                                                                                                                         -->
 <!-- *********************************************************************************************************************************  -->
-<!-- ****************************************************** Import RVIZ Materials*****************************************************  -->
-  <xacro:include filename="$(find robot_gazebo)/xacro/common_rviz_materials.xacro" />
-<!-- ****************************************************** Base Footprint Link ******************************************************  -->
-  <link name="base_footprint"/>
-<!-- ****************************************************** Base Joint ***************************************************************  -->
-  <joint name="base_joint" type="fixed">
-    <parent link="base_footprint"/>
-    <child link="base_link" />
-    <origin xyz="0 0 0.010" rpy="0 0 0"/>
-  </joint>
 <!-- ****************************************************** Base Link ****************************************************************  -->
-  <link name="base_link">
-    <visual>
-      <origin xyz="-0.064 0 0.0" rpy="0 0 0"/>
-      <geometry>
-        <mesh filename="package://robot_gazebo/meshes/tb3/waffle_pi_base.stl" scale="0.001 0.001 0.001"/>
-      </geometry>
-      <material name="blue"/>
-    </visual>
-    <collision>
-      <origin xyz="-0.064 0 0.047" rpy="0 0 0"/>
-      <geometry>
-        <box size="0.266 0.266 0.094"/>
-      </geometry>
-    </collision>
-    <inertial>
-      <origin xyz="0 0 0" rpy="0 0 0"/>
-      <mass value="1.3729096e+00"/>
-      <inertia ixx="8.7002718e-03" ixy="-4.7576583e-05" ixz="1.1160499e-04"
-               iyy="8.6195418e-03" iyz="-3.5422299e-06"
-               izz="1.4612727e-02" />
-    </inertial>
-  </link>
   <gazebo reference="base_link">
     <material>Gazebo/Blue</material>
   </gazebo>
-<!-- ****************************************************** Wheel Left Joint *********************************************************  -->
-  <joint name="wheel_left_joint" type="continuous">
-    <parent link="base_link"/>
-    <child link="wheel_left_link"/>
-    <origin xyz="0.0 0.144 0.023" rpy="-1.57 0 0"/>
-    <axis xyz="0 0 1"/>
-  </joint>
 <!-- ****************************************************** Wheel Left Link **********************************************************  -->
-  <link name="wheel_left_link">
-    <visual>
-      <origin xyz="0 0 0" rpy="1.57 0 0"/>
-      <geometry>
-        <mesh filename="package://robot_gazebo/meshes/tb3/left_tire.stl" scale="0.001 0.001 0.001"/>
-      </geometry>
-      <material name="black"/>
-    </visual>
-    <collision>
-      <origin xyz="0 0 0" rpy="0 0 0"/>
-      <geometry>
-        <cylinder length="0.018" radius="0.033"/>
-      </geometry>
-    </collision>
-    <inertial>
-      <origin xyz="0 0 0" />
-      <mass value="2.8498940e-02" />
-      <inertia ixx="1.1175580e-05" ixy="-4.2369783e-11" ixz="-5.9381719e-09"
-               iyy="1.1192413e-05" iyz="-1.4400107e-11"
-               izz="2.0712558e-05" />
-      </inertial>
-  </link>
   <gazebo reference="wheel_left_link">
     <material>Gazebo/FlatBlack</material>
   </gazebo>
-<!-- ****************************************************** Wheel Right Joint ********************************************************  -->
-  <joint name="wheel_right_joint" type="continuous">
-    <parent link="base_link"/>
-    <child link="wheel_right_link"/>
-    <origin xyz="0.0 -0.144 0.023" rpy="-1.57 0 0"/>
-    <axis xyz="0 0 1"/>
-  </joint>
 <!-- ****************************************************** Wheel Right Link *********************************************************  -->
-  <link name="wheel_right_link">
-    <visual>
-      <origin xyz="0 0 0" rpy="1.57 0 0"/>
-      <geometry>
-        <mesh filename="package://robot_gazebo/meshes/tb3/right_tire.stl" scale="0.001 0.001 0.001"/>
-      </geometry>
-      <material name="black"/>
-    </visual>
-    <collision>
-      <origin xyz="0 0 0" rpy="0 0 0"/>
-      <geometry>
-        <cylinder length="0.018" radius="0.033"/>
-      </geometry>
-    </collision>
-    <inertial>
-      <origin xyz="0 0 0" />
-      <mass value="2.8498940e-02" />
-      <inertia ixx="1.1175580e-05" ixy="-4.2369783e-11" ixz="-5.9381719e-09"
-               iyy="1.1192413e-05" iyz="-1.4400107e-11"
-               izz="2.0712558e-05" />
-      </inertial>
-  </link>
   <gazebo reference="wheel_right_link">
     <material>Gazebo/FlatBlack</material>
   </gazebo>
-<!-- ****************************************************** Caster Back Right Joint **************************************************  -->
-  <joint name="caster_back_right_joint" type="fixed">
-    <parent link="base_link"/>
-    <child link="caster_back_right_link"/>
-    <origin xyz="-0.177 -0.064 -0.004" rpy="-1.57 0 0"/>
-  </joint>
 <!-- ****************************************************** Caster Back Right Link ***************************************************  -->
-  <link name="caster_back_right_link">
-    <visual>
-      <geometry>
-        <sphere radius="0.007"/>
-      </geometry>
-      <material name="white"/>
-    </visual>
-    <collision>
-      <origin xyz="0 0.001 0" rpy="0 0 0"/>
-      <geometry>
-        <box size="0.030 0.009 0.020"/>
-      </geometry>
-    </collision>
-    <inertial>
-      <origin xyz="0 0 0" />
-      <mass value="0.005" />
-      <inertia ixx="0.001" ixy="0.0" ixz="0.0"
-               iyy="0.001" iyz="0.0"
-               izz="0.001" />
-    </inertial>
-  </link>
   <gazebo reference="caster_back_right_link">
     <material>Gazebo/White</material>
   </gazebo>
-<!-- ****************************************************** Caster Back Left Joint ***************************************************  -->
-  <joint name="caster_back_left_joint" type="fixed">
-    <parent link="base_link"/>
-    <child link="caster_back_left_link"/>
-    <origin xyz="-0.177 0.064 -0.004" rpy="-1.57 0 0"/>
-  </joint>
 <!-- ****************************************************** Caster Back Left Link ****************************************************  -->
-  <link name="caster_back_left_link">
-    <visual>
-      <geometry>
-        <sphere radius="0.007"/>
-      </geometry>
-      <material name="white"/>
-    </visual>
-    <collision>
-      <origin xyz="0 0.001 0" rpy="0 0 0"/>
-      <geometry>
-        <box size="0.030 0.009 0.020"/>
-      </geometry>
-    </collision>
-    <inertial>
-      <origin xyz="0 0 0" />
-      <mass value="0.005" />
-      <inertia ixx="0.001" ixy="0.0" ixz="0.0"
-               iyy="0.001" iyz="0.0"
-               izz="0.001" />
-    </inertial>
-  </link>
   <gazebo reference="caster_back_left_link">
     <material>Gazebo/White</material>
   </gazebo>
-<!-- ****************************************************** IMU Joint ****************************************************************  -->
-  <joint name="imu_joint" type="fixed">
-    <parent link="base_link"/>
-    <child link="imu_link"/>
-    <origin xyz="0.0 0 0.068" rpy="0 0 0"/>
-  </joint>
-<!-- ****************************************************** IMU Link *****************************************************************  -->
-  <link name="imu_link"/>
-<!-- ****************************************************** Laser Scan Joint *********************************************************  -->
-  <joint name="scan_joint" type="fixed">
-    <parent link="base_link"/>
-    <child link="base_scan"/>
-    <origin xyz="-0.064 0 0.122" rpy="0 0 0"/>
-  </joint>
 <!-- ****************************************************** Laser Scan Link **********************************************************  -->
-  <link name="base_scan">
-    <visual>
-      <origin xyz="0 0 0.0" rpy="0 0 0"/>
-      <geometry>
-        <mesh filename="package://robot_gazebo/meshes/tb3/lds.stl" scale="0.001 0.001 0.001"/>
-      </geometry>
-      <material name="green"/>
-    </visual>
-    <collision>
-      <origin xyz="0.015 0 -0.0065" rpy="0 0 0"/>
-      <geometry>
-        <cylinder length="0.0315" radius="0.055"/>
-      </geometry>
-    </collision>
-    <inertial>
-      <mass value="0.114" />
-      <origin xyz="0 0 0" />
-      <inertia ixx="0.001" ixy="0.0" ixz="0.0"
-               iyy="0.001" iyz="0.0"
-               izz="0.001" />
-    </inertial>
-  </link>
   <gazebo reference="base_scan">
     <material>Gazebo/Green</material>
   </gazebo>
-<!-- ****************************************************** Camera Joint ************************************************************* -->
-  <joint name="camera_joint" type="fixed">
-    <origin xyz="0.073 -0.011 0.084" rpy="0 0 0"/>
-    <parent link="base_link"/>
-    <child link="camera_link"/>
-  </joint>
-<!-- ****************************************************** Camera Link **************************************************************  -->
-  <link name="camera_link">
-    <collision>
-      <origin xyz="0.005 0.011 0.013" rpy="0 0 0"/>
-      <geometry>
-        <box size="0.015 0.030 0.027"/>
-      </geometry>
-    </collision>
-  </link>
-<!-- ****************************************************** RGB Camera Joint *********************************************************  -->
-  <joint name="camera_rgb_joint" type="fixed">
-    <origin xyz="0.003 0.011 0.009" rpy="0 0 0"/>
-    <parent link="camera_link"/>
-    <child link="camera_rgb_frame"/>
-  </joint>
-<!-- ****************************************************** RGB Camera Frame Link ****************************************************  -->
-  <link name="camera_rgb_frame"/>
-<!-- ****************************************************** RGB Camera Optical Joint *************************************************  -->
-  <joint name="camera_rgb_optical_joint" type="fixed">
-    <origin xyz="0 0 0" rpy="-1.57 0 -1.57"/>
-    <parent link="camera_rgb_frame"/>
-    <child link="camera_rgb_optical_frame"/>
-  </joint>
-  <link name="camera_rgb_optical_frame"/>
 <!-- *********************************************************************************************************************************  -->
 </robot>

File: xacro/tb3_burger.xacro (robot description, xacro)
@@ -5,6 +5,7 @@
 <!-- March 2022                                                                                                                         -->
 <!-- *********************************************************************************************************************************  -->
-<!-- ****************************************************** Import RVIZ Materials*****************************************************  -->
-  <xacro:include filename="$(find robot_gazebo)/xacro/common_rviz_materials.xacro" />
+<!-- ****************************************************** Includes *****************************************************************  -->
+  <xacro:include filename="$(find robot_gazebo)/xacro/common_rviz_materials.xacro" />   <!-- RVIZ Colors                                -->
+  <xacro:include filename="$(find robot_gazebo)/gazebo/gz_tb3_burger.xacro" />          <!-- Gazebo                                     -->
 <!-- ****************************************************** Base Footprint Link ******************************************************  -->
   <link name="base_footprint"/>
@@ -38,7 +39,4 @@
     </inertial>
   </link>
-  <gazebo reference="base_link">
-    <material>Gazebo/Blue</material>
-  </gazebo>
 <!-- ****************************************************** Wheel Left Joint *********************************************************  -->
   <joint name="wheel_left_joint" type="continuous">
@@ -71,7 +69,4 @@
     </inertial>
   </link>
-  <gazebo reference="wheel_left_link">
-    <material>Gazebo/FlatBlack</material>
-  </gazebo>
 <!-- ****************************************************** Wheel Right Joint ********************************************************  -->
   <joint name="wheel_right_joint" type="continuous">
@@ -83,5 +78,5 @@
 <!-- ****************************************************** Wheel Right Link *********************************************************  -->
   <link name="wheel_right_link">
-    <visual>
+      <visual>
       <origin xyz="0 0 0" rpy="1.57 0 0"/>
       <geometry>
@@ -104,7 +99,4 @@
     </inertial>
   </link>
-  <gazebo reference="wheel_right_link">
-    <material>Gazebo/FlatBlack</material>
-  </gazebo>
 <!-- ****************************************************** Caster Back Joint ********************************************************  -->
   <joint name="caster_back_joint" type="fixed">
@@ -135,7 +127,4 @@
     </inertial>
   </link>
-  <gazebo reference="caster_back_link">
-    <material>Gazebo/White</material>
-  </gazebo>
 <!-- ****************************************************** IMU Joint ****************************************************************  -->
   <joint name="imu_joint" type="fixed">
@@ -175,7 +164,4 @@
     </inertial>
   </link>
-  <gazebo reference="base_scan">
-    <material>Gazebo/Green</material>
-  </gazebo>
 <!-- *********************************************************************************************************************************  -->
 </robot>

File: xacro/tb3_waffle.xacro (robot description, xacro)
@@ -5,6 +5,7 @@
 <!-- March 2022                                                                                                                         -->
 <!-- *********************************************************************************************************************************  -->
-<!-- ****************************************************** Import RVIZ Materials*****************************************************  -->
-  <xacro:include filename="$(find robot_gazebo)/xacro/common_rviz_materials.xacro" />
+<!-- ****************************************************** Includes *****************************************************************  -->
+  <xacro:include filename="$(find robot_gazebo)/xacro/common_rviz_materials.xacro" />   <!-- RVIZ Colors                                -->
+  <xacro:include filename="$(find robot_gazebo)/gazebo/gz_tb3_affle.xacro" />           <!-- Gazebo                                     -->
 <!-- ****************************************************** Base Footprint Link ******************************************************  -->
   <link name="base_footprint"/>

File: xacro/tb3_waffle_pi.xacro (robot description, xacro)
@@ -5,6 +5,7 @@
 <!-- March 2022                                                                                                                         -->
 <!-- *********************************************************************************************************************************  -->
-<!-- ****************************************************** Import RVIZ Materials*****************************************************  -->
-  <xacro:include filename="$(find robot_gazebo)/xacro/common_rviz_materials.xacro" />
+<!-- ****************************************************** Includes *****************************************************************  -->
+  <xacro:include filename="$(find robot_gazebo)/xacro/common_rviz_materials.xacro" />   <!-- RVIZ Colors                                -->
+  <xacro:include filename="$(find robot_gazebo)/gazebo/gz_tb3_waffle_pi.xacro" />       <!-- Gazebo                                     -->
 <!-- ****************************************************** Base Footprint Link ******************************************************  -->
   <link name="base_footprint"/>
@@ -38,7 +39,4 @@
     </inertial>
   </link>
-  <gazebo reference="base_link">
-    <material>Gazebo/Blue</material>
-  </gazebo>
 <!-- ****************************************************** Wheel Left Joint *********************************************************  -->
   <joint name="wheel_left_joint" type="continuous">
@@ -71,7 +69,4 @@
       </inertial>
   </link>
-  <gazebo reference="wheel_left_link">
-    <material>Gazebo/FlatBlack</material>
-  </gazebo>
 <!-- ****************************************************** Wheel Right Joint ********************************************************  -->
   <joint name="wheel_right_joint" type="continuous">
@@ -104,7 +99,4 @@
       </inertial>
   </link>
-  <gazebo reference="wheel_right_link">
-    <material>Gazebo/FlatBlack</material>
-  </gazebo>
 <!-- ****************************************************** Caster Back Right Joint **************************************************  -->
   <joint name="caster_back_right_joint" type="fixed">
@@ -135,7 +127,4 @@
     </inertial>
   </link>
-  <gazebo reference="caster_back_right_link">
-    <material>Gazebo/White</material>
-  </gazebo>
 <!-- ****************************************************** Caster Back Left Joint ***************************************************  -->
   <joint name="caster_back_left_joint" type="fixed">
@@ -166,7 +155,4 @@
     </inertial>
   </link>
-  <gazebo reference="caster_back_left_link">
-    <material>Gazebo/White</material>
-  </gazebo>
 <!-- ****************************************************** IMU Joint ****************************************************************  -->
   <joint name="imu_joint" type="fixed">
@@ -206,7 +192,4 @@
     </inertial>
   </link>
-  <gazebo reference="base_scan">
-    <material>Gazebo/Green</material>
-  </gazebo>
 <!-- ****************************************************** Camera Joint ************************************************************* -->
   <joint name="camera_joint" type="fixed">
