Commit message: u

File: gazebo/gz_bocbot.xacro (robot description, xacro)
@@ -1,4 +1,13 @@
 <?xml version="1.0"?>
 <robot>
+  <gazebo reference="chassis">
+    <material>Gazebo/Blue</material>
+  </gazebo>
+  <gazebo reference="camera">
+    <material>Gazebo/Red</material>
+  </gazebo>
+  <gazebo reference="hokuyo">
+    <material>Gazebo/Black</material>
+  </gazebo>
   <!--skid_steer_drive_controller-->
   <gazebo>

File: xacro/bocbot.xacro (robot description, xacro)
@@ -1,6 +1,14 @@
 <?xml version='1.0'?>
-<robot name="bocbot"
-  xmlns:xacro="http://www.ros.org/wiki/xacro">
-  <xacro:include filename="bocbot.gazebo" />
+<robot name="bocbot" xmlns:xacro="http://www.ros.org/wiki/xacro">
+<!-- ****************************************************** diffbot Robot ************************************************************  -->
+<!-- Muthanna Alwahash                                                                                                                  -->
+<!-- March 2022                                                                                                                         -->
+<!-- *********************************************************************************************************************************  -->
+<!-- ****************************************************** Parameters ***************************************************************  -->
+  <xacro:property name="mesh_path"      value="package://robot_gazebo/meshes/bocbot/"/>
+<!-- ****************************************************** Includes *****************************************************************  -->
+  <xacro:include filename="$(find robot_gazebo)/xacro/common_rviz_materials.xacro" />   <!-- RVIZ Colors                                -->
+  <xacro:include filename="$(find robot_gazebo)/gazebo/gz_bocbot.xacro" />              <!-- Gazebo                                     -->
+<!-- ****************************************************** Base Footprint ***********************************************************  -->
   <link name="robot_footprint"></link>
   <joint name="robot_footprint_joint" type="fixed">
@@ -133,6 +141,6 @@
       <origin xyz="0 0 0" rpy="0 0 0" />
       <geometry>
-        <!-- <mesh filename="$(find bocbot)/meshes/hokuyo.dae"/> -->
-        <box size="0.05 0.05 0.05"/>
+        <mesh filename="${mesh_path}hokuyo.dae"/>
+        <!-- <box size="0.05 0.05 0.05"/> -->
       </geometry>
     </visual>
@@ -188,12 +196,3 @@
     <axis xyz="0 1 0" rpy="0 0 0"/>
   </joint>
-  <gazebo reference="chassis">
-    <material>Gazebo/Blue</material>
-  </gazebo>
-  <gazebo reference="camera">
-    <material>Gazebo/Red</material>
-  </gazebo>
-  <gazebo reference="hokuyo">
-    <material>Gazebo/Black</material>
-  </gazebo>
 </robot>

Commit message: u

File: gazebo/gz_bocbot.xacro (robot description, xacro)
@@ -4,9 +4,21 @@
     <material>Gazebo/Blue</material>
   </gazebo>
+  <gazebo reference="front_left_wheel">
+    <material>Gazebo/Gray</material>
+  </gazebo>
+  <gazebo reference="back_left_wheel">
+    <material>Gazebo/Gray</material>
+  </gazebo>
+  <gazebo reference="front_right_wheel">
+    <material>Gazebo/Gray</material>
+  </gazebo>
+  <gazebo reference="back_right_wheel">
+    <material>Gazebo/Gray</material>
+  </gazebo>
   <gazebo reference="camera">
-    <material>Gazebo/Red</material>
+    <material>Gazebo/Green</material>
   </gazebo>
   <gazebo reference="hokuyo">
-    <material>Gazebo/Black</material>
+    <material>Gazebo/Red</material>
   </gazebo>
   <!--skid_steer_drive_controller-->

File: xacro/bocbot.xacro (robot description, xacro)
@@ -35,4 +35,5 @@
         <box size=".4 .2 .1"/>
       </geometry>
+      <material name="blue"/>
     </visual>
   </link>
@@ -48,4 +49,5 @@
         <cylinder length="0.05" radius="0.1"/>
       </geometry>
+      <material name="grey"/>
     </visual>
     <collision>
@@ -67,4 +69,5 @@
         <cylinder length="0.05" radius="0.1"/>
       </geometry>
+      <material name="grey"/>
     </visual>
     <collision>
@@ -86,4 +89,5 @@
         <cylinder length="0.05" radius="0.1"/>
       </geometry>
+      <material name="grey"/>
     </visual>
     <collision>
@@ -105,4 +109,5 @@
         <cylinder length="0.05" radius="0.1"/>
       </geometry>
+      <material name="grey"/>
     </visual>
     <collision>
@@ -124,4 +129,5 @@
         <box size="0.05 0.05 0.05"/>
       </geometry>
+      <material name="green"/>
     </visual>
     <collision name="camera_colision">
@@ -144,4 +150,5 @@
         <!-- <box size="0.05 0.05 0.05"/> -->
       </geometry>
+      <material name="red"/>
     </visual>
     <collision name="hokuyo_colision">

Commit message: u

File: gazebo/gz_bocbot.xacro (robot description, xacro)
@@ -1,5 +1,9 @@
 <?xml version="1.0"?>
-<robot>
-  <gazebo reference="chassis">
+<robot name="bocbot" xmlns:xacro="http://www.ros.org/wiki/xacro">
+<!-- ****************************************************** bocbot Robot *************************************************************  -->
+<!-- Muthanna Alwahash                                                                                                                  -->
+<!-- March 2022                                                                                                                         -->
+<!-- *********************************************************************************************************************************  -->
+  <gazebo reference="base">
     <material>Gazebo/Blue</material>
   </gazebo>
@@ -22,4 +26,5 @@
     <material>Gazebo/Red</material>
   </gazebo>
+<!-- ******************************************************  *************************************************************************  -->
   <!--skid_steer_drive_controller-->
   <gazebo>
@@ -41,5 +46,5 @@
       <wheel_separation>0.4</wheel_separation>
       <wheel_diameter>0.2</wheel_diameter>
-      <robot_base_frame>robot_footprint</robot_base_frame>
+      <robot_base_frame>footprint</robot_base_frame>
       <max_wheel_torque>20</max_wheel_torque>
       <publish_odom>true</publish_odom>
@@ -49,4 +54,5 @@
     </plugin>
   </gazebo>
+<!-- ******************************************************  *************************************************************************  -->
   <!-- camera -->
   <gazebo reference="camera">
@@ -86,4 +92,5 @@
     </sensor>
   </gazebo>
+<!-- ******************************************************  *************************************************************************  -->
   <!-- hokuyo -->
   <gazebo reference="hokuyo">
@@ -126,3 +133,4 @@
     </sensor>
   </gazebo>
+<!-- ******************************************************  *************************************************************************  -->
 </robot>

File: xacro/bocbot.xacro (robot description, xacro)
@@ -1,5 +1,5 @@
 <?xml version='1.0'?>
 <robot name="bocbot" xmlns:xacro="http://www.ros.org/wiki/xacro">
-<!-- ****************************************************** diffbot Robot ************************************************************  -->
+<!-- ****************************************************** bocbot Robot *************************************************************  -->
 <!-- Muthanna Alwahash                                                                                                                  -->
 <!-- March 2022                                                                                                                         -->
@@ -11,11 +11,7 @@
   <xacro:include filename="$(find robot_gazebo)/gazebo/gz_bocbot.xacro" />              <!-- Gazebo                                     -->
 <!-- ****************************************************** Base Footprint ***********************************************************  -->
-  <link name="robot_footprint"></link>
-  <joint name="robot_footprint_joint" type="fixed">
-    <origin xyz="0 0 0" rpy="0 0 0" />
-    <parent link="robot_footprint"/>
-    <child link="chassis" />
-  </joint>
-  <link name='chassis'>
+  <link name="footprint"></link>
+<!-- ******************************************************  *************************************************************************  -->
+  <link name='base'>
     <pose>0 0 0.1 0 0 0</pose>
     <inertial>
@@ -30,5 +26,5 @@
       </geometry>
     </collision>
-    <visual name='chassis_visual'>
+    <visual name='base_visual'>
       <origin xyz="0 0 0" rpy=" 0 0 0"/>
       <geometry>
@@ -38,4 +34,5 @@
     </visual>
   </link>
+<!-- ******************************************************  *************************************************************************  -->
   <link name="front_left_wheel">
     <inertial>
@@ -58,4 +55,5 @@
     </collision>
   </link>
+<!-- ******************************************************  *************************************************************************  -->
   <link name="back_left_wheel">
     <inertial>
@@ -78,4 +76,5 @@
     </collision>
   </link>
+<!-- ******************************************************  *************************************************************************  -->
   <link name="front_right_wheel">
     <inertial>
@@ -98,4 +97,5 @@
     </collision>
   </link>
+<!-- ******************************************************  *************************************************************************  -->
   <link name="back_right_wheel">
     <inertial>
@@ -118,4 +118,5 @@
     </collision>
   </link>
+<!-- ******************************************************  *************************************************************************  -->
   <link name="camera">
     <inertial>
@@ -138,4 +139,5 @@
     </collision>
   </link>
+<!-- ******************************************************  *************************************************************************  -->
   <link name="hokuyo">
     <inertial>
@@ -159,47 +161,60 @@
     </collision>
   </link>
+<!-- ******************************************************  *************************************************************************  -->
+  <joint type="fixed" name="footprint_joint" >
+    <origin xyz="0 0 0" rpy="0 0 0" />
+    <parent link="footprint"/>
+    <child link="base" />
+  </joint>
+<!-- ******************************************************  *************************************************************************  -->
   <joint type="continuous" name="front_left_wheel_joint">
     <origin xyz="0.12 0.15 0" rpy="0 0 0"/>
     <child link="front_left_wheel"/>
-    <parent link="chassis"/>
-    <axis xyz="0 1 0" rpy="0 0 0"/>
-    <limit effort="10000" velocity="1000"/>
-    <dynamics damping="1.0" friction="1.0"/>
-  </joint>
+    <parent link="base"/>
+    <axis xyz="0 1 0" rpy="0 0 0"/>
+    <limit effort="10000" velocity="1000"/>
+    <dynamics damping="1.0" friction="1.0"/>
+  </joint>
+<!-- ******************************************************  *************************************************************************  -->
   <joint type="continuous" name="front_right_wheel_joint">
     <origin xyz="0.12 -0.15 0" rpy="0 0 0"/>
     <child link="front_right_wheel"/>
-    <parent link="chassis"/>
-    <axis xyz="0 1 0" rpy="0 0 0"/>
-    <limit effort="10000" velocity="1000"/>
-    <dynamics damping="1.0" friction="1.0"/>
-  </joint>
+    <parent link="base"/>
+    <axis xyz="0 1 0" rpy="0 0 0"/>
+    <limit effort="10000" velocity="1000"/>
+    <dynamics damping="1.0" friction="1.0"/>
+  </joint>
+<!-- ******************************************************  *************************************************************************  -->
   <joint type="continuous" name="back_left_wheel_joint">
     <origin xyz="-0.12 0.15 0" rpy="0 0 0"/>
     <child link="back_left_wheel"/>
-    <parent link="chassis"/>
-    <axis xyz="0 1 0" rpy="0 0 0"/>
-    <limit effort="10000" velocity="1000"/>
-    <dynamics damping="1.0" friction="1.0"/>
-  </joint>
+    <parent link="base"/>
+    <axis xyz="0 1 0" rpy="0 0 0"/>
+    <limit effort="10000" velocity="1000"/>
+    <dynamics damping="1.0" friction="1.0"/>
+  </joint>
+<!-- ******************************************************  *************************************************************************  -->
   <joint type="continuous" name="back_right_wheel_joint">
     <origin xyz="-0.12 -0.15 0" rpy="0 0 0"/>
     <child link="back_right_wheel"/>
-    <parent link="chassis"/>
-    <axis xyz="0 1 0" rpy="0 0 0"/>
-    <limit effort="10000" velocity="1000"/>
-    <dynamics damping="1.0" friction="1.0"/>
-  </joint>
+    <parent link="base"/>
+    <axis xyz="0 1 0" rpy="0 0 0"/>
+    <limit effort="10000" velocity="1000"/>
+    <dynamics damping="1.0" friction="1.0"/>
+  </joint>
+<!-- ******************************************************  *************************************************************************  -->
   <joint type="fixed" name="camera_joint">
     <origin xyz="0.2 0 0" rpy="0 0 0"/>
     <child link="camera"/>
-    <parent link="chassis"/>
-    <axis xyz="0 1 0" rpy="0 0 0"/>
-  </joint>
+    <parent link="base"/>
+    <axis xyz="0 1 0" rpy="0 0 0"/>
+  </joint>
+<!-- ******************************************************  *************************************************************************  -->
   <joint type="fixed" name="hokuyo_joint">
     <origin xyz="0.15 0 0.1" rpy="0 0 0"/>
     <child link="hokuyo"/>
-    <parent link="chassis"/>
-    <axis xyz="0 1 0" rpy="0 0 0"/>
-  </joint>
+    <parent link="base"/>
+    <axis xyz="0 1 0" rpy="0 0 0"/>
+  </joint>
+<!-- ******************************************************  *************************************************************************  -->
 </robot>

Commit message: u

File: gazebo/gz_bocbot.xacro (robot description, xacro)
@@ -5,24 +5,23 @@
 <!-- March 2022                                                                                                                         -->
 <!-- *********************************************************************************************************************************  -->
+<!-- ******************************************************  *************************************************************************  -->
   <gazebo reference="base">
     <material>Gazebo/Blue</material>
   </gazebo>
+<!-- ******************************************************  *************************************************************************  -->
   <gazebo reference="front_left_wheel">
     <material>Gazebo/Gray</material>
   </gazebo>
+<!-- ******************************************************  *************************************************************************  -->
   <gazebo reference="back_left_wheel">
     <material>Gazebo/Gray</material>
   </gazebo>
+<!-- ******************************************************  *************************************************************************  -->
   <gazebo reference="front_right_wheel">
     <material>Gazebo/Gray</material>
   </gazebo>
+<!-- ******************************************************  *************************************************************************  -->
   <gazebo reference="back_right_wheel">
     <material>Gazebo/Gray</material>
-  </gazebo>
-  <gazebo reference="camera">
-    <material>Gazebo/Green</material>
-  </gazebo>
-  <gazebo reference="hokuyo">
-    <material>Gazebo/Red</material>
   </gazebo>
 <!-- ******************************************************  *************************************************************************  -->
@@ -91,4 +90,5 @@
       </plugin>
     </sensor>
+    <material>Gazebo/Green</material>
   </gazebo>
 <!-- ******************************************************  *************************************************************************  -->
@@ -132,4 +132,5 @@
       </plugin>
     </sensor>
+    <material>Gazebo/Red</material>
   </gazebo>
 <!-- ******************************************************  *************************************************************************  -->

Commit message: u

File: gazebo/gz_bocbot.xacro (robot description, xacro)
@@ -25,6 +25,5 @@
     <material>Gazebo/Gray</material>
   </gazebo>
-<!-- ******************************************************  *************************************************************************  -->
-  <!--skid_steer_drive_controller-->
+<!-- ******************************************************  Skid Steer Drive Controller *********************************************  -->
   <gazebo>
     <plugin name="skid_steer_drive_controller" filename="libgazebo_ros_diff_drive.so">
@@ -53,8 +52,17 @@
     </plugin>
   </gazebo>
-<!-- ******************************************************  *************************************************************************  -->
-  <!-- camera -->
+<!-- ******************************************************  Camera ******************************************************************  -->
   <gazebo reference="camera">
     <sensor type="camera" name="camera_sensor">
+      <plugin name="camera_controller" filename="libgazebo_ros_camera.so">
+        <ros>
+          <namespace>/bocbot</namespace>
+          <argument>camera/image_raw:=/bocbot/camera/image</argument>
+          <argument>camera/camera_info:=/bocbot/camera/image/camera_info</argument>
+        </ros>
+        <camera_name>camera</camera_name>
+        <frame_name>camera</frame_name>
+        <hack_baseline>0.07</hack_baseline>
+      </plugin>
       <update_rate>30.0</update_rate>
       <always_on>1</always_on>
@@ -79,19 +87,8 @@
         </distortion>
       </camera>
-      <plugin name="camera_controller" filename="libgazebo_ros_camera.so">
-        <ros>
-          <namespace>/bocbot</namespace>
-          <argument>camera/image_raw:=/bocbot/camera/image</argument>
-          <argument>camera/camera_info:=/bocbot/camera/image/camera_info</argument>
-        </ros>
-        <camera_name>camera</camera_name>
-        <frame_name>camera</frame_name>
-        <hack_baseline>0.07</hack_baseline>
-      </plugin>
     </sensor>
     <material>Gazebo/Green</material>
   </gazebo>
-<!-- ******************************************************  *************************************************************************  -->
-  <!-- hokuyo -->
+<!-- ****************************************************** hokuyo  ******************************************************************  -->
   <gazebo reference="hokuyo">
     <sensor type="ray" name="head_hokuyo_sensor">
@@ -113,10 +110,8 @@
           <resolution>0.01</resolution>
         </range>
+<!-- Noise parameters based on published spec for Hokuyo laser achieving "+-30mm" accuracy at range < 10m.  A mean of 0.0m and stddev   -->
+<!-- of 0.01m will put 99.7% of samples within 0.03m of the true reading.                                                               -->
         <noise>
           <type>gaussian</type>
-          <!-- Noise parameters based on published spec for Hokuyo laser
-                achieving "+-30mm" accuracy at range < 10m.  A mean of 0.0m and
-                stddev of 0.01m will put 99.7% of samples within 0.03m of the true
-                reading. -->
           <mean>0.0</mean>
           <stddev>0.01</stddev>
@@ -134,4 +129,4 @@
     <material>Gazebo/Red</material>
   </gazebo>
-<!-- ******************************************************  *************************************************************************  -->
+<!-- ****************************************************** end **********************************************************************  -->
 </robot>

File: urdf/bocbot.urdf (robot description, URDF)
Before this commit: robot bocbot, 8 links, 7 joints
Links:
- removed link chassis
- removed link robot_footprint
- added link base, mass 15.0; collision box size=.4 .2 .1; visual box size=.4 .2 .1
- added link footprint
Joints:
- removed joint robot_footprint_joint
- added joint footprint_joint: type fixed, parent footprint, child base, origin xyz=0 0 0 rpy=0 0 0
- joint back_left_wheel_joint: parent chassis -> base
- joint back_right_wheel_joint: parent chassis -> base
- joint camera_joint: parent chassis -> base
- joint front_left_wheel_joint: parent chassis -> base
- joint front_right_wheel_joint: parent chassis -> base
- joint hokuyo_joint: parent chassis -> base
