Commit message: u

File: gazebo/gz_bocbot.xacro (robot description, xacro)
@@ -44,12 +44,15 @@
       </ros>
       <update_rate>100.0</update_rate>
+      <odometry_frame>odom</odometry_frame>
       <num_wheel_pairs>2</num_wheel_pairs>
-      <odometry_frame>odom</odometry_frame>
       <left_joint>front_left_wheel_joint</left_joint>
+      <right_joint>front_right_wheel_joint</right_joint>
+      <wheel_separation>0.4</wheel_separation>
+      <wheel_diameter>"${(wheel_radius*2)}</wheel_diameter>
+      <max_wheel_torque>20</max_wheel_torque>
       <left_joint>back_left_wheel_joint</left_joint>
-      <right_joint>front_right_wheel_joint</right_joint>
       <right_joint>back_right_wheel_joint</right_joint>
       <wheel_separation>0.4</wheel_separation>
-      <wheel_diameter>0.2</wheel_diameter>
+      <wheel_diameter>"${(wheel_radius*2)}</wheel_diameter>
       <max_wheel_torque>20</max_wheel_torque>
       <robot_base_frame>footprint</robot_base_frame>
@@ -63,5 +66,5 @@
   <gazebo reference="camera">
     <sensor type="camera" name="camera_sensor">
-      <plugin name="camera_controller" filename="libgazebo_ros_camera.so">
+      <plugin name="camera" filename="libgazebo_ros_camera.so">
         <ros>
           <namespace>bocbot</namespace>
@@ -101,7 +104,14 @@
   <gazebo reference="hokuyo">
     <sensor type="ray" name="head_hokuyo_sensor">
+      <plugin name="hokuyo" filename="libgazebo_ros_ray_sensor.so">
+        <ros>
+          <namespace>bocbot</namespace>
+          <argument>--remap ~/out:=scan</argument>
+        </ros>
+        <output_type>sensor_msgs/LaserScan</output_type>
+      </plugin>
+      <update_rate>30</update_rate>
       <pose>0 0 0 0 0 0</pose>
       <visualize>false</visualize>
-      <update_rate>40</update_rate>
       <ray>
         <scan>
@@ -126,12 +136,4 @@
         </noise>
       </ray>
-      <update_rate>30</update_rate>
-      <plugin name="gazebo_ros_head_hokuyo_controller" filename="libgazebo_ros_ray_sensor.so">
-        <ros>
-          <namespace>bocbot</namespace>
-          <argument>--remap ~/out:=scan</argument>
-        </ros>
-        <output_type>sensor_msgs/LaserScan</output_type>
-      </plugin>
     </sensor>
     <material>Gazebo/Red</material>

File: urdf/bocbot.urdf (robot description, URDF)
Before this commit: robot bocbot, 8 links, 7 joints
Links:
- link hokuyo: mass 1e-5 -> 1e-05; geometry collision mesh filename=package://robot_gazebo/meshes/bocbot/hokuyo.dae; visual mesh filename=package://robot_gazebo/meshes/bocbot/hokuyo.dae

File: xacro/bocbot.xacro (robot description, xacro)
@@ -29,5 +29,11 @@
 <!-- ****************************************************** Base Footprint ***********************************************************  -->
   <link name="footprint"></link>
-<!-- ****************************************************** Base *********************************************************************  -->
+<!-- ****************************************************** Footprint Joint **********************************************************  -->
+  <joint type="fixed" name="footprint_joint" >
+    <origin xyz="0 0 0" rpy="0 0 0" />
+    <parent link="footprint"/>
+    <child link="base" />
+  </joint>
+<!-- ****************************************************** Base Link ****************************************************************  -->
   <link name='base'>
     <pose>0 0 0.1 0 0 0</pose>
@@ -51,89 +57,44 @@
     </visual>
   </link>
-<!-- ****************************************************** Front Left Wheel *********************************************************  -->
-  <link name="front_left_wheel">
-    <inertial>
-      <mass value="${base_mass}"/>
-      <origin xyz="0 0 0" rpy=" 0 ${radians(90)} ${radians(90)}"/>
-      <inertia ixx="0.1" ixy="0" ixz="0" iyy="0.1" iyz="0" izz="0.1" />
-    </inertial>
-    <visual>
-      <origin xyz="0 0 0" rpy=" 0 ${radians(90)} ${radians(90)}"/>
-      <geometry>
-        <cylinder length="${wheel_width}" radius="${wheel_radius}"/>
-      </geometry>
-      <material name="grey"/>
-    </visual>
-    <collision>
-      <origin xyz="0 0 0" rpy=" 0 ${radians(90)} ${radians(90)}"/>
-      <geometry>
-        <cylinder length="${wheel_width}" radius="${wheel_radius}"/>
-      </geometry>
-    </collision>
-  </link>
-<!-- ****************************************************** Back Left Wheel **********************************************************  -->
-  <link name="back_left_wheel">
-    <inertial>
-      <mass value="${base_mass}"/>
-      <origin xyz="0 0 0" rpy=" 0 ${radians(90)} ${radians(90)}"/>
-      <inertia ixx="0.1" ixy="0" ixz="0" iyy="0.1" iyz="0" izz="0.1" />
-    </inertial>
-    <visual>
-      <origin xyz="0 0 0" rpy=" 0 ${radians(90)} ${radians(90)}"/>
-      <geometry>
-        <cylinder length="${wheel_width}" radius="${wheel_radius}"/>
-      </geometry>
-      <material name="grey"/>
-    </visual>
-    <collision>
-      <origin xyz="0 0 0" rpy=" 0 ${radians(90)} ${radians(90)}"/>
-      <geometry>
-        <cylinder length="${wheel_width}" radius="${wheel_radius}"/>
-      </geometry>
-    </collision>
-  </link>
-<!-- ****************************************************** Front Right Wheel ********************************************************  -->
-  <link name="front_right_wheel">
-    <inertial>
-      <mass value="${base_mass}"/>
-      <origin xyz="0 0 0" rpy=" 0 ${radians(90)} ${radians(90)}"/>
-      <inertia ixx="0.1" ixy="0" ixz="0" iyy="0.1" iyz="0" izz="0.1" />
-    </inertial>
-    <visual>
-      <origin xyz="0 0 0" rpy=" 0 ${radians(90)} ${radians(90)}"/>
-      <geometry>
-        <cylinder length="${wheel_width}" radius="${wheel_radius}"/>
-      </geometry>
-      <material name="grey"/>
-    </visual>
-    <collision>
-      <origin xyz="0 0 0" rpy=" 0 ${radians(90)} ${radians(90)}"/>
-      <geometry>
-        <cylinder length="${wheel_width}" radius="${wheel_radius}"/>
-      </geometry>
-    </collision>
-  </link>
-<!-- ****************************************************** Back Right Wheel *********************************************************  -->
-  <link name="back_right_wheel">
-    <inertial>
-      <mass value="${base_mass}"/>
-      <origin xyz="0 0 0" rpy=" 0 ${radians(90)} ${radians(90)}"/>
-      <inertia ixx="0.1" ixy="0" ixz="0" iyy="0.1" iyz="0" izz="0.1" />
-    </inertial>
-    <visual>
-      <origin xyz="0 0 0" rpy=" 0 ${radians(90)} ${radians(90)}"/>
-      <geometry>
-        <cylinder length="${wheel_width}" radius="${wheel_radius}"/>
-      </geometry>
-      <material name="grey"/>
-    </visual>
-    <collision>
-      <origin xyz="0 0 0" rpy=" 0 ${radians(90)} ${radians(90)}"/>
-      <geometry>
-        <cylinder length="${wheel_width}" radius="${wheel_radius}"/>
-      </geometry>
-    </collision>
-  </link>
-<!-- ****************************************************** Camera *******************************************************************  -->
+<!-- ****************************************************** Wheels Macro *************************************************************  -->
+  <xacro:macro name="wheel" params="position side x y">
+<!-- ****************************************************** Wheel Link ***************************************************************  -->
+    <link name="${position}_${side}_wheel">
+      <inertial>
+        <mass value="${base_mass}"/>
+        <origin xyz="0 0 0" rpy=" 0 ${radians(90)} ${radians(90)}"/>
+        <inertia ixx="0.1" ixy="0" ixz="0" iyy="0.1" iyz="0" izz="0.1" />
+      </inertial>
+      <visual>
+        <origin xyz="0 0 0" rpy=" 0 ${radians(90)} ${radians(90)}"/>
+        <geometry>
+          <cylinder length="${wheel_width}" radius="${wheel_radius}"/>
+        </geometry>
+        <material name="grey"/>
+      </visual>
+      <collision>
+        <origin xyz="0 0 0" rpy=" 0 ${radians(90)} ${radians(90)}"/>
+        <geometry>
+          <cylinder length="${wheel_width}" radius="${wheel_radius}"/>
+        </geometry>
+      </collision>
+    </link>
+<!-- ****************************************************** Wheel Joint **************************************************************  -->
+    <joint type="continuous" name="${position}_${side}_wheel_joint">
+        <origin xyz="${x} ${y} 0.15 0" rpy="0 0 0"/>
+        <child link="front_left_wheel"/>
+        <parent link="base"/>
+        <axis xyz="0 1 0" rpy="0 0 0"/>
+        <limit effort="10000" velocity="1000"/>
+        <dynamics damping="1.0" friction="1.0"/>
+    </joint>
+<!-- ****************************************************** End of Macro *************************************************************  -->
+  </xacro:macro>
+<!-- ****************************************************** Expand Wheels Macro ******************************************************  -->
+<xacro:wheel position="front" side="right" x=" 0.12" y="-0.15" />
+<xacro:wheel position="front" side="left"  x=" 0.12" y=" 0.15" />
+<xacro:wheel position="back"  side="right" x="-0.12" y="-0.15" />
+<xacro:wheel position="back"  side="left"  x="-0.12" y=" 0.15" />
+<!-- ****************************************************** Camera Link **************************************************************  -->
   <link name="camera">
     <inertial>
@@ -156,5 +117,12 @@
     </collision>
   </link>
-<!-- ****************************************************** Hokuyo *******************************************************************  -->
+<!-- ****************************************************** Camera Joint *************************************************************  -->
+  <joint type="fixed" name="camera_joint">
+    <origin xyz="0.2 0 0" rpy="0 0 0"/>
+    <child link="camera"/>
+    <parent link="base"/>
+    <axis xyz="0 1 0" rpy="0 0 0"/>
+  </joint>
+<!-- ****************************************************** Hokuyo Link **************************************************************  -->
   <link name="hokuyo">
     <inertial>
@@ -177,53 +145,4 @@
     </collision>
   </link>
-<!-- ****************************************************** Footprint Joint **********************************************************  -->
-  <joint type="fixed" name="footprint_joint" >
-    <origin xyz="0 0 0" rpy="0 0 0" />
-    <parent link="footprint"/>
-    <child link="base" />
-  </joint>
-<!-- ****************************************************** Front Left Wheel Joint ***************************************************  -->
-  <joint type="continuous" name="front_left_wheel_joint">
-    <origin xyz="0.12 0.15 0" rpy="0 0 0"/>
-    <child link="front_left_wheel"/>
-    <parent link="base"/>
-    <axis xyz="0 1 0" rpy="0 0 0"/>
-    <limit effort="10000" velocity="1000"/>
-    <dynamics damping="1.0" friction="1.0"/>
-  </joint>
-<!-- ****************************************************** Front Right Wheel Joint **************************************************  -->
-  <joint type="continuous" name="front_right_wheel_joint">
-    <origin xyz="0.12 -0.15 0" rpy="0 0 0"/>
-    <child link="front_right_wheel"/>
-    <parent link="base"/>
-    <axis xyz="0 1 0" rpy="0 0 0"/>
-    <limit effort="10000" velocity="1000"/>
-    <dynamics damping="1.0" friction="1.0"/>
-  </joint>
-<!-- ****************************************************** Back Left Wheel Joint ****************************************************  -->
-  <joint type="continuous" name="back_left_wheel_joint">
-    <origin xyz="-0.12 0.15 0" rpy="0 0 0"/>
-    <child link="back_left_wheel"/>
-    <parent link="base"/>
-    <axis xyz="0 1 0" rpy="0 0 0"/>
-    <limit effort="10000" velocity="1000"/>
-    <dynamics damping="1.0" friction="1.0"/>
-  </joint>
-<!-- ****************************************************** Back Right Wheel Joint ***************************************************  -->
-  <joint type="continuous" name="back_right_wheel_joint">
-    <origin xyz="-0.12 -0.15 0" rpy="0 0 0"/>
-    <child link="back_right_wheel"/>
-    <parent link="base"/>
-    <axis xyz="0 1 0" rpy="0 0 0"/>
-    <limit effort="10000" velocity="1000"/>
-    <dynamics damping="1.0" friction="1.0"/>
-  </joint>
-<!-- ****************************************************** Camera Joint *************************************************************  -->
-  <joint type="fixed" name="camera_joint">
-    <origin xyz="0.2 0 0" rpy="0 0 0"/>
-    <child link="camera"/>
-    <parent link="base"/>
-    <axis xyz="0 1 0" rpy="0 0 0"/>
-  </joint>
 <!-- ****************************************************** Hokuyo Joint *************************************************************  -->
   <joint type="fixed" name="hokuyo_joint">

Commit message: u

File: gazebo/gz_bocbot.xacro (robot description, xacro)
@@ -28,4 +28,7 @@
   <gazebo>
     <plugin name="joint_states_pub" filename="libgazebo_ros_joint_state_publisher.so">
+      <ros>
+        <namespace>bocbot</namespace>
+      </ros>
       <joint_name>front_left_wheel_joint</joint_name>
       <joint_name>back_left_wheel_joint</joint_name>
@@ -49,10 +52,10 @@
       <right_joint>front_right_wheel_joint</right_joint>
       <wheel_separation>0.4</wheel_separation>
-      <wheel_diameter>"${(wheel_radius*2)}</wheel_diameter>
+      <wheel_diameter>${(wheel_radius*2)}</wheel_diameter>
       <max_wheel_torque>20</max_wheel_torque>
       <left_joint>back_left_wheel_joint</left_joint>
       <right_joint>back_right_wheel_joint</right_joint>
       <wheel_separation>0.4</wheel_separation>
-      <wheel_diameter>"${(wheel_radius*2)}</wheel_diameter>
+      <wheel_diameter>${(wheel_radius*2)}</wheel_diameter>
       <max_wheel_torque>20</max_wheel_torque>
       <robot_base_frame>footprint</robot_base_frame>

File: xacro/bocbot.xacro (robot description, xacro)
@@ -82,6 +82,6 @@
 <!-- ****************************************************** Wheel Joint **************************************************************  -->
     <joint type="continuous" name="${position}_${side}_wheel_joint">
-        <origin xyz="${x} ${y} 0.15 0" rpy="0 0 0"/>
-        <child link="front_left_wheel"/>
+        <origin xyz="${x} ${y} 0" rpy="0 0 0"/>
+        <child link="${position}_${side}_wheel"/>
         <parent link="base"/>
         <axis xyz="0 1 0" rpy="0 0 0"/>

Commit message: u

File: gazebo/gz_bocbot.xacro (robot description, xacro)
@@ -7,5 +7,5 @@
 <!-- ****************************************************** Base *********************************************************************  -->
   <gazebo reference="base">
-    <material>Gazebo/Blue</material>
+    <material>Gazebo/Orange</material>
   </gazebo>
 <!-- ****************************************************** Front Left Wheel *********************************************************  -->
