Commit message: u

File: gazebo/gz_skidbot.xacro (robot description, xacro)
@@ -1,5 +1,5 @@
 <?xml version="1.0"?>
-<robot name="bocbot" xmlns:xacro="http://www.ros.org/wiki/xacro">
-<!-- ****************************************************** bocbot Robot *************************************************************  -->
+<robot name="skidbot" xmlns:xacro="http://www.ros.org/wiki/xacro">
+<!-- ****************************************************** skidbot Robot *************************************************************  -->
 <!-- Muthanna Alwahash                                                                                                                  -->
 <!-- March 2022                                                                                                                         -->
@@ -29,5 +29,5 @@
     <plugin name="joint_states_pub" filename="libgazebo_ros_joint_state_publisher.so">
       <ros>
-        <namespace>bocbot</namespace>
+        <namespace>skidbot</namespace>
       </ros>
       <joint_name>front_left_wheel_joint</joint_name>
@@ -40,12 +40,10 @@
 <!-- ******************************************************  Skid Steer Drive Controller *********************************************  -->
   <gazebo>
-    <plugin name="diff_drive" filename="libgazebo_ros_diff_drive.so">
+    <plugin name="skid_drive" filename="libgazebo_ros_diff_drive.so">
       <ros>
-        <namespace>bocbot</namespace>
+        <namespace>skidbot</namespace>
         <argument>--remap cmd_vel:=cme_vel</argument>
         <argument>--remap odom:=odom</argument>
       </ros>
-      <update_rate>100.0</update_rate>
-      <odometry_frame>odom</odometry_frame>
       <num_wheel_pairs>2</num_wheel_pairs>
       <left_joint>front_left_wheel_joint</left_joint>
@@ -53,5 +51,4 @@
       <wheel_separation>0.4</wheel_separation>
       <wheel_diameter>${(wheel_radius*2)}</wheel_diameter>
-      <max_wheel_torque>20</max_wheel_torque>
       <left_joint>back_left_wheel_joint</left_joint>
       <right_joint>back_right_wheel_joint</right_joint>
@@ -59,9 +56,11 @@
       <wheel_diameter>${(wheel_radius*2)}</wheel_diameter>
       <max_wheel_torque>20</max_wheel_torque>
+      <max_wheel_acceleration>1.0</max_wheel_acceleration>
+      <update_rate>100.0</update_rate>
       <robot_base_frame>footprint</robot_base_frame>
+      <odometry_frame>odom</odometry_frame>
       <publish_odom>true</publish_odom>
       <publish_odom_tf>true</publish_odom_tf>
       <publish_wheel_tf>true</publish_wheel_tf>
-      <odometry_source>world</odometry_source>
     </plugin>
   </gazebo>
@@ -71,5 +70,5 @@
       <plugin name="camera" filename="libgazebo_ros_camera.so">
         <ros>
-          <namespace>bocbot</namespace>
+          <namespace>skidbot</namespace>
           <argument>--remap camera/image_raw:=camera/image_raw</argument>
           <argument>--remap camera/camera_info:=camera/camera_info</argument>
@@ -109,5 +108,5 @@
       <plugin name="hokuyo" filename="libgazebo_ros_ray_sensor.so">
         <ros>
-          <namespace>bocbot</namespace>
+          <namespace>skidbot</namespace>
           <argument>--remap ~/out:=scan</argument>
         </ros>

File: xacro/skidbot.xacro (robot description, xacro)
@@ -1,10 +1,10 @@
 <?xml version='1.0'?>
-<robot name="bocbot" xmlns:xacro="http://www.ros.org/wiki/xacro">
-<!-- ****************************************************** bocbot Robot *************************************************************  -->
+<robot name="skidbot" xmlns:xacro="http://www.ros.org/wiki/xacro">
+<!-- ****************************************************** skidbot Robot *************************************************************  -->
 <!-- Muthanna Alwahash                                                                                                                  -->
 <!-- March 2022                                                                                                                         -->
 <!-- *********************************************************************************************************************************  -->
 <!-- ****************************************************** Parameters ***************************************************************  -->
-  <xacro:property name="mesh_path"      value="package://robot_gazebo/meshes/bocbot/"/>
+  <xacro:property name="mesh_path"      value="package://robot_gazebo/meshes/skidbot/"/>
   <xacro:property name="base_mass"      value="15.0"                              /> <!-- arbitrary mass value                          -->
   <xacro:property name="base_width"     value="0.20"                              />
@@ -26,5 +26,5 @@
 <!-- ****************************************************** Includes *****************************************************************  -->
   <xacro:include filename="$(find robot_gazebo)/xacro/common_rviz_materials.xacro" />   <!-- RVIZ Colors                                -->
-  <xacro:include filename="$(find robot_gazebo)/gazebo/gz_bocbot.xacro" />              <!-- Gazebo                                     -->
+  <xacro:include filename="$(find robot_gazebo)/gazebo/gz_skidbot.xacro" />              <!-- Gazebo                                     -->
 <!-- ****************************************************** Base Footprint ***********************************************************  -->
   <link name="footprint"></link>

Commit message: u

File: gazebo/gz_skidbot.xacro (robot description, xacro)
@@ -40,5 +40,5 @@
 <!-- ******************************************************  Skid Steer Drive Controller *********************************************  -->
   <gazebo>
-    <plugin name="skid_drive" filename="libgazebo_ros_diff_drive.so">
+    <plugin name="skid_drive" filename="libgazebo_ros_skid_steer_drive.so">
       <ros>
         <namespace>skidbot</namespace>
@@ -47,8 +47,10 @@
       </ros>
       <num_wheel_pairs>2</num_wheel_pairs>
+      <!-- 1st Set -->
       <left_joint>front_left_wheel_joint</left_joint>
       <right_joint>front_right_wheel_joint</right_joint>
       <wheel_separation>0.4</wheel_separation>
       <wheel_diameter>${(wheel_radius*2)}</wheel_diameter>
+      <!-- 2nd Set -->
       <left_joint>back_left_wheel_joint</left_joint>
       <right_joint>back_right_wheel_joint</right_joint>

File: xacro/skidbot.xacro (robot description, xacro)
@@ -14,4 +14,6 @@
   <xacro:property name="wheel_width"    value="0.05"                              />
   <xacro:property name="wheel_radius"   value="0.10"                              />
+  <xacro:property name="wheel_x"        value="0.12"                              />
+  <xacro:property name="wheel_y"        value="0.15"                              />
   <xacro:property name="camera_mass"    value="0.1"                               />
   <xacro:property name="camera_width"   value="0.05"                              />
@@ -22,6 +24,4 @@
   <xacro:property name="hokuyo_length"  value="0.05"                              />
   <xacro:property name="hokuyo_height"  value="0.080165"                          />
-  <xacro:property name="y_offset"       value="${(base_width+wheel_width*1.2)/2}" />
-  <xacro:property name="z_offset"       value="${base_height/2}"                  />
 <!-- ****************************************************** Includes *****************************************************************  -->
   <xacro:include filename="$(find robot_gazebo)/xacro/common_rviz_materials.xacro" />   <!-- RVIZ Colors                                -->
@@ -92,8 +92,8 @@
   </xacro:macro>
 <!-- ****************************************************** Expand Wheels Macro ******************************************************  -->
-<xacro:wheel position="front" side="right" x=" 0.12" y="-0.15" />
-<xacro:wheel position="front" side="left"  x=" 0.12" y=" 0.15" />
-<xacro:wheel position="back"  side="right" x="-0.12" y="-0.15" />
-<xacro:wheel position="back"  side="left"  x="-0.12" y=" 0.15" />
+<xacro:wheel position="front" side="right" x=" ${wheel_x}" y="-${wheel_y}" />
+<xacro:wheel position="front" side="left"  x=" ${wheel_x}" y=" ${wheel_y}" />
+<xacro:wheel position="back"  side="right" x="-${wheel_x}" y="-${wheel_y}" />
+<xacro:wheel position="back"  side="left"  x="-${wheel_x}" y=" ${wheel_y}" />
 <!-- ****************************************************** Camera Link **************************************************************  -->
   <link name="camera">

Commit message: U

File: gazebo/gz_skidbot.xacro (robot description, xacro)
@@ -47,10 +47,10 @@
       </ros>
       <num_wheel_pairs>2</num_wheel_pairs>
-      <!-- 1st Set -->
+      <!-- 1st Wheels Set -->
       <left_joint>front_left_wheel_joint</left_joint>
       <right_joint>front_right_wheel_joint</right_joint>
       <wheel_separation>0.4</wheel_separation>
       <wheel_diameter>${(wheel_radius*2)}</wheel_diameter>
-      <!-- 2nd Set -->
+      <!-- 2nd Wheels Set -->
       <left_joint>back_left_wheel_joint</left_joint>
       <right_joint>back_right_wheel_joint</right_joint>

File: xacro/skidbot.xacro (robot description, xacro)
@@ -7,21 +7,24 @@
 <!-- ****************************************************** Parameters ***************************************************************  -->
   <xacro:property name="mesh_path"      value="package://robot_gazebo/meshes/skidbot/"/>
-  <xacro:property name="base_mass"      value="15.0"                              /> <!-- arbitrary mass value                          -->
-  <xacro:property name="base_width"     value="0.20"                              />
-  <xacro:property name="base_length"    value="0.40"                              />
-  <xacro:property name="base_height"    value="0.10"                              />
-  <xacro:property name="wheel_mass"     value="5.0"                               />
-  <xacro:property name="wheel_width"    value="0.05"                              />
-  <xacro:property name="wheel_radius"   value="0.10"                              />
-  <xacro:property name="wheel_x"        value="0.12"                              />
-  <xacro:property name="wheel_y"        value="0.15"                              />
-  <xacro:property name="camera_mass"    value="0.1"                               />
-  <xacro:property name="camera_width"   value="0.05"                              />
-  <xacro:property name="camera_length"  value="0.05"                              />
-  <xacro:property name="camera_height"  value="0.05"                              />
-  <xacro:property name="hokuyo_mass"    value="1e-5"                              />
-  <xacro:property name="hokuyo_width"   value="0.05"                              />
-  <xacro:property name="hokuyo_length"  value="0.05"                              />
-  <xacro:property name="hokuyo_height"  value="0.080165"                          />
+  <xacro:property name="base_mass"      value="15.0"     /> <!-- arbitrary mass value -->
+  <xacro:property name="base_width"     value="0.20"     />
+  <xacro:property name="base_length"    value="0.40"     />
+  <xacro:property name="base_height"    value="0.10"     />
+  <xacro:property name="wheel_mass"     value="5.0"      />
+  <xacro:property name="wheel_width"    value="0.05"     />
+  <xacro:property name="wheel_radius"   value="0.10"     />
+  <xacro:property name="wheel_x"        value="0.12"     />
+  <xacro:property name="wheel_y"        value="0.15"     />
+  <xacro:property name="camera_mass"    value="0.1"      />
+  <xacro:property name="camera_width"   value="0.05"     />
+  <xacro:property name="camera_length"  value="0.05"     />
+  <xacro:property name="camera_height"  value="0.05"     />
+  <xacro:property name="camera_x"       value="0.2"      />
+  <xacro:property name="hokuyo_mass"    value="1e-5"     />
+  <xacro:property name="hokuyo_width"   value="0.05"     />
+  <xacro:property name="hokuyo_length"  value="0.05"     />
+  <xacro:property name="hokuyo_height"  value="0.080165" />
+  <xacro:property name="hokuyo_x"       value="0.15"     />
+  <xacro:property name="hokuyo_z"       value="0.05"     />
 <!-- ****************************************************** Includes *****************************************************************  -->
   <xacro:include filename="$(find robot_gazebo)/xacro/common_rviz_materials.xacro" />   <!-- RVIZ Colors                                -->
@@ -119,5 +122,5 @@
 <!-- ****************************************************** Camera Joint *************************************************************  -->
   <joint type="fixed" name="camera_joint">
-    <origin xyz="0.2 0 0" rpy="0 0 0"/>
+    <origin xyz="${camera_x} 0 0" rpy="0 0 0"/>
     <child link="camera"/>
     <parent link="base"/>
@@ -147,5 +150,5 @@
 <!-- ****************************************************** Hokuyo Joint *************************************************************  -->
   <joint type="fixed" name="hokuyo_joint">
-    <origin xyz="0.15 0 0.1" rpy="0 0 0"/>
+    <origin xyz="${hokuyo_x} 0 ${hokuyo_Z}" rpy="0 0 0"/>
     <child link="hokuyo"/>
     <parent link="base"/>

Commit message: u

File: gazebo/gz_skidbot.xacro (robot description, xacro)
@@ -29,5 +29,5 @@
     <plugin name="joint_states_pub" filename="libgazebo_ros_joint_state_publisher.so">
       <ros>
-        <namespace>skidbot</namespace>
+        <namespace>${name_space}</namespace>
       </ros>
       <joint_name>front_left_wheel_joint</joint_name>
@@ -42,5 +42,5 @@
     <plugin name="skid_drive" filename="libgazebo_ros_diff_drive.so">
       <ros>
-        <namespace>skidbot</namespace>
+        <namespace>${name_space}</namespace>
         <argument>--remap cmd_vel:=cme_vel</argument>
         <argument>--remap odom:=odom</argument>
@@ -72,5 +72,5 @@
       <plugin name="camera" filename="libgazebo_ros_camera.so">
         <ros>
-          <namespace>skidbot</namespace>
+          <namespace>${name_space}</namespace>
           <argument>--remap camera/image_raw:=camera/image_raw</argument>
           <argument>--remap camera/camera_info:=camera/camera_info</argument>
@@ -110,5 +110,5 @@
       <plugin name="hokuyo" filename="libgazebo_ros_ray_sensor.so">
         <ros>
-          <namespace>skidbot</namespace>
+          <namespace>${name_space}</namespace>
           <argument>--remap ~/out:=scan</argument>
         </ros>

File: xacro/skidbot.xacro (robot description, xacro)
@@ -7,4 +7,5 @@
 <!-- ****************************************************** Parameters ***************************************************************  -->
   <xacro:property name="mesh_path"      value="package://robot_gazebo/meshes/skidbot/"/>
+  <xacro:property name="name_space"     value="skidbot"  />
   <xacro:property name="base_mass"      value="15.0"     /> <!-- arbitrary mass value -->
   <xacro:property name="base_width"     value="0.20"     />
@@ -140,5 +141,5 @@
         <mesh filename="${mesh_path}hokuyo.dae"/> <!--  <box size="${hokuyo_length} ${hokuyo_width} ${hokuyo_height}"/> -->
       </geometry>
-      <material name="red"/>
+      <!-- <material name="red"/> -->
     </visual>
     <collision name="hokuyo_colision">

Commit message: u

File: gazebo/gz_skidbot.xacro (robot description, xacro)
@@ -111,5 +111,5 @@
         <ros>
           <namespace>${name_space}</namespace>
-          <argument>--remap ~/out:=scan</argument>
+          <argument>--remap out:=scan</argument>
         </ros>
         <output_type>sensor_msgs/LaserScan</output_type>
@@ -123,6 +123,6 @@
             <samples>720</samples>
             <resolution>1</resolution>
-            <min_angle>-1.570796</min_angle>
-            <max_angle>1.570796</max_angle>
+            <min_angle>-${radians(90)}</min_angle>
+            <max_angle> ${radians(90)}</max_angle>
           </horizontal>
         </scan>
@@ -141,5 +141,5 @@
       </ray>
     </sensor>
-    <material>Gazebo/Red</material>
+    <!-- <material>Gazebo/Red</material> -->
   </gazebo>
 <!-- ****************************************************** end **********************************************************************  -->

Commit message: u

File: gazebo/gz_skidbot.xacro (robot description, xacro)
@@ -7,21 +7,5 @@
 <!-- ****************************************************** Base *********************************************************************  -->
   <gazebo reference="base">
-    <material>Gazebo/Orange</material>
-  </gazebo>
-<!-- ****************************************************** Front Left Wheel *********************************************************  -->
-  <gazebo reference="front_left_wheel">
-    <material>Gazebo/Gray</material>
-  </gazebo>
-<!-- ****************************************************** Back Left Wheel **********************************************************  -->
-  <gazebo reference="back_left_wheel">
-    <material>Gazebo/Gray</material>
-  </gazebo>
-<!-- ****************************************************** Front Right Wheel ********************************************************  -->
-  <gazebo reference="front_right_wheel">
-    <material>Gazebo/Gray</material>
-  </gazebo>
-<!-- ****************************************************** Back Right Wheel *********************************************************  -->
-  <gazebo reference="back_right_wheel">
-    <material>Gazebo/Gray</material>
+    <material>Gazebo/Blue</material>
   </gazebo>
 <!-- ******************************************************  Joint States Publisher **************************************************  -->
