Commit message: u

File: gazebo/gz_cart_effort.xacro (robot description, xacro)
@@ -1,8 +1,16 @@
 <?xml version="1.0" ?>
 <robot name="cart" xmlns:xacro="http://ros.org/wiki/xacro">
+<!-- ****************************************************** slideBar Link ************************************************************ -->
+  <gazebo reference="slideBar">
+    <material>Gazebo/Orange</material>
+  </gazebo>
+<!-- ****************************************************** cart Link **************************************************************** -->
+  <gazebo reference="cart">
+    <material>Gazebo/Red</material>
+  </gazebo>
 <!-- ****************************************************** Gazebo ROS2 Plugin ******************************************************* -->
   <gazebo>
     <plugin filename="libgazebo_ros2_control.so" name="gazebo_ros2_control">
-      <parameters>$(find cart)/config/cartpole_controller_effort.yaml</parameters>
+      <parameters>$(find bots)/config/cartpole_controller_effort.yaml</parameters>
     </plugin>
   </gazebo>

File: gazebo/gz_cart_position.xacro (robot description, xacro)
@@ -1,8 +1,16 @@
 <?xml version="1.0" ?>
 <robot name="cart" xmlns:xacro="http://ros.org/wiki/xacro">
+<!-- ****************************************************** slideBar Link ************************************************************ -->
+  <gazebo reference="slideBar">
+    <material>Gazebo/Orange</material>
+  </gazebo>
+<!-- ****************************************************** cart Link **************************************************************** -->
+  <gazebo reference="cart">
+    <material>Gazebo/Red</material>
+  </gazebo>
 <!-- ****************************************************** Gazebo ROS2 Plugin ******************************************************* -->
   <gazebo>
     <plugin filename="libgazebo_ros2_control.so" name="gazebo_ros2_control">
-      <parameters>$(find cart)/config/cartpole_controller.yaml</parameters>
+      <parameters>$(find bots)/config/cartpole_controller.yaml</parameters>
     </plugin>
   </gazebo>

File: gazebo/gz_cart_velocity.xacro (robot description, xacro)
@@ -1,8 +1,16 @@
 <?xml version="1.0" ?>
 <robot name="cart" xmlns:xacro="http://ros.org/wiki/xacro">
+<!-- ****************************************************** slideBar Link ************************************************************ -->
+  <gazebo reference="slideBar">
+    <material>Gazebo/Orange</material>
+  </gazebo>
+<!-- ****************************************************** cart Link **************************************************************** -->
+  <gazebo reference="cart">
+    <material>Gazebo/Red</material>
+  </gazebo>
 <!-- ****************************************************** Gazebo ROS2 Plugin ******************************************************* -->
   <gazebo>
     <plugin filename="libgazebo_ros2_control.so" name="gazebo_ros2_control">
-      <parameters>$(find cart)/config/cartpole_controller_velocity.yaml</parameters>
+      <parameters>$(find bots)/config/cartpole_controller_velocity.yaml</parameters>
     </plugin>
   </gazebo>

File: xacro/cart_position.xacro (robot description, xacro)
@@ -12,7 +12,7 @@
 <!-- ****************************************************** Includes *****************************************************************  -->
     <xacro:include filename="${pkg_path}/xacro/common_rviz_materials.xacro" />  <!--  RVIZ Colors  -->
-    <xacro:include filename="${pkg_path}/xacro/urdf_cart.xacro" />             <!--  Robot URDF   -->
-    <xacro:include filename="${pkg_path}/gazebo/gz_cart_position.xacro" />              <!--  Gazebo Sim   -->
-    <xacro:include filename="${pkg_path}/r2c/r2c_cart_position.xacro" />                <!--  ROS2_Control -->
+    <xacro:include filename="${pkg_path}/xacro/urdf_cart.xacro" />              <!--  Robot URDF   -->
+    <xacro:include filename="${pkg_path}/gazebo/gz_cart_position.xacro" />      <!--  Gazebo Sim   -->
+    <xacro:include filename="${pkg_path}/r2c/r2c_cart_position.xacro" />        <!--  ROS2_Control -->
 <!-- ****************************************************** END **********************************************************************  -->
 </robot>

File: xacro/urdf_cart.xacro (robot description, xacro)
@@ -19,7 +19,4 @@
     </inertial>
   </link>
-  <gazebo reference="slideBar">
-    <material>Gazebo/Orange</material>
-  </gazebo>
 <!-- ****************************************************** cart Link **************************************************************** -->
   <link name="cart">
@@ -38,7 +35,4 @@
     </inertial>
   </link>
-  <gazebo reference="cart">
-    <material>Gazebo/Red</material>
-  </gazebo>
 <!-- ****************************************************** world to slideBar Joint ************************************************** -->
   <joint name="world_to_base" type="fixed">

Commit message: u

File: gazebo/gz_cart_effort.xacro (robot description, xacro)
@@ -12,5 +12,5 @@
   <gazebo>
     <plugin filename="libgazebo_ros2_control.so" name="gazebo_ros2_control">
-      <parameters>$(find bots)/config/cart_effort.yaml</parameters>
+      <parameters>${config_path}cart_effort.yaml</parameters>
     </plugin>
   </gazebo>

File: gazebo/gz_cart_position.xacro (robot description, xacro)
@@ -12,5 +12,5 @@
   <gazebo>
     <plugin filename="libgazebo_ros2_control.so" name="gazebo_ros2_control">
-      <parameters>$(find bots)/config/cart_position.yaml</parameters>
+      <parameters>${config_path}cart_position.yaml</parameters>
     </plugin>
   </gazebo>

File: gazebo/gz_cart_velocity.xacro (robot description, xacro)
@@ -12,5 +12,5 @@
   <gazebo>
     <plugin filename="libgazebo_ros2_control.so" name="gazebo_ros2_control">
-      <parameters>$(find bots)/config/cart_velocity.yaml</parameters>
+      <parameters>${config_path}cart_velocity.yaml</parameters>
     </plugin>
   </gazebo>

File: xacro/cart_effort.xacro (robot description, xacro)
@@ -8,4 +8,5 @@
     <xacro:property name="pkg_path"     value="$(find bots)"                />
     <xacro:property name="mesh_path"    value="${pkg_path}/meshes/cart/"    />
+    <xacro:property name="config_path"  value="${pkg_path}/config/"         />
     <xacro:property name="name_space"   value="cart" />
     <xacro:property name="prefix"       value=""      />

File: xacro/cart_position.xacro (robot description, xacro)
@@ -8,4 +8,5 @@
     <xacro:property name="pkg_path"     value="$(find bots)"                />
     <xacro:property name="mesh_path"    value="${pkg_path}/meshes/cart/"    />
+    <xacro:property name="config_path"  value="${pkg_path}/config/"         />
     <xacro:property name="name_space"   value="cart" />
     <xacro:property name="prefix"       value=""      />

File: xacro/cart_velocity.xacro (robot description, xacro)
@@ -8,4 +8,5 @@
     <xacro:property name="pkg_path"     value="$(find bots)"                />
     <xacro:property name="mesh_path"    value="${pkg_path}/meshes/cart/"    />
+    <xacro:property name="config_path"  value="${pkg_path}/config/"         />
     <xacro:property name="name_space"   value="cart" />
     <xacro:property name="prefix"       value=""      />

File: xacro/rrbot.xacro (robot description, xacro)
@@ -7,5 +7,6 @@
 <!-- ****************************************************** Parameters ***************************************************************  -->
     <xacro:property name="pkg_path"     value="$(find bots)"                />
-    <xacro:property name="mesh_path"    value="${pkg_path}/meshes/rrbot/"    />
+    <xacro:property name="mesh_path"    value="${pkg_path}/meshes/rrbot/"   />
+    <xacro:property name="config_path"  value="${pkg_path}/config/"         />
     <xacro:property name="name_space"   value="rrbot" />
     <xacro:property name="prefix"       value=""      />
