Commit message: u

File: gazebo/gz_rrbot.xacro (robot description, xacro)
@@ -5,185 +5,26 @@
 <!-- March 2022                                                                                                                         -->
 <!-- *********************************************************************************************************************************  -->
-<!-- ****************************************************** Parameters ***************************************************************  -->
-    <xacro:property name="mesh_path"    value="package://robot_gazebo/meshes/rrbot/" />
-    <xacro:property name="mass"         value="1"     /> <!-- arbitrary value for mass -->
-    <xacro:property name="width"        value="0.1"   /> <!-- Square dimensions (widthxwidth) of beams -->
-    <xacro:property name="height1"      value="2"     /> <!-- Link 1 -->
-    <xacro:property name="height2"      value="1"     /> <!-- Link 2 -->
-    <xacro:property name="height3"      value="1"     /> <!-- Link 3 -->
-    <xacro:property name="camera_link"  value="0.05"  /> <!-- Size of square 'camera' box -->
-    <xacro:property name="axel_offset"  value="0.05"  /> <!-- Space btw top of beam and the each joint -->
-<!-- ****************************************************** Import RVIZ Materials*****************************************************  -->
-  <xacro:include filename="$(find robot_gazebo)/xacro/common_rviz_materials.xacro" />
 <!-- ****************************************************** Macro ********************************************************************  -->
-  <xacro:macro name="rrbot" params="parent prefix">
-<!-- ****************************************************** Base Joint ***************************************************************  -->
-    <joint name="${prefix}base_joint" type="fixed">
-      <origin xyz="0 0 0" rpy="0 0 0" />
-      <parent link="${parent}"/>
-      <child link="${prefix}base_link" />
-    </joint>
+  <xacro:macro name="rrbot_gz" params="prefix">
 <!-- ****************************************************** Base Link ****************************************************************  -->
-    <link name="${prefix}base_link">
-      <collision>
-        <origin xyz="0 0 ${height1/2}" rpy="0 0 0"/>
-        <geometry>
-          <box size="${width} ${width} ${height1}"/>
-        </geometry>
-      </collision>
-      <visual>
-        <origin xyz="0 0 ${height1/2}" rpy="0 0 0"/>
-        <geometry>
-          <box size="${width} ${width} ${height1}"/>
-        </geometry>
-        <material name="orange"/>
-      </visual>
-      <inertial>
-        <origin xyz="0 0 ${height1/2}" rpy="0 0 0"/>
-        <mass value="${mass}"/>
-        <inertia
-          ixx="${mass / 12.0 * (width*width + height1*height1)}" ixy="0.0" ixz="0.0"
-          iyy="${mass / 12.0 * (height1*height1 + width*width)}" iyz="0.0"
-          izz="${mass / 12.0 * (width*width + width*width)}"/>
-      </inertial>
-    </link>
-<!-- ****************************************************** Joint 1 ******************************************************************  -->
-    <joint name="${prefix}joint1" type="continuous">
-      <parent link="${prefix}base_link"/>
-      <child link="${prefix}link1"/>
-      <origin xyz="0 ${width} ${height1 - axel_offset}" rpy="0 0 0"/>
-      <axis xyz="0 1 0"/>
-      <dynamics damping="0.7"/>
-    </joint>
+    <gazebo reference="${prefix}base_link">
+        <material>Gazebo/Orange</material>
+    </gazebo>
 <!-- ****************************************************** Link 1 *******************************************************************  -->
-    <link name="${prefix}link1">
-      <collision>
-        <origin xyz="0 0 ${height2/2 - axel_offset}" rpy="0 0 0"/>
-        <geometry>
-          <box size="${width} ${width} ${height2}"/>
-        </geometry>
-      </collision>
-      <visual>
-        <origin xyz="0 0 ${height2/2 - axel_offset}" rpy="0 0 0"/>
-        <geometry>
-          <box size="${width} ${width} ${height2}"/>
-        </geometry>
-        <material name="yellow"/>
-      </visual>
-      <inertial>
-        <origin xyz="0 0 ${height2/2 - axel_offset}" rpy="0 0 0"/>
-        <mass value="${mass}"/>
-        <inertia
-          ixx="${mass / 12.0 * (width*width + height2*height2)}" ixy="0.0" ixz="0.0"
-          iyy="${mass / 12.0 * (height2*height2 + width*width)}" iyz="0.0"
-          izz="${mass / 12.0 * (width*width + width*width)}"/>
-      </inertial>
-    </link>
-<!-- ****************************************************** Joint 2 ******************************************************************  -->
-    <joint name="${prefix}joint2" type="continuous">
-      <parent link="${prefix}link1"/>
-      <child link="${prefix}link2"/>
-      <origin xyz="0 ${width} ${height2 - axel_offset*2}" rpy="0 0 0"/>
-      <axis xyz="0 1 0"/>
-      <dynamics damping="0.7"/>
-    </joint>
+    <gazebo reference="${prefix}link1">
+        <material>Gazebo/Red</material>
+    </gazebo>
 <!-- ****************************************************** Link 2 *******************************************************************  -->
-    <link name="${prefix}link2">
-      <collision>
-        <origin xyz="0 0 ${height3/2 - axel_offset}" rpy="0 0 0"/>
-        <geometry>
-          <box size="${width} ${width} ${height3}"/>
-        </geometry>
-      </collision>
-      <visual>
-        <origin xyz="0 0 ${height3/2 - axel_offset}" rpy="0 0 0"/>
-        <geometry>
-          <box size="${width} ${width} ${height3}"/>
-        </geometry>
-        <material name="orange"/>
-      </visual>
-      <inertial>
-        <origin xyz="0 0 ${height3/2 - axel_offset}" rpy="0 0 0"/>
-        <mass value="${mass}"/>
-        <inertia
-          ixx="${mass / 12.0 * (width*width + height3*height3)}" ixy="0.0" ixz="0.0"
-          iyy="${mass / 12.0 * (height3*height3 + width*width)}" iyz="0.0"
-          izz="${mass / 12.0 * (width*width + width*width)}"/>
-      </inertial>
-    </link>
-<!-- ****************************************************** Tool Joint ***************************************************************  -->
-    <joint name="${prefix}tool_joint" type="fixed">
-      <origin xyz="0 0 1" rpy="0 0 0" />
-      <parent link="${prefix}link2"/>
-      <child link="${prefix}tool_link" />
-    </joint>
-<!-- ****************************************************** Tool Link ****************************************************************  -->
-    <link name="${prefix}tool_link" />
-<!-- ****************************************************** Hokuyo Joint *************************************************************  -->
-    <joint name="${prefix}hokuyo_joint" type="fixed">
-      <axis xyz="0 1 0" />
-      <origin xyz="0 0 ${height3 - axel_offset/2}" rpy="0 0 0"/>
-      <parent link="${prefix}link2"/>
-      <child link="${prefix}hokuyo_link"/>
-    </joint>
+    <gazebo reference="${prefix}link2">
+        <material>Gazebo/Orange</material>
+    </gazebo>
 <!-- ****************************************************** Hokuyo Link **************************************************************  -->
-    <link name="${prefix}hokuyo_link">
-      <collision>
-        <origin xyz="0 0 0" rpy="0 0 0"/>
-        <geometry>
-          <box size="0.1 0.1 0.1"/>
-        </geometry>
-      </collision>
-      <visual>
-        <origin xyz="0 0 0" rpy="0 0 0"/>
-        <geometry>
-          <mesh filename="${mesh_path}hokuyo.dae"/>
-        </geometry>
-      </visual>
-      <inertial>
-        <mass value="1e-5" />
-        <origin xyz="0 0 0" rpy="0 0 0"/>
-        <inertia ixx="1e-6" ixy="0" ixz="0" iyy="1e-6" iyz="0" izz="1e-6" />
-      </inertial>
-    </link>
-<!-- ****************************************************** Camera Joint *************************************************************  -->
-    <joint name="${prefix}camera_joint" type="fixed">
-      <axis xyz="0 1 0" />
-      <origin xyz="${camera_link} 0 ${height3 - axel_offset*2}" rpy="0 0 0"/>
-      <parent link="${prefix}link2"/>
-      <child link="${prefix}camera_link"/>
-    </joint>
+    <gazebo reference="${prefix}hokuyo_link">
+        <material>Gazebo/Green</material>
+    </gazebo>
 <!-- ****************************************************** Camera Link **************************************************************  -->
-    <link name="${prefix}camera_link">
-      <collision>
-        <origin xyz="0 0 0" rpy="0 0 0"/>
-        <geometry>
-          <box size="${camera_link} ${camera_link} ${camera_link}"/>
-        </geometry>
-      </collision>
-      <visual>
-        <origin xyz="0 0 0" rpy="0 0 0"/>
-        <geometry>
-          <box size="${camera_link} ${camera_link} ${camera_link}"/>
-        </geometry>
-        <material name="red"/>
-      </visual>
-      <inertial>
-        <mass value="1e-5" />
-        <origin xyz="0 0 0" rpy="0 0 0"/>
-        <inertia ixx="1e-6" ixy="0" ixz="0" iyy="1e-6" iyz="0" izz="1e-6" />
-      </inertial>
-    </link>
-<!-- ****************************************************** Camera Optical Joint *****************************************************  -->
-<!-- generate an optical frame http://www.ros.org/reps/rep-0103.html#suffix-frames so that ros and opencv can operate on the camera     -->
-<!-- frame correctly. these values have to be these values otherwise the gazebo camera image won't be aligned properly with the frame   -->
-<!-- it is supposedly originating from                                                                                                  -->                                                                                                                   -->
-    <joint name="${prefix}camera_optical_joint" type="fixed">
-      <origin xyz="0 0 0" rpy="${-pi/2} 0 ${-pi/2}"/>
-      <parent link="${prefix}camera_link"/>
-      <child link="${prefix}camera_link_optical"/>
-    </joint>
-<!-- ****************************************************** Camera Optical Link ******************************************************  -->
-    <link name="${prefix}camera_link_optical"/>
+    <gazebo reference="${prefix}camera_link">
+        <material>Gazebo/Green</material>
+    </gazebo>
 <!-- ****************************************************** End Macro ****************************************************************  -->
   </xacro:macro>
@@ -194,5 +35,5 @@
   </gazebo>
 <!-- ****************************************************** Expand Macro *************************************************************  -->
-  <xacro:rrbot parent="world" prefix="" />
+  <xacro:rrbot_gz prefix="" />
 <!-- ****************************************************** END **********************************************************************  -->
 </robot>

File: xacro/rrbot.xacro (robot description, xacro)
@@ -14,6 +14,7 @@
     <xacro:property name="camera_link"  value="0.05"  /> <!-- Size of square 'camera' box -->
     <xacro:property name="axel_offset"  value="0.05"  /> <!-- Space btw top of beam and the each joint -->
-<!-- ****************************************************** Import RVIZ Materials*****************************************************  -->
-  <xacro:include filename="$(find robot_gazebo)/xacro/common_rviz_materials.xacro" />
+<!-- ****************************************************** Includes *****************************************************************  -->
+  <xacro:include filename="$(find robot_gazebo)/xacro/common_rviz_materials.xacro" />   <!-- RVIZ Colors                                -->
+  <xacro:include filename="$(find robot_gazebo)/gazebo/gz_rrbot.xacro" />               <!-- Gazebo                                     -->
 <!-- ****************************************************** Macro ********************************************************************  -->
   <xacro:macro name="rrbot" params="parent prefix">
@@ -188,9 +189,4 @@
 <!-- ****************************************************** End Macro ****************************************************************  -->
   </xacro:macro>
-<!-- ****************************************************** World Link ****************************************************************  -->
-  <link name="world"/>
-  <gazebo reference="world">
-    <static>true</static>
-  </gazebo>
 <!-- ****************************************************** Expand Macro *************************************************************  -->
   <xacro:rrbot parent="world" prefix="" />

Commit message: u

File: gazebo/gz_rrbot.xacro (robot description, xacro)
@@ -5,28 +5,20 @@
 <!-- March 2022                                                                                                                         -->
 <!-- *********************************************************************************************************************************  -->
-<!-- ****************************************************** Macro ********************************************************************  -->
-  <xacro:macro name="rrbot_gz" params="prefix">
 <!-- ****************************************************** Base Link ****************************************************************  -->
-    <gazebo reference="${prefix}base_link">
-        <material>Gazebo/Orange</material>
-    </gazebo>
+  <gazebo reference="${prefix}base_link">
+      <material>Gazebo/Orange</material>
+  </gazebo>
 <!-- ****************************************************** Link 1 *******************************************************************  -->
-    <gazebo reference="${prefix}link1">
-        <material>Gazebo/Red</material>
-    </gazebo>
+  <gazebo reference="${prefix}link1">
+      <material>Gazebo/Orange</material>
+  </gazebo>
 <!-- ****************************************************** Link 2 *******************************************************************  -->
-    <gazebo reference="${prefix}link2">
-        <material>Gazebo/Orange</material>
-    </gazebo>
-<!-- ****************************************************** Hokuyo Link **************************************************************  -->
-    <gazebo reference="${prefix}hokuyo_link">
-        <material>Gazebo/Green</material>
-    </gazebo>
+  <gazebo reference="${prefix}link2">
+      <material>Gazebo/Orange</material>
+  </gazebo>
 <!-- ****************************************************** Camera Link **************************************************************  -->
-    <gazebo reference="${prefix}camera_link">
-        <material>Gazebo/Green</material>
-    </gazebo>
-<!-- ****************************************************** End Macro ****************************************************************  -->
-  </xacro:macro>
+  <gazebo reference="${prefix}camera_link">
+      <material>Gazebo/Green</material>
+  </gazebo>
 <!-- ****************************************************** World Link ****************************************************************  -->
   <link name="world"/>
@@ -34,6 +26,4 @@
     <static>true</static>
   </gazebo>
-<!-- ****************************************************** Expand Macro *************************************************************  -->
-  <xacro:rrbot_gz prefix="" />
 <!-- ****************************************************** END **********************************************************************  -->
 </robot>

File: xacro/rrbot.xacro (robot description, xacro)
@@ -7,4 +7,6 @@
 <!-- ****************************************************** Parameters ***************************************************************  -->
     <xacro:property name="mesh_path"    value="package://robot_gazebo/meshes/rrbot/" />
+    <xacro:property name="name_space"     value="rrbot"  />
+    <xacro:property name="prefix"         value=""  />
     <xacro:property name="mass"         value="1"     /> <!-- arbitrary value for mass -->
     <xacro:property name="width"        value="0.1"   /> <!-- Square dimensions (widthxwidth) of beams -->
@@ -17,10 +19,8 @@
   <xacro:include filename="$(find robot_gazebo)/xacro/common_rviz_materials.xacro" />   <!-- RVIZ Colors                                -->
   <xacro:include filename="$(find robot_gazebo)/gazebo/gz_rrbot.xacro" />               <!-- Gazebo                                     -->
-<!-- ****************************************************** Macro ********************************************************************  -->
-  <xacro:macro name="rrbot" params="parent prefix">
 <!-- ****************************************************** Base Joint ***************************************************************  -->
     <joint name="${prefix}base_joint" type="fixed">
       <origin xyz="0 0 0" rpy="0 0 0" />
-      <parent link="${parent}"/>
+      <parent link="world"/>
       <child link="${prefix}base_link" />
     </joint>
@@ -187,8 +187,4 @@
 <!-- ****************************************************** Camera Optical Link ******************************************************  -->
     <link name="${prefix}camera_link_optical"/>
-<!-- ****************************************************** End Macro ****************************************************************  -->
-  </xacro:macro>
-<!-- ****************************************************** Expand Macro *************************************************************  -->
-  <xacro:rrbot parent="world" prefix="" />
 <!-- ****************************************************** END **********************************************************************  -->
 </robot>
