Commit message: u

File: gazebo/gz_rrbot.xacro (robot description, xacro)
@@ -6,5 +6,5 @@
 <!-- *********************************************************************************************************************************  -->
 <!-- ****************************************************** Base Link ****************************************************************  -->
-  <gazebo reference="${prefix}base_link">
+  <gazebo reference="${prefix}base">
       <material>Gazebo/Orange</material>
   </gazebo>
@@ -18,5 +18,5 @@
   </gazebo>
 <!-- ****************************************************** Camera Link **************************************************************  -->
-  <gazebo reference="${prefix}camera_link">
+  <gazebo reference="${prefix}camera">
       <material>Gazebo/Green</material>
   </gazebo>

File: xacro/rrbot.xacro (robot description, xacro)
@@ -6,185 +6,190 @@
 <!-- *********************************************************************************************************************************  -->
 <!-- ****************************************************** Parameters ***************************************************************  -->
-    <xacro:property name="mesh_path"    value="package://robot_gazebo/meshes/rrbot/" />
-    <xacro:property name="name_space"     value="rrbot"  />
-    <xacro:property name="prefix"         value=""  />
-    <xacro:property name="mass"         value="1"     /> <!-- arbitrary value for mass -->
-    <xacro:property name="width"        value="0.1"   /> <!-- Square dimensions (widthxwidth) of beams -->
-    <xacro:property name="height1"      value="2"     /> <!-- Link 1 -->
-    <xacro:property name="height2"      value="1"     /> <!-- Link 2 -->
-    <xacro:property name="height3"      value="1"     /> <!-- Link 3 -->
-    <xacro:property name="camera_link"  value="0.05"  /> <!-- Size of square 'camera' box -->
-    <xacro:property name="axel_offset"  value="0.05"  /> <!-- Space btw top of beam and the each joint -->
+  <xacro:property name="mesh_path"    value="package://robot_gazebo/meshes/rrbot/" />
+  <xacro:property name="name_space"     value="rrbot"  />
+  <xacro:property name="prefix"         value=""  />
+  <xacro:property name="mass"         value="1"     /> <!-- arbitrary value for mass -->
+  <xacro:property name="width"        value="0.1"   /> <!-- Square dimensions (widthxwidth) of beams -->
+  <xacro:property name="height1"      value="2"     /> <!-- Link 1 -->
+  <xacro:property name="height2"      value="1"     /> <!-- Link 2 -->
+  <xacro:property name="height3"      value="1"     /> <!-- Link 3 -->
+  <xacro:property name="camera_mass"    value="1e-5"     />
+  <xacro:property name="camera_width"   value="0.05"     />
+  <xacro:property name="camera_length"  value="0.05"     />
+  <xacro:property name="camera_height"  value="0.05"     />
+  <xacro:property name="camera_x"       value="0.05"     />
+  <xacro:property name="camera_z"       value="${height3 - axel_offset*2}" />
+  <xacro:property name="axel_offset"  value="0.05"  /> <!-- Space btw top of beam and the each joint -->
 <!-- ****************************************************** Includes *****************************************************************  -->
   <xacro:include filename="$(find robot_gazebo)/xacro/common_rviz_materials.xacro" />   <!-- RVIZ Colors                                -->
   <xacro:include filename="$(find robot_gazebo)/gazebo/gz_rrbot.xacro" />               <!-- Gazebo                                     -->
 <!-- ****************************************************** Base Joint ***************************************************************  -->
-    <joint name="${prefix}base_joint" type="fixed">
-      <origin xyz="0 0 0" rpy="0 0 0" />
-      <parent link="world"/>
-      <child link="${prefix}base_link" />
-    </joint>
+  <joint name="${prefix}base_joint" type="fixed">
+    <origin xyz="0 0 0" rpy="0 0 0" />
+    <parent link="world"/>
+    <child link="${prefix}base" />
+  </joint>
 <!-- ****************************************************** Base Link ****************************************************************  -->
-    <link name="${prefix}base_link">
-      <collision>
-        <origin xyz="0 0 ${height1/2}" rpy="0 0 0"/>
-        <geometry>
-          <box size="${width} ${width} ${height1}"/>
-        </geometry>
-      </collision>
-      <visual>
-        <origin xyz="0 0 ${height1/2}" rpy="0 0 0"/>
-        <geometry>
-          <box size="${width} ${width} ${height1}"/>
-        </geometry>
-        <material name="orange"/>
-      </visual>
-      <inertial>
-        <origin xyz="0 0 ${height1/2}" rpy="0 0 0"/>
-        <mass value="${mass}"/>
-        <inertia
-          ixx="${mass / 12.0 * (width*width + height1*height1)}" ixy="0.0" ixz="0.0"
-          iyy="${mass / 12.0 * (height1*height1 + width*width)}" iyz="0.0"
-          izz="${mass / 12.0 * (width*width + width*width)}"/>
-      </inertial>
-    </link>
+  <link name="${prefix}base">
+    <collision>
+      <origin xyz="0 0 ${height1/2}" rpy="0 0 0"/>
+      <geometry>
+        <box size="${width} ${width} ${height1}"/>
+      </geometry>
+    </collision>
+    <visual>
+      <origin xyz="0 0 ${height1/2}" rpy="0 0 0"/>
+      <geometry>
+        <box size="${width} ${width} ${height1}"/>
+      </geometry>
+      <material name="orange"/>
+    </visual>
+    <inertial>
+      <origin xyz="0 0 ${height1/2}" rpy="0 0 0"/>
+      <mass value="${mass}"/>
+      <inertia
+        ixx="${mass / 12.0 * (width*width + height1*height1)}" ixy="0.0" ixz="0.0"
+        iyy="${mass / 12.0 * (height1*height1 + width*width)}" iyz="0.0"
+        izz="${mass / 12.0 * (width*width + width*width)}"/>
+    </inertial>
+  </link>
 <!-- ****************************************************** Joint 1 ******************************************************************  -->
-    <joint name="${prefix}joint1" type="continuous">
-      <parent link="${prefix}base_link"/>
-      <child link="${prefix}link1"/>
-      <origin xyz="0 ${width} ${height1 - axel_offset}" rpy="0 0 0"/>
-      <axis xyz="0 1 0"/>
-      <dynamics damping="0.7"/>
-    </joint>
+  <joint name="${prefix}joint1" type="continuous">
+    <parent link="${prefix}base"/>
+    <child link="${prefix}link1"/>
+    <origin xyz="0 ${width} ${height1 - axel_offset}" rpy="0 0 0"/>
+    <axis xyz="0 1 0"/>
+    <dynamics damping="0.7"/>
+  </joint>
 <!-- ****************************************************** Link 1 *******************************************************************  -->
-    <link name="${prefix}link1">
-      <collision>
-        <origin xyz="0 0 ${height2/2 - axel_offset}" rpy="0 0 0"/>
-        <geometry>
-          <box size="${width} ${width} ${height2}"/>
-        </geometry>
-      </collision>
-      <visual>
-        <origin xyz="0 0 ${height2/2 - axel_offset}" rpy="0 0 0"/>
-        <geometry>
-          <box size="${width} ${width} ${height2}"/>
-        </geometry>
-        <material name="yellow"/>
-      </visual>
-      <inertial>
-        <origin xyz="0 0 ${height2/2 - axel_offset}" rpy="0 0 0"/>
-        <mass value="${mass}"/>
-        <inertia
-          ixx="${mass / 12.0 * (width*width + height2*height2)}" ixy="0.0" ixz="0.0"
-          iyy="${mass / 12.0 * (height2*height2 + width*width)}" iyz="0.0"
-          izz="${mass / 12.0 * (width*width + width*width)}"/>
-      </inertial>
-    </link>
+  <link name="${prefix}link1">
+    <collision>
+      <origin xyz="0 0 ${height2/2 - axel_offset}" rpy="0 0 0"/>
+      <geometry>
+        <box size="${width} ${width} ${height2}"/>
+      </geometry>
+    </collision>
+    <visual>
+      <origin xyz="0 0 ${height2/2 - axel_offset}" rpy="0 0 0"/>
+      <geometry>
+        <box size="${width} ${width} ${height2}"/>
+      </geometry>
+      <material name="yellow"/>
+    </visual>
+    <inertial>
+      <origin xyz="0 0 ${height2/2 - axel_offset}" rpy="0 0 0"/>
+      <mass value="${mass}"/>
+      <inertia
+        ixx="${mass / 12.0 * (width*width + height2*height2)}" ixy="0.0" ixz="0.0"
+        iyy="${mass / 12.0 * (height2*height2 + width*width)}" iyz="0.0"
+        izz="${mass / 12.0 * (width*width + width*width)}"/>
+    </inertial>
+  </link>
 <!-- ****************************************************** Joint 2 ******************************************************************  -->
-    <joint name="${prefix}joint2" type="continuous">
-      <parent link="${prefix}link1"/>
-      <child link="${prefix}link2"/>
-      <origin xyz="0 ${width} ${height2 - axel_offset*2}" rpy="0 0 0"/>
-      <axis xyz="0 1 0"/>
-      <dynamics damping="0.7"/>
-    </joint>
+  <joint name="${prefix}joint2" type="continuous">
+    <parent link="${prefix}link1"/>
+    <child link="${prefix}link2"/>
+    <origin xyz="0 ${width} ${height2 - axel_offset*2}" rpy="0 0 0"/>
+    <axis xyz="0 1 0"/>
+    <dynamics damping="0.7"/>
+  </joint>
 <!-- ****************************************************** Link 2 *******************************************************************  -->
-    <link name="${prefix}link2">
-      <collision>
-        <origin xyz="0 0 ${height3/2 - axel_offset}" rpy="0 0 0"/>
-        <geometry>
-          <box size="${width} ${width} ${height3}"/>
-        </geometry>
-      </collision>
-      <visual>
-        <origin xyz="0 0 ${height3/2 - axel_offset}" rpy="0 0 0"/>
-        <geometry>
-          <box size="${width} ${width} ${height3}"/>
-        </geometry>
-        <material name="orange"/>
-      </visual>
-      <inertial>
-        <origin xyz="0 0 ${height3/2 - axel_offset}" rpy="0 0 0"/>
-        <mass value="${mass}"/>
-        <inertia
-          ixx="${mass / 12.0 * (width*width + height3*height3)}" ixy="0.0" ixz="0.0"
-          iyy="${mass / 12.0 * (height3*height3 + width*width)}" iyz="0.0"
-          izz="${mass / 12.0 * (width*width + width*width)}"/>
-      </inertial>
-    </link>
+  <link name="${prefix}link2">
+    <collision>
+      <origin xyz="0 0 ${height3/2 - axel_offset}" rpy="0 0 0"/>
+      <geometry>
+        <box size="${width} ${width} ${height3}"/>
+      </geometry>
+    </collision>
+    <visual>
+      <origin xyz="0 0 ${height3/2 - axel_offset}" rpy="0 0 0"/>
+      <geometry>
+        <box size="${width} ${width} ${height3}"/>
+      </geometry>
+      <material name="orange"/>
+    </visual>
+    <inertial>
+      <origin xyz="0 0 ${height3/2 - axel_offset}" rpy="0 0 0"/>
+      <mass value="${mass}"/>
+      <inertia
+        ixx="${mass / 12.0 * (width*width + height3*height3)}" ixy="0.0" ixz="0.0"
+        iyy="${mass / 12.0 * (height3*height3 + width*width)}" iyz="0.0"
+        izz="${mass / 12.0 * (width*width + width*width)}"/>
+    </inertial>
+  </link>
 <!-- ****************************************************** Tool Joint ***************************************************************  -->
-    <joint name="${prefix}tool_joint" type="fixed">
-      <origin xyz="0 0 1" rpy="0 0 0" />
-      <parent link="${prefix}link2"/>
-      <child link="${prefix}tool_link" />
-    </joint>
+  <joint name="${prefix}tool_joint" type="fixed">
+    <origin xyz="0 0 1" rpy="0 0 0" />
+    <parent link="${prefix}link2"/>
+    <child link="${prefix}tool" />
+  </joint>
 <!-- ****************************************************** Tool Link ****************************************************************  -->
-    <link name="${prefix}tool_link" />
+  <link name="${prefix}tool" />
 <!-- ****************************************************** Hokuyo Joint *************************************************************  -->
-    <joint name="${prefix}hokuyo_joint" type="fixed">
-      <axis xyz="0 1 0" />
-      <origin xyz="0 0 ${height3 - axel_offset/2}" rpy="0 0 0"/>
-      <parent link="${prefix}link2"/>
-      <child link="${prefix}hokuyo_link"/>
-    </joint>
+  <joint name="${prefix}hokuyo_joint" type="fixed">
+    <axis xyz="0 1 0" />
+    <origin xyz="0 0 ${height3 - axel_offset/2}" rpy="0 0 0"/>
+    <parent link="${prefix}link2"/>
+    <child link="${prefix}hokuyo"/>
+  </joint>
 <!-- ****************************************************** Hokuyo Link **************************************************************  -->
-    <link name="${prefix}hokuyo_link">
-      <collision>
-        <origin xyz="0 0 0" rpy="0 0 0"/>
-        <geometry>
-          <box size="0.1 0.1 0.1"/>
-        </geometry>
-      </collision>
-      <visual>
-        <origin xyz="0 0 0" rpy="0 0 0"/>
-        <geometry>
-          <mesh filename="${mesh_path}hokuyo.dae"/>
-        </geometry>
-      </visual>
-      <inertial>
-        <mass value="1e-5" />
-        <origin xyz="0 0 0" rpy="0 0 0"/>
-        <inertia ixx="1e-6" ixy="0" ixz="0" iyy="1e-6" iyz="0" izz="1e-6" />
-      </inertial>
-    </link>
+  <link name="${prefix}hokuyo">
+    <collision>
+      <origin xyz="0 0 0" rpy="0 0 0"/>
+      <geometry>
+        <box size="0.1 0.1 0.1"/>
+      </geometry>
+    </collision>
+    <visual>
+      <origin xyz="0 0 0" rpy="0 0 0"/>
+      <geometry>
+        <mesh filename="${mesh_path}hokuyo.dae"/>
+      </geometry>
+    </visual>
+    <inertial>
+      <mass value="1e-5" />
+      <origin xyz="0 0 0" rpy="0 0 0"/>
+      <inertia ixx="1e-6" ixy="0" ixz="0" iyy="1e-6" iyz="0" izz="1e-6" />
+    </inertial>
+  </link>
 <!-- ****************************************************** Camera Joint *************************************************************  -->
-    <joint name="${prefix}camera_joint" type="fixed">
-      <axis xyz="0 1 0" />
-      <origin xyz="${camera_link} 0 ${height3 - axel_offset*2}" rpy="0 0 0"/>
-      <parent link="${prefix}link2"/>
-      <child link="${prefix}camera_link"/>
-    </joint>
+  <joint name="${prefix}camera_joint" type="fixed">
+    <axis xyz="0 1 0" />
+    <origin xyz="${camera_x} 0 ${camera_z}" rpy="0 0 0"/>
+    <parent link="${prefix}link2"/>
+    <child link="${prefix}camera"/>
+  </joint>
 <!-- ****************************************************** Camera Link **************************************************************  -->
-    <link name="${prefix}camera_link">
-      <collision>
-        <origin xyz="0 0 0" rpy="0 0 0"/>
-        <geometry>
-          <box size="${camera_link} ${camera_link} ${camera_link}"/>
-        </geometry>
-      </collision>
-      <visual>
-        <origin xyz="0 0 0" rpy="0 0 0"/>
-        <geometry>
-          <box size="${camera_link} ${camera_link} ${camera_link}"/>
-        </geometry>
-        <material name="red"/>
-      </visual>
-      <inertial>
-        <mass value="1e-5" />
-        <origin xyz="0 0 0" rpy="0 0 0"/>
-        <inertia ixx="1e-6" ixy="0" ixz="0" iyy="1e-6" iyz="0" izz="1e-6" />
-      </inertial>
-    </link>
+<link name="${prefix}camera">
+  <inertial>
+    <mass value="${camera_mass}"/>
+    <origin xyz="0 0 0" rpy=" 0 0 0"/>
+    <inertia ixx="1e-6" ixy="0" ixz="0" iyy="1e-6" iyz="0" izz="1e-6" />
+  </inertial>
+  <visual name="camera_visual">
+    <origin xyz="0 0 0" rpy="0 0 0" />
+    <geometry>
+      <box size="${camera_length} ${camera_width} ${camera_height}"/>
+    </geometry>
+    <material name="green"/>
+  </visual>
+  <collision name="camera_colision">
+    <origin xyz="0 0 0" rpy="0 0 0" />
+    <geometry>
+      <box size="${camera_length} ${camera_width} ${camera_height}"/>
+    </geometry>
+  </collision>
+</link>
 <!-- ****************************************************** Camera Optical Joint *****************************************************  -->
 <!-- generate an optical frame http://www.ros.org/reps/rep-0103.html#suffix-frames so that ros and opencv can operate on the camera     -->
 <!-- frame correctly. these values have to be these values otherwise the gazebo camera image won't be aligned properly with the frame   -->
 <!-- it is supposedly originating from                                                                                                  -->                                                                                                                   -->
-    <joint name="${prefix}camera_optical_joint" type="fixed">
-      <origin xyz="0 0 0" rpy="${-pi/2} 0 ${-pi/2}"/>
-      <parent link="${prefix}camera_link"/>
-      <child link="${prefix}camera_link_optical"/>
-    </joint>
+  <joint name="${prefix}camera_optical_joint" type="fixed">
+    <origin xyz="0 0 0" rpy="${-pi/2} 0 ${-pi/2}"/>
+    <parent link="${prefix}camera"/>
+    <child link="${prefix}camera_optical"/>
+  </joint>
 <!-- ****************************************************** Camera Optical Link ******************************************************  -->
-    <link name="${prefix}camera_link_optical"/>
+  <link name="${prefix}camera_optical"/>
 <!-- ****************************************************** END **********************************************************************  -->
 </robot>

File: xacro/skidbot.xacro (robot description, xacro)
@@ -19,5 +19,5 @@
   <xacro:property name="wheel_x"        value="0.12"     /> <!-- x offset from base center -->
   <xacro:property name="wheel_y"        value="${(base_width+wheel_width)/2+wheel_gap}" />
-  <xacro:property name="camera_mass"    value="0.1"      />
+  <xacro:property name="camera_mass"    value="1e-5"     />
   <xacro:property name="camera_width"   value="0.05"     />
   <xacro:property name="camera_length"  value="0.05"     />
