Commit message: u

File: gazebo/gz_rrbot.xacro (robot description, xacro)
@@ -10,9 +10,9 @@
   </gazebo>
 <!-- ****************************************************** Link 1 *******************************************************************  -->
-  <gazebo reference="${prefix}link1">
+  <gazebo reference="${prefix}link2">
       <material>Gazebo/Orange</material>
   </gazebo>
 <!-- ****************************************************** Link 2 *******************************************************************  -->
-  <gazebo reference="${prefix}link2">
+  <gazebo reference="${prefix}link3">
       <material>Gazebo/Orange</material>
   </gazebo>

File: urdf/rrbot.urdf (robot description, URDF)
Before this commit: robot rrbot, 8 links, 7 joints
Links:
- removed link link1
- added link link3, mass 1; collision box size=0.1 0.1 1; visual box size=0.1 0.1 1
- link hokuyo: mass 1e-5 -> 1e-05; geometry collision mesh filename=package://robot_gazebo/meshes/rrbot/hokuyo.dae; visual mesh filename=package://robot_gazebo/meshes/rrbot/hokuyo.dae
Joints:
- joint camera_joint: origin xyz=0.05 0 0.9 rpy=0 0 0 -> xyz=0.07500000000000001 0 0.9 rpy=0 0 0; parent link2 -> link3
- joint hokuyo_joint: parent link2 -> link3
- joint joint1: child link1 -> link2
- joint joint2: child link2 -> link3; parent link1 -> link2
- joint tool_joint: parent link2 -> link3

File: xacro/rrbot.xacro (robot description, xacro)
@@ -9,16 +9,26 @@
   <xacro:property name="name_space"     value="rrbot"  />
   <xacro:property name="prefix"         value=""  />
-  <xacro:property name="mass"         value="1"     /> <!-- arbitrary value for mass -->
-  <xacro:property name="width"        value="0.1"   /> <!-- Square dimensions (widthxwidth) of beams -->
-  <xacro:property name="height1"      value="2"     /> <!-- Link 1 -->
-  <xacro:property name="height2"      value="1"     /> <!-- Link 2 -->
-  <xacro:property name="height3"      value="1"     /> <!-- Link 3 -->
+  <xacro:property name="mass"           value="1"     /> <!-- arbitrary value for mass -->
+  <xacro:property name="width"          value="0.1"   /> <!-- Square dimensions (widthxwidth) of beams -->
+  <xacro:property name="height1"        value="2"     /> <!-- Link 1 (Base) -->
+  <xacro:property name="height2"        value="1"     /> <!-- Link 2 -->
+  <xacro:property name="height3"        value="1"     /> <!-- Link 3 -->
+  <xacro:property name="joint_gap"      value="0.05"                   /> <!-- Space btw top of beam and the each joint -->
+  <xacro:property name="joint1_y"       value="${width}"               />
+  <xacro:property name="joint1_z"       value="${height1-joint_gap}"   />
+  <xacro:property name="joint2_y"       value="${width}"               />
+  <xacro:property name="joint2_z"       value="${height2-joint_gap*2}" />
   <xacro:property name="camera_mass"    value="1e-5"     />
   <xacro:property name="camera_width"   value="0.05"     />
   <xacro:property name="camera_length"  value="0.05"     />
   <xacro:property name="camera_height"  value="0.05"     />
-  <xacro:property name="camera_x"       value="0.05"     />
-  <xacro:property name="camera_z"       value="${height3 - axel_offset*2}" />
-  <xacro:property name="axel_offset"  value="0.05"  /> <!-- Space btw top of beam and the each joint -->
+  <xacro:property name="camera_x"       value="${(width+camera_width)/2}" />
+  <xacro:property name="camera_z"       value="${height3-joint_gap*2}" />
+  <xacro:property name="hokuyo_mass"    value="1e-5"     />
+  <xacro:property name="hokuyo_width"   value="0.05"     />
+  <xacro:property name="hokuyo_length"  value="0.05"     />
+  <xacro:property name="hokuyo_height"  value="0.0706"   />
+  <xacro:property name="hokuyo_z"       value="${height3-joint_gap/2}" />
+  <xacro:property name="tool_z"         value="${height3}" />
 <!-- ****************************************************** Includes *****************************************************************  -->
   <xacro:include filename="$(find robot_gazebo)/xacro/common_rviz_materials.xacro" />   <!-- RVIZ Colors                                -->
@@ -57,13 +67,13 @@
   <joint name="${prefix}joint1" type="continuous">
     <parent link="${prefix}base"/>
-    <child link="${prefix}link1"/>
-    <origin xyz="0 ${width} ${height1 - axel_offset}" rpy="0 0 0"/>
+    <child link="${prefix}link2"/>
+    <origin xyz="0 ${joint1_y} ${joint1_z}" rpy="0 0 0"/>
     <axis xyz="0 1 0"/>
     <dynamics damping="0.7"/>
   </joint>
-<!-- ****************************************************** Link 1 *******************************************************************  -->
-  <link name="${prefix}link1">
-    <collision>
-      <origin xyz="0 0 ${height2/2 - axel_offset}" rpy="0 0 0"/>
+<!-- ****************************************************** Link 2 *******************************************************************  -->
+  <link name="${prefix}link2">
+    <collision>
+      <origin xyz="0 0 ${height2/2 - joint_gap}" rpy="0 0 0"/>
       <geometry>
         <box size="${width} ${width} ${height2}"/>
@@ -71,5 +81,5 @@
     </collision>
     <visual>
-      <origin xyz="0 0 ${height2/2 - axel_offset}" rpy="0 0 0"/>
+      <origin xyz="0 0 ${height2/2 - joint_gap}" rpy="0 0 0"/>
       <geometry>
         <box size="${width} ${width} ${height2}"/>
@@ -78,5 +88,5 @@
     </visual>
     <inertial>
-      <origin xyz="0 0 ${height2/2 - axel_offset}" rpy="0 0 0"/>
+      <origin xyz="0 0 ${height2/2 - joint_gap}" rpy="0 0 0"/>
       <mass value="${mass}"/>
       <inertia
@@ -88,14 +98,14 @@
 <!-- ****************************************************** Joint 2 ******************************************************************  -->
   <joint name="${prefix}joint2" type="continuous">
-    <parent link="${prefix}link1"/>
-    <child link="${prefix}link2"/>
-    <origin xyz="0 ${width} ${height2 - axel_offset*2}" rpy="0 0 0"/>
+    <parent link="${prefix}link2"/>
+    <child link="${prefix}link3"/>
+    <origin xyz="0 ${joint2_y} ${joint2_z}" rpy="0 0 0"/>
     <axis xyz="0 1 0"/>
     <dynamics damping="0.7"/>
   </joint>
-<!-- ****************************************************** Link 2 *******************************************************************  -->
-  <link name="${prefix}link2">
-    <collision>
-      <origin xyz="0 0 ${height3/2 - axel_offset}" rpy="0 0 0"/>
+<!-- ****************************************************** Link 3 *******************************************************************  -->
+  <link name="${prefix}link3">
+    <collision>
+      <origin xyz="0 0 ${height3/2 - joint_gap}" rpy="0 0 0"/>
       <geometry>
         <box size="${width} ${width} ${height3}"/>
@@ -103,5 +113,5 @@
     </collision>
     <visual>
-      <origin xyz="0 0 ${height3/2 - axel_offset}" rpy="0 0 0"/>
+      <origin xyz="0 0 ${height3/2 - joint_gap}" rpy="0 0 0"/>
       <geometry>
         <box size="${width} ${width} ${height3}"/>
@@ -110,5 +120,5 @@
     </visual>
     <inertial>
-      <origin xyz="0 0 ${height3/2 - axel_offset}" rpy="0 0 0"/>
+      <origin xyz="0 0 ${height3/2 - joint_gap}" rpy="0 0 0"/>
       <mass value="${mass}"/>
       <inertia
@@ -120,42 +130,15 @@
 <!-- ****************************************************** Tool Joint ***************************************************************  -->
   <joint name="${prefix}tool_joint" type="fixed">
-    <origin xyz="0 0 1" rpy="0 0 0" />
-    <parent link="${prefix}link2"/>
+    <origin xyz="0 0 ${tool_z}" rpy="0 0 0" />
+    <parent link="${prefix}link3"/>
     <child link="${prefix}tool" />
   </joint>
 <!-- ****************************************************** Tool Link ****************************************************************  -->
   <link name="${prefix}tool" />
-<!-- ****************************************************** Hokuyo Joint *************************************************************  -->
-  <joint name="${prefix}hokuyo_joint" type="fixed">
-    <axis xyz="0 1 0" />
-    <origin xyz="0 0 ${height3 - axel_offset/2}" rpy="0 0 0"/>
-    <parent link="${prefix}link2"/>
-    <child link="${prefix}hokuyo"/>
-  </joint>
-<!-- ****************************************************** Hokuyo Link **************************************************************  -->
-  <link name="${prefix}hokuyo">
-    <collision>
-      <origin xyz="0 0 0" rpy="0 0 0"/>
-      <geometry>
-        <box size="0.1 0.1 0.1"/>
-      </geometry>
-    </collision>
-    <visual>
-      <origin xyz="0 0 0" rpy="0 0 0"/>
-      <geometry>
-        <mesh filename="${mesh_path}hokuyo.dae"/>
-      </geometry>
-    </visual>
-    <inertial>
-      <mass value="1e-5" />
-      <origin xyz="0 0 0" rpy="0 0 0"/>
-      <inertia ixx="1e-6" ixy="0" ixz="0" iyy="1e-6" iyz="0" izz="1e-6" />
-    </inertial>
-  </link>
 <!-- ****************************************************** Camera Joint *************************************************************  -->
   <joint name="${prefix}camera_joint" type="fixed">
     <axis xyz="0 1 0" />
     <origin xyz="${camera_x} 0 ${camera_z}" rpy="0 0 0"/>
-    <parent link="${prefix}link2"/>
+    <parent link="${prefix}link3"/>
     <child link="${prefix}camera"/>
   </joint>
@@ -186,5 +169,5 @@
 <!-- it is supposedly originating from                                                                                                  -->                                                                                                                   -->
   <joint name="${prefix}camera_optical_joint" type="fixed">
-    <origin xyz="0 0 0" rpy="${-pi/2} 0 ${-pi/2}"/>
+    <origin xyz="0 0 0" rpy="${-radians(90)} 0 ${-radians(90)}"/>
     <parent link="${prefix}camera"/>
     <child link="${prefix}camera_optical"/>
@@ -192,4 +175,31 @@
 <!-- ****************************************************** Camera Optical Link ******************************************************  -->
   <link name="${prefix}camera_optical"/>
+<!-- ****************************************************** Hokuyo Joint *************************************************************  -->
+  <joint name="${prefix}hokuyo_joint" type="fixed">
+    <axis xyz="0 1 0" />
+    <origin xyz="0 0 ${hokuyo_z}" rpy="0 0 0"/>
+    <parent link="${prefix}link3"/>
+    <child link="${prefix}hokuyo"/>
+  </joint>
+<!-- ****************************************************** Hokuyo Link **************************************************************  -->
+  <link name="${prefix}hokuyo">
+    <collision>
+      <origin xyz="0 0 0" rpy="0 0 0"/>
+      <geometry>
+        <mesh filename="${mesh_path}hokuyo.dae"/> <!--  <box size="${hokuyo_length} ${hokuyo_width} ${hokuyo_height}"/> -->
+      </geometry>
+    </collision>
+    <visual>
+      <origin xyz="0 0 0" rpy="0 0 0"/>
+      <geometry>
+        <mesh filename="${mesh_path}hokuyo.dae"/> <!--  <box size="${hokuyo_length} ${hokuyo_width} ${hokuyo_height}"/> -->
+      </geometry>
+    </visual>
+    <inertial>
+      <mass value="${hokuyo_mass}" />
+      <origin xyz="0 0 0" rpy="0 0 0"/>
+      <inertia ixx="1e-6" ixy="0" ixz="0" iyy="1e-6" iyz="0" izz="1e-6" />
+    </inertial>
+  </link>
 <!-- ****************************************************** END **********************************************************************  -->
 </robot>

Commit message: u

File: gazebo/gz_rrbot.xacro (robot description, xacro)
@@ -26,4 +26,92 @@
     <static>true</static>
   </gazebo>
+<!-- ******************************************************  Camera ******************************************************************  -->
+  <gazebo reference="${prefix}camera">
+    <sensor type="camera" name="camera">
+      <update_rate>30.0</update_rate>
+      <camera name="head">
+        <horizontal_fov>${radians(80)}</horizontal_fov>
+        <image>
+          <width>1280</width>
+          <height>720</height>
+          <format>R8G8B8</format>
+        </image>
+        <clip>
+          <near>0.02</near>
+          <far>300</far>
+        </clip>
+        <noise>
+          <type>gaussian</type>
+          <!-- Noise is sampled independently per pixel on each frame.
+          That pixel's noise value is added to each of its color
+          channels, which at that point lie in the range [0,1]. -->
+          <mean>0.0</mean>
+          <stddev>0.007</stddev>
+        </noise>
+      </camera>
+      <plugin name="camera_controller" filename="libgazebo_ros_camera.so">
+        <ros>
+          <namespace>${name_space}</namespace>
+        </ros>
+        <alwaysOn>true</alwaysOn>
+        <updateRate>0.0</updateRate>
+        <cameraName>camera</cameraName>
+        <imageTopicName>image_raw</imageTopicName>
+        <cameraInfoTopicName>camera_info</cameraInfoTopicName>
+        <frameName>camera_optical</frameName>
+        <!-- setting hackBaseline to anything but 0.0 will cause a misalignment
+        between the gazebo sensor image and the frame it is supposed to
+        be attached to -->
+        <hackBaseline>0.0</hackBaseline>
+        <distortionK1>0.0</distortionK1>
+        <distortionK2>0.0</distortionK2>
+        <distortionK3>0.0</distortionK3>
+        <distortionT1>0.0</distortionT1>
+        <distortionT2>0.0</distortionT2>
+        <CxPrime>0</CxPrime>
+        <Cx>0.0</Cx>
+        <Cy>0.0</Cy>
+        <focalLength>0.0</focalLength>
+      </plugin>
+    </sensor>
+    <material>Gazebo/Green</material>
+  </gazebo>
+<!-- ****************************************************** hokuyo  ******************************************************************  -->
+  <gazebo reference="${prefix}hokuyo">
+    <sensor type="ray" name="head_hokuyo_sensor">
+      <plugin name="hokuyo" filename="libgazebo_ros_ray_sensor.so">
+        <ros>
+          <namespace>${name_space}</namespace>
+        </ros>
+        <output_type>sensor_msgs/LaserScan</output_type>
+      </plugin>
+      <update_rate>30</update_rate>
+      <pose>0 0 0 0 0 0</pose>
+      <visualize>false</visualize>
+      <ray>
+        <scan>
+          <horizontal>
+            <samples>720</samples>
+            <resolution>1</resolution>
+            <min_angle>-${radians(180)}</min_angle>
+            <max_angle> ${radians(180)}</max_angle>
+          </horizontal>
+        </scan>
+        <range>
+          <min>0.10</min>
+          <max>30.0</max>
+          <resolution>0.01</resolution>
+        </range>
+<!-- Noise parameters based on published spec for Hokuyo laser achieving "+-30mm" accuracy at range < 10m.  A mean of 0.0m and stddev   -->
+<!-- of 0.01m will put 99.7% of samples within 0.03m of the true reading.                                                               -->
+        <noise>
+          <type>gaussian</type>
+          <mean>0.0</mean>
+          <stddev>0.01</stddev>
+        </noise>
+      </ray>
+    </sensor>
+    <!-- <material>Gazebo/Red</material> -->
+  </gazebo>
 <!-- ****************************************************** END **********************************************************************  -->
 </robot>

File: gazebo/gz_skidbot.xacro (robot description, xacro)
@@ -53,16 +53,7 @@
 <!-- ******************************************************  Camera ******************************************************************  -->
   <gazebo reference="${prefix}camera">
-    <sensor type="camera" name="camera_sensor">
-      <plugin name="camera" filename="libgazebo_ros_camera.so">
-        <ros>
-          <namespace>${name_space}</namespace>
-        </ros>
-        <camera_name>camera</camera_name>
-        <frame_name>camera</frame_name>
-        <hack_baseline>0.07</hack_baseline>
-      </plugin>
+    <sensor type="camera" name="camera">
       <update_rate>30.0</update_rate>
-      <always_on>1</always_on>
-      <camera name="camera">
+      <camera name="head">
         <horizontal_fov>${radians(80)}</horizontal_fov>
         <image>
@@ -75,13 +66,37 @@
           <far>300</far>
         </clip>
-        <distortion>
-          <k1>0.0</k1>
-          <k2>0.0</k2>
-          <k3>0.0</k3>
-          <p1>0.0</p1>
-          <p2>0.0</p2>
-          <center>0.5 0.5</center>
-        </distortion>
+        <noise>
+          <type>gaussian</type>
+          <!-- Noise is sampled independently per pixel on each frame.
+          That pixel's noise value is added to each of its color
+          channels, which at that point lie in the range [0,1]. -->
+          <mean>0.0</mean>
+          <stddev>0.007</stddev>
+        </noise>
       </camera>
+      <plugin name="camera_controller" filename="libgazebo_ros_camera.so">
+        <ros>
+          <namespace>${name_space}</namespace>
+        </ros>
+        <alwaysOn>true</alwaysOn>
+        <updateRate>0.0</updateRate>
+        <cameraName>camera</cameraName>
+        <imageTopicName>image_raw</imageTopicName>
+        <cameraInfoTopicName>camera_info</cameraInfoTopicName>
+        <frameName>camera_optical</frameName>
+        <!-- setting hackBaseline to anything but 0.0 will cause a misalignment
+        between the gazebo sensor image and the frame it is supposed to
+        be attached to -->
+        <hackBaseline>0.0</hackBaseline>
+        <distortionK1>0.0</distortionK1>
+        <distortionK2>0.0</distortionK2>
+        <distortionK3>0.0</distortionK3>
+        <distortionT1>0.0</distortionT1>
+        <distortionT2>0.0</distortionT2>
+        <CxPrime>0</CxPrime>
+        <Cx>0.0</Cx>
+        <Cy>0.0</Cy>
+        <focalLength>0.0</focalLength>
+      </plugin>
     </sensor>
     <material>Gazebo/Green</material>
@@ -104,6 +119,6 @@
             <samples>720</samples>
             <resolution>1</resolution>
-            <min_angle>-${radians(90)}</min_angle>
-            <max_angle> ${radians(90)}</max_angle>
+            <min_angle>-${radians(180)}</min_angle>
+            <max_angle> ${radians(180)}</max_angle>
           </horizontal>
         </scan>

Commit message: u

File: gazebo/gz_rrbot.xacro (robot description, xacro)
@@ -26,4 +26,17 @@
     <static>true</static>
   </gazebo>
+<!-- ******************************************************  Joint States Publisher **************************************************  -->
+  <gazebo>
+    <plugin name="joint_states_pub" filename="libgazebo_ros_joint_state_publisher.so">
+      <ros>
+        <namespace>${name_space}</namespace>
+      </ros>
+      <joint_name>${prefix}base_joint</joint_name>
+      <joint_name>${prefix}joint1</joint_name>
+      <joint_name>${prefix}joint2</joint_name>
+      <joint_name>${prefix}tool_joint</joint_name>
+      <update_rate>100.0</update_rate>
+    </plugin>
+ </gazebo>
 <!-- ******************************************************  Camera ******************************************************************  -->
   <gazebo reference="${prefix}camera">

File: urdf/diffbot.urdf (robot description, URDF)
Before this commit: robot diffbot, 7 links, 6 joints
Links:
- added link camera_optical
Joints:
- added joint camera_optical_joint: type fixed, parent camera, child camera_optical, origin xyz=0 0 0 rpy=-1.5707963267948966 0 -1.5707963267948966

File: xacro/rrbot.xacro (robot description, xacro)
@@ -7,6 +7,6 @@
 <!-- ****************************************************** Parameters ***************************************************************  -->
   <xacro:property name="mesh_path"      value="package://robot_gazebo/meshes/rrbot/" />
-  <xacro:property name="name_space"     default="rrbot"  />
-  <xacro:property name="prefix"         default=""  />
+  <xacro:property name="name_space"     value="rrbot" />
+  <xacro:property name="prefix"         value=""      />
   <xacro:property name="mass"           value="1"     /> <!-- arbitrary value for mass -->
   <xacro:property name="width"          value="0.1"   /> <!-- Square dimensions (widthxwidth) of beams -->

Commit message: u

File: gazebo/gz_rrbot.xacro (robot description, xacro)
@@ -37,5 +37,5 @@
   <gazebo>
     <plugin name="gz_ros2_control" filename="libgazebo_ros2_control.so">
-      <parameters>${config_path}rrbot_forward_position.yaml</parameters>
+      <!--<parameters>${config_path}rrbot_forward_position.yaml</parameters>-->
     </plugin>
   </gazebo>
@@ -126,5 +126,4 @@
       </ray>
     </sensor>
-    <!-- <material>Gazebo/Red</material> -->
   </gazebo>
 <!-- ****************************************************** END **********************************************************************  -->
