Commit message: u

File: gazebo/gz_gripper.xacro (robot description, xacro)
@@ -18,5 +18,5 @@
       <robot_param>robot_description</robot_param>
       <robot_param_node>robot_state_publisher</robot_param_node>
-      <parameters>$(find bots)/config/gripper.yaml</parameters>
+      <parameters>${config_path}config/gripper.yaml</parameters>
     </plugin>
   </gazebo>

File: xacro/gripper.xacro (robot description, xacro)
@@ -7,5 +7,6 @@
 <!-- ****************************************************** Parameters ***************************************************************  -->
     <xacro:property name="pkg_path"     value="$(find bots)"                />
-    <xacro:property name="mesh_path"    value="${pkg_path}/meshes/gripper/"    />
+    <xacro:property name="mesh_path"    value="${pkg_path}/meshes/gripper/" />
+    <xacro:property name="config_path"  value="${pkg_path}/config/"         />
     <xacro:property name="name_space"   value="cart" />
     <xacro:property name="prefix"       value=""      />
