Commit message: u

File: gazebo/gz_diffbot.xacro (robot description, xacro)
@@ -1,171 +1,30 @@
 <?xml version="1.0"?>
-<robot name="diffbot" xmlns:xacro="http://www.ros.org/wiki/xacro">
+<robot xmlns:xacro="http://www.ros.org/wiki/xacro">
 <!-- ****************************************************** diffbot Robot ************************************************************  -->
 <!-- Muthanna Alwahash                                                                                                                  -->
 <!-- March 2022                                                                                                                         -->
 <!-- *********************************************************************************************************************************  -->
-<!-- ****************************************************** Parameters ***************************************************************  -->
-  <xacro:property name="base_mass"            value="0.3"               /> <!-- arbitrary value for base mass             -->
-  <xacro:property name="base_width"           value="0.1"               />
-  <xacro:property name="base_length"          value="0.1"               />
-  <xacro:property name="base_height"          value="0.05"              />
-  <xacro:property name="wheel_mass"           value="0.3"               /> <!-- arbitrary value for wheel mass            -->
-  <xacro:property name="wheel_len"            value="0.020"             />
-  <xacro:property name="wheel_radius"         value="0.015"             />
-  <xacro:property name="caster_wheel_mass"    value="0.1"               /> <!-- arbitrary value for caster wheel mass     -->
-  <xacro:property name="caster_wheel_radius"  value="0.015"             />
-  <xacro:property name="z_offset"             value="-${base_height/2}" /> <!-- Space btw top of beam and the each joint  -->
-<!-- ****************************************************** Import RVIZ Materials*****************************************************  -->
-  <xacro:include filename="$(find robot_gazebo)/xacro/common_rviz_materials.xacro" />
 <!-- ****************************************************** Macro ********************************************************************  -->
   <xacro:macro name="diffbot" params="prefix">
 <!-- ****************************************************** Base Link ****************************************************************  -->
-  <link name="${prefix}base_link">
-    <collision>
-      <origin xyz="0 0 0" rpy="0 0 0"/>
-      <geometry>
-        <box size="${base_width} ${base_length} ${base_height}"/>
-      </geometry>
-    </collision>
-    <visual>
-      <origin xyz="0 0 ${base_height/2}" rpy="0 0 0"/>
-      <geometry>
-        <box size="${base_width} ${base_length} ${base_height}"/>
-      </geometry>
-      <material name="orange"/>
-    </visual>
-    <inertial>
-      <origin xyz="0 0 0" rpy="0 0 0"/>
-      <mass value="${base_mass}"/>
-      <inertia
-        ixx="${base_mass / 12.0 * (base_length*base_length + base_height*base_height)}" ixy="0.0" ixz="0.0"
-        iyy="${base_mass / 12.0 * (base_height*base_height + base_width*base_width)}" iyz="0.0"
-        izz="${base_mass / 12.0 * (base_width*base_width + base_length*base_length)}"/>
-    </inertial>
-  </link>
-<!-- ****************************************************** Left Wheel Joint *********************************************************  -->
-    <joint name="${prefix}left_wheel_joint" type="continuous">
-      <parent link="${prefix}base_link"/>
-      <child link="${prefix}left_wheel"/>
-      <origin xyz="0 -${base_width/2} ${z_offset}" rpy="0 0 0"/>
-      <axis xyz="0 1 0"/>
-      <dynamics damping="0.2"/>
-    </joint>
+    <gazebo reference="${prefix}base_link">
+      <material>Gazebo/Blue</material>
+    </gazebo>
 <!-- ****************************************************** Left Wheel Link **********************************************************  -->
-    <link name="${prefix}left_wheel">
-      <collision>
-        <origin xyz="0 0 0" rpy="${pi/2} 0 0"/>
-        <geometry>
-          <cylinder length="${wheel_len}" radius="${wheel_radius}"/>
-        </geometry>
-      </collision>
-      <visual>
-        <origin xyz="0 0 0" rpy="${pi/2} 0 0"/>
-        <geometry>
-          <cylinder length="${wheel_len}" radius="${wheel_radius}"/>
-        </geometry>
-        <material name="black"/>
-      </visual>
-      <inertial>
-        <origin xyz="0 0 0" rpy="${pi/2} 0 0"/>
-        <mass value="${wheel_mass}"/>
-        <inertia
-          ixx="${wheel_mass / 12.0 * (3*wheel_radius + wheel_len*wheel_len)}" ixy="0.0" ixz="0.0"
-          iyy="${wheel_mass / 12.0 * wheel_radius*wheel_radius}" iyz="0.0"
-          izz="${wheel_mass / 12.0 * wheel_radius*wheel_radius}"/>
-      </inertial>
-    </link>
-<!-- ****************************************************** Right Wheel Joint ********************************************************  -->
-    <joint name="${prefix}right_wheel_joint" type="continuous">
-      <parent link="${prefix}base_link"/>
-      <child link="${prefix}right_wheel"/>
-      <origin xyz="0 ${base_width/2} ${z_offset}" rpy="0 0 0"/>
-      <axis xyz="0 1 0"/>
-      <dynamics damping="0.2"/>
-    </joint>
+    <gazebo reference="${prefix}left_wheel">
+      <material>Gazebo/Black</material>
+    </gazebo>
 <!-- ****************************************************** Right Wheel Link ********************************************************  -->
-    <link name="${prefix}right_wheel">
-      <collision>
-        <origin xyz="0 0 0" rpy="${pi/2} 0 0"/>
-        <geometry>
-          <cylinder length="${wheel_len}" radius="${wheel_radius}"/>
-        </geometry>
-      </collision>
-      <visual>
-        <origin xyz="0 0 0" rpy="${pi/2} 0 0"/>
-        <geometry>
-          <cylinder length="${wheel_len}" radius="${wheel_radius}"/>
-        </geometry>
-        <material name="black"/>
-      </visual>
-      <inertial>
-        <origin xyz="0 0 0" rpy="${pi/2} 0 0"/>
-        <mass value="${wheel_mass}"/>
-        <inertia
-          ixx="${wheel_mass / 12.0 * (3*wheel_radius + wheel_len*wheel_len)}" ixy="0.0" ixz="0.0"
-          iyy="${wheel_mass / 12.0 * wheel_radius*wheel_radius}" iyz="0.0"
-          izz="${wheel_mass / 12.0 * wheel_radius*wheel_radius}"/>
-      </inertial>
-    </link>
-<!-- ****************************************************** Front caster joint *******************************************************  -->
-    <joint name="${prefix}caster_frontal_wheel_joint" type="fixed">
-      <parent link="${prefix}base_link"/>
-      <child link="${prefix}caster_frontal_wheel"/>
-      <origin xyz="${base_width/2 - caster_wheel_radius} 0 ${z_offset}" rpy="0 0 0"/>
-    </joint>
+    <gazebo reference="${prefix}right_wheel">
+      <material>Gazebo/Black</material>
+    </gazebo>
 <!-- ****************************************************** Front caster Link ********************************************************  -->
-    <link name="${prefix}caster_frontal_wheel">
-      <collision>
-        <origin xyz="0 0 0" rpy="0 0 0"/>
-        <geometry>
-          <sphere radius="${caster_wheel_radius}"/>
-        </geometry>
-      </collision>
-      <visual>
-        <origin xyz="0 0 0" rpy="0 0 0"/>
-        <geometry>
-          <sphere radius="${caster_wheel_radius}"/>
-        </geometry>
-        <material name="white"/>
-      </visual>
-      <inertial>
-        <origin xyz="0 0 0" rpy="0 0 0"/>
-        <mass value="${caster_wheel_mass}"/>
-        <inertia
-          ixx="${caster_wheel_mass * 0.4 * (caster_wheel_radius * caster_wheel_radius)}" ixy="0.0" ixz="0.0"
-          iyy="${caster_wheel_mass * 0.4 * (caster_wheel_radius * caster_wheel_radius)}" iyz="0.0"
-          izz="${caster_wheel_mass * 0.4 * (caster_wheel_radius * caster_wheel_radius)}"/>
-      </inertial>
-    </link>
-<!-- ****************************************************** Rear Caster Joint ********************************************************  -->
-    <joint name="${prefix}caster_rear_wheel_joint" type="fixed">
-      <parent link="${prefix}base_link"/>
-      <child link="${prefix}caster_rear_wheel"/>
-      <origin xyz="${-base_width/2 + caster_wheel_radius} 0 ${z_offset}" rpy="0 0 0"/>
-    </joint>
+    <gazebo reference="${prefix}caster_frontal_wheel">
+      <material>Gazebo/White</material>
+    </gazebo>
 <!-- ****************************************************** Rear Caster Link *********************************************************  -->
-    <link name="${prefix}caster_rear_wheel">
-      <collision>
-        <origin xyz="0 0 0" rpy="0 0 0"/>
-        <geometry>
-          <sphere radius="${caster_wheel_radius}"/>
-        </geometry>
-      </collision>
-      <visual>
-        <origin xyz="0 0 0" rpy="0 0 0"/>
-        <geometry>
-          <sphere radius="${caster_wheel_radius}"/>
-        </geometry>
-        <material name="white"/>
-      </visual>
-      <inertial>
-        <origin xyz="0 0 0" rpy="0 0 0"/>
-        <mass value="${caster_wheel_mass}"/>
-        <inertia
-          ixx="${caster_wheel_mass * 0.4 * (caster_wheel_radius * caster_wheel_radius)}" ixy="0.0" ixz="0.0"
-          iyy="${caster_wheel_mass * 0.4 * (caster_wheel_radius * caster_wheel_radius)}" iyz="0.0"
-          izz="${caster_wheel_mass * 0.4 * (caster_wheel_radius * caster_wheel_radius)}"/>
-      </inertial>
-    </link>
+    <gazebo reference="${prefix}caster_rear_wheel">
+      <material>Gazebo/White</material>
+    </gazebo>
 <!-- ****************************************************** End Macro ****************************************************************  -->
   </xacro:macro>

File: xacro/diffbot.xacro (robot description, xacro)
@@ -16,6 +16,7 @@
   <xacro:property name="caster_wheel_radius"  value="0.015"             />
   <xacro:property name="z_offset"             value="-${base_height/2}" /> <!-- Space btw top of beam and the each joint  -->
-<!-- ****************************************************** Import RVIZ Materials*****************************************************  -->
-  <xacro:include filename="$(find robot_gazebo)/xacro/common_rviz_materials.xacro" />
+<!-- ****************************************************** Includes *****************************************************************  -->
+  <xacro:include filename="$(find robot_gazebo)/xacro/common_rviz_materials.xacro" />   <!-- RVIZ Colors                                -->
+  <xacro:include filename="$(find robot_gazebo)/gazebo/gz_diffbot.xacro" />             <!-- Gazebo                                     -->
 <!-- ****************************************************** Macro ********************************************************************  -->
   <xacro:macro name="diffbot" params="prefix">

Commit message: u

File: gazebo/gz_diffbot.xacro (robot description, xacro)
@@ -6,5 +6,5 @@
 <!-- *********************************************************************************************************************************  -->
 <!-- ****************************************************** Macro ********************************************************************  -->
-  <xacro:macro name="diffbot" params="prefix">
+  <xacro:macro name="diffbot_gz" params="prefix">
 <!-- ****************************************************** Base Link ****************************************************************  -->
     <gazebo reference="${prefix}base_link">
@@ -20,9 +20,9 @@
     </gazebo>
 <!-- ****************************************************** Front caster Link ********************************************************  -->
-    <gazebo reference="${prefix}caster_frontal_wheel">
+    <gazebo reference="${prefix}front_caster">
       <material>Gazebo/White</material>
     </gazebo>
 <!-- ****************************************************** Rear Caster Link *********************************************************  -->
-    <gazebo reference="${prefix}caster_rear_wheel">
+    <gazebo reference="${prefix}rear_caster">
       <material>Gazebo/White</material>
     </gazebo>
@@ -30,5 +30,5 @@
   </xacro:macro>
 <!-- ****************************************************** Expand Macro *************************************************************  -->
-  <xacro:diffbot prefix="" />
+  <xacro:diffbot_gz prefix="" />
 <!-- ****************************************************** END **********************************************************************  -->
 </robot>

File: urdf/diffbot.urdf (robot description, URDF)
Before this commit: robot diffbot, 6 links, 5 joints
Links:
- removed link caster_frontal_wheel
- removed link caster_rear_wheel
- added link front_caster, mass 0.1; collision sphere radius=0.05; visual sphere radius=0.05
- added link rear_caster, mass 0.1; collision sphere radius=0.05; visual sphere radius=0.05
- link left_wheel: geometry collision cylinder length=0.02 radius=0.05; visual cylinder length=0.02 radius=0.05
- link right_wheel: geometry collision cylinder length=0.02 radius=0.05; visual cylinder length=0.02 radius=0.05
Joints:
- removed joint caster_frontal_wheel_joint
- removed joint caster_rear_wheel_joint
- added joint front_caster_joint: type fixed, parent base_link, child front_caster, origin xyz=0.0 0 -0.025 rpy=0 0 0
- added joint rear_caster_joint: type fixed, parent base_link, child rear_caster, origin xyz=0.0 0 -0.025 rpy=0 0 0
- joint left_wheel_joint: origin xyz=0 -0.05 -0.025 rpy=0 0 0 -> xyz=0 -0.060000000000000005 -0.025 rpy=0 0 0
- joint right_wheel_joint: origin xyz=0 0.05 -0.025 rpy=0 0 0 -> xyz=0 0.060000000000000005 -0.025 rpy=0 0 0

File: xacro/diffbot.xacro (robot description, xacro)
@@ -7,12 +7,12 @@
 <!-- ****************************************************** Parameters ***************************************************************  -->
   <xacro:property name="base_mass"            value="0.3"               /> <!-- arbitrary value for base mass             -->
-  <xacro:property name="base_width"           value="0.1"               />
-  <xacro:property name="base_length"          value="0.1"               />
+  <xacro:property name="base_width"           value="0.10"              />
+  <xacro:property name="base_length"          value="0.20"              />
   <xacro:property name="base_height"          value="0.05"              />
   <xacro:property name="wheel_mass"           value="0.3"               /> <!-- arbitrary value for wheel mass            -->
-  <xacro:property name="wheel_len"            value="0.020"             />
-  <xacro:property name="wheel_radius"         value="0.015"             />
+  <xacro:property name="wheel_width"          value="0.010"             />
+  <xacro:property name="wheel_radius"         value="0.025"             />
   <xacro:property name="caster_wheel_mass"    value="0.1"               /> <!-- arbitrary value for caster wheel mass     -->
-  <xacro:property name="caster_wheel_radius"  value="0.015"             />
+  <xacro:property name="caster_wheel_radius"  value="${wheel_radius}"   />
   <xacro:property name="z_offset"             value="-${base_height/2}" /> <!-- Space btw top of beam and the each joint  -->
 <!-- ****************************************************** Includes *****************************************************************  -->
@@ -22,5 +22,5 @@
   <xacro:macro name="diffbot" params="prefix">
 <!-- ****************************************************** Base Footprint ***********************************************************  -->
-    <link name="base_footprint"/>
+    <link name="${prefix}base_footprint"/>
 <!-- ****************************************************** Base Joint ***************************************************************  -->
     <joint name="base_joint" type="fixed">
@@ -40,5 +40,5 @@
       <origin xyz="0 0 0" rpy="0 0 0"/>
       <geometry>
-        <box size="${base_width} ${base_length} ${base_height}"/>
+        <box size="${base_length} ${base_width} ${base_height}"/>
       </geometry>
       <material name="orange"/>
@@ -57,5 +57,5 @@
       <parent link="${prefix}base_link"/>
       <child link="${prefix}left_wheel"/>
-      <origin xyz="0 -${base_width/2} ${z_offset}" rpy="0 0 0"/>
+      <origin xyz="0 -${(base_width+wheel_width)/2} ${z_offset}" rpy="0 0 0"/>
       <axis xyz="0 1 0"/>
       <dynamics damping="0.2"/>
@@ -66,5 +66,5 @@
         <origin xyz="0 0 0" rpy="${pi/2} 0 0"/>
         <geometry>
-          <cylinder length="${wheel_len}" radius="${wheel_radius}"/>
+          <cylinder length="${wheel_width}" radius="${wheel_radius}"/>
         </geometry>
       </collision>
@@ -72,5 +72,5 @@
         <origin xyz="0 0 0" rpy="${pi/2} 0 0"/>
         <geometry>
-          <cylinder length="${wheel_len}" radius="${wheel_radius}"/>
+          <cylinder length="${wheel_width}" radius="${wheel_radius}"/>
         </geometry>
         <material name="black"/>
@@ -80,5 +80,5 @@
         <mass value="${wheel_mass}"/>
         <inertia
-          ixx="${wheel_mass / 12.0 * (3*wheel_radius + wheel_len*wheel_len)}" ixy="0.0" ixz="0.0"
+          ixx="${wheel_mass / 12.0 * (3*wheel_radius + wheel_width*wheel_width)}" ixy="0.0" ixz="0.0"
           iyy="${wheel_mass / 12.0 * wheel_radius*wheel_radius}" iyz="0.0"
           izz="${wheel_mass / 12.0 * wheel_radius*wheel_radius}"/>
@@ -89,5 +89,5 @@
       <parent link="${prefix}base_link"/>
       <child link="${prefix}right_wheel"/>
-      <origin xyz="0 ${base_width/2} ${z_offset}" rpy="0 0 0"/>
+      <origin xyz="0 ${(base_width+wheel_width)/2} ${z_offset}" rpy="0 0 0"/>
       <axis xyz="0 1 0"/>
       <dynamics damping="0.2"/>
@@ -98,5 +98,5 @@
         <origin xyz="0 0 0" rpy="${pi/2} 0 0"/>
         <geometry>
-          <cylinder length="${wheel_len}" radius="${wheel_radius}"/>
+          <cylinder length="${wheel_width}" radius="${wheel_radius}"/>
         </geometry>
       </collision>
@@ -104,5 +104,5 @@
         <origin xyz="0 0 0" rpy="${pi/2} 0 0"/>
         <geometry>
-          <cylinder length="${wheel_len}" radius="${wheel_radius}"/>
+          <cylinder length="${wheel_width}" radius="${wheel_radius}"/>
         </geometry>
         <material name="black"/>
@@ -112,5 +112,5 @@
         <mass value="${wheel_mass}"/>
         <inertia
-          ixx="${wheel_mass / 12.0 * (3*wheel_radius + wheel_len*wheel_len)}" ixy="0.0" ixz="0.0"
+          ixx="${wheel_mass / 12.0 * (3*wheel_radius + wheel_width*wheel_width)}" ixy="0.0" ixz="0.0"
           iyy="${wheel_mass / 12.0 * wheel_radius*wheel_radius}" iyz="0.0"
           izz="${wheel_mass / 12.0 * wheel_radius*wheel_radius}"/>
@@ -118,11 +118,11 @@
     </link>
 <!-- ****************************************************** Front caster joint *******************************************************  -->
-    <joint name="${prefix}caster_frontal_wheel_joint" type="fixed">
+    <joint name="${prefix}front_caster_joint" type="fixed">
       <parent link="${prefix}base_link"/>
-      <child link="${prefix}caster_frontal_wheel"/>
-      <origin xyz="${base_width/2 - caster_wheel_radius} 0 ${z_offset}" rpy="0 0 0"/>
+      <child link="${prefix}front_caster"/>
+      <origin xyz="${base_length/2 - caster_wheel_radius} 0 ${z_offset}" rpy="0 0 0"/>
     </joint>
 <!-- ****************************************************** Front caster Link ********************************************************  -->
-    <link name="${prefix}caster_frontal_wheel">
+    <link name="${prefix}front_caster">
       <collision>
         <origin xyz="0 0 0" rpy="0 0 0"/>
@@ -148,11 +148,11 @@
     </link>
 <!-- ****************************************************** Rear Caster Joint ********************************************************  -->
-    <joint name="${prefix}caster_rear_wheel_joint" type="fixed">
+    <joint name="${prefix}rear_caster_joint" type="fixed">
       <parent link="${prefix}base_link"/>
-      <child link="${prefix}caster_rear_wheel"/>
-      <origin xyz="${-base_width/2 + caster_wheel_radius} 0 ${z_offset}" rpy="0 0 0"/>
+      <child link="${prefix}rear_caster"/>
+      <origin xyz="${-base_length/2 + caster_wheel_radius} 0 ${z_offset}" rpy="0 0 0"/>
     </joint>
 <!-- ****************************************************** Rear Caster Link *********************************************************  -->
-    <link name="${prefix}caster_rear_wheel">
+    <link name="${prefix}rear_caster">
       <collision>
         <origin xyz="0 0 0" rpy="0 0 0"/>

File: xacro/twr.xacro (robot description, xacro)
@@ -56,5 +56,5 @@
   <link name="base_link">
     <visual>
-      <origin xyz="0 0 -0.05" rpy="1.5707963267949 0 3.141592654"/>
+      <origin xyz="0 0 -0.05" rpy="${radians(90)} 0 ${radians(180)}"/>
       <geometry>
         <mesh filename="${mesh_path}robot_base.stl" />
@@ -73,5 +73,5 @@
     <link name="${prefix}_link">
       <visual>
-        <origin xyz="0 0 0" rpy="1.5707963267949 0 0"/>
+        <origin xyz="0 0 0" rpy="${radians(90)} 0 0"/>
         <geometry>
             <cylinder radius="${wheel_radius}" length="${wheel_width}"/>

Commit message: u

File: gazebo/gz_diffbot.xacro (robot description, xacro)
@@ -9,13 +9,13 @@
 <!-- ****************************************************** Base Link ****************************************************************  -->
     <gazebo reference="${prefix}base_link">
-      <material>Gazebo/Blue</material>
+      <material>Gazebo/Orange</material>
     </gazebo>
 <!-- ****************************************************** Left Wheel Link **********************************************************  -->
     <gazebo reference="${prefix}left_wheel">
-      <material>Gazebo/Black</material>
+      <material>Gazebo/Gray</material>
     </gazebo>
 <!-- ****************************************************** Right Wheel Link ********************************************************  -->
     <gazebo reference="${prefix}right_wheel">
-      <material>Gazebo/Black</material>
+      <material>Gazebo/Gray</material>
     </gazebo>
 <!-- ****************************************************** Front caster Link ********************************************************  -->

Commit message: u

File: gazebo/gz_diffbot.xacro (robot description, xacro)
@@ -13,9 +13,9 @@
 <!-- ****************************************************** Left Wheel Link **********************************************************  -->
     <gazebo reference="${prefix}left_wheel">
-      <material>Gazebo/Gray</material>
+      <material>Gazebo/Red</material>
     </gazebo>
 <!-- ****************************************************** Right Wheel Link ********************************************************  -->
     <gazebo reference="${prefix}right_wheel">
-      <material>Gazebo/Gray</material>
+      <material>Gazebo/Red</material>
     </gazebo>
 <!-- ****************************************************** Front caster Link ********************************************************  -->
