Commit message: u

File: gazebo/gz_diffbot.xacro (robot description, xacro)
@@ -13,9 +13,9 @@
 <!-- ****************************************************** Left Wheel Link **********************************************************  -->
     <gazebo reference="${prefix}left_wheel">
-      <material>Gazebo/Red</material>
+      <material>Gazebo/Gray</material>
     </gazebo>
 <!-- ****************************************************** Right Wheel Link ********************************************************  -->
     <gazebo reference="${prefix}right_wheel">
-      <material>Gazebo/Red</material>
+      <material>Gazebo/Gray</material>
     </gazebo>
 <!-- ****************************************************** Front caster Link ********************************************************  -->

Commit message: u

File: gazebo/gz_diffbot.xacro (robot description, xacro)
@@ -9,5 +9,5 @@
 <!-- ****************************************************** Base Link ****************************************************************  -->
     <gazebo reference="${prefix}base_link">
-      <material>Gazebo/Orange</material>
+      <material>Gazebo/Blue</material>
     </gazebo>
 <!-- ****************************************************** Left Wheel Link **********************************************************  -->

File: urdf/diffbot.urdf (robot description, URDF)
Before this commit: robot diffbot, 6 links, 5 joints
Links:
- link front_caster: geometry collision sphere radius=0.08; visual sphere radius=0.08
- link left_wheel: mass 0.3 -> 5.0; geometry collision cylinder length=0.05 radius=0.08; visual cylinder length=0.05 radius=0.08
- link rear_caster: geometry collision sphere radius=0.08; visual sphere radius=0.08
- link right_wheel: mass 0.3 -> 5.0; geometry collision cylinder length=0.05 radius=0.08; visual cylinder length=0.05 radius=0.08
Joints:
- joint base_joint: origin xyz=0.0 0.0 0.1 rpy=0.0 0.0 0.0 -> xyz=0.0 0.0 0.10500000000000001 rpy=0.0 0.0 0.0
- joint front_caster_joint: origin xyz=0.15000000000000002 0 -0.05 rpy=0 0 0 -> xyz=0.114 0 -0.025 rpy=0 0 0
- joint left_wheel_joint: origin xyz=0 -0.11800000000000001 -0.05 rpy=0 0 0 -> xyz=0 -0.135 -0.025 rpy=0 0 0
- joint rear_caster_joint: origin xyz=-0.15000000000000002 0 -0.05 rpy=0 0 0 -> xyz=-0.114 0 -0.025 rpy=0 0 0
- joint right_wheel_joint: origin xyz=0 0.11800000000000001 -0.05 rpy=0 0 0 -> xyz=0 0.135 -0.025 rpy=0 0 0

File: xacro/diffbot.xacro (robot description, xacro)
@@ -7,15 +7,19 @@
 <!-- ****************************************************** Parameters ***************************************************************  -->
   <xacro:property name="mesh_path"      value="package://robot_gazebo/meshes/diffbot/"/>
+  <xacro:property name="name_space"     value="diffbot"  />
   <xacro:property name="base_mass"      value="0.6"                               />  <!-- arbitrary value for base mass                -->
   <xacro:property name="base_width"     value="0.20"                              />
   <xacro:property name="base_length"    value="0.40"                              />
   <xacro:property name="base_height"    value="0.10"                              />
-  <xacro:property name="wheel_mass"     value="0.3"                               />  <!-- arbitrary value for wheel mass               -->
-  <xacro:property name="wheel_width"    value="0.030"                             />
-  <xacro:property name="wheel_radius"   value="0.050"                             />
+  <xacro:property name="wheel_mass"     value="5.0"                               />
+  <xacro:property name="wheel_width"    value="0.05"                              />
+  <xacro:property name="wheel_radius"   value="0.08"                              />
+  <xacro:property name="wheel_gap"      value="0.01"                              /> <!-- Gap between wheels and base                   -->
+  <xacro:property name="wheel_y"        value="${(base_width+wheel_width)/2+wheel_gap}" />
+  <xacro:property name="wheel_z"        value="${base_height/4}"                  />  <!-- Space btw top of beam and the each joint     -->
   <xacro:property name="caster_mass"    value="0.1"                               />  <!-- arbitrary value for caster wheel mass        -->
-  <xacro:property name="caster_radius"  value="${wheel_radius}"                   />
-  <xacro:property name="y_offset"       value="${(base_width+wheel_width*1.2)/2}" />
-  <xacro:property name="z_offset"       value="${base_height/2}"                  />  <!-- Space btw top of beam and the each joint     -->
+  <xacro:property name="caster_radius"  value="${wheel_radius-wheel_z}"           />
+  <xacro:property name="caster_x"       value="${(base_length/2 - caster_radius)*0.95}" />
+  <xacro:property name="caster_z"       value="${base_height/2}"/>
 <!-- ****************************************************** Includes *****************************************************************  -->
   <xacro:include filename="$(find robot_gazebo)/xacro/common_rviz_materials.xacro" />   <!-- RVIZ Colors                                -->
@@ -29,5 +33,5 @@
         <parent link="base_footprint"/>
         <child link="${prefix}base_link"/>
-        <origin xyz="0.0 0.0 ${(wheel_radius+z_offset)}" rpy="0.0 0.0 0.0"/>
+        <origin xyz="0.0 0.0 ${(wheel_radius+wheel_z)}" rpy="0.0 0.0 0.0"/>
     </joint>
 <!-- ****************************************************** Base Link ****************************************************************  -->
@@ -44,5 +48,5 @@
         <mesh filename="${mesh_path}base.stl" scale="1 1 1"/>  <!--  <box size="${base_length} ${base_width} ${base_height}"/> -->
       </geometry>
-      <material name="orange"/>
+      <material name="blue"/>
     </visual>
     <inertial>
@@ -59,5 +63,5 @@
       <parent link="${prefix}base_link"/>
       <child link="${prefix}left_wheel"/>
-      <origin xyz="0 -${y_offset} -${z_offset}" rpy="0 0 0"/>
+      <origin xyz="0 -${wheel_y} -${wheel_z}" rpy="0 0 0"/>
       <limit upper="${radians(180)}" lower="-${radians(180)}" effort="30" velocity="5.0"/>
       <axis xyz="0 1 0"/>
@@ -92,5 +96,5 @@
       <parent link="${prefix}base_link"/>
       <child link="${prefix}right_wheel"/>
-      <origin xyz="0 ${y_offset} -${z_offset}" rpy="0 0 0"/>
+      <origin xyz="0 ${wheel_y} -${wheel_z}" rpy="0 0 0"/>
       <limit upper="${radians(180)}" lower="-${radians(180)}" effort="30" velocity="5.0"/>
       <axis xyz="0 1 0"/>
@@ -125,5 +129,5 @@
       <parent link="${prefix}base_link"/>
       <child link="${prefix}front_caster"/>
-      <origin xyz="${base_length/2 - caster_radius} 0 ${-z_offset}" rpy="0 0 0"/>
+      <origin xyz="${caster_x} 0 ${-caster_z}" rpy="0 0 0"/>
     </joint>
 <!-- ****************************************************** Front caster Link ********************************************************  -->
@@ -155,5 +159,5 @@
       <parent link="${prefix}base_link"/>
       <child link="${prefix}rear_caster"/>
-      <origin xyz="${-base_length/2 + caster_radius} 0 ${-z_offset}" rpy="0 0 0"/>
+      <origin xyz="${-caster_x} 0 ${-caster_z}" rpy="0 0 0"/>
     </joint>
 <!-- ****************************************************** Rear Caster Link *********************************************************  -->

Commit message: u

File: gazebo/gz_diffbot.xacro (robot description, xacro)
@@ -5,17 +5,7 @@
 <!-- March 2022                                                                                                                         -->
 <!-- *********************************************************************************************************************************  -->
-<!-- ****************************************************** Macro ********************************************************************  -->
-  <xacro:macro name="diffbot_gz" params="prefix">
 <!-- ****************************************************** Base Link ****************************************************************  -->
     <gazebo reference="${prefix}base_link">
       <material>Gazebo/Blue</material>
-    </gazebo>
-<!-- ****************************************************** Left Wheel Link **********************************************************  -->
-    <gazebo reference="${prefix}left_wheel">
-      <material>Gazebo/Gray</material>
-    </gazebo>
-<!-- ****************************************************** Right Wheel Link ********************************************************  -->
-    <gazebo reference="${prefix}right_wheel">
-      <material>Gazebo/Gray</material>
     </gazebo>
 <!-- ****************************************************** Front caster Link ********************************************************  -->
@@ -27,8 +17,4 @@
       <material>Gazebo/White</material>
     </gazebo>
-<!-- ****************************************************** End Macro ****************************************************************  -->
-  </xacro:macro>
-<!-- ****************************************************** Expand Macro *************************************************************  -->
-  <xacro:diffbot_gz prefix="" />
 <!-- ****************************************************** END **********************************************************************  -->
 </robot>

File: gazebo/gz_skidbot.xacro (robot description, xacro)
@@ -6,5 +6,5 @@
 <!-- *********************************************************************************************************************************  -->
 <!-- ****************************************************** Base *********************************************************************  -->
-  <gazebo reference="base">
+  <gazebo reference="${prefix}base">
     <material>Gazebo/Blue</material>
   </gazebo>
@@ -15,8 +15,8 @@
         <namespace>${name_space}</namespace>
       </ros>
-      <joint_name>front_left_wheel_joint</joint_name>
-      <joint_name>back_left_wheel_joint</joint_name>
-      <joint_name>front_right_wheel_joint</joint_name>
-      <joint_name>back_right_wheel_joint</joint_name>
+      <joint_name>${prefix}front_left_wheel_joint</joint_name>
+      <joint_name>${prefix}back_left_wheel_joint</joint_name>
+      <joint_name>${prefix}front_right_wheel_joint</joint_name>
+      <joint_name>${prefix}back_right_wheel_joint</joint_name>
       <update_rate>100.0</update_rate>
     </plugin>
@@ -30,11 +30,11 @@
       <num_wheel_pairs>2</num_wheel_pairs>
       <!-- 1st Wheels Set -->
-      <left_joint>front_left_wheel_joint</left_joint>
-      <right_joint>front_right_wheel_joint</right_joint>
+      <left_joint>${prefix}front_left_wheel_joint</left_joint>
+      <right_joint>${prefix}front_right_wheel_joint</right_joint>
       <wheel_separation>${wheel_y*2}</wheel_separation>
       <wheel_diameter>${wheel_radius*2}</wheel_diameter>
       <!-- 2nd Wheels Set -->
-      <left_joint>back_left_wheel_joint</left_joint>
-      <right_joint>back_right_wheel_joint</right_joint>
+      <left_joint>${prefix}back_left_wheel_joint</left_joint>
+      <right_joint>${prefix}back_right_wheel_joint</right_joint>
       <wheel_separation>${wheel_y*2}</wheel_separation>
       <wheel_diameter>${wheel_radius*2}</wheel_diameter>
@@ -42,5 +42,5 @@
       <max_wheel_acceleration>1.0</max_wheel_acceleration>
       <update_rate>100.0</update_rate>
-      <robot_base_frame>footprint</robot_base_frame>
+      <robot_base_frame>${prefix}footprint</robot_base_frame>
       <odometry_frame>odom</odometry_frame>
       <publish_odom>true</publish_odom>
@@ -50,5 +50,5 @@
   </gazebo>
 <!-- ******************************************************  Camera ******************************************************************  -->
-  <gazebo reference="camera">
+  <gazebo reference="${prefix}camera">
     <sensor type="camera" name="camera_sensor">
       <plugin name="camera" filename="libgazebo_ros_camera.so">
@@ -86,5 +86,5 @@
   </gazebo>
 <!-- ****************************************************** hokuyo  ******************************************************************  -->
-  <gazebo reference="hokuyo">
+  <gazebo reference="${prefix}hokuyo">
     <sensor type="ray" name="head_hokuyo_sensor">
       <plugin name="hokuyo" filename="libgazebo_ros_ray_sensor.so">

File: urdf/diffbot.urdf (robot description, URDF)
Before this commit: robot diffbot, 6 links, 5 joints
Links:
- added link hokuyo, mass 1e-05; collision mesh filename=package://robot_gazebo/meshes/diffbot/hokuyo.dae; visual mesh filename=package://robot_gazebo/meshes/diffbot/hokuyo.dae
Joints:
- added joint hokuyo_joint: type fixed, parent base_link, child hokuyo, origin xyz=0.11 0 0.0853 rpy=0 0 0, axis 0 1 0

File: xacro/diffbot.xacro (robot description, xacro)
@@ -8,4 +8,5 @@
   <xacro:property name="mesh_path"      value="package://robot_gazebo/meshes/diffbot/"/>
   <xacro:property name="name_space"     value="diffbot"  />
+  <xacro:property name="prefix"         value=""  />
   <xacro:property name="base_mass"      value="0.6"                               />  <!-- arbitrary value for base mass                -->
   <xacro:property name="base_width"     value="0.20"                              />
@@ -31,6 +32,4 @@
   <xacro:include filename="$(find robot_gazebo)/xacro/common_rviz_materials.xacro" />   <!-- RVIZ Colors                                -->
   <xacro:include filename="$(find robot_gazebo)/gazebo/gz_diffbot.xacro" />             <!-- Gazebo                                     -->
-<!-- ****************************************************** Macro ********************************************************************  -->
-  <xacro:macro name="diffbot" params="prefix">
 <!-- ****************************************************** Base Footprint ***********************************************************  -->
     <link name="${prefix}base_footprint"/>
@@ -216,11 +215,7 @@
     <origin xyz="${hokuyo_x} 0 ${hokuyo_z}" rpy="0 0 0"/>
     <child link="${prefix}hokuyo"/>
-    <parent link="${prefix}base"/>
+    <parent link="${prefix}base_link"/>
     <axis xyz="0 1 0" rpy="0 0 0"/>
   </joint>
-<!-- ****************************************************** End Macro ****************************************************************  -->
-  </xacro:macro>
-<!-- ****************************************************** Expand Macro *************************************************************  -->
-  <xacro:diffbot prefix="" />
 <!-- ****************************************************** END **********************************************************************  -->
 </robot>

File: xacro/skidbot.xacro (robot description, xacro)
@@ -8,4 +8,5 @@
   <xacro:property name="mesh_path"      value="package://robot_gazebo/meshes/skidbot/"/>
   <xacro:property name="name_space"     value="skidbot"  />
+  <xacro:property name="prefix"         value=""  />
   <xacro:property name="base_mass"      value="15.0"     /> <!-- arbitrary mass value -->
   <xacro:property name="base_width"     value="0.20"     />
@@ -33,13 +34,13 @@
   <xacro:include filename="$(find robot_gazebo)/gazebo/gz_skidbot.xacro" />             <!-- Gazebo                                     -->
 <!-- ****************************************************** Base Footprint ***********************************************************  -->
-  <link name="footprint"></link>
+  <link name="${prefix}footprint"></link>
 <!-- ****************************************************** Footprint Joint **********************************************************  -->
-  <joint type="fixed" name="footprint_joint" >
+  <joint type="fixed" name="${prefix}footprint_joint" >
     <origin xyz="0 0 0" rpy="0 0 0" />
-    <parent link="footprint"/>
-    <child link="base" />
+    <parent link="${prefix}footprint"/>
+    <child link="${prefix}base" />
   </joint>
 <!-- ****************************************************** Base Link ****************************************************************  -->
-  <link name='base'>
+  <link name='${prefix}base'>
     <pose>0 0 0 0 0 0</pose>
     <inertial>
@@ -65,5 +66,5 @@
   <xacro:macro name="wheel" params="position side x y">
 <!-- ****************************************************** Wheel Link ***************************************************************  -->
-    <link name="${position}_${side}_wheel">
+    <link name="${prefix}${prefix}${position}_${side}_wheel">
       <inertial>
         <mass value="${base_mass}"/>
@@ -86,5 +87,5 @@
     </link>
 <!-- ****************************************************** Wheel Joint **************************************************************  -->
-    <joint type="continuous" name="${position}_${side}_wheel_joint">
+    <joint type="continuous" name="${prefix}${position}_${side}_wheel_joint">
         <origin xyz="${x} ${y} 0" rpy="0 0 0"/>
         <child link="${position}_${side}_wheel"/>
@@ -102,5 +103,5 @@
 <xacro:wheel position="back"  side="left"  x="-${wheel_x}" y=" ${wheel_y}" />
 <!-- ****************************************************** Camera Link **************************************************************  -->
-  <link name="camera">
+  <link name="${prefix}camera">
     <inertial>
       <mass value="${camera_mass}"/>
@@ -123,12 +124,12 @@
   </link>
 <!-- ****************************************************** Camera Joint *************************************************************  -->
-  <joint type="fixed" name="camera_joint">
+  <joint type="fixed" name="${prefix}camera_joint">
     <origin xyz="${camera_x} 0 0" rpy="0 0 0"/>
-    <child link="camera"/>
-    <parent link="base"/>
+    <child link="${prefix}camera"/>
+    <parent link="${prefix}base"/>
     <axis xyz="0 1 0" rpy="0 0 0"/>
   </joint>
 <!-- ****************************************************** Hokuyo Link **************************************************************  -->
-  <link name="hokuyo">
+  <link name="${prefix}hokuyo">
     <inertial>
       <mass value="${hokuyo_mass}"/>
@@ -151,8 +152,8 @@
   </link>
 <!-- ****************************************************** Hokuyo Joint *************************************************************  -->
-  <joint type="fixed" name="hokuyo_joint">
+  <joint type="fixed" name="${prefix}hokuyo_joint">
     <origin xyz="${hokuyo_x} 0 ${hokuyo_z}" rpy="0 0 0"/>
-    <child link="hokuyo"/>
-    <parent link="base"/>
+    <child link="${prefix}hokuyo"/>
+    <parent link="${prefix}base"/>
     <axis xyz="0 1 0" rpy="0 0 0"/>
   </joint>
