Commit message: u

File: gazebo/gz_diffbot.xacro (robot description, xacro)
@@ -6,5 +6,5 @@
 <!-- *********************************************************************************************************************************  -->
 <!-- ****************************************************** Base Link ****************************************************************  -->
-    <gazebo reference="${prefix}base_link">
+    <gazebo reference="${prefix}base">
       <material>Gazebo/Blue</material>
     </gazebo>
@@ -17,4 +17,110 @@
       <material>Gazebo/White</material>
     </gazebo>
+<!-- ******************************************************  Joint States Publisher **************************************************  -->
+  <gazebo>
+    <plugin name="joint_states_pub" filename="libgazebo_ros_joint_state_publisher.so">
+      <ros>
+        <namespace>${name_space}</namespace>
+      </ros>
+      <joint_name>${prefix}right_wheel_joint</joint_name>
+      <joint_name>${prefix}left_wheel_joint</joint_name>
+      <update_rate>100.0</update_rate>
+    </plugin>
+ </gazebo>
+<!-- ******************************************************  Skid Steer Drive Controller *********************************************  -->
+  <gazebo>
+    <plugin name="skid_drive" filename="libgazebo_ros_diff_drive.so">
+      <ros>
+        <namespace>${name_space}</namespace>
+      </ros>
+      <num_wheel_pairs>1</num_wheel_pairs>
+      <!-- 1st Wheels Set -->
+      <right_joint>${prefix}right_wheel_joint</right_joint>
+      <left_joint>${prefix}left_wheel_joint</left_joint>
+      <wheel_separation>${wheel_y*2}</wheel_separation>
+      <wheel_diameter>${wheel_radius*2}</wheel_diameter>
+      <max_wheel_torque>20</max_wheel_torque>
+      <max_wheel_acceleration>1.0</max_wheel_acceleration>
+      <update_rate>100.0</update_rate>
+      <robot_base_frame>${prefix}footprint</robot_base_frame>
+      <odometry_frame>odom</odometry_frame>
+      <publish_odom>true</publish_odom>
+      <publish_odom_tf>true</publish_odom_tf>
+      <publish_wheel_tf>true</publish_wheel_tf>
+    </plugin>
+  </gazebo>
+<!-- ******************************************************  Camera ******************************************************************  -->
+  <gazebo reference="${prefix}camera">
+    <sensor type="camera" name="camera_sensor">
+      <plugin name="camera" filename="libgazebo_ros_camera.so">
+        <ros>
+          <namespace>${name_space}</namespace>
+        </ros>
+        <camera_name>camera</camera_name>
+        <frame_name>camera</frame_name>
+        <hack_baseline>0.07</hack_baseline>
+      </plugin>
+      <update_rate>30.0</update_rate>
+      <always_on>1</always_on>
+      <camera name="camera">
+        <horizontal_fov>${radians(80)}</horizontal_fov>
+        <image>
+          <width>1280</width>
+          <height>720</height>
+          <format>R8G8B8</format>
+        </image>
+        <clip>
+          <near>0.02</near>
+          <far>300</far>
+        </clip>
+        <distortion>
+          <k1>0.0</k1>
+          <k2>0.0</k2>
+          <k3>0.0</k3>
+          <p1>0.0</p1>
+          <p2>0.0</p2>
+          <center>0.5 0.5</center>
+        </distortion>
+      </camera>
+    </sensor>
+    <material>Gazebo/Green</material>
+  </gazebo>
+<!-- ****************************************************** hokuyo  ******************************************************************  -->
+  <gazebo reference="${prefix}hokuyo">
+    <sensor type="ray" name="head_hokuyo_sensor">
+      <plugin name="hokuyo" filename="libgazebo_ros_ray_sensor.so">
+        <ros>
+          <namespace>${name_space}</namespace>
+        </ros>
+        <output_type>sensor_msgs/LaserScan</output_type>
+      </plugin>
+      <update_rate>30</update_rate>
+      <pose>0 0 0 0 0 0</pose>
+      <visualize>false</visualize>
+      <ray>
+        <scan>
+          <horizontal>
+            <samples>720</samples>
+            <resolution>1</resolution>
+            <min_angle>-${radians(180)}</min_angle>
+            <max_angle> ${radians(180)}</max_angle>
+          </horizontal>
+        </scan>
+        <range>
+          <min>0.10</min>
+          <max>30.0</max>
+          <resolution>0.01</resolution>
+        </range>
+<!-- Noise parameters based on published spec for Hokuyo laser achieving "+-30mm" accuracy at range < 10m.  A mean of 0.0m and stddev   -->
+<!-- of 0.01m will put 99.7% of samples within 0.03m of the true reading.                                                               -->
+        <noise>
+          <type>gaussian</type>
+          <mean>0.0</mean>
+          <stddev>0.01</stddev>
+        </noise>
+      </ray>
+    </sensor>
+    <!-- <material>Gazebo/Red</material> -->
+  </gazebo>
 <!-- ****************************************************** END **********************************************************************  -->
 </robot>

File: gazebo/gz_skidbot.xacro (robot description, xacro)
@@ -39,7 +39,9 @@
       <wheel_separation>${wheel_y*2}</wheel_separation>
       <wheel_diameter>${wheel_radius*2}</wheel_diameter>
+      <!---->
       <max_wheel_torque>20</max_wheel_torque>
       <max_wheel_acceleration>1.0</max_wheel_acceleration>
       <update_rate>100.0</update_rate>
+      <!---->
       <robot_base_frame>${prefix}footprint</robot_base_frame>
       <odometry_frame>odom</odometry_frame>

File: xacro/diffbot.xacro (robot description, xacro)
@@ -32,14 +32,14 @@
   <xacro:include filename="$(find robot_gazebo)/xacro/common_rviz_materials.xacro" />   <!-- RVIZ Colors                                -->
   <xacro:include filename="$(find robot_gazebo)/gazebo/gz_diffbot.xacro" />             <!-- Gazebo                                     -->
-<!-- ****************************************************** Base Footprint ***********************************************************  -->
-    <link name="${prefix}base_footprint"/>
+<!-- ****************************************************** Footprint ****************************************************************  -->
+    <link name="${prefix}footprint"/>
 <!-- ****************************************************** Base Joint ***************************************************************  -->
-    <joint name="base_joint" type="fixed">
-        <parent link="base_footprint"/>
-        <child link="${prefix}base_link"/>
+    <joint name="footprint_joint" type="fixed">
+        <parent link="footprint"/>
+        <child link="${prefix}base"/>
         <origin xyz="0.0 0.0 ${(wheel_radius+wheel_z)}" rpy="0.0 0.0 0.0"/>
     </joint>
 <!-- ****************************************************** Base Link ****************************************************************  -->
-  <link name="${prefix}base_link">
+  <link name="${prefix}base">
     <collision>
       <origin xyz="0 0 0" rpy="0 0 0"/>
@@ -66,5 +66,5 @@
 <!-- ****************************************************** Right Wheel Joint ********************************************************  -->
     <joint name="${prefix}right_wheel_joint" type="continuous">
-      <parent link="${prefix}base_link"/>
+      <parent link="${prefix}base"/>
       <child link="${prefix}right_wheel"/>
       <origin xyz="0 ${wheel_y} -${wheel_z}" rpy="0 0 0"/>
@@ -99,5 +99,5 @@
 <!-- ****************************************************** Left Wheel Joint *********************************************************  -->
     <joint name="${prefix}left_wheel_joint" type="continuous">
-      <parent link="${prefix}base_link"/>
+      <parent link="${prefix}base"/>
       <child link="${prefix}left_wheel"/>
       <origin xyz="0 -${wheel_y} -${wheel_z}" rpy="0 0 0"/>
@@ -132,5 +132,5 @@
 <!-- ****************************************************** Front caster joint *******************************************************  -->
     <joint name="${prefix}front_caster_joint" type="fixed">
-      <parent link="${prefix}base_link"/>
+      <parent link="${prefix}base"/>
       <child link="${prefix}front_caster"/>
       <origin xyz="${caster_x} 0 ${-caster_z}" rpy="0 0 0"/>
@@ -162,5 +162,5 @@
 <!-- ****************************************************** Rear Caster Joint ********************************************************  -->
     <joint name="${prefix}rear_caster_joint" type="fixed">
-      <parent link="${prefix}base_link"/>
+      <parent link="${prefix}base"/>
       <child link="${prefix}rear_caster"/>
       <origin xyz="${-caster_x} 0 ${-caster_z}" rpy="0 0 0"/>
@@ -190,4 +190,32 @@
       </inertial>
     </link>
+<!-- ****************************************************** Camera Link **************************************************************  -->
+  <link name="${prefix}camera">
+    <inertial>
+      <mass value="${camera_mass}"/>
+      <origin xyz="0 0 0" rpy=" 0 0 0"/>
+      <inertia ixx="1e-6" ixy="0" ixz="0" iyy="1e-6" iyz="0" izz="1e-6" />
+    </inertial>
+    <visual name="camera_visual">
+      <origin xyz="0 0 0" rpy="0 0 0" />
+      <geometry>
+        <box size="${camera_length} ${camera_width} ${camera_height}"/>
+      </geometry>
+      <material name="green"/>
+    </visual>
+    <collision name="camera_colision">
+      <origin xyz="0 0 0" rpy="0 0 0" />
+      <geometry>
+        <box size="${camera_length} ${camera_width} ${camera_height}"/>
+      </geometry>
+    </collision>
+  </link>
+<!-- ****************************************************** Camera Joint *************************************************************  -->
+  <joint type="fixed" name="${prefix}camera_joint">
+    <origin xyz="${camera_x} 0 0" rpy="0 0 0"/>
+    <child link="${prefix}camera"/>
+    <parent link="${prefix}base"/>
+    <axis xyz="0 1 0" rpy="0 0 0"/>
+  </joint>
 <!-- ****************************************************** Hokuyo Link **************************************************************  -->
   <link name="${prefix}hokuyo">
@@ -215,5 +243,5 @@
     <origin xyz="${hokuyo_x} 0 ${hokuyo_z}" rpy="0 0 0"/>
     <child link="${prefix}hokuyo"/>
-    <parent link="${prefix}base_link"/>
+    <parent link="${prefix}base"/>
     <axis xyz="0 1 0" rpy="0 0 0"/>
   </joint>

Commit message: u

File: gazebo/gz_diffbot.xacro (robot description, xacro)
@@ -11,8 +11,4 @@
 <!-- ****************************************************** Front caster Link ********************************************************  -->
     <gazebo reference="${prefix}front_caster">
-      <material>Gazebo/White</material>
-    </gazebo>
-<!-- ****************************************************** Rear Caster Link *********************************************************  -->
-    <gazebo reference="${prefix}rear_caster">
       <material>Gazebo/White</material>
     </gazebo>

File: urdf/diffbot.urdf (robot description, URDF)
Before this commit: robot diffbot, 8 links, 7 joints
Links:
- removed link rear_caster
Joints:
- removed joint rear_caster_joint
- joint front_caster_joint: origin xyz=0.13775 0 -0.04 rpy=0 0 0 -> xyz=0.14500000000000002 0 -0.05 rpy=0 0 0
- joint left_wheel_joint: origin xyz=0 -0.135 -0.025 rpy=0 0 0 -> xyz=-0.12 -0.135 -0.025 rpy=0 0 0
- joint right_wheel_joint: origin xyz=0 0.135 -0.025 rpy=0 0 0 -> xyz=-0.12 0.135 -0.025 rpy=0 0 0

File: xacro/diffbot.xacro (robot description, xacro)
@@ -17,10 +17,11 @@
   <xacro:property name="wheel_radius"   value="0.08"                              />
   <xacro:property name="wheel_gap"      value="0.01"                              /> <!-- Gap between wheels and base                   -->
+  <xacro:property name="wheel_x"        value="0.12"                              /> <!-- x offset from base center -->
   <xacro:property name="wheel_y"        value="${(base_width+wheel_width)/2+wheel_gap}" />
   <xacro:property name="wheel_z"        value="${base_height/4}"                  />  <!-- Space btw top of beam and the each joint     -->
   <xacro:property name="caster_mass"    value="0.1"                               />  <!-- arbitrary value for caster wheel mass        -->
   <xacro:property name="caster_radius"  value="${wheel_radius-wheel_z}"           />
-  <xacro:property name="caster_x"       value="${(base_length/2 - caster_radius)*0.95}" />
-  <xacro:property name="caster_z"       value="${base_height/2-0.01}"/>
+  <xacro:property name="caster_x"       value="${(base_length/2 - caster_radius)}" />
+  <xacro:property name="caster_z"       value="${base_height/2}"/>
   <xacro:property name="camera_mass"    value="0.1"      />
   <xacro:property name="camera_width"   value="0.05"     />
@@ -73,5 +74,5 @@
       <parent link="${prefix}base"/>
       <child link="${prefix}right_wheel"/>
-      <origin xyz="0 ${wheel_y} -${wheel_z}" rpy="0 0 0"/>
+      <origin xyz="-${wheel_x} ${wheel_y} -${wheel_z}" rpy="0 0 0"/>
       <limit upper="${radians(180)}" lower="-${radians(180)}" effort="30" velocity="5.0"/>
       <axis xyz="0 1 0"/>
@@ -106,5 +107,5 @@
       <parent link="${prefix}base"/>
       <child link="${prefix}left_wheel"/>
-      <origin xyz="0 -${wheel_y} -${wheel_z}" rpy="0 0 0"/>
+      <origin xyz="-${wheel_x} -${wheel_y} -${wheel_z}" rpy="0 0 0"/>
       <limit upper="${radians(180)}" lower="-${radians(180)}" effort="30" velocity="5.0"/>
       <axis xyz="0 1 0"/>
@@ -143,34 +144,4 @@
 <!-- ****************************************************** Front caster Link ********************************************************  -->
     <link name="${prefix}front_caster">
-      <collision>
-        <origin xyz="0 0 0" rpy="0 0 0"/>
-        <geometry>
-          <sphere radius="${caster_radius}"/>
-        </geometry>
-      </collision>
-      <visual>
-        <origin xyz="0 0 0" rpy="0 0 0"/>
-        <geometry>
-          <sphere radius="${caster_radius}"/>
-        </geometry>
-        <material name="white"/>
-      </visual>
-      <inertial>
-        <origin xyz="0 0 0" rpy="0 0 0"/>
-        <mass value="${caster_mass}"/>
-        <inertia
-          ixx="${caster_mass * 0.4 * (caster_radius * caster_radius)}" ixy="0.0" ixz="0.0"
-          iyy="${caster_mass * 0.4 * (caster_radius * caster_radius)}" iyz="0.0"
-          izz="${caster_mass * 0.4 * (caster_radius * caster_radius)}"/>
-      </inertial>
-    </link>
-<!-- ****************************************************** Rear Caster Joint ********************************************************  -->
-    <joint name="${prefix}rear_caster_joint" type="fixed">
-      <parent link="${prefix}base"/>
-      <child link="${prefix}rear_caster"/>
-      <origin xyz="${-caster_x} 0 ${-caster_z}" rpy="0 0 0"/>
-    </joint>
-<!-- ****************************************************** Rear Caster Link *********************************************************  -->
-    <link name="${prefix}rear_caster">
       <collision>
         <origin xyz="0 0 0" rpy="0 0 0"/>

Commit message: u

File: gazebo/gz_diffbot.xacro (robot description, xacro)
@@ -48,16 +48,7 @@
 <!-- ******************************************************  Camera ******************************************************************  -->
   <gazebo reference="${prefix}camera">
-    <sensor type="camera" name="camera_sensor">
-      <plugin name="camera" filename="libgazebo_ros_camera.so">
-        <ros>
-          <namespace>${name_space}</namespace>
-        </ros>
-        <camera_name>camera</camera_name>
-        <frame_name>camera</frame_name>
-        <hack_baseline>0.07</hack_baseline>
-      </plugin>
+    <sensor type="camera" name="camera">
       <update_rate>30.0</update_rate>
-      <always_on>1</always_on>
-      <camera name="camera">
+      <camera name="head">
         <horizontal_fov>${radians(80)}</horizontal_fov>
         <image>
@@ -70,13 +61,37 @@
           <far>300</far>
         </clip>
-        <distortion>
-          <k1>0.0</k1>
-          <k2>0.0</k2>
-          <k3>0.0</k3>
-          <p1>0.0</p1>
-          <p2>0.0</p2>
-          <center>0.5 0.5</center>
-        </distortion>
+        <noise>
+          <type>gaussian</type>
+          <!-- Noise is sampled independently per pixel on each frame.
+          That pixel's noise value is added to each of its color
+          channels, which at that point lie in the range [0,1]. -->
+          <mean>0.0</mean>
+          <stddev>0.007</stddev>
+        </noise>
       </camera>
+      <plugin name="camera_controller" filename="libgazebo_ros_camera.so">
+        <ros>
+          <namespace>${name_space}</namespace>
+        </ros>
+        <alwaysOn>true</alwaysOn>
+        <updateRate>0.0</updateRate>
+        <cameraName>camera</cameraName>
+        <imageTopicName>image_raw</imageTopicName>
+        <cameraInfoTopicName>camera_info</cameraInfoTopicName>
+        <frameName>camera_optical</frameName>
+        <!-- setting hackBaseline to anything but 0.0 will cause a misalignment
+        between the gazebo sensor image and the frame it is supposed to
+        be attached to -->
+        <hackBaseline>0.0</hackBaseline>
+        <distortionK1>0.0</distortionK1>
+        <distortionK2>0.0</distortionK2>
+        <distortionK3>0.0</distortionK3>
+        <distortionT1>0.0</distortionT1>
+        <distortionT2>0.0</distortionT2>
+        <CxPrime>0</CxPrime>
+        <Cx>0.0</Cx>
+        <Cy>0.0</Cy>
+        <focalLength>0.0</focalLength>
+      </plugin>
     </sensor>
     <material>Gazebo/Green</material>

File: xacro/rrbot.xacro (robot description, xacro)
@@ -8,5 +8,5 @@
   <xacro:property name="mesh_path"      value="package://robot_gazebo/meshes/rrbot/" />
   <xacro:property name="name_space"     default="rrbot"  />
-  <xacro:property name="prefix"         defaut=""  />
+  <xacro:property name="prefix"         default=""  />
   <xacro:property name="mass"           value="1"     /> <!-- arbitrary value for mass -->
   <xacro:property name="width"          value="0.1"   /> <!-- Square dimensions (widthxwidth) of beams -->
