Commit message: u

File: gazebo/gz_diffbot.xacro (robot description, xacro)
@@ -15,6 +15,97 @@
 <!-- ******************************************************  Joint States Publisher **************************************************  -->
 <!-- ******************************************************  Skid Steer Drive Controller *********************************************  -->
+<!-- ****************************************************** ROS Control Plugin *******************************************************  -->
+  <gazebo>
+    <plugin name="gz_ros2_control" filename="libgazebo_ros2_control.so">
+      <!--<parameters>${config_path}diffbot.yaml</parameters>-->
+    </plugin>
+  </gazebo>
 <!-- ******************************************************  Camera ******************************************************************  -->
+  <gazebo reference="${prefix}camera">
+    <sensor type="camera" name="camera">
+      <update_rate>30.0</update_rate>
+      <camera name="head">
+        <horizontal_fov>${radians(80)}</horizontal_fov>
+        <image>
+          <width>1280</width>
+          <height>720</height>
+          <format>R8G8B8</format>
+        </image>
+        <clip>
+          <near>0.02</near>
+          <far>300</far>
+        </clip>
+        <noise>
+          <type>gaussian</type>
+          <!-- Noise is sampled independently per pixel on each frame.
+          That pixel's noise value is added to each of its color
+          channels, which at that point lie in the range [0,1]. -->
+          <mean>0.0</mean>
+          <stddev>0.007</stddev>
+        </noise>
+      </camera>
+      <plugin name="camera_controller" filename="libgazebo_ros_camera.so">
+        <ros>
+          <namespace>${name_space}</namespace>
+        </ros>
+        <alwaysOn>true</alwaysOn>
+        <updateRate>0.0</updateRate>
+        <cameraName>camera</cameraName>
+        <imageTopicName>image_raw</imageTopicName>
+        <cameraInfoTopicName>camera_info</cameraInfoTopicName>
+        <frameName>camera_optical</frameName>
+        <!-- setting hackBaseline to anything but 0.0 will cause a misalignment
+        between the gazebo sensor image and the frame it is supposed to
+        be attached to -->
+        <hackBaseline>0.0</hackBaseline>
+        <distortionK1>0.0</distortionK1>
+        <distortionK2>0.0</distortionK2>
+        <distortionK3>0.0</distortionK3>
+        <distortionT1>0.0</distortionT1>
+        <distortionT2>0.0</distortionT2>
+        <CxPrime>0</CxPrime>
+        <Cx>0.0</Cx>
+        <Cy>0.0</Cy>
+        <focalLength>0.0</focalLength>
+      </plugin>
+    </sensor>
+    <material>Gazebo/Green</material>
+  </gazebo>
 <!-- ****************************************************** hokuyo  ******************************************************************  -->
+  <gazebo reference="${prefix}hokuyo">
+    <sensor type="ray" name="head_hokuyo_sensor">
+      <plugin name="hokuyo" filename="libgazebo_ros_ray_sensor.so">
+        <ros>
+          <namespace>${name_space}</namespace>
+        </ros>
+        <output_type>sensor_msgs/LaserScan</output_type>
+      </plugin>
+      <update_rate>30</update_rate>
+      <pose>0 0 0 0 0 0</pose>
+      <visualize>false</visualize>
+      <ray>
+        <scan>
+          <horizontal>
+            <samples>720</samples>
+            <resolution>1</resolution>
+            <min_angle>-${radians(180)}</min_angle>
+            <max_angle> ${radians(180)}</max_angle>
+          </horizontal>
+        </scan>
+        <range>
+          <min>0.10</min>
+          <max>30.0</max>
+          <resolution>0.01</resolution>
+        </range>
+<!-- Noise parameters based on published spec for Hokuyo laser achieving "+-30mm" accuracy at range < 10m.  A mean of 0.0m and stddev   -->
+<!-- of 0.01m will put 99.7% of samples within 0.03m of the true reading.                                                               -->
+        <noise>
+          <type>gaussian</type>
+          <mean>0.0</mean>
+          <stddev>0.01</stddev>
+        </noise>
+      </ray>
+    </sensor>
+  </gazebo>
 <!-- ****************************************************** END **********************************************************************  -->
 </robot>

File: gazebo/gz_skidbot.xacro (robot description, xacro)
@@ -15,6 +15,97 @@
 <!-- ******************************************************  Joint States Publisher **************************************************  -->
 <!-- ******************************************************  Diff Steer Drive Controller *********************************************  -->
+<!-- ****************************************************** ROS Control Plugin *******************************************************  -->
+  <gazebo>
+    <plugin name="gz_ros2_control" filename="libgazebo_ros2_control.so">
+      <!--<parameters>${config_path}skidbot.yaml</parameters>-->
+    </plugin>
+  </gazebo>
 <!-- ******************************************************  Camera ******************************************************************  -->
+  <gazebo reference="${prefix}camera">
+    <sensor type="camera" name="camera">
+      <update_rate>30.0</update_rate>
+      <camera name="head">
+        <horizontal_fov>${radians(80)}</horizontal_fov>
+        <image>
+          <width>1280</width>
+          <height>720</height>
+          <format>R8G8B8</format>
+        </image>
+        <clip>
+          <near>0.02</near>
+          <far>300</far>
+        </clip>
+        <noise>
+          <type>gaussian</type>
+          <!-- Noise is sampled independently per pixel on each frame.
+          That pixel's noise value is added to each of its color
+          channels, which at that point lie in the range [0,1]. -->
+          <mean>0.0</mean>
+          <stddev>0.007</stddev>
+        </noise>
+      </camera>
+      <plugin name="camera_controller" filename="libgazebo_ros_camera.so">
+        <ros>
+          <namespace>${name_space}</namespace>
+        </ros>
+        <alwaysOn>true</alwaysOn>
+        <updateRate>0.0</updateRate>
+        <cameraName>camera</cameraName>
+        <imageTopicName>image_raw</imageTopicName>
+        <cameraInfoTopicName>camera_info</cameraInfoTopicName>
+        <frameName>camera_optical</frameName>
+        <!-- setting hackBaseline to anything but 0.0 will cause a misalignment
+        between the gazebo sensor image and the frame it is supposed to
+        be attached to -->
+        <hackBaseline>0.0</hackBaseline>
+        <distortionK1>0.0</distortionK1>
+        <distortionK2>0.0</distortionK2>
+        <distortionK3>0.0</distortionK3>
+        <distortionT1>0.0</distortionT1>
+        <distortionT2>0.0</distortionT2>
+        <CxPrime>0</CxPrime>
+        <Cx>0.0</Cx>
+        <Cy>0.0</Cy>
+        <focalLength>0.0</focalLength>
+      </plugin>
+    </sensor>
+    <material>Gazebo/Green</material>
+  </gazebo>
 <!-- ****************************************************** hokuyo  ******************************************************************  -->
+  <gazebo reference="${prefix}hokuyo">
+    <sensor type="ray" name="head_hokuyo_sensor">
+      <plugin name="hokuyo" filename="libgazebo_ros_ray_sensor.so">
+        <ros>
+          <namespace>${name_space}</namespace>
+        </ros>
+        <output_type>sensor_msgs/LaserScan</output_type>
+      </plugin>
+      <update_rate>30</update_rate>
+      <pose>0 0 0 0 0 0</pose>
+      <visualize>false</visualize>
+      <ray>
+        <scan>
+          <horizontal>
+            <samples>720</samples>
+            <resolution>1</resolution>
+            <min_angle>-${radians(180)}</min_angle>
+            <max_angle> ${radians(180)}</max_angle>
+          </horizontal>
+        </scan>
+        <range>
+          <min>0.10</min>
+          <max>30.0</max>
+          <resolution>0.01</resolution>
+        </range>
+<!-- Noise parameters based on published spec for Hokuyo laser achieving "+-30mm" accuracy at range < 10m.  A mean of 0.0m and stddev   -->
+<!-- of 0.01m will put 99.7% of samples within 0.03m of the true reading.                                                               -->
+        <noise>
+          <type>gaussian</type>
+          <mean>0.0</mean>
+          <stddev>0.01</stddev>
+        </noise>
+      </ray>
+    </sensor>
+  </gazebo>
 <!-- ****************************************************** END **********************************************************************  -->
 </robot>
