Commit message: u

File: r2c/r2c_diffbot.xacro (robot description, xacro)
@@ -2,5 +2,5 @@
 <robot xmlns:xacro="http://www.ros.org/wiki/xacro">
     <ros2_control name="diffbot" type="system">
-      <joint name="${prefix}joint1">
+      <joint name="${prefix}right_wheel_joint">
         <command_interface name="position">
           <param name="min">-1</param>
@@ -9,5 +9,5 @@
         <state_interface name="position"/>
       </joint>
-      <joint name="${prefix}joint2">
+      <joint name="${prefix}left_wheel_joint">
         <command_interface name="position">
           <param name="min">-1</param>
